Commit message: torso and arm origins are calibratable in calibration.urdf.xacro

File: cob_hardware_config/cob3-3/calibration/calibration.urdf.xacro (robot description, xacro)
@@ -1,4 +1,20 @@
-<?xml version="1.0"?>
-<robot>
+<?xml version="1.0" ?><robot>
+	<!-- ***************** -->
+	<!-- robot calibration -->
+	<!-- ***************** -->
+	<!-- torso mount positions | relative to base_link -->
+	<property name="torso_x" value="0.155"/>
+	<property name="torso_y" value="0.0"/>
+	<property name="torso_z" value="0.892"/>
+	<property name="torso_roll" value="1.5708"/>
+	<property name="torso_pitch" value="0.0"/>
+	<property name="torso_yaw" value="0.0"/>
+	<!-- arm mount positions | relative to base_link -->
+	<property name="arm_x" value="-0.015982"/>
+	<property name="arm_y" value="-0.080992"/>
+	<property name="arm_z" value="0.875995"/>
+	<property name="arm_roll" value="0.7854"/>
+	<property name="arm_pitch" value="0.0"/>
+	<property name="arm_yaw" value="-0.2618"/>
 	<!-- *********************************** -->
 	<!-- kinematic chain reference positions -->

File: cob_hardware_config/cob3-3/urdf/cob3-3.urdf.xacro (robot description, xacro)
@@ -25,8 +25,8 @@
   <xacro:cob_base name="base"/>
   <xacro:cob_torso_v1 name="torso" parent="base_link">
-    <origin xyz="0.155 0 0.892" rpy="1.5708 0 0" />
+    <origin xyz="${torso_x} ${torso_y} ${torso_z}" rpy="${torso_roll} ${torso_pitch} ${torso_yaw}" />
   </xacro:cob_torso_v1>
   <xacro:cob_lbr name="arm" parent="base_link">
-    <origin xyz="-0.015982 -0.080992 0.875995" rpy="0.7854 0.0 -0.2618" />
+    <origin xyz="${arm_x} ${arm_y} ${arm_z}" rpy="${arm_roll} ${arm_pitch} ${arm_yaw}" />
   </xacro:cob_lbr>
   <xacro:cob_head_v3 name="head" parent="torso_upper_neck_tilt_link">
