Commit message: cob3-2 update, calibration and urdf file

File: cob_hardware_config/cob3-2/calibration/calibration.urdf.xacro (robot description, xacro)
@@ -1,3 +1,4 @@
-<?xml version="1.0" ?><robot>
+<?xml version="1.0"?>
+<robot>
 	<!-- ***************** -->
 	<!-- robot calibration -->
@@ -7,5 +8,5 @@
 	<property name="torso_y" value="0.0"/>
 	<property name="torso_z" value="0.892"/>
-	<property name="torso_roll" value="1.5708"/>
+	<property name="torso_roll" value="3.1415926"/>
 	<property name="torso_pitch" value="0.0"/>
 	<property name="torso_yaw" value="0.0"/>
@@ -17,53 +18,44 @@
 	<property name="arm_pitch" value="0.0"/>
 	<property name="arm_yaw" value="-0.2618"/>
-	<!-- *********************************** -->
-	<!-- kinematic chain reference positions -->
-	<!-- *********************************** -->
-	<!-- torso chain calibration_offest! | relative to reference position (see below)-->
-	<!-- not used right now
-	<property name="torso_lower_neck_tilt_cal_offset" value="0.0"/>
-	<property name="torso_pan_cal_offset" value="0.0"/>
-	<property name="torso_upper_neck_tilt_cal_offset" value="0.0"/>
-	-->
-	<!-- torso reference positions | used as calibration_rising for torso chain -->
-	<!-- ! set these values to make torso straight with (0, 0, 0) joint angles ! -->
-	<property name="torso_lower_neck_tilt_ref" value="-0.24501037"/>
-	<property name="torso_pan_ref" value="-0.0146"/>
-	<property name="torso_upper_neck_tilt_ref" value="+0.14419551"/>
-	<!-- tray reference position | used as calibration_rising for tray chain -->
-	<property name="torso_tray_ref" value="3.14"/>
-	<!-- head camera axis reference position | used as calibration_rising for head axis chain -->
-	<property name="head_axis_ref" value="-0.1"/>
-	<!-- arm reference positions | used as calibration_rising for arm chain-->
-	<property name="arm_1_ref" value="0.0"/>
-	<property name="arm_2_ref" value="0.0"/>
-	<property name="arm_3_ref" value="0.0"/>
-	<property name="arm_4_ref" value="0.0"/>
-	<property name="arm_5_ref" value="0.0"/>
-	<property name="arm_6_ref" value="0.0"/>
-	<property name="arm_7_ref" value="0.0"/>
-	<!-- ***************************** -->
+	<!-- common properties -->
+	<property name="M_PI" value="3.1415926535897931" />
+	<!-- torso reference positions -->
+	<property name="torso_lower_neck_pan_ref" value="-0.5470" />
+	<property name="torso_lower_neck_tilt_ref" value="0.0344" />
+	<property name="torso_upper_neck_pan_ref" value="0.0247" />
+	<property name="torso_upper_neck_tilt_ref" value="0.02201" />
+	<!-- tray reference position -->
+	<property name="torso_tray_ref" value="4.1451" />
+	<!-- head camera axis reference position -->
+	<property name="head_axis_ref" value="+3.14" />
+	<!-- arm reference positions -->
+	<property name="arm_1_ref" value="-2.8761" />
+	<property name="arm_2_ref" value="-0.1687" />
+	<property name="arm_3_ref" value="-0.0274" />
+	<property name="arm_4_ref" value="-1.7193" />
+	<property name="arm_5_ref" value="0.0342" />
+	<property name="arm_6_ref" value="-1.6959" />
+	<property name="arm_7_ref" value="1.8707" />
 	<!-- camera calibration properties -->
-	<!-- ***************************** -->
-	<!-- left | handeye calibration | relative to head_axis_link -->
-	<property name="cam_l_x" value="-0.035"/>
-	<property name="cam_l_y" value="-0.0065"/>
-	<property name="cam_l_z" value="-0.06"/>
-	<property name="cam_l_roll" value="0.0"/>
-	<property name="cam_l_pitch" value="-1.5708"/>
-	<property name="cam_l_yaw" value="0.0"/>
-	<!-- right | stereo baseline calibration | relative to left camera -->
-	<property name="cam_r_x" value="0.12"/>
-	<property name="cam_r_y" value="0.0"/>
-	<property name="cam_r_z" value="0.0"/>
-	<property name="cam_r_roll" value="0.0"/>
-	<property name="cam_r_pitch" value="0.0"/>
-	<property name="cam_r_yaw" value="0.0"/>
-	<!-- cam3d | handeye calibration | relative to head_axis_link -->
-	<property name="cam3d_x" value="-0.05"/>
-	<property name="cam3d_y" value="-0.04"/>
-	<property name="cam3d_z" value="-0.01"/>
-	<property name="cam3d_roll" value="0.0"/>
-	<property name="cam3d_pitch" value="-1.5708"/>
-	<property name="cam3d_yaw" value="0.0"/>
+	<!-- hand eye calibration -->
+	<property name="cam_l_x" value="0.0" />
+	<property name="cam_l_y" value="0.0" />
+	<property name="cam_l_z" value="0.0" />
+	<property name="cam_l_roll" value="0.0" />
+	<property name="cam_l_pitch" value="0.0" />
+	<property name="cam_l_yaw" value="0.0" />
+	<!-- right to left calibration -->
+	<property name="cam_r_x" value="0.0" />
+	<property name="cam_r_y" value="0.0" />
+	<property name="cam_r_z" value="0.0" />
+	<property name="cam_r_roll" value="0.0" />
+	<property name="cam_r_pitch" value="0.0" />
+	<property name="cam_r_yaw" value="0.0" />
+	<!-- cam3d to left calibration -->
+	<property name="cam3d_x" value="0.0" />
+	<property name="cam3d_y" value="0.0" />
+	<property name="cam3d_z" value="0.0" />
+	<property name="cam3d_roll" value="0.0" />
+	<property name="cam3d_pitch" value="0.0" />
+	<property name="cam3d_yaw" value="0.0" />
 </robot>

File: cob_hardware_config/cob3-2/calibration/default/calibration.urdf.xacro (robot description, xacro)
@@ -21,14 +21,9 @@
 	<!-- *********************************** -->
 	<!-- torso chain calibration_offest! | relative to reference position (see below)-->
-	<!-- not used right now
-	<property name="torso_lower_neck_tilt_cal_offset" value="0.0"/>
-	<property name="torso_pan_cal_offset" value="0.0"/>
-	<property name="torso_upper_neck_tilt_cal_offset" value="0.0"/>
-	-->
-	<!-- torso reference positions | used as calibration_rising for torso chain -->
-	<!-- ! set these values to make torso straight with (0, 0, 0) joint angles ! -->
-	<property name="torso_lower_neck_tilt_ref" value="-0.24501037"/>
-	<property name="torso_pan_ref" value="-0.0146"/>
-	<property name="torso_upper_neck_tilt_ref" value="+0.14419551"/>
+	<!-- not used right now -->
+	<property name="torso_lower_neck_pan_ref" value="0" />
+	<property name="torso_lower_neck_tilt_ref" value="0" />
+	<property name="torso_upper_neck_pan_ref" value="0" />
+	<property name="torso_upper_neck_tilt_ref" value="0" />
 	<!-- tray reference position | used as calibration_rising for tray chain -->
 	<property name="torso_tray_ref" value="3.14"/>

File: cob_hardware_config/cob3-2/urdf/cob3-2.urdf.xacro (robot description, xacro)
@@ -10,11 +10,10 @@
   <!-- calibration -->
   <include filename="$(find cob_hardware_config)/cob3-2/calibration/calibration.urdf.xacro" />
-  <include filename="$(find cob_description)/calibration/cob3-2.urdf.xacro" />
   <!-- base -->
   <include filename="$(find cob_description)/urdf/base/base.urdf.xacro" />
   <!-- torso -->
-  <include filename="$(find cob_description)/urdf/torso_v1/torso.urdf.xacro" />
+  <include filename="$(find cob_description)/urdf/torso_v0/torso.urdf.xacro" />
   <!-- head -->
-  <include filename="$(find cob_description)/urdf/head_v3/head.urdf.xacro" />
+  <include filename="$(find cob_description)/urdf/head_v2/head.urdf.xacro" />
   <!-- arm -->
   <include filename="$(find cob_description)/urdf/lbr/lbr.urdf.xacro" />
@@ -25,13 +24,13 @@
   <!-- composition of the robot -->
   <xacro:cob_base name="base"/>
-  <xacro:cob_torso_v1 name="torso" parent="base_link">
+  <xacro:cob_torso_v0 name="torso" parent="base_link">
     <origin xyz="${torso_x} ${torso_y} ${torso_z}" rpy="${torso_roll} ${torso_pitch} ${torso_yaw}" />
-  </xacro:cob_torso_v1>
+  </xacro:cob_torso_v0>
   <xacro:cob_lbr name="arm" parent="base_link">
     <origin xyz="${arm_x} ${arm_y} ${arm_z}" rpy="${arm_roll} ${arm_pitch} ${arm_yaw}" />
   </xacro:cob_lbr>
-  <xacro:cob_head_v3 name="head" parent="torso_upper_neck_tilt_link">
-    <origin xyz="0 0.173 0" rpy="0 0 0" />
-  </xacro:cob_head_v3>
+  <xacro:cob_head_v2 name="head" parent="torso_upper_neck_tilt_link">
+    <origin xyz="0 -0.154 0" rpy="3.14159 0 0" />
+  </xacro:cob_head_v2>
   <xacro:schunk_sdh name="sdh" parent="arm_7_link">
     <origin xyz="0 0 0.032" rpy="0 0 1.5708" />

Commit message: cob3-2 with schunk lwa

File: cob_hardware_config/cob3-2/calibration/calibration.urdf.xacro (robot description, xacro)
@@ -12,10 +12,10 @@
 	<property name="torso_yaw" value="0.0"/>
 	<!-- arm mount positions | relative to base_link -->
-	<property name="arm_x" value="-0.015982"/>
-	<property name="arm_y" value="-0.080992"/>
-	<property name="arm_z" value="0.875995"/>
-	<property name="arm_roll" value="0.7854"/>
-	<property name="arm_pitch" value="0.0"/>
-	<property name="arm_yaw" value="-0.2618"/>
+	<property name="arm_x" value="0.040"/>
+	<property name="arm_y" value="-0.005"/>
+	<property name="arm_z" value="0.83637"/>
+	<property name="arm_roll" value="3.1415926"/>
+	<property name="arm_pitch" value="0.7854"/>
+	<property name="arm_yaw" value="-1.8326"/>
 	<!-- common properties -->
 	<property name="M_PI" value="3.1415926535897931" />

File: cob_hardware_config/cob3-2/urdf/cob3-2.urdf.xacro (robot description, xacro)
@@ -17,5 +17,5 @@
   <include filename="$(find cob_description)/urdf/head_v2/head.urdf.xacro" />
   <!-- arm -->
-  <include filename="$(find cob_description)/urdf/lbr/lbr.urdf.xacro" />
+  <include filename="$(find schunk_description)/urdf/lwa/lwa.urdf.xacro" />
   <!-- sdh -->
   <include filename="$(find schunk_description)/urdf/sdh/sdh.urdf.xacro" />
@@ -27,12 +27,12 @@
     <origin xyz="${torso_x} ${torso_y} ${torso_z}" rpy="${torso_roll} ${torso_pitch} ${torso_yaw}" />
   </xacro:cob_torso_v0>
-  <xacro:cob_lbr name="arm" parent="base_link">
+  <xacro:schunk_lwa name="arm" parent="base_link">
     <origin xyz="${arm_x} ${arm_y} ${arm_z}" rpy="${arm_roll} ${arm_pitch} ${arm_yaw}" />
-  </xacro:cob_lbr>
+  </xacro:schunk_lwa>
   <xacro:cob_head_v2 name="head" parent="torso_upper_neck_tilt_link">
     <origin xyz="0 -0.154 0" rpy="3.14159 0 0" />
   </xacro:cob_head_v2>
   <xacro:schunk_sdh name="sdh" parent="arm_7_link">
-    <origin xyz="0 0 0.032" rpy="0 0 1.5708" />
+    <origin xyz="0 0 0" rpy="0 3.1415926 0" />
   </xacro:schunk_sdh>
 </robot>
