Commit message: load new calibration structure for cob3-4

File: cob_hardware_config/cob3-4/urdf/cob3-4.urdf.xacro (robot description, xacro)
@@ -25,14 +25,14 @@
   <xacro:cob_base name="base"/>
   <xacro:cob_torso_v1 name="torso" parent="base_link">
-    <origin xyz="0.155 0 0.892" rpy="1.5708 0 0" />
+    <origin xyz="${torso_x} ${torso_y} ${torso_z}" rpy="${torso_roll} ${torso_pitch} ${torso_yaw}" />
   </xacro:cob_torso_v1>
   <xacro:cob_lbr name="arm" parent="base_link">
-    <origin xyz="-0.015982 -0.080992 0.875995" rpy="0.7854 0.0 -0.2618" />
+    <origin xyz="${arm_x} ${arm_y} ${arm_z}" rpy="${arm_roll} ${arm_pitch} ${arm_yaw}" />
   </xacro:cob_lbr>
   <xacro:cob_head_v3 name="head" parent="torso_upper_neck_tilt_link">
-    <origin xyz="0 0.154 0" rpy="0 0 0" />
+    <origin xyz="0 0.173 0" rpy="0 0 0" />
   </xacro:cob_head_v3>
   <xacro:schunk_sdh name="sdh" parent="arm_7_link">
-    <origin xyz="0 0 0.02" rpy="0 0 1.5708" />
+    <origin xyz="0 0 0.032" rpy="0 0 1.5708" />
   </xacro:schunk_sdh>
 </robot>
