Commit message: urdf structure change: tray can be calibrated now

File: cob_hardware_config/cob3-1/calibration/calibration.urdf.xacro (robot description, xacro)
@@ -25,7 +25,14 @@
 	<property name="laser_top_pitch" value="0"/>
 	<property name="laser_top_yaw" value="0"/>
-	<!-- ***************** -->
-	<!-- robot calibration -->
-	<!-- ***************** -->
+	<!-- *********************** -->
+	<!-- upper robot calibration -->
+	<!-- *********************** -->
+	<!-- tray mount positions | relative to base_link -->"0.2406 0.1900 0.7320" rpy="2.3561 0 0" />
+	<property name="tray_x" value="0.2406"/>
+	<property name="tray_y" value="0.1900"/>
+	<property name="tray_z" value="0.7320"/>
+	<property name="tray_roll" value="2.3561"/>
+	<property name="tray_pitch" value="0"/>
+	<property name="tray_yaw" value="0"/>
 	<!-- torso mount positions | relative to base_link -->
 	<property name="torso_x" value="0.1523087993"/>
@@ -51,4 +58,6 @@
 	<property name="torso_upper_neck_tilt_cal_offset" value="0.0"/>
 	-->
+	<!-- torso reference positions | used as calibration_rising for torso chain -->
+	<!-- ! set these values to make torso straight with (0, 0, 0) joint angles ! -->
 	<property name="torso_lower_neck_pan_ref" value="-0.5470" />
 	<property name="torso_lower_neck_tilt_ref" value="0.0344" />
@@ -56,5 +65,5 @@
 	<property name="torso_upper_neck_tilt_ref" value="0.02201" />
 	<!-- tray reference position | used as calibration_rising for tray chain -->
-	<property name="torso_tray_ref" value="-0.2"/>
+	<property name="tray_ref" value="-0.2"/>
 	<!-- head camera axis reference position | used as calibration_rising for head axis chain -->
 	<property name="head_axis_ref" value="-0.1"/>

File: cob_hardware_config/cob3-1/urdf/cob3-1.urdf.xacro (robot description, xacro)
@@ -12,4 +12,6 @@
   <!-- base -->
   <include filename="$(find cob_description)/urdf/base/base.urdf.xacro" />
+  <!-- tray -->
+  <include filename="$(find cob_description)/urdf/tray/tray.urdf.xacro" />
   <!-- torso -->
   <include filename="$(find cob_description)/urdf/torso_v0/torso.urdf.xacro" />
@@ -24,5 +26,8 @@
   <!-- composition of the robot -->
   <xacro:cob_base name="base"/>
-  <xacro:cob_torso_v0 name="torso" parent="base_link">
+  <xacro:cob_tray name="tray" parent="base_link">
+    <origin xyz="${tray_x} ${tray_y} ${tray_z}" rpy="${tray_roll} ${tray_pitch} ${tray_yaw}" />
+  </xacro:cob_tray>
+  <xacro:cob_torso_v1 name="torso" parent="base_link">
     <origin xyz="${torso_x} ${torso_y} ${torso_z}" rpy="${torso_roll} ${torso_pitch} ${torso_yaw}" />
   </xacro:cob_torso_v0>

File: cob_hardware_config/cob3-2/calibration/calibration.urdf.xacro (robot description, xacro)
@@ -25,7 +25,14 @@
 	<property name="laser_top_pitch" value="0"/>
 	<property name="laser_top_yaw" value="0"/>
-	<!-- ***************** -->
-	<!-- robot calibration -->
-	<!-- ***************** -->
+	<!-- *********************** -->
+	<!-- upper robot calibration -->
+	<!-- *********************** -->
+	<!-- tray mount positions | relative to base_link -->"0.2406 0.1900 0.7320" rpy="2.3561 0 0" />
+	<property name="tray_x" value="0.2406"/>
+	<property name="tray_y" value="0.1900"/>
+	<property name="tray_z" value="0.7320"/>
+	<property name="tray_roll" value="2.3561"/>
+	<property name="tray_pitch" value="0"/>
+	<property name="tray_yaw" value="0"/>
 	<!-- torso mount positions | relative to base_link -->
 	<property name="torso_x" value="0.155"/>
@@ -59,5 +66,5 @@
 	<property name="torso_upper_neck_tilt_ref" value="0.02201" />
 	<!-- tray reference position | used as calibration_rising for tray chain -->
-	<property name="torso_tray_ref" value="4.1451" />
+	<property name="tray_ref" value="4.1451" />
 	<!-- head camera axis reference position | used as calibration_rising for head axis chain -->
 	<property name="head_axis_ref" value="+3.14" />

File: cob_hardware_config/cob3-2/calibration/default/calibration.urdf.xacro (robot description, xacro)
@@ -27,5 +27,5 @@
 	<property name="torso_upper_neck_tilt_ref" value="0" />
 	<!-- tray reference position | used as calibration_rising for tray chain -->
-	<property name="torso_tray_ref" value="3.14"/>
+	<property name="tray_ref" value="3.14"/>
 	<!-- head camera axis reference position | used as calibration_rising for head axis chain -->
 	<property name="head_axis_ref" value="-0.1"/>

File: cob_hardware_config/cob3-2/urdf/cob3-2.urdf.xacro (robot description, xacro)
@@ -12,4 +12,6 @@
   <!-- base -->
   <include filename="$(find cob_description)/urdf/base/base.urdf.xacro" />
+  <!-- tray -->
+  <include filename="$(find cob_description)/urdf/tray/tray.urdf.xacro" />
   <!-- torso -->
   <include filename="$(find cob_description)/urdf/torso_v0/torso.urdf.xacro" />
@@ -24,5 +26,8 @@
   <!-- composition of the robot -->
   <xacro:cob_base name="base"/>
-  <xacro:cob_torso_v0 name="torso" parent="base_link">
+  <xacro:cob_tray name="tray" parent="base_link">
+    <origin xyz="${tray_x} ${tray_y} ${tray_z}" rpy="${tray_roll} ${tray_pitch} ${tray_yaw}" />
+  </xacro:cob_tray>
+  <xacro:cob_torso_v1 name="torso" parent="base_link">
     <origin xyz="${torso_x} ${torso_y} ${torso_z}" rpy="${torso_roll} ${torso_pitch} ${torso_yaw}" />
   </xacro:cob_torso_v0>

File: cob_hardware_config/cob3-3/calibration/calibration.urdf.xacro (robot description, xacro)
@@ -25,7 +25,14 @@
 	<property name="laser_top_pitch" value="0"/>
 	<property name="laser_top_yaw" value="0"/>
-	<!-- ***************** -->
-	<!-- robot calibration -->
-	<!-- ***************** -->
+	<!-- *********************** -->
+	<!-- upper robot calibration -->
+	<!-- *********************** -->
+	<!-- tray mount positions | relative to base_link -->"0.2406 0.1900 0.7320" rpy="2.3561 0 0" />
+	<property name="tray_x" value="0.2406"/>
+	<property name="tray_y" value="0.1900"/>
+	<property name="tray_z" value="0.7320"/>
+	<property name="tray_roll" value="2.3561"/>
+	<property name="tray_pitch" value="0"/>
+	<property name="tray_yaw" value="0"/>
 	<!-- torso mount positions | relative to base_link -->
 	<property name="torso_x" value="0.1523087993"/>
@@ -57,5 +64,5 @@
 	<property name="torso_upper_neck_tilt_ref" value="9.81040327"/>
 	<!-- tray reference position | used as calibration_rising for tray chain -->
-	<property name="torso_tray_ref" value="-0.2"/>
+	<property name="tray_ref" value="-0.2"/>
 	<!-- head camera axis reference position | used as calibration_rising for head axis chain -->
 	<property name="head_axis_ref" value="-0.1"/>

File: cob_hardware_config/cob3-3/calibration/default/calibration.urdf.xacro (robot description, xacro)
@@ -32,5 +32,5 @@
 	<property name="torso_upper_neck_tilt_ref" value="+0.14419551"/>
 	<!-- tray reference position | used as calibration_rising for tray chain -->
-	<property name="torso_tray_ref" value="3.14"/>
+	<property name="tray_ref" value="3.14"/>
 	<!-- head camera axis reference position | used as calibration_rising for head axis chain -->
 	<property name="head_axis_ref" value="-0.1"/>

File: cob_hardware_config/cob3-3/urdf/cob3-3.urdf.xacro (robot description, xacro)
@@ -12,4 +12,6 @@
   <!-- base -->
   <include filename="$(find cob_description)/urdf/base/base.urdf.xacro" />
+  <!-- tray -->
+  <include filename="$(find cob_description)/urdf/tray/tray.urdf.xacro" />
   <!-- torso -->
   <include filename="$(find cob_description)/urdf/torso_v1/torso.urdf.xacro" />
@@ -24,4 +26,7 @@
   <!-- composition of the robot -->
   <xacro:cob_base name="base"/>
+  <xacro:cob_tray name="tray" parent="base_link">
+    <origin xyz="${tray_x} ${tray_y} ${tray_z}" rpy="${tray_roll} ${tray_pitch} ${tray_yaw}" />
+  </xacro:cob_tray>
   <xacro:cob_torso_v1 name="torso" parent="base_link">
     <origin xyz="${torso_x} ${torso_y} ${torso_z}" rpy="${torso_roll} ${torso_pitch} ${torso_yaw}" />

File: cob_hardware_config/cob3-4/calibration/calibration.urdf.xacro (robot description, xacro)
@@ -25,7 +25,14 @@
 	<property name="laser_top_pitch" value="0"/>
 	<property name="laser_top_yaw" value="0"/>
-	<!-- ***************** -->
-	<!-- robot calibration -->
-	<!-- ***************** -->
+	<!-- *********************** -->
+	<!-- upper robot calibration -->
+	<!-- *********************** -->
+	<!-- tray mount positions | relative to base_link -->"0.2406 0.1900 0.7320" rpy="2.3561 0 0" />
+	<property name="tray_x" value="0.2406"/>
+	<property name="tray_y" value="0.1900"/>
+	<property name="tray_z" value="0.7320"/>
+	<property name="tray_roll" value="2.3561"/>
+	<property name="tray_pitch" value="0"/>
+	<property name="tray_yaw" value="0"/>
 	<!-- torso mount positions | relative to base_link -->
 	<property name="torso_x" value="0.1535525935"/>
@@ -57,5 +64,5 @@
 	<property name="torso_upper_neck_tilt_ref" value="+0.14419551"/>
 	<!-- tray reference position | used as calibration_rising for tray chain -->
-	<property name="torso_tray_ref" value="-0.2"/>
+	<property name="tray_ref" value="-0.2"/>
 	<!-- head camera axis reference position | used as calibration_rising for head axis chain -->
 	<property name="head_axis_ref" value="-0.1"/>

File: cob_hardware_config/cob3-4/urdf/cob3-4.urdf.xacro (robot description, xacro)
@@ -12,4 +12,6 @@
   <!-- base -->
   <include filename="$(find cob_description)/urdf/base/base.urdf.xacro" />
+  <!-- tray -->
+  <include filename="$(find cob_description)/urdf/tray/tray.urdf.xacro" />
   <!-- torso -->
   <include filename="$(find cob_description)/urdf/torso_v1/torso.urdf.xacro" />
@@ -24,4 +26,7 @@
   <!-- composition of the robot -->
   <xacro:cob_base name="base"/>
+  <xacro:cob_tray name="tray" parent="base_link">
+    <origin xyz="${tray_x} ${tray_y} ${tray_z}" rpy="${tray_roll} ${tray_pitch} ${tray_yaw}" />
+  </xacro:cob_tray>
   <xacro:cob_torso_v1 name="torso" parent="base_link">
     <origin xyz="${torso_x} ${torso_y} ${torso_z}" rpy="${torso_roll} ${torso_pitch} ${torso_yaw}" />
