Commit message: almost final raw3-1 hardware setup

File: cob_hardware_config/raw3-1/calibration/calibration.urdf.xacro (robot description, xacro)
@@ -10,3 +10,6 @@
 	<property name="arm_4_ref" value="0" />
 	<property name="arm_5_ref" value="0" />
+        <property name="torso_lower_neck_tilt_ref" value="0.1"/>
+        <property name="torso_pan_ref" value="0.0"/>
+        <property name="torso_upper_neck_tilt_ref" value="0.0"/>
 </robot>

File: cob_hardware_config/raw3-1/urdf/raw3-1.urdf.xacro (robot description, xacro)
@@ -14,4 +14,6 @@
   <!-- generic simulator_gazebo plugins for starting mechanism control, ros time, ros battery -->
   <include filename="$(find cob_description)/gazebo/gazebo.urdf.xacro" />
+  <!-- torso -->
+  <include filename="$(find raw_description)/urdf/torso/torso.urdf.xacro" />
   <!-- ur_arm -->
  <!--include filename="$(find raw_description)/urdf/arm_ur/arm.urdf.xacro" /-->
@@ -22,7 +24,10 @@
     <origin xyz="0.62 0.00 0.88" rpy="0 0 0" />
   </xacro:frida-->
+  <xacro:cob_torso_v1 name="torso" parent="base_link">
+    <origin xyz="0 0 1.0" rpy="0 0 0" />
+  </xacro:cob_torso_v1>
   <xacro:ur5_robot prefix="arm_"/>
   <joint name="arm_base_joint" type="fixed" >
-		 <origin xyz="0.32 0.03 0.48" rpy="0 0 -0.79" />
+		 <origin xyz="0.3235 -0.191 0.58" rpy="0 0 -0.79" />
 		<parent link="base_link" />
 		<child link="arm_base_link" />

Commit message: small modifications for raw

File: cob_hardware_config/raw3-1/calibration/calibration.urdf.xacro (robot description, xacro)
@@ -13,3 +13,27 @@
         <property name="torso_pan_ref" value="0.0"/>
         <property name="torso_upper_neck_tilt_ref" value="0.0"/>
+	<!-- ***************************** -->
+	<!-- camera calibration properties -->
+	<!-- ***************************** -->
+	<!-- left | handeye calibration | relative to head_axis_link -->
+	<property name="cam_l_x" value="-0.0171250371"/>
+	<property name="cam_l_y" value="-0.0389120491"/>
+	<property name="cam_l_z" value="-0.12027305"/>
+	<property name="cam_l_roll" value="2.149627771"/>
+	<property name="cam_l_pitch" value="-1.5608998734"/>
+	<property name="cam_l_yaw" value="-2.2074792588"/>
+	<!-- right | stereo baseline calibration | relative to left camera -->
+	<property name="cam_r_x" value="0.121342166993"/>
+	<property name="cam_r_y" value="0.000964077625598"/>
+	<property name="cam_r_z" value="-0.00119322781437"/>
+	<property name="cam_r_roll" value="0.004726030387"/>
+	<property name="cam_r_pitch" value="0.0169849756686"/>
+	<property name="cam_r_yaw" value="0.0118232483039"/>
+	<!-- cam3d | handeye calibration | relative to head_axis_link -->
+	<property name="cam3d_x" value="-0.0392332921"/>
+	<property name="cam3d_y" value="-0.0725275279"/>
+	<property name="cam3d_z" value="-0.041924241"/>
+	<property name="cam3d_roll" value="0.0974172003"/>
+	<property name="cam3d_pitch" value="-1.5456482961"/>
+	<property name="cam3d_yaw" value="-0.1128148583"/>
 </robot>

File: cob_hardware_config/raw3-1/urdf/raw3-1.urdf.xacro (robot description, xacro)
@@ -25,5 +25,5 @@
   </xacro:frida-->
   <xacro:cob_torso_v1 name="torso" parent="base_link">
-    <origin xyz="0 0 1.0" rpy="0 0 0" />
+    <origin xyz="0.166 0.2175 0.5405" rpy="0 0 0" />
   </xacro:cob_torso_v1>
   <xacro:ur5_robot prefix="arm_"/>
