Commit message: add controllers for cob3-6

File: cob_hardware_config/cob3-6/calibration/calibration.urdf.xacro (robot description, xacro)
@@ -43,10 +43,10 @@
 	<property name="torso_yaw" value="0.0660275925"/>
 	<!-- arm mount positions | relative to base_link -->
-	<property name="arm_x" value="-0.0135247781"/>
-	<property name="arm_y" value="-0.0461165405"/>
-	<property name="arm_z" value="0.8737003446"/>
-	<property name="arm_roll" value="0.8188441679"/>
-	<property name="arm_pitch" value="0.0073986966"/>
-	<property name="arm_yaw" value="-0.2545901695"/>
+	<property name="arm_x" value="0.040"/>
+	<property name="arm_y" value="-0.005"/>
+	<property name="arm_z" value="0.83637"/>
+	<property name="arm_roll" value="3.1415926"/>
+	<property name="arm_pitch" value="0.7854"/>
+	<property name="arm_yaw" value="-1.8326"/>
 	<!-- *********************************** -->
 	<!-- kinematic chain reference positions -->

File: cob_hardware_config/cob3-6/urdf/cob3-6.urdf.xacro (robot description, xacro)
@@ -4,5 +4,5 @@
        xmlns:interface="http://playerstage.sourceforge.net/gazebo/xmlschema/#interface"
        xmlns:xacro="http://playerstage.sourceforge.net/gazebo/xmlschema/#interface"
-       name="cob3_4" >
+       name="cob3_6" >
   <!-- common stuff -->
   <include filename="$(find cob_description)/urdf/common.xacro" />
@@ -39,5 +39,5 @@
   </xacro:cob_head_v3>
   <xacro:schunk_sdh name="sdh" parent="arm_7_link">
-    <origin xyz="0 0 0.032" rpy="0 0 1.5708" />
+    <origin xyz="0 0 0" rpy="0 3.1415926 0" />
   </xacro:schunk_sdh>
 </robot>
