Commit message: new tower description

File: cob_hardware_config/raw3-6/urdf/raw3-6.urdf.xacro (robot description, xacro)
@@ -4,5 +4,5 @@
        xmlns:interface="http://playerstage.sourceforge.net/gazebo/xmlschema/#interface"
        xmlns:xacro="http://playerstage.sourceforge.net/gazebo/xmlschema/#interface"
-       name="raw3-1" >
+       name="raw3-6" >
   <!-- common stuff -->
   <include filename="$(find cob_description)/urdf/common.xacro" />
@@ -10,7 +10,12 @@
   <include filename="$(find cob_calibration_data)/raw3-6/calibration/calibration.urdf.xacro" />
   <!-- raw base -->
-  <include filename="$(find raw_description)/urdf/base/base.urdf.xacro" />
+  <include filename="$(find raw_description)/urdf/base_long/base.urdf.xacro" />
+  <!-- raw tower -->
+  <include filename="$(find raw_description)/urdf/tower_symetric/tower.urdf.xacro" />
   <!-- generic simulator_gazebo plugins for starting mechanism control, ros time, ros battery -->
   <include filename="$(find cob_description)/gazebo/gazebo.urdf.xacro" />
-  <xacro:raw_base name="base"/>	<!--with new collision_model, but no platform_controller available yet-->
+  <xacro:raw_base name="base"/>	<!--with new collision_model-->
+  <xacro:tower_symetric name="tower" parent="base_link">
+    <origin xyz="0.361 0.0 0.306"/>
+  </xacro:tower_symetric>
   </robot>
