Commit message: change desire arm_left and arm_right

File: cob_hardware_config/desire/urdf/desire.urdf.xacro (robot description, xacro)
@@ -31,9 +31,8 @@
   <xacro:desire_base name="base"/>
   <xacro:cob_lbr name="arm_left" parent="base_link">
-    <!--origin xyz="0.35 0.0 1.25239" rpy="3.1415926 0.7854 -1.8326" /-->
-    <origin xyz="0.3 -0.2 1.36" rpy="0.82 0 0" />
+    <origin xyz="0.3 0.2 1.36" rpy="-0.82 0 0" />
   </xacro:cob_lbr>
   <xacro:cob_lbr name="arm_right" parent="base_link">
-    <origin xyz="0.3 0.2 1.36" rpy="-0.82 0 0" />
+    <origin xyz="0.3 -0.2 1.36" rpy="0.82 0 0" />
   </xacro:cob_lbr>
   <xacro:head_desire name="head" parent="base_link">

Commit message: replace all hardcoded mounting values with respective macros in cob_calibration_data

File: cob_hardware_config/desire/urdf/desire.urdf.xacro (robot description, xacro)
@@ -32,17 +32,17 @@
   <xacro:desire_base name="base"/>
   <xacro:cob_lbr name="arm_left" parent="base_link">
-    <origin xyz="0.3 0.2 1.36" rpy="-0.82 0 0" />
+    <origin xyz="${arm_left_x} ${arm_left_y} ${arm_left_z}" rpy="${arm_left_roll} ${arm_left_pitch} ${arm_left_yaw}" />
   </xacro:cob_lbr>
   <xacro:cob_lbr name="arm_right" parent="base_link">
-    <origin xyz="0.3 -0.2 1.36" rpy="0.82 0 0" />
+    <origin xyz="${arm_right_x} ${arm_right_y} ${arm_right_z}" rpy="${arm_right_roll} ${arm_right_pitch} ${arm_right_yaw}" />
   </xacro:cob_lbr>
   <xacro:head_desire name="head" parent="base_link">
-    <origin xyz="0.40 0 1.4246" rpy="3.14159 0 0" />
+    <origin xyz="${head_x} ${head_y} ${head_z}" rpy="${head_roll} ${head_pitch} ${head_yaw}" />
   </xacro:head_desire>
   <xacro:schunk_sdh name="sdh_left" parent="arm_left_7_link">
-    <origin xyz="0 0 0.032" rpy="0 0 1.5708" />
+    <origin xyz="${sdh_left_x} ${sdh_left_y} ${sdh_left_z}" rpy="${sdh_left_roll} ${sdh_left_pitch} ${sdh_left_yaw}" />
   </xacro:schunk_sdh>
   <xacro:schunk_sdh name="sdh_right" parent="arm_right_7_link">
-    <origin xyz="0 0 0.032" rpy="0 0 1.5708" />
+    <origin xyz="${sdh_right_x} ${sdh_right_y} ${sdh_right_z}" rpy="${sdh_right_roll} ${sdh_right_pitch} ${sdh_right_yaw}" />
   </xacro:schunk_sdh>
 </robot>

File: cob_hardware_config/raw3-1/urdf/raw3-1.urdf.xacro (robot description, xacro)
@@ -18,26 +18,14 @@
   <include filename="$(find raw_description)/urdf/torso/torso.urdf.xacro" />
   <!-- ur_arm -->
-  <include filename="$(find ur10_description)/urdf/model.urdf.xacro" />
+  <include filename="$(find raw_description)/urdf/ur_arm/ur10_arm.urdf.xacro" />
   <xacro:raw_base name="base"/>	<!--with new collision_model, but no platform_controller available yet-->
-  <xacro:macro name="ur_arm_base_joint" >
-  <joint name="arm_base_joint" type="fixed" >
-    <origin xyz="${arm_x} ${arm_y} ${arm_z}" rpy="${arm_roll} ${arm_roll} ${arm_yaw}" />
-    <parent link="base_link" />
-    <child link="arm_base_link" />
-  </joint>
-  </xacro:macro>
- <xacro:ur_arm_base_joint/>
- <xacro:ur10_robot prefix="arm_"/>
+  <xacro:cob_ur10 name="arm" parent="base_link">
+      <origin xyz="${arm_x} ${arm_y} ${arm_z}" rpy="${arm_roll} ${arm_pitch} ${arm_yaw}" />
+  </xacro:cob_ur10>
   <xacro:raw_torso name="torso" parent="base_link">
       <origin xyz="${torso_x} ${torso_y} ${torso_z}" rpy="${torso_roll} ${torso_pitch} ${torso_yaw}" />
   </xacro:raw_torso>
-  <!--link name="arm_ee_link"/-->
-  <!--joint name ="arm_ee_joint" type="fixed">
-	  <origin xyz="0.0 0.090 0" rpy="-1.570796 0 0" />
-	  <parent link="arm_wrist_3_link" />
-	  <child link="arm_ee_link" />
-  </joint-->
   <xacro:raw_boxgripper name="gripper" parent="arm_ee_link">
-	<origin xyz="0.00 0.0 0.0" rpy="0 0 0" />
+      <origin xyz="${gripper_x} ${gripper_y} ${gripper_z}" rpy="${gripper_roll} ${gripper_pitch} ${gripper_yaw}" />
   </xacro:raw_boxgripper>
   </robot>

File: cob_hardware_config/raw3-2/urdf/raw3-2.urdf.xacro (robot description, xacro)
@@ -4,11 +4,9 @@
        xmlns:interface="http://playerstage.sourceforge.net/gazebo/xmlschema/#interface"
        xmlns:xacro="http://playerstage.sourceforge.net/gazebo/xmlschema/#interface"
-       name="icob" >
+       name="raw3-2" >
   <!-- common stuff -->
   <include filename="$(find cob_description)/urdf/common.xacro" />
   <include filename="$(find cob_description)/urdf/materials.urdf.xacro" />
   <include filename="$(find cob_calibration_data)/raw3-2/calibration/calibration.urdf.xacro" />
-  <!-- icob base -->
-  <!--include filename="$(find icob_description)/ros/urdf/base_v1/base.urdf.xacro" /-->	<!-- fxm: old	-->
   <include filename="$(find raw_description)/urdf/base/base.urdf.xacro" />
   <!-- generic simulator_gazebo plugins for starting mechanism control, ros time, ros battery -->

File: cob_hardware_config/raw3-3/urdf/raw3-3.urdf.xacro (robot description, xacro)
@@ -21,15 +21,15 @@
   <xacro:raw_base name="base"/>	<!--with new collision_model, but no platform_controller available yet-->
   <xacro:tower_symetric name="tower" parent="base_link">
-    <origin xyz="0.221 0.0 0.306"/>
+      <origin xyz="${tower_x} ${tower_y} ${tower_z}" rpy="${tower_roll} ${tower_pitch} ${tower_yaw}" />
   </xacro:tower_symetric>
-  <xacro:frida parent="base_link" name="arm">
-    <origin xyz="0.24 0.0 0.48" rpy="0 0 0" />
+  <xacro:frida name="arm" parent="base_link">
+      <origin xyz="${arm_x} ${arm_y} ${arm_z}" rpy="${arm_roll} ${arm_pitch} ${arm_yaw}" />
   </xacro:frida>
  <!--
   <xacro:prace_gripper name="gripper_left" parent="arm_left_7_link">
-    <origin xyz="0.0 0.0 0.0561" rpy="0 0 0" />
+      <origin xyz="${gripper_left_x} ${gripper_left_y} ${gripper_left_z}" rpy="${gripper_left_roll} ${gripper_left_pitch} ${gripper_left_yaw}" />
   </xacro:prace_gripper>
   <xacro:prace_gripper name="gripper_right" parent="arm_right_7_link">
-    <origin xyz="0.0 0.0 0.0561" rpy="0 0 0" />
+      <origin xyz="${gripper_right_x} ${gripper_right_y} ${gripper_right_z}" rpy="${gripper_right_roll} ${gripper_right_pitch} ${gripper_right_yaw}" />
   </xacro:prace_gripper>
 -->

File: cob_hardware_config/raw3-4/urdf/raw3-4.urdf.xacro (robot description, xacro)
@@ -4,11 +4,9 @@
        xmlns:interface="http://playerstage.sourceforge.net/gazebo/xmlschema/#interface"
        xmlns:xacro="http://playerstage.sourceforge.net/gazebo/xmlschema/#interface"
-       name="icob" >
+       name="raw3-4" >
   <!-- common stuff -->
   <include filename="$(find cob_description)/urdf/common.xacro" />
   <include filename="$(find cob_description)/urdf/materials.urdf.xacro" />
   <include filename="$(find cob_calibration_data)/raw3-4/calibration/calibration.urdf.xacro" />
-  <!-- icob base -->
-  <!--include filename="$(find icob_description)/ros/urdf/base_v1/base.urdf.xacro" /-->	<!-- fxm: old	-->
   <include filename="$(find raw_description)/urdf/base/base.urdf.xacro" />
   <!-- generic simulator_gazebo plugins for starting mechanism control, ros time, ros battery -->

File: cob_hardware_config/raw3-5/urdf/raw3-5.urdf.xacro (robot description, xacro)
@@ -4,5 +4,5 @@
        xmlns:interface="http://playerstage.sourceforge.net/gazebo/xmlschema/#interface"
        xmlns:xacro="http://playerstage.sourceforge.net/gazebo/xmlschema/#interface"
-       name="icob" >
+       name="raw3-5" >
   <!-- common stuff -->
   <include filename="$(find cob_description)/urdf/common.xacro" />

File: cob_hardware_config/raw3-6/urdf/raw3-6.urdf.xacro (robot description, xacro)
@@ -17,5 +17,5 @@
   <xacro:raw_base name="base"/>	<!--with new collision_model-->
   <xacro:tower_symetric name="tower" parent="base_link">
-    <origin xyz="0.361 0.0 0.306"/>
+      <origin xyz="${tower_x} ${tower_y} ${tower_z}" rpy="${tower_roll} ${tower_pitch} ${tower_yaw}" />
   </xacro:tower_symetric>
   </robot>
