Commit message: tosro urdf change: moved head axis up (as in cad)

File: cob_hardware_config/cob3-3/urdf/cob3-3.urdf.xacro (robot description, xacro)
@@ -31,5 +31,5 @@
   </xacro:cob_lbr>
   <xacro:cob_head_v3 name="head" parent="torso_upper_neck_tilt_link">
-    <origin xyz="0 0.154 0" rpy="0 0 0" />
+    <origin xyz="0 0.173 0" rpy="0 0 0" />
   </xacro:cob_head_v3>
   <xacro:schunk_sdh name="sdh" parent="arm_7_link">

Commit message: moved sdh up by 1.2cm to correct mount position

File: cob_hardware_config/cob3-3/urdf/cob3-3.urdf.xacro (robot description, xacro)
@@ -34,5 +34,5 @@
   </xacro:cob_head_v3>
   <xacro:schunk_sdh name="sdh" parent="arm_7_link">
-    <origin xyz="0 0 0.02" rpy="0 0 1.5708" />
+    <origin xyz="0 0 0.032" rpy="0 0 1.5708" />
   </xacro:schunk_sdh>
 </robot>

Commit message: add tests for cob3-5

File: cob_hardware_config/cob3-3/urdf/cob3-3.urdf.xacro (robot description, xacro)
@@ -39,5 +39,5 @@
   </xacro:cob_head_v3>
   <xacro:schunk_sdh name="sdh" parent="arm_7_link">
-    <origin xyz="0 0 0.032" rpy="0 0 1.5708" />
+    <origin xyz="0 0 0.032" rpy="0 0 ${M_PI/2}" />
   </xacro:schunk_sdh>
 </robot>

File: cob_hardware_config/cob3-6/urdf/cob3-6.urdf.xacro (robot description, xacro)
@@ -39,5 +39,5 @@
   </xacro:cob_head_v3>
   <xacro:schunk_sdh name="sdh" parent="arm_7_link">
-    <origin xyz="0 0 0" rpy="0 3.1415926 0" />
+    <origin xyz="0 0 0" rpy="0 ${M_PI} 0" />
   </xacro:schunk_sdh>
 </robot>

Commit message: fixed direction of translation for head link. due to last commit

File: cob_hardware_config/cob3-3/urdf/cob3-3.urdf.xacro (robot description, xacro)
@@ -36,5 +36,5 @@
   </xacro:cob_lbr>
   <xacro:cob_head_v3 name="head" parent="head_cover_link">
-    <origin xyz="0 0.173 0" rpy="0 0 0" />
+    <origin xyz="0 -0.173 0" rpy="0 0 0" />
   </xacro:cob_head_v3>
   <xacro:schunk_sdh name="sdh" parent="arm_7_link">

File: cob_hardware_config/cob3-6/urdf/cob3-6.urdf.xacro (robot description, xacro)
@@ -36,5 +36,5 @@
   </xacro:schunk_lwa>
   <xacro:cob_head_v3 name="head" parent="head_cover_link">
-    <origin xyz="0 0.173 0" rpy="0 0 0" />
+    <origin xyz="0 -0.173 0" rpy="0 0 0" />
   </xacro:cob_head_v3>
   <xacro:schunk_sdh name="sdh" parent="arm_7_link">

Commit message: head mount calibration

File: cob_hardware_config/cob3-3/urdf/cob3-3.urdf.xacro (robot description, xacro)
@@ -36,5 +36,5 @@
   </xacro:cob_lbr>
   <xacro:cob_head_v3 name="head" parent="head_cover_link">
-    <origin xyz="0 -0.173 0" rpy="0 0 0" />
+    <origin xyz="${head_x} ${head_y} ${head_z}" rpy="${head_roll} ${head_pitch} ${head_yaw}" />
   </xacro:cob_head_v3>
   <xacro:schunk_sdh name="sdh" parent="arm_7_link">

File: cob_hardware_config/cob3-5/urdf/cob3-5.urdf.xacro (robot description, xacro)
@@ -35,6 +35,6 @@
     <origin xyz="${arm_x} ${arm_y} ${arm_z}" rpy="${arm_roll} ${arm_pitch} ${arm_yaw}" />
   </xacro:schunk_lwa>
-  <xacro:cob_head_v3 name="head" parent="torso_upper_neck_tilt_link">
-    <origin xyz="0 0.173 0" rpy="0 0 0" />
+  <xacro:cob_head_v3 name="head" parent="head_cover_link">
+    <origin xyz="${head_x} ${head_y} ${head_z}" rpy="${head_roll} ${head_pitch} ${head_yaw}" />
   </xacro:cob_head_v3>
   <xacro:schunk_sdh name="sdh" parent="arm_7_link">

Commit message: new reference for head due to change in cob_common

File: cob_hardware_config/cob3-3/urdf/cob3-3.urdf.xacro (robot description, xacro)
@@ -35,5 +35,5 @@
     <origin xyz="${arm_x} ${arm_y} ${arm_z}" rpy="${arm_roll} ${arm_pitch} ${arm_yaw}" />
   </xacro:cob_lbr>
-  <xacro:cob_head_v3 name="head" parent="head_cover_link">
+  <xacro:cob_head_v3 name="head" parent="torso_upper_neck_tilt_link">
     <origin xyz="${head_x} ${head_y} ${head_z}" rpy="${head_roll} ${head_pitch} ${head_yaw}" />
   </xacro:cob_head_v3>

File: cob_hardware_config/cob3-5/urdf/cob3-5.urdf.xacro (robot description, xacro)
@@ -35,5 +35,5 @@
     <origin xyz="${arm_x} ${arm_y} ${arm_z}" rpy="${arm_roll} ${arm_pitch} ${arm_yaw}" />
   </xacro:schunk_lwa>
-  <xacro:cob_head_v3 name="head" parent="head_cover_link">
+  <xacro:cob_head_v3 name="head" parent="torso_upper_neck_tilt_link">
     <origin xyz="${head_x} ${head_y} ${head_z}" rpy="${head_roll} ${head_pitch} ${head_yaw}" />
   </xacro:cob_head_v3>

File: cob_hardware_config/cob3-6/urdf/cob3-6.urdf.xacro (robot description, xacro)
@@ -35,6 +35,6 @@
     <origin xyz="${arm_x} ${arm_y} ${arm_z}" rpy="${arm_roll} ${arm_pitch} ${arm_yaw}" />
   </xacro:schunk_lwa>
-  <xacro:cob_head_v3 name="head" parent="head_cover_link">
-    <origin xyz="0 -0.173 0" rpy="0 0 0" />
+  <xacro:cob_head_v3 name="head" parent="torso_upper_neck_tilt_link">
+    <origin xyz="0 0.173 0" rpy="0 0 0" />
   </xacro:cob_head_v3>
   <xacro:schunk_sdh name="sdh" parent="arm_7_link">

Commit message: add lookat component to cob3-3

File: cob_hardware_config/cob3-3/urdf/cob3-3.urdf.xacro (robot description, xacro)
@@ -19,4 +19,5 @@
   <!-- head -->
   <include filename="$(find cob_description)/urdf/head_v3/head.urdf.xacro" />
+  <include filename="$(find cob_description)/urdf/lookat/lookat.urdf.xacro" />
   <!-- arm -->
   <include filename="$(find cob_description)/urdf/lbr/lbr.urdf.xacro" />
@@ -39,4 +40,8 @@
     <origin xyz="${head_x} ${head_y} ${head_z}" rpy="${head_roll} ${head_pitch} ${head_yaw}" />
   </xacro:cob_head_v3>
+  <xacro:cob_lookat name="lookat" parent="torso_upper_neck_tilt_link">
+    <origin xyz="${head_x} ${head_y} ${head_z}" rpy="${head_roll} ${head_pitch} ${head_yaw}" />
+    <axis xyz="-1 0 0"/>
+  </xacro:cob_lookat>
   <xacro:schunk_sdh name="sdh" parent="arm_7_link">
     <origin xyz="${sdh_x} ${sdh_y} ${sdh_z}" rpy="${sdh_roll} ${sdh_pitch} ${sdh_yaw}" />
