Commit message: Added powerball tray

File: cob_hardware_config/cob3-5/urdf/cob3-5.urdf.xacro (robot description, xacro)
@@ -14,5 +14,5 @@
   <include filename="$(find cob_description)/urdf/base/base.urdf.xacro" />
   <!-- tray -->
-  <include filename="$(find cob_description)/urdf/tray/tray.urdf.xacro" />
+  <include filename="$(find cob_description)/urdf/tray_powerball/tray.urdf.xacro" />
   <!-- torso -->
   <include filename="$(find cob_description)/urdf/torso_v1/torso.urdf.xacro" />
@@ -27,7 +27,7 @@
   <!-- composition of the robot -->
   <xacro:cob_base name="base"/>
-  <xacro:cob_tray name="tray" parent="base_link">
+  <xacro:cob_tray_powerball name="tray" parent="base_link">
     <origin xyz="${tray_x} ${tray_y} ${tray_z}" rpy="${tray_roll} ${tray_pitch} ${tray_yaw}" />
-  </xacro:cob_tray>
+  </xacro:cob_tray_powerball>
   <xacro:cob_torso_v1 name="torso" parent="base_link">
     <origin xyz="${torso_x} ${torso_y} ${torso_z}" rpy="${torso_roll} ${torso_pitch} ${torso_yaw}" />
@@ -37,5 +37,5 @@
   </xacro:schunk_lwa>
   <xacro:cob_head_v3 name="head" parent="torso_upper_neck_tilt_link">
-    <origin xyz="${head_x} ${head_y} ${head_z}" rpy="${head_roll} ${head_pitch} ${head_yaw}" />
+    <origin xyz="0 0.173 0" rpy="0 0 0" />
   </xacro:cob_head_v3>
   <xacro:schunk_sdh name="sdh" parent="arm_7_link">

Commit message: fix cob3-5 urdf for head

File: cob_hardware_config/cob3-5/urdf/cob3-5.urdf.xacro (robot description, xacro)
@@ -37,5 +37,5 @@
   </xacro:schunk_lwa>
   <xacro:cob_head_v3 name="head" parent="torso_upper_neck_tilt_link">
-    <origin xyz="0 0.173 0" rpy="0 0 0" />
+    <origin xyz="${head_x} ${head_y} ${head_z}" rpy="${head_roll} ${head_pitch} ${head_yaw}" />
   </xacro:cob_head_v3>
   <xacro:schunk_sdh name="sdh" parent="arm_7_link">
