Commit message: update cob3-7

File: cob_hardware_config/cob3-7/urdf/cob3-7.urdf.xacro (robot description, xacro)
@@ -19,6 +19,8 @@
   <!-- head -->
   <include filename="$(find cob_description)/urdf/head_v3/head.urdf.xacro" />
-  <!-- sdh -->
-  <include filename="$(find schunk_description)/urdf/sdh/sdh.urdf.xacro" />
+  <!-- ur_conector -->
+  <include filename="$(find cob_description)/urdf/ur_conector/ur_conector.urdf.xacro" />
+  <!-- arm -->
+  <include filename="$(find cob_description)/urdf/ur_arm/ur5_arm.urdf.xacro"/>
   <!-- generic simulator_gazebo plugins for starting mechanism control, ros time, ros battery -->
   <include filename="$(find cob_description)/gazebo/gazebo.urdf.xacro" />
@@ -34,3 +36,9 @@
     <origin xyz="${head_x} ${head_y} ${head_z}" rpy="${head_roll} ${head_pitch} ${head_yaw}" />
   </xacro:cob_head_v3>
+  <xacro:cob_ur_conector name="ur_conector" parent="base_link">
+    <origin xyz="${ur_conector_x} ${ur_conector_y} ${ur_conector_z}" rpy="${ur_conector_roll} ${ur_conector_pitch} ${ur_conector_yaw}" />
+  </xacro:cob_ur_conector>
+  <xacro:cob_ur5 name="arm" parent="ur_conector_link">
+      <origin xyz="${arm_x} ${arm_y} ${arm_z}" rpy="${arm_roll} ${arm_pitch} ${arm_yaw}" />
+  </xacro:cob_ur5>
 </robot>

Commit message: Update cob3-7

File: cob_hardware_config/cob3-7/urdf/cob3-7.urdf.xacro (robot description, xacro)
@@ -19,6 +19,6 @@
   <!-- head -->
   <include filename="$(find cob_description)/urdf/head_v3/head.urdf.xacro" />
-  <!-- ur_conector -->
-  <include filename="$(find cob_description)/urdf/ur_conector/ur_conector.urdf.xacro" />
+  <!-- ur_connector -->
+  <include filename="$(find cob_description)/urdf/ur_connector/ur_connector.urdf.xacro" />
   <!-- arm -->
   <include filename="$(find cob_description)/urdf/ur_arm/ur5_arm.urdf.xacro"/>
@@ -36,8 +36,8 @@
     <origin xyz="${head_x} ${head_y} ${head_z}" rpy="${head_roll} ${head_pitch} ${head_yaw}" />
   </xacro:cob_head_v3>
-  <xacro:cob_ur_conector name="ur_conector" parent="base_link">
-    <origin xyz="${ur_conector_x} ${ur_conector_y} ${ur_conector_z}" rpy="${ur_conector_roll} ${ur_conector_pitch} ${ur_conector_yaw}" />
-  </xacro:cob_ur_conector>
-  <xacro:cob_ur5 name="arm" parent="ur_conector_link">
+  <xacro:cob_ur_connector name="ur_connector" parent="base_link">
+    <origin xyz="${ur_connector_x} ${ur_connector_y} ${ur_connector_z}" rpy="${ur_connector_roll} ${ur_connector_pitch} ${ur_connector_yaw}" />
+  </xacro:cob_ur_connector>
+  <xacro:cob_ur5 name="arm" parent="ur_connector_link">
       <origin xyz="${arm_x} ${arm_y} ${arm_z}" rpy="${arm_roll} ${arm_pitch} ${arm_yaw}" />
   </xacro:cob_ur5>

Commit message: merge with ipa320-groovy_dev

File: cob_hardware_config/cob3-7/urdf/cob3-7.urdf.xacro (robot description, xacro)
@@ -19,6 +19,8 @@
   <!-- head -->
   <include filename="$(find cob_description)/urdf/head_v3/head.urdf.xacro" />
-  <!-- sdh -->
-  <include filename="$(find schunk_description)/urdf/sdh/sdh.urdf.xacro" />
+  <!-- ur_connector -->
+  <include filename="$(find cob_description)/urdf/ur_connector/ur_connector.urdf.xacro" />
+  <!-- arm -->
+  <include filename="$(find cob_description)/urdf/ur_arm/ur5_arm.urdf.xacro"/>
   <!-- generic simulator_gazebo plugins for starting mechanism control, ros time, ros battery -->
   <include filename="$(find cob_description)/gazebo/gazebo.urdf.xacro" />
@@ -34,3 +36,9 @@
     <origin xyz="${head_x} ${head_y} ${head_z}" rpy="${head_roll} ${head_pitch} ${head_yaw}" />
   </xacro:cob_head_v3>
+  <xacro:cob_ur_connector name="ur_connector" parent="base_link">
+    <origin xyz="${ur_connector_x} ${ur_connector_y} ${ur_connector_z}" rpy="${ur_connector_roll} ${ur_connector_pitch} ${ur_connector_yaw}" />
+  </xacro:cob_ur_connector>
+  <xacro:cob_ur5 name="arm" parent="ur_connector_link">
+      <origin xyz="${arm_x} ${arm_y} ${arm_z}" rpy="${arm_roll} ${arm_pitch} ${arm_yaw}" />
+  </xacro:cob_ur5>
 </robot>
