Commit message: cob3-8 has pg70 as gripper

File: cob_hardware_config/cob3-8/urdf/calibration_default.urdf.xacro (robot description, xacro)
@@ -56,11 +56,11 @@
 	<property name="def_arm_pitch" value="0.7854"/>
 	<property name="def_arm_yaw" value="-1.8326"/>
-	<!-- sdh mount positions | relative to arm_7_link -->
-	<property name="def_sdh_x" value="0.0"/>
-	<property name="def_sdh_y" value="0.0"/>
-	<property name="def_sdh_z" value="0.0"/>
-	<property name="def_sdh_roll" value="0.0"/>
-	<property name="def_sdh_pitch" value="3.1415926"/>
-	<property name="def_sdh_yaw" value="0.0"/>
+	<!-- pg70 mount positions | relative to arm_7_link -->
+	<property name="def_pg70_x" value="0.0"/>
+	<property name="def_pg70_y" value="0.0"/>
+	<property name="def_pg70_z" value="0.0"/>
+	<property name="def_pg70_roll" value="0.0"/>
+	<property name="def_pg70_pitch" value="3.1415926"/>
+	<property name="def_pg70_yaw" value="0.0"/>
 	<!-- *********************************** -->
 	<!-- kinematic chain reference positions -->

File: cob_hardware_config/cob3-8/urdf/cob3-8.urdf.xacro (robot description, xacro)
@@ -20,5 +20,5 @@
   <xacro:include filename="$(find schunk_description)/urdf/lwa/lwa.urdf.xacro" />
   <!-- sdh -->
-  <xacro:include filename="$(find schunk_description)/urdf/sdh/sdh.urdf.xacro" />
+  <xacro:include filename="$(find schunk_description)/urdf/pg70/pg70.urdf.xacro" />
   <!-- generic simulator_gazebo plugins for starting mechanism control, ros time, ros battery -->
   <xacro:include filename="$(find cob_description)/gazebo/gazebo.urdf.xacro" />
@@ -41,6 +41,6 @@
     <axis xyz="-1 0 0"/>
   </xacro:lookat>
-  <xacro:schunk_sdh name="sdh" parent="arm_7_link">
-    <origin xyz="${sdh_x} ${sdh_y} ${sdh_z}" rpy="${sdh_roll} ${sdh_pitch} ${sdh_yaw}" />
-  </xacro:schunk_sdh>
+  <xacro:schunk_pg70 name="pg70" parent="arm_7_link">
+    <origin xyz="${pg70_x} ${pg70_y} ${pg70_z}" rpy="${pg70_roll} ${pg70_pitch} ${pg70_yaw}" />
+  </xacro:schunk_pg70>
 </robot>

File: cob_hardware_config/cob3-8/urdf/properties.urdf.xacro (robot description, xacro)
@@ -58,11 +58,11 @@
 	<property name="arm_pitch" value="${def_arm_pitch+offset_arm_pitch}"/>
 	<property name="arm_yaw" value="${def_arm_yaw+offset_arm_yaw}"/>
-	<!-- sdh mount positions | relative to arm_7_link -->
-	<property name="sdh_x" value="${def_sdh_x+offset_sdh_x}"/>
-	<property name="sdh_y" value="${def_sdh_y+offset_sdh_y}"/>
-	<property name="sdh_z" value="${def_sdh_z+offset_sdh_z}"/>
-	<property name="sdh_roll" value="${def_sdh_roll+offset_sdh_roll}"/>
-	<property name="sdh_pitch" value="${def_sdh_pitch+offset_sdh_pitch}"/>
-	<property name="sdh_yaw" value="${def_sdh_yaw+offset_sdh_yaw}"/>
+	<!-- pg70 mount positions | relative to arm_7_link -->
+	<property name="pg70_x" value="${def_pg70_x+offset_pg70_x}"/>
+	<property name="pg70_y" value="${def_pg70_y+offset_pg70_y}"/>
+	<property name="pg70_z" value="${def_pg70_z+offset_pg70_z}"/>
+	<property name="pg70_roll" value="${def_pg70_roll+offset_pg70_roll}"/>
+	<property name="pg70_pitch" value="${def_pg70_pitch+offset_pg70_pitch}"/>
+	<property name="pg70_yaw" value="${def_pg70_yaw+offset_pg70_yaw}"/>
 	<!-- *********************************** -->
 	<!-- kinematic chain reference positions -->

Commit message: setup cob3-8

File: cob_hardware_config/cob3-8/urdf/calibration_default.urdf.xacro (robot description, xacro)
@@ -36,15 +36,15 @@
 	<property name="def_tray_yaw" value="0.0"/>
 	<!-- torso mount positions | relative to base_link -->
-	<property name="def_torso_x" value="0.155"/>
+	<property name="def_torso_x" value="0.1505153138"/>
 	<property name="def_torso_y" value="0.0"/>
-	<property name="def_torso_z" value="0.892"/>
-	<property name="def_torso_roll" value="3.1415926"/>
-	<property name="def_torso_pitch" value="0.0"/>
-	<property name="def_torso_yaw" value="0.0"/>
+	<property name="def_torso_z" value="0.8602400721"/>
+	<property name="def_torso_roll" value="1.563226442"/>
+	<property name="def_torso_pitch" value="0.0346163655"/>
+	<property name="def_torso_yaw" value="0.0107070343"/>
 	<!-- head mount positions | relative to head_cover_link -->
 	<property name="def_head_x" value="0.0"/>
-	<property name="def_head_y" value="-0.154"/>
+	<property name="def_head_y" value="0.173"/>
 	<property name="def_head_z" value="0.0"/>
-	<property name="def_head_roll" value="3.14159"/>
+	<property name="def_head_roll" value="0.0"/>
 	<property name="def_head_pitch" value="0.0"/>
 	<property name="def_head_yaw" value="0.0"/>
@@ -67,20 +67,19 @@
 	<!-- *********************************** -->
 	<!-- torso chain calibration_offest! | relative to reference position (see below)-->
-	<property name="def_torso_lower_neck_pan_ref" value="-0.00018174503929913044" />
-	<property name="def_torso_lower_neck_tilt_ref" value="0.048314183950424194" />
-	<property name="def_torso_upper_neck_pan_ref" value="0.0022084463853389025" />
-	<property name="def_torso_upper_neck_tilt_ref" value="0.0073217283934354782" />
+	<property name="def_torso_lower_neck_tilt_ref" value="0.0"/>
+	<property name="def_torso_pan_ref" value="0.0"/>
+	<property name="def_torso_upper_neck_tilt_ref" value="0.0"/>
 	<!-- tray reference position | used as calibration_rising for tray chain -->
 	<property name="def_tray_ref" value="4.2"/>
 	<!-- head camera axis reference position | used as calibration_rising for head axis chain -->
-	<property name="def_head_axis_ref" value="3.29"/>
+	<property name="def_head_axis_ref" value="0.1"/>
 	<!-- arm reference positions | used as calibration_rising for arm chain-->
-	<property name="def_arm_1_ref" value="3.403339959" />
-	<property name="def_arm_2_ref" value="-0.180424702" />
-	<property name="def_arm_3_ref" value="-1.62660" />
-	<property name="def_arm_4_ref" value="1.36543799" />
-	<property name="def_arm_5_ref" value="0.00185081481" />
-	<property name="def_arm_6_ref" value="7549.28222" />
-	<property name="def_arm_7_ref" value="-0.41888" />
+	<property name="def_arm_1_ref" value="-0.29616492077091777" />
+	<property name="def_arm_2_ref" value="0" />
+	<property name="def_arm_3_ref" value="0" />
+	<property name="def_arm_4_ref" value="0" />
+	<property name="def_arm_5_ref" value="0" />
+	<property name="def_arm_6_ref" value="0" />
+	<property name="def_arm_7_ref" value="0" />
 	<!-- ***************************** -->
 	<!-- camera calibration properties -->

File: cob_hardware_config/cob3-8/urdf/cob3-8.urdf.xacro (robot description, xacro)
@@ -13,5 +13,5 @@
   <xacro:include filename="$(find cob_description)/urdf/cob3_tray/tray.urdf.xacro" />
   <!-- torso -->
-  <xacro:include filename="$(find cob_description)/urdf/cob3_torso/torso_v1.urdf.xacro" />
+  <xacro:include filename="$(find cob_description)/urdf/cob3_torso/torso_v2.urdf.xacro" />
   <!-- head -->
   <xacro:include filename="$(find cob_description)/urdf/cob3_head/head_kinect.urdf.xacro" />
@@ -37,8 +37,4 @@
     <origin xyz="${head_x} ${head_y} ${head_z}" rpy="${head_roll} ${head_pitch} ${head_yaw}" />
   </xacro:head>
-  <xacro:lookat name="lookat" parent="torso_upper_neck_tilt_link" lower="-5.0" upper="5.0">
-    <origin xyz="${head_x} ${head_y} ${head_z}" rpy="${head_roll} ${head_pitch} ${head_yaw}" />
-    <axis xyz="-1 0 0"/>
-  </xacro:lookat>
   <xacro:schunk_pg70 name="pg70" parent="arm_7_link">
     <origin xyz="${pg70_x} ${pg70_y} ${pg70_z}" rpy="${pg70_roll} ${pg70_pitch} ${pg70_yaw}" />

File: cob_hardware_config/cob3-8/urdf/properties.urdf.xacro (robot description, xacro)
@@ -71,8 +71,7 @@
 	<!-- torso reference positions | used as calibration_rising for torso chain -->
 	<!-- ! set these values to make torso straight with (0, 0, 0) joint angles ! -->
-	<property name="torso_lower_neck_pan_ref" value="${def_torso_lower_neck_pan_ref+offset_torso_lower_neck_pan_ref}" />
-	<property name="torso_lower_neck_tilt_ref" value="${def_torso_lower_neck_tilt_ref+offset_torso_lower_neck_tilt_ref}" />
-	<property name="torso_upper_neck_pan_ref" value="${def_torso_upper_neck_pan_ref+offset_torso_upper_neck_pan_ref}" />
-	<property name="torso_upper_neck_tilt_ref" value="${def_torso_upper_neck_tilt_ref+offset_torso_upper_neck_tilt_ref}" />
+	<property name="torso_lower_neck_tilt_ref" value="${def_torso_lower_neck_tilt_ref+offset_torso_lower_neck_tilt_ref}"/>
+	<property name="torso_pan_ref" value="${def_torso_pan_ref+offset_torso_pan_ref}"/>
+	<property name="torso_upper_neck_tilt_ref" value="${def_torso_upper_neck_tilt_ref+offset_torso_upper_neck_tilt_ref}"/>
 	<!-- tray reference position | used as calibration_rising for tray chain -->
 	<property name="tray_ref" value="${def_tray_ref+offset_tray_ref}"/>
