Commit message: update cob3-1 urdf

File: cob_hardware_config/cob3-1/urdf/cob3-1.urdf.xacro (robot description, xacro)
@@ -36,5 +36,5 @@
   </xacro:cob_lbr>
   <xacro:cob_head_v1 name="head" parent="torso_upper_neck_tilt_link">
-    <origin xyz="0 -0.154 0" rpy="3.1415926 0 0" />
+    <origin xyz="0 -0.154 0" rpy="3.1415926 3.1415926 0" />
   </xacro:cob_head_v1>
   <xacro:schunk_sdh name="sdh" parent="arm_7_link">

Commit message: replace all hardcoded mounting values with respective macros in cob_calibration_data

File: cob_hardware_config/cob3-1/urdf/cob3-1.urdf.xacro (robot description, xacro)
@@ -37,8 +37,8 @@
   </xacro:cob_lbr>
   <xacro:cob_head_v1 name="head" parent="torso_upper_neck_tilt_link">
-    <origin xyz="0 -0.154 0" rpy="3.1415926 3.1415926 0" />
+    <origin xyz="${head_x} ${head_y} ${head_z}" rpy="${head_roll} ${head_pitch} ${head_yaw}" />
   </xacro:cob_head_v1>
   <xacro:schunk_sdh name="sdh" parent="arm_7_link">
-    <origin xyz="0 0 0.032" rpy="0 0 1.5708" />
+    <origin xyz="${sdh_x} ${sdh_y} ${sdh_z}" rpy="${sdh_roll} ${sdh_pitch} ${sdh_yaw}" />
   </xacro:schunk_sdh>
 </robot>

File: cob_hardware_config/cob3-2/urdf/cob3-2.urdf.xacro (robot description, xacro)
@@ -37,8 +37,8 @@
   </xacro:schunk_lwa>
   <xacro:cob_head_v2 name="head" parent="torso_upper_neck_tilt_link">
-    <origin xyz="0 -0.154 0" rpy="3.14159 0 0" />
+    <origin xyz="${head_x} ${head_y} ${head_z}" rpy="${head_roll} ${head_pitch} ${head_yaw}" />
   </xacro:cob_head_v2>
   <xacro:schunk_sdh name="sdh" parent="arm_7_link">
-    <origin xyz="0 0 0" rpy="0 3.1415926 0" />
+    <origin xyz="${sdh_x} ${sdh_y} ${sdh_z}" rpy="${sdh_roll} ${sdh_pitch} ${sdh_yaw}" />
   </xacro:schunk_sdh>
 </robot>

File: cob_hardware_config/cob3-3/urdf/cob3-3.urdf.xacro (robot description, xacro)
@@ -40,5 +40,5 @@
   </xacro:cob_head_v3>
   <xacro:schunk_sdh name="sdh" parent="arm_7_link">
-    <origin xyz="0 0 0.032" rpy="0 0 ${M_PI/2}" />
+    <origin xyz="${sdh_x} ${sdh_y} ${sdh_z}" rpy="${sdh_roll} ${sdh_pitch} ${sdh_yaw}" />
   </xacro:schunk_sdh>
 </robot>

File: cob_hardware_config/cob3-4/urdf/cob3-4.urdf.xacro (robot description, xacro)
@@ -37,8 +37,8 @@
   </xacro:cob_lbr>
   <xacro:cob_head_v3 name="head" parent="torso_upper_neck_tilt_link">
-    <origin xyz="0 0.173 0" rpy="0 0 0" />
+    <origin xyz="${head_x} ${head_y} ${head_z}" rpy="${head_roll} ${head_pitch} ${head_yaw}" />
   </xacro:cob_head_v3>
   <xacro:schunk_sdh name="sdh" parent="arm_7_link">
-    <origin xyz="0 0 0.032" rpy="0 0 1.5708" />
+    <origin xyz="${sdh_x} ${sdh_y} ${sdh_z}" rpy="${sdh_roll} ${sdh_pitch} ${sdh_yaw}" />
   </xacro:schunk_sdh>
 </robot>

File: cob_hardware_config/cob3-5/urdf/cob3-5.urdf.xacro (robot description, xacro)
@@ -40,5 +40,5 @@
   </xacro:cob_head_v3>
   <xacro:schunk_sdh name="sdh" parent="arm_7_link">
-    <origin xyz="0 0 0" rpy="0 ${M_PI} 0" />
+    <origin xyz="${sdh_x} ${sdh_y} ${sdh_z}" rpy="${sdh_roll} ${sdh_pitch} ${sdh_yaw}" />
   </xacro:schunk_sdh>
 </robot>

File: cob_hardware_config/cob3-6/urdf/cob3-6.urdf.xacro (robot description, xacro)
@@ -37,8 +37,8 @@
   </xacro:schunk_lwa>
   <xacro:cob_head_v3 name="head" parent="torso_upper_neck_tilt_link">
-    <origin xyz="0 0.173 0" rpy="0 0 0" />
+    <origin xyz="${head_x} ${head_y} ${head_z}" rpy="${head_roll} ${head_pitch} ${head_yaw}" />
   </xacro:cob_head_v3>
   <xacro:schunk_sdh name="sdh" parent="arm_7_link">
-    <origin xyz="0 0 0" rpy="0 ${M_PI} 0" />
+    <origin xyz="${sdh_x} ${sdh_y} ${sdh_z}" rpy="${sdh_roll} ${sdh_pitch} ${sdh_yaw}" />
   </xacro:schunk_sdh>
 </robot>
