Commit message: add lookat to all cobs + some fixes in calibration values

File: cob_hardware_config/cob3-1/urdf/cob3-1.urdf.xacro (robot description, xacro)
@@ -4,5 +4,5 @@
        xmlns:interface="http://playerstage.sourceforge.net/gazebo/xmlschema/#interface"
        xmlns:xacro="http://playerstage.sourceforge.net/gazebo/xmlschema/#interface"
-       name="cob3_1" >
+       name="cob3-1" >
   <!-- common stuff -->
   <include filename="$(find cob_description)/urdf/common.xacro" />
@@ -19,4 +19,5 @@
   <!-- head -->
   <include filename="$(find cob_description)/urdf/head_v1/head.urdf.xacro" />
+  <include filename="$(find cob_description)/urdf/lookat/lookat.urdf.xacro" />
   <!-- arm -->
   <include filename="$(find cob_description)/urdf/lbr/lbr.urdf.xacro" />
@@ -39,4 +40,8 @@
     <origin xyz="${head_x} ${head_y} ${head_z}" rpy="${head_roll} ${head_pitch} ${head_yaw}" />
   </xacro:cob_head_v1>
+  <xacro:cob_lookat name="lookat" parent="torso_upper_neck_tilt_link">
+    <origin xyz="${head_x} ${head_y} ${head_z}" rpy="${head_roll} ${head_pitch} ${head_yaw}" />
+    <axis xyz="-1 0 0"/>
+  </xacro:cob_lookat>
   <xacro:schunk_sdh name="sdh" parent="arm_7_link">
     <origin xyz="${sdh_x} ${sdh_y} ${sdh_z}" rpy="${sdh_roll} ${sdh_pitch} ${sdh_yaw}" />

File: cob_hardware_config/cob3-2/urdf/calibration_default.urdf.xacro (robot description, xacro)
@@ -87,11 +87,4 @@
 	<!-- ***************************** -->
 	<!-- left | handeye calibration | relative to head_axis_link -->
-	<property name="def_cam_reference_x" value="0.0"/>
-	<property name="def_cam_reference_y" value="0.0"/>
-	<property name="def_cam_reference_z" value="0.0"/>
-	<property name="def_cam_reference_roll" value="0.6254583135"/>
-	<property name="def_cam_reference_pitch" value="-1.5196809763"/>
-	<property name="def_cam_reference_yaw" value="-0.8146938173"/>
-	<!-- left | handeye calibration | relative to head_axis_link -->
 	<property name="def_cam_l_x" value="0"/>
 	<property name="def_cam_l_y" value="0"/>
@@ -100,17 +93,24 @@
 	<property name="def_cam_l_pitch" value="0"/>
 	<property name="def_cam_l_yaw" value="0"/>
+	<!-- left | handeye calibration | relative to head_axis_link -->
+	<property name="def_cam_reference_x" value="-0.05"/>
+	<property name="def_cam_reference_y" value="-0.02"/>
+	<property name="def_cam_reference_z" value="-0.07"/>
+	<property name="def_cam_reference_roll" value="0"/>
+	<property name="def_cam_reference_pitch" value="-1.5563904314"/>
+	<property name="def_cam_reference_yaw" value="0"/>
 	<!-- right | stereo baseline calibration | relative to left camera -->
-	<property name="def_cam_r_x" value="0.0"/>
-	<property name="def_cam_r_y" value="0.0"/>
-	<property name="def_cam_r_z" value="0.0"/>
-	<property name="def_cam_r_roll" value="0.0"/>
-	<property name="def_cam_r_pitch" value="0.0"/>
-	<property name="def_cam_r_yaw" value="0.0116886166619"/>
-	<!-- cam3d | handeye calibration | relative to left camera -->
-	<property name="def_cam3d_x" value="0.0"/>
-	<property name="def_cam3d_y" value="0.0"/>
-	<property name="def_cam3d_z" value="0.0"/>
-	<property name="def_cam3d_roll" value="0.512574156"/>
-	<property name="def_cam3d_pitch" value="-1.5250630397"/>
-	<property name="def_cam3d_yaw" value="-0.6569406141"/>
+	<property name="def_cam_r_x" value="0.12"/>
+	<property name="def_cam_r_y" value="0"/>
+	<property name="def_cam_r_z" value="0"/>
+	<property name="def_cam_r_roll" value="0"/>
+	<property name="def_cam_r_pitch" value="0"/>
+	<property name="def_cam_r_yaw" value="0"/>
+	<!-- cam3d | handeye calibration | relative to head_axis_link -->
+	<property name="def_cam3d_x" value="0.06"/>
+	<property name="def_cam3d_y" value="-0.03"/>
+	<property name="def_cam3d_z" value="0"/>
+	<property name="def_cam3d_roll" value="0"/>
+	<property name="def_cam3d_pitch" value="0"/>
+	<property name="def_cam3d_yaw" value="0"/>
 </robot>

File: cob_hardware_config/cob3-2/urdf/cob3-2.urdf.xacro (robot description, xacro)
@@ -4,5 +4,5 @@
        xmlns:interface="http://playerstage.sourceforge.net/gazebo/xmlschema/#interface"
        xmlns:xacro="http://playerstage.sourceforge.net/gazebo/xmlschema/#interface"
-       name="cob3_2" >
+       name="cob3-2" >
   <!-- common stuff -->
   <include filename="$(find cob_description)/urdf/common.xacro" />
@@ -19,4 +19,5 @@
   <!-- head -->
   <include filename="$(find cob_description)/urdf/head_v2/head.urdf.xacro" />
+  <include filename="$(find cob_description)/urdf/lookat/lookat.urdf.xacro" />
   <!-- arm -->
   <include filename="$(find schunk_description)/urdf/lwa/lwa.urdf.xacro" />
@@ -39,4 +40,8 @@
     <origin xyz="${head_x} ${head_y} ${head_z}" rpy="${head_roll} ${head_pitch} ${head_yaw}" />
   </xacro:cob_head_v2>
+  <xacro:cob_lookat name="lookat" parent="torso_upper_neck_tilt_link">
+    <origin xyz="${head_x} ${head_y} ${head_z}" rpy="${head_roll} ${head_pitch} ${head_yaw}" />
+    <axis xyz="-1 0 0"/>
+  </xacro:cob_lookat>
   <xacro:schunk_sdh name="sdh" parent="arm_7_link">
     <origin xyz="${sdh_x} ${sdh_y} ${sdh_z}" rpy="${sdh_roll} ${sdh_pitch} ${sdh_yaw}" />

File: cob_hardware_config/cob3-3/urdf/cob3-3.urdf.xacro (robot description, xacro)
@@ -4,5 +4,5 @@
        xmlns:interface="http://playerstage.sourceforge.net/gazebo/xmlschema/#interface"
        xmlns:xacro="http://playerstage.sourceforge.net/gazebo/xmlschema/#interface"
-       name="cob3_3" >
+       name="cob3-3" >
   <!-- common stuff -->
   <include filename="$(find cob_description)/urdf/common.xacro" />

File: cob_hardware_config/cob3-4/urdf/calibration_default.urdf.xacro (robot description, xacro)
@@ -75,21 +75,14 @@
 	<property name="def_head_axis_ref" value="0.14"/>
 	<!-- arm reference positions | used as calibration_rising for arm chain-->
-	<property name="def_arm_1_ref" value="0"/>
-	<property name="def_arm_2_ref" value="0"/>
-	<property name="def_arm_3_ref" value="0"/>
-	<property name="def_arm_4_ref" value="0"/>
-	<property name="def_arm_5_ref" value="0"/>
-	<property name="def_arm_6_ref" value="0"/>
-	<property name="def_arm_7_ref" value="0"/>
+	<property name="def_arm_1_ref" value="0.0"/>
+	<property name="def_arm_2_ref" value="0.0"/>
+	<property name="def_arm_3_ref" value="0.0"/>
+	<property name="def_arm_4_ref" value="0.0"/>
+	<property name="def_arm_5_ref" value="0.0"/>
+	<property name="def_arm_6_ref" value="0.0"/>
+	<property name="def_arm_7_ref" value="0.0"/>
 	<!-- ***************************** -->
 	<!-- camera calibration properties -->
 	<!-- ***************************** -->
-	<!-- left | handeye calibration | relative to head_axis_link -->
-	<property name="def_cam_reference_x" value="-0.0168918076"/>
-	<property name="def_cam_reference_y" value="-0.0331605618"/>
-	<property name="def_cam_reference_z" value="-0.1227576067"/>
-	<property name="def_cam_reference_roll" value="0.8665791516"/>
-	<property name="def_cam_reference_pitch" value="-1.5610273707"/>
-	<property name="def_cam_reference_yaw" value="-0.9246703056"/>
 	<!-- left | handeye calibration | relative to head_axis_link -->
 	<property name="def_cam_l_x" value="0"/>
@@ -99,17 +92,24 @@
 	<property name="def_cam_l_pitch" value="0"/>
 	<property name="def_cam_l_yaw" value="0"/>
+	<!-- left | handeye calibration | relative to head_axis_link -->
+	<property name="def_cam_reference_x" value="-0.05"/>
+	<property name="def_cam_reference_y" value="-0.02"/>
+	<property name="def_cam_reference_z" value="-0.07"/>
+	<property name="def_cam_reference_roll" value="0"/>
+	<property name="def_cam_reference_pitch" value="-1.5563904314"/>
+	<property name="def_cam_reference_yaw" value="0"/>
 	<!-- right | stereo baseline calibration | relative to left camera -->
-	<property name="def_cam_r_x" value="0.120625576659"/>
-	<property name="def_cam_r_y" value="0.00069791469442"/>
-	<property name="def_cam_r_z" value="-0.000529628535957"/>
-	<property name="def_cam_r_roll" value="0.00400056610075"/>
-	<property name="def_cam_r_pitch" value="0.0120185944721"/>
-	<property name="def_cam_r_yaw" value="0.0118234806514"/>
+	<property name="def_cam_r_x" value="0.12"/>
+	<property name="def_cam_r_y" value="0"/>
+	<property name="def_cam_r_z" value="0"/>
+	<property name="def_cam_r_roll" value="0"/>
+	<property name="def_cam_r_pitch" value="0"/>
+	<property name="def_cam_r_yaw" value="0"/>
 	<!-- cam3d | handeye calibration | relative to head_axis_link -->
-	<property name="def_cam3d_x" value="-0.037555729"/>
-	<property name="def_cam3d_y" value="-0.0651598868"/>
-	<property name="def_cam3d_z" value="-0.0442883082"/>
-	<property name="def_cam3d_roll" value="-0.0652253986"/>
-	<property name="def_cam3d_pitch" value="-1.5552469375"/>
-	<property name="def_cam3d_yaw" value="0.0523406338"/>
+	<property name="def_cam3d_x" value="0.06"/>
+	<property name="def_cam3d_y" value="-0.03"/>
+	<property name="def_cam3d_z" value="0"/>
+	<property name="def_cam3d_roll" value="0"/>
+	<property name="def_cam3d_pitch" value="0"/>
+	<property name="def_cam3d_yaw" value="0"/>
 </robot>

File: cob_hardware_config/cob3-4/urdf/cob3-4.urdf.xacro (robot description, xacro)
@@ -4,5 +4,5 @@
        xmlns:interface="http://playerstage.sourceforge.net/gazebo/xmlschema/#interface"
        xmlns:xacro="http://playerstage.sourceforge.net/gazebo/xmlschema/#interface"
-       name="cob3_4" >
+       name="cob3-4" >
   <!-- common stuff -->
   <include filename="$(find cob_description)/urdf/common.xacro" />
@@ -19,4 +19,5 @@
   <!-- head -->
   <include filename="$(find cob_description)/urdf/head_v3/head.urdf.xacro" />
+  <include filename="$(find cob_description)/urdf/lookat/lookat.urdf.xacro" />
   <!-- arm -->
   <include filename="$(find cob_description)/urdf/lbr/lbr.urdf.xacro" />
@@ -39,4 +40,8 @@
     <origin xyz="${head_x} ${head_y} ${head_z}" rpy="${head_roll} ${head_pitch} ${head_yaw}" />
   </xacro:cob_head_v3>
+  <xacro:cob_lookat name="lookat" parent="torso_upper_neck_tilt_link">
+    <origin xyz="${head_x} ${head_y} ${head_z}" rpy="${head_roll} ${head_pitch} ${head_yaw}" />
+    <axis xyz="-1 0 0"/>
+  </xacro:cob_lookat>
   <xacro:schunk_sdh name="sdh" parent="arm_7_link">
     <origin xyz="${sdh_x} ${sdh_y} ${sdh_z}" rpy="${sdh_roll} ${sdh_pitch} ${sdh_yaw}" />

File: cob_hardware_config/cob3-5/urdf/calibration_default.urdf.xacro (robot description, xacro)
@@ -29,10 +29,10 @@
 	<!-- *********************** -->
 	<!-- tray mount positions | relative to base_link -->
-	<property name="def_tray_x" value="0.2406"/>
-	<property name="def_tray_y" value="0.1900"/>
-	<property name="def_tray_z" value="0.7320"/>
-	<property name="def_tray_roll" value="2.3561"/>
-	<property name="def_tray_pitch" value="0.0"/>
-	<property name="def_tray_yaw" value="0.0"/>
+	<property name="def_tray_x" value="0.186"/>
+	<property name="def_tray_y" value="0.113"/>
+	<property name="def_tray_z" value="0.721"/>
+	<property name="def_tray_roll" value="-1.5707"/>
+	<property name="def_tray_pitch" value="0.35"/>
+	<property name="def_tray_yaw" value="0"/>
 	<!-- torso mount positions | relative to base_link -->
 	<property name="def_torso_x" value="0.1535525935"/>
@@ -88,11 +88,4 @@
 	<!-- ***************************** -->
 	<!-- left | handeye calibration | relative to head_axis_link -->
-	<property name="def_cam_reference_x" value="-0.0168918076"/>
-	<property name="def_cam_reference_y" value="-0.0331605618"/>
-	<property name="def_cam_reference_z" value="-0.1227576067"/>
-	<property name="def_cam_reference_roll" value="0.8665791516"/>
-	<property name="def_cam_reference_pitch" value="-1.5610273707"/>
-	<property name="def_cam_reference_yaw" value="-0.9246703056"/>
-	<!-- left | handeye calibration | relative to head_axis_link -->
 	<property name="def_cam_l_x" value="0"/>
 	<property name="def_cam_l_y" value="0"/>
@@ -101,17 +94,24 @@
 	<property name="def_cam_l_pitch" value="0"/>
 	<property name="def_cam_l_yaw" value="0"/>
+	<!-- left | handeye calibration | relative to head_axis_link -->
+	<property name="def_cam_reference_x" value="-0.05"/>
+	<property name="def_cam_reference_y" value="-0.02"/>
+	<property name="def_cam_reference_z" value="-0.07"/>
+	<property name="def_cam_reference_roll" value="0"/>
+	<property name="def_cam_reference_pitch" value="-1.5563904314"/>
+	<property name="def_cam_reference_yaw" value="0"/>
 	<!-- right | stereo baseline calibration | relative to left camera -->
-	<property name="def_cam_r_x" value="0.120625576659"/>
-	<property name="def_cam_r_y" value="0.00069791469442"/>
-	<property name="def_cam_r_z" value="-0.000529628535957"/>
-	<property name="def_cam_r_roll" value="0.00400056610075"/>
-	<property name="def_cam_r_pitch" value="0.0120185944721"/>
-	<property name="def_cam_r_yaw" value="0.0118234806514"/>
+	<property name="def_cam_r_x" value="0.12"/>
+	<property name="def_cam_r_y" value="0"/>
+	<property name="def_cam_r_z" value="0"/>
+	<property name="def_cam_r_roll" value="0"/>
+	<property name="def_cam_r_pitch" value="0"/>
+	<property name="def_cam_r_yaw" value="0"/>
 	<!-- cam3d | handeye calibration | relative to head_axis_link -->
-	<property name="def_cam3d_x" value="-0.037555729"/>
-	<property name="def_cam3d_y" value="-0.0651598868"/>
-	<property name="def_cam3d_z" value="-0.0442883082"/>
-	<property name="def_cam3d_roll" value="-0.0652253986"/>
-	<property name="def_cam3d_pitch" value="-1.5552469375"/>
-	<property name="def_cam3d_yaw" value="0.0523406338"/>
+	<property name="def_cam3d_x" value="0.06"/>
+	<property name="def_cam3d_y" value="-0.03"/>
+	<property name="def_cam3d_z" value="0"/>
+	<property name="def_cam3d_roll" value="0"/>
+	<property name="def_cam3d_pitch" value="0"/>
+	<property name="def_cam3d_yaw" value="0"/>
 </robot>

File: cob_hardware_config/cob3-5/urdf/cob3-5.urdf.xacro (robot description, xacro)
@@ -4,5 +4,5 @@
        xmlns:interface="http://playerstage.sourceforge.net/gazebo/xmlschema/#interface"
        xmlns:xacro="http://playerstage.sourceforge.net/gazebo/xmlschema/#interface"
-       name="cob3_5" >
+       name="cob3-5" >
   <!-- common stuff -->
   <include filename="$(find cob_description)/urdf/common.xacro" />
@@ -19,4 +19,5 @@
   <!-- head -->
   <include filename="$(find cob_description)/urdf/head_v3/head.urdf.xacro" />
+  <include filename="$(find cob_description)/urdf/lookat/lookat.urdf.xacro" />
   <!-- arm -->
   <include filename="$(find schunk_description)/urdf/lwa/lwa.urdf.xacro" />
@@ -39,4 +40,8 @@
     <origin xyz="${head_x} ${head_y} ${head_z}" rpy="${head_roll} ${head_pitch} ${head_yaw}" />
   </xacro:cob_head_v3>
+  <xacro:cob_lookat name="lookat" parent="torso_upper_neck_tilt_link">
+    <origin xyz="${head_x} ${head_y} ${head_z}" rpy="${head_roll} ${head_pitch} ${head_yaw}" />
+    <axis xyz="-1 0 0"/>
+  </xacro:cob_lookat>
   <xacro:schunk_sdh name="sdh" parent="arm_7_link">
     <origin xyz="${sdh_x} ${sdh_y} ${sdh_z}" rpy="${sdh_roll} ${sdh_pitch} ${sdh_yaw}" />

File: cob_hardware_config/cob3-6/urdf/calibration_default.urdf.xacro (robot description, xacro)
@@ -88,11 +88,4 @@
 	<!-- ***************************** -->
 	<!-- left | handeye calibration | relative to head_axis_link -->
-	<property name="def_cam_reference_x" value="-0.0168918076"/>
-	<property name="def_cam_reference_y" value="-0.0331605618"/>
-	<property name="def_cam_reference_z" value="-0.1227576067"/>
-	<property name="def_cam_reference_roll" value="0.8665791516"/>
-	<property name="def_cam_reference_pitch" value="-1.5610273707"/>
-	<property name="def_cam_reference_yaw" value="-0.9246703056"/>
-	<!-- left | handeye calibration | relative to head_axis_link -->
 	<property name="def_cam_l_x" value="0"/>
 	<property name="def_cam_l_y" value="0"/>
@@ -101,17 +94,24 @@
 	<property name="def_cam_l_pitch" value="0"/>
 	<property name="def_cam_l_yaw" value="0"/>
+	<!-- left | handeye calibration | relative to head_axis_link -->
+	<property name="def_cam_reference_x" value="-0.05"/>
+	<property name="def_cam_reference_y" value="-0.02"/>
+	<property name="def_cam_reference_z" value="-0.07"/>
+	<property name="def_cam_reference_roll" value="0"/>
+	<property name="def_cam_reference_pitch" value="-1.5563904314"/>
+	<property name="def_cam_reference_yaw" value="0"/>
 	<!-- right | stereo baseline calibration | relative to left camera -->
-	<property name="def_cam_r_x" value="0.120625576659"/>
-	<property name="def_cam_r_y" value="0.00069791469442"/>
-	<property name="def_cam_r_z" value="-0.000529628535957"/>
-	<property name="def_cam_r_roll" value="0.00400056610075"/>
-	<property name="def_cam_r_pitch" value="0.0120185944721"/>
-	<property name="def_cam_r_yaw" value="0.0118234806514"/>
+	<property name="def_cam_r_x" value="0.12"/>
+	<property name="def_cam_r_y" value="0"/>
+	<property name="def_cam_r_z" value="0"/>
+	<property name="def_cam_r_roll" value="0"/>
+	<property name="def_cam_r_pitch" value="0"/>
+	<property name="def_cam_r_yaw" value="0"/>
 	<!-- cam3d | handeye calibration | relative to head_axis_link -->
-	<property name="def_cam3d_x" value="-0.037555729"/>
-	<property name="def_cam3d_y" value="-0.0651598868"/>
-	<property name="def_cam3d_z" value="-0.0442883082"/>
-	<property name="def_cam3d_roll" value="-0.0652253986"/>
-	<property name="def_cam3d_pitch" value="-1.5552469375"/>
-	<property name="def_cam3d_yaw" value="0.0523406338"/>
+	<property name="def_cam3d_x" value="0.06"/>
+	<property name="def_cam3d_y" value="-0.03"/>
+	<property name="def_cam3d_z" value="0"/>
+	<property name="def_cam3d_roll" value="0"/>
+	<property name="def_cam3d_pitch" value="0"/>
+	<property name="def_cam3d_yaw" value="0"/>
 </robot>

File: cob_hardware_config/cob3-6/urdf/cob3-6.urdf.xacro (robot description, xacro)
@@ -4,5 +4,5 @@
        xmlns:interface="http://playerstage.sourceforge.net/gazebo/xmlschema/#interface"
        xmlns:xacro="http://playerstage.sourceforge.net/gazebo/xmlschema/#interface"
-       name="cob3_6" >
+       name="cob3-6" >
   <!-- common stuff -->
   <include filename="$(find cob_description)/urdf/common.xacro" />
@@ -19,4 +19,5 @@
   <!-- head -->
   <include filename="$(find cob_description)/urdf/head_v3/head.urdf.xacro" />
+  <include filename="$(find cob_description)/urdf/lookat/lookat.urdf.xacro" />
   <!-- arm -->
   <include filename="$(find schunk_description)/urdf/lwa/lwa.urdf.xacro" />
@@ -39,4 +40,8 @@
     <origin xyz="${head_x} ${head_y} ${head_z}" rpy="${head_roll} ${head_pitch} ${head_yaw}" />
   </xacro:cob_head_v3>
+  <xacro:cob_lookat name="lookat" parent="torso_upper_neck_tilt_link">
+    <origin xyz="${head_x} ${head_y} ${head_z}" rpy="${head_roll} ${head_pitch} ${head_yaw}" />
+    <axis xyz="-1 0 0"/>
+  </xacro:cob_lookat>
   <xacro:schunk_sdh name="sdh" parent="arm_7_link">
     <origin xyz="${sdh_x} ${sdh_y} ${sdh_z}" rpy="${sdh_roll} ${sdh_pitch} ${sdh_yaw}" />

File: cob_hardware_config/cob3-7/urdf/calibration_default.urdf.xacro (robot description, xacro)
@@ -98,11 +98,4 @@
 	<!-- ***************************** -->
 	<!-- left | handeye calibration | relative to head_axis_link -->
-	<property name="def_cam_reference_x" value="-0.0168918076"/>
-	<property name="def_cam_reference_y" value="-0.0331605618"/>
-	<property name="def_cam_reference_z" value="-0.1227576067"/>
-	<property name="def_cam_reference_roll" value="0.8665791516"/>
-	<property name="def_cam_reference_pitch" value="-1.5610273707"/>
-	<property name="def_cam_reference_yaw" value="-0.9246703056"/>
-	<!-- left | handeye calibration | relative to head_axis_link -->
 	<property name="def_cam_l_x" value="0"/>
 	<property name="def_cam_l_y" value="0"/>
@@ -111,17 +104,24 @@
 	<property name="def_cam_l_pitch" value="0"/>
 	<property name="def_cam_l_yaw" value="0"/>
+	<!-- left | handeye calibration | relative to head_axis_link -->
+	<property name="def_cam_reference_x" value="-0.05"/>
+	<property name="def_cam_reference_y" value="-0.02"/>
+	<property name="def_cam_reference_z" value="-0.07"/>
+	<property name="def_cam_reference_roll" value="0"/>
+	<property name="def_cam_reference_pitch" value="-1.5563904314"/>
+	<property name="def_cam_reference_yaw" value="0"/>
 	<!-- right | stereo baseline calibration | relative to left camera -->
-	<property name="def_cam_r_x" value="0.120625576659"/>
-	<property name="def_cam_r_y" value="0.00069791469442"/>
-	<property name="def_cam_r_z" value="-0.000529628535957"/>
-	<property name="def_cam_r_roll" value="0.00400056610075"/>
-	<property name="def_cam_r_pitch" value="0.0120185944721"/>
-	<property name="def_cam_r_yaw" value="0.0118234806514"/>
+	<property name="def_cam_r_x" value="0.12"/>
+	<property name="def_cam_r_y" value="0"/>
+	<property name="def_cam_r_z" value="0"/>
+	<property name="def_cam_r_roll" value="0"/>
+	<property name="def_cam_r_pitch" value="0"/>
+	<property name="def_cam_r_yaw" value="0"/>
 	<!-- cam3d | handeye calibration | relative to head_axis_link -->
-	<property name="def_cam3d_x" value="-0.037555729"/>
-	<property name="def_cam3d_y" value="-0.0651598868"/>
-	<property name="def_cam3d_z" value="-0.0442883082"/>
-	<property name="def_cam3d_roll" value="-0.0652253986"/>
-	<property name="def_cam3d_pitch" value="-1.5552469375"/>
-	<property name="def_cam3d_yaw" value="0.0523406338"/>
+	<property name="def_cam3d_x" value="0.06"/>
+	<property name="def_cam3d_y" value="-0.03"/>
+	<property name="def_cam3d_z" value="0"/>
+	<property name="def_cam3d_roll" value="0"/>
+	<property name="def_cam3d_pitch" value="0"/>
+	<property name="def_cam3d_yaw" value="0"/>
 </robot>

File: cob_hardware_config/cob3-7/urdf/cob3-7.urdf.xacro (robot description, xacro)
@@ -4,5 +4,5 @@
        xmlns:interface="http://playerstage.sourceforge.net/gazebo/xmlschema/#interface"
        xmlns:xacro="http://playerstage.sourceforge.net/gazebo/xmlschema/#interface"
-       name="cob3_7" >
+       name="cob3-7" >
   <!-- common stuff -->
   <include filename="$(find cob_description)/urdf/common.xacro" />
@@ -19,4 +19,5 @@
   <!-- head -->
   <include filename="$(find cob_description)/urdf/head_v3/head.urdf.xacro" />
+  <include filename="$(find cob_description)/urdf/lookat/lookat.urdf.xacro" />
   <!-- ur_connector -->
   <include filename="$(find cob_description)/urdf/ur_connector/ur_connector.urdf.xacro" />
@@ -36,4 +37,8 @@
     <origin xyz="${head_x} ${head_y} ${head_z}" rpy="${head_roll} ${head_pitch} ${head_yaw}" />
   </xacro:cob_head_v3>
+  <xacro:cob_lookat name="lookat" parent="torso_upper_neck_tilt_link">
+    <origin xyz="${head_x} ${head_y} ${head_z}" rpy="${head_roll} ${head_pitch} ${head_yaw}" />
+    <axis xyz="-1 0 0"/>
+  </xacro:cob_lookat>
   <xacro:cob_ur_connector name="ur_connector" parent="base_link">
     <origin xyz="${ur_connector_x} ${ur_connector_y} ${ur_connector_z}" rpy="${ur_connector_roll} ${ur_connector_pitch} ${ur_connector_yaw}" />
