Commit message: remove unused and not existing lookat(.urdf.xacro) tags

File: cob_hardware_config/cob3-1/urdf/cob3-1.urdf.xacro (robot description, xacro)
@@ -16,5 +16,4 @@
   <!-- head -->
   <xacro:include filename="$(find cob_description)/urdf/head_v1/head.urdf.xacro" />
-  <xacro:include filename="$(find cob_description)/urdf/lookat/lookat.urdf.xacro" />
   <!-- arm -->
   <xacro:include filename="$(find cob_description)/urdf/lbr/lbr.urdf.xacro" />
@@ -37,8 +36,4 @@
     <origin xyz="${head_x} ${head_y} ${head_z}" rpy="${head_roll} ${head_pitch} ${head_yaw}" />
   </xacro:cob_head_v1>
-  <xacro:cob_lookat name="lookat" parent="torso_upper_neck_tilt_link" lower="-5.0" upper="5.0">
-    <origin xyz="${head_x} ${head_y} ${head_z}" rpy="${head_roll} ${head_pitch} ${head_yaw}" />
-    <axis xyz="-1 0 0"/>
-  </xacro:cob_lookat>
   <xacro:schunk_sdh name="sdh" parent="arm_7_link">
     <origin xyz="${sdh_x} ${sdh_y} ${sdh_z}" rpy="${sdh_roll} ${sdh_pitch} ${sdh_yaw}" />

Commit message: consequently remove lookat and hybrid stuff from cob3-X robots

File: cob_hardware_config/cob3-1/urdf/cob3-1.urdf.xacro (robot description, xacro)
@@ -16,5 +16,4 @@
   <!-- head -->
   <xacro:include filename="$(find cob_description)/urdf/cob3_head/head_prosilicas_kinect.urdf.xacro" />
-  <xacro:include filename="$(find cob_description)/urdf/lookat/lookat.urdf.xacro" />
   <!-- arm -->
   <xacro:include filename="$(find cob_description)/urdf/lbr/lbr.urdf.xacro" />
@@ -37,8 +36,4 @@
     <origin xyz="${head_x} ${head_y} ${head_z}" rpy="${head_roll} ${head_pitch} ${head_yaw}" />
   </xacro:head>
-  <xacro:lookat name="lookat" parent="torso_upper_neck_tilt_link" lower="-5.0" upper="5.0">
-    <origin xyz="${head_x} ${head_y} ${head_z}" rpy="${head_roll} ${head_pitch} ${head_yaw}" />
-    <axis xyz="-1 0 0"/>
-  </xacro:lookat>
   <xacro:schunk_sdh name="sdh" parent="arm_7_link">
     <origin xyz="${sdh_x} ${sdh_y} ${sdh_z}" rpy="${sdh_roll} ${sdh_pitch} ${sdh_yaw}" />

File: cob_hardware_config/cob3-2/urdf/cob3-2.urdf.xacro (robot description, xacro)
@@ -16,5 +16,4 @@
   <!-- head -->
   <xacro:include filename="$(find cob_description)/urdf/cob3_head/head_prosilicas_kinect.urdf.xacro" />
-  <xacro:include filename="$(find cob_description)/urdf/lookat/lookat.urdf.xacro" />
   <!-- arm -->
   <xacro:include filename="$(find schunk_description)/urdf/lwa/lwa.urdf.xacro" />
@@ -37,8 +36,4 @@
     <origin xyz="${head_x} ${head_y} ${head_z}" rpy="${head_roll} ${head_pitch} ${head_yaw}" />
   </xacro:head>
-  <xacro:lookat name="lookat" parent="torso_upper_neck_tilt_link" lower="-5.0" upper="5.0">
-    <origin xyz="${head_x} ${head_y} ${head_z}" rpy="${head_roll} ${head_pitch} ${head_yaw}" />
-    <axis xyz="-1 0 0"/>
-  </xacro:lookat>
   <xacro:schunk_sdh name="sdh" parent="arm_7_link">
     <origin xyz="${sdh_x} ${sdh_y} ${sdh_z}" rpy="${sdh_roll} ${sdh_pitch} ${sdh_yaw}" />

File: cob_hardware_config/cob3-3/urdf/cob3-3.urdf.xacro (robot description, xacro)
@@ -16,5 +16,4 @@
   <!-- head -->
   <xacro:include filename="$(find cob_description)/urdf/cob3_head/head_prosilicas_kinect.urdf.xacro" />
-  <xacro:include filename="$(find cob_description)/urdf/lookat/lookat.urdf.xacro" />
   <!-- arm -->
   <xacro:include filename="$(find cob_description)/urdf/lbr/lbr.urdf.xacro" />
@@ -37,8 +36,4 @@
     <origin xyz="${head_x} ${head_y} ${head_z}" rpy="${head_roll} ${head_pitch} ${head_yaw}" />
   </xacro:head>
-  <xacro:lookat name="lookat" parent="torso_upper_neck_tilt_link" lower="-5.0" upper="5.0">
-    <origin xyz="${head_x} ${head_y} ${head_z}" rpy="${head_roll} ${head_pitch} ${head_yaw}" />
-    <axis xyz="-1 0 0"/>
-  </xacro:lookat>
   <xacro:schunk_sdh name="sdh" parent="arm_7_link">
     <origin xyz="${sdh_x} ${sdh_y} ${sdh_z}" rpy="${sdh_roll} ${sdh_pitch} ${sdh_yaw}" />

File: cob_hardware_config/cob3-4/urdf/cob3-4.urdf.xacro (robot description, xacro)
@@ -16,5 +16,4 @@
   <!-- head -->
   <xacro:include filename="$(find cob_description)/urdf/cob3_head/head_prosilicas_kinect.urdf.xacro" />
-  <xacro:include filename="$(find cob_description)/urdf/lookat/lookat.urdf.xacro" />
   <!-- arm -->
   <xacro:include filename="$(find cob_description)/urdf/lbr/lbr.urdf.xacro" />
@@ -37,8 +36,4 @@
     <origin xyz="${head_x} ${head_y} ${head_z}" rpy="${head_roll} ${head_pitch} ${head_yaw}" />
   </xacro:head>
-  <xacro:lookat name="lookat" parent="torso_upper_neck_tilt_link" lower="-5.0" upper="5.0">
-    <origin xyz="${head_x} ${head_y} ${head_z}" rpy="${head_roll} ${head_pitch} ${head_yaw}" />
-    <axis xyz="-1 0 0"/>
-  </xacro:lookat>
   <xacro:schunk_sdh name="sdh" parent="arm_7_link">
     <origin xyz="${sdh_x} ${sdh_y} ${sdh_z}" rpy="${sdh_roll} ${sdh_pitch} ${sdh_yaw}" />

File: cob_hardware_config/cob3-5/urdf/cob3-5.urdf.xacro (robot description, xacro)
@@ -16,5 +16,4 @@
   <!-- head -->
   <xacro:include filename="$(find cob_description)/urdf/cob3_head/head_prosilicas_kinect.urdf.xacro" />
-  <xacro:include filename="$(find cob_description)/urdf/lookat/lookat.urdf.xacro" />
   <!-- arm -->
   <xacro:include filename="$(find schunk_description)/urdf/lwa/lwa.urdf.xacro" />
@@ -37,8 +36,4 @@
     <origin xyz="${head_x} ${head_y} ${head_z}" rpy="${head_roll} ${head_pitch} ${head_yaw}" />
   </xacro:head>
-  <xacro:lookat name="lookat" parent="torso_upper_neck_tilt_link" lower="-5.0" upper="5.0">
-    <origin xyz="${head_x} ${head_y} ${head_z}" rpy="${head_roll} ${head_pitch} ${head_yaw}" />
-    <axis xyz="-1 0 0"/>
-  </xacro:lookat>
   <xacro:schunk_sdh name="sdh" parent="arm_7_link">
     <origin xyz="${sdh_x} ${sdh_y} ${sdh_z}" rpy="${sdh_roll} ${sdh_pitch} ${sdh_yaw}" />

File: cob_hardware_config/cob3-6/urdf/cob3-6.urdf.xacro (robot description, xacro)
@@ -16,5 +16,4 @@
   <!-- head -->
   <xacro:include filename="$(find cob_description)/urdf/cob3_head/head_prosilicas_kinect.urdf.xacro" />
-  <xacro:include filename="$(find cob_description)/urdf/lookat/lookat.urdf.xacro" />
   <!-- arm -->
   <xacro:include filename="$(find schunk_description)/urdf/lwa/lwa.urdf.xacro" />
@@ -37,8 +36,4 @@
     <origin xyz="${head_x} ${head_y} ${head_z}" rpy="${head_roll} ${head_pitch} ${head_yaw}" />
   </xacro:head>
-  <xacro:lookat name="lookat" parent="torso_upper_neck_tilt_link" lower="-5.0" upper="5.0">
-    <origin xyz="${head_x} ${head_y} ${head_z}" rpy="${head_roll} ${head_pitch} ${head_yaw}" />
-    <axis xyz="-1 0 0"/>
-  </xacro:lookat>
   <xacro:schunk_sdh name="sdh" parent="arm_7_link">
     <origin xyz="${sdh_x} ${sdh_y} ${sdh_z}" rpy="${sdh_roll} ${sdh_pitch} ${sdh_yaw}" />

File: cob_hardware_config/cob3-7/urdf/cob3-7.urdf.xacro (robot description, xacro)
@@ -16,5 +16,4 @@
   <!-- head -->
   <xacro:include filename="$(find cob_description)/urdf/cob3_head/head_prosilicas_kinect.urdf.xacro" />
-  <xacro:include filename="$(find cob_description)/urdf/lookat/lookat.urdf.xacro" />
   <!-- ur_connector -->
   <xacro:include filename="$(find cob_description)/urdf/ur_connector/ur_connector.urdf.xacro" />
@@ -34,8 +33,4 @@
     <origin xyz="${head_x} ${head_y} ${head_z}" rpy="${head_roll} ${head_pitch} ${head_yaw}" />
   </xacro:head>
-  <xacro:lookat name="lookat" parent="torso_upper_neck_tilt_link" lower="-5.0" upper="5.0">
-    <origin xyz="${head_x} ${head_y} ${head_z}" rpy="${head_roll} ${head_pitch} ${head_yaw}" />
-    <axis xyz="-1 0 0"/>
-  </xacro:lookat>
   <xacro:ur_connector name="ur_connector" parent="base_link">
     <origin xyz="${ur_connector_x} ${ur_connector_y} ${ur_connector_z}" rpy="${ur_connector_roll} ${ur_connector_pitch} ${ur_connector_yaw}" />

File: cob_hardware_config/cob3-8/urdf/cob3-8.urdf.xacro (robot description, xacro)
@@ -16,5 +16,4 @@
   <!-- head -->
   <xacro:include filename="$(find cob_description)/urdf/cob3_head/head_kinect.urdf.xacro" />
-  <xacro:include filename="$(find cob_description)/urdf/lookat/lookat.urdf.xacro" />
   <!-- arm -->
   <xacro:include filename="$(find schunk_description)/urdf/lwa4d/lwa4d.urdf.xacro" />
@@ -37,5 +36,6 @@
     <origin xyz="${head_x} ${head_y} ${head_z}" rpy="${head_roll} ${head_pitch} ${head_yaw}" />
   </xacro:head>
-  <xacro:schunk_pg70 name="pg70" parent="arm_7_link">
+  <xacro:schunk_pg70 name="pg70" parent="arm_7_link" pg70_finger_left_ref="${pg70_finger_left_ref}"
+            pg70_finger_right_ref="${pg70_finger_right_ref}" >
     <origin xyz="${pg70_x} ${pg70_y} ${pg70_z}" rpy="${pg70_roll} ${pg70_pitch} ${pg70_yaw}" />
   </xacro:schunk_pg70>

Commit message: Revert "[Indigo] Velocity interface controller indigo"

File: cob_hardware_config/cob3-1/urdf/cob3-1.urdf.xacro (robot description, xacro)
@@ -16,4 +16,5 @@
   <!-- head -->
   <xacro:include filename="$(find cob_description)/urdf/cob3_head/head_prosilicas_kinect.urdf.xacro" />
+  <xacro:include filename="$(find cob_description)/urdf/lookat/lookat.urdf.xacro" />
   <!-- arm -->
   <xacro:include filename="$(find cob_description)/urdf/lbr/lbr.urdf.xacro" />
@@ -36,4 +37,8 @@
     <origin xyz="${head_x} ${head_y} ${head_z}" rpy="${head_roll} ${head_pitch} ${head_yaw}" />
   </xacro:head>
+  <xacro:lookat name="lookat" parent="torso_upper_neck_tilt_link" lower="-5.0" upper="5.0">
+    <origin xyz="${head_x} ${head_y} ${head_z}" rpy="${head_roll} ${head_pitch} ${head_yaw}" />
+    <axis xyz="-1 0 0"/>
+  </xacro:lookat>
   <xacro:schunk_sdh name="sdh" parent="arm_7_link">
     <origin xyz="${sdh_x} ${sdh_y} ${sdh_z}" rpy="${sdh_roll} ${sdh_pitch} ${sdh_yaw}" />

File: cob_hardware_config/cob3-2/urdf/cob3-2.urdf.xacro (robot description, xacro)
@@ -16,4 +16,5 @@
   <!-- head -->
   <xacro:include filename="$(find cob_description)/urdf/cob3_head/head_prosilicas_kinect.urdf.xacro" />
+  <xacro:include filename="$(find cob_description)/urdf/lookat/lookat.urdf.xacro" />
   <!-- arm -->
   <xacro:include filename="$(find schunk_description)/urdf/lwa/lwa.urdf.xacro" />
@@ -36,4 +37,8 @@
     <origin xyz="${head_x} ${head_y} ${head_z}" rpy="${head_roll} ${head_pitch} ${head_yaw}" />
   </xacro:head>
+  <xacro:lookat name="lookat" parent="torso_upper_neck_tilt_link" lower="-5.0" upper="5.0">
+    <origin xyz="${head_x} ${head_y} ${head_z}" rpy="${head_roll} ${head_pitch} ${head_yaw}" />
+    <axis xyz="-1 0 0"/>
+  </xacro:lookat>
   <xacro:schunk_sdh name="sdh" parent="arm_7_link">
     <origin xyz="${sdh_x} ${sdh_y} ${sdh_z}" rpy="${sdh_roll} ${sdh_pitch} ${sdh_yaw}" />

File: cob_hardware_config/cob3-3/urdf/cob3-3.urdf.xacro (robot description, xacro)
@@ -16,4 +16,5 @@
   <!-- head -->
   <xacro:include filename="$(find cob_description)/urdf/cob3_head/head_prosilicas_kinect.urdf.xacro" />
+  <xacro:include filename="$(find cob_description)/urdf/lookat/lookat.urdf.xacro" />
   <!-- arm -->
   <xacro:include filename="$(find cob_description)/urdf/lbr/lbr.urdf.xacro" />
@@ -36,4 +37,8 @@
     <origin xyz="${head_x} ${head_y} ${head_z}" rpy="${head_roll} ${head_pitch} ${head_yaw}" />
   </xacro:head>
+  <xacro:lookat name="lookat" parent="torso_upper_neck_tilt_link" lower="-5.0" upper="5.0">
+    <origin xyz="${head_x} ${head_y} ${head_z}" rpy="${head_roll} ${head_pitch} ${head_yaw}" />
+    <axis xyz="-1 0 0"/>
+  </xacro:lookat>
   <xacro:schunk_sdh name="sdh" parent="arm_7_link">
     <origin xyz="${sdh_x} ${sdh_y} ${sdh_z}" rpy="${sdh_roll} ${sdh_pitch} ${sdh_yaw}" />

File: cob_hardware_config/cob3-4/urdf/cob3-4.urdf.xacro (robot description, xacro)
@@ -16,4 +16,5 @@
   <!-- head -->
   <xacro:include filename="$(find cob_description)/urdf/cob3_head/head_prosilicas_kinect.urdf.xacro" />
+  <xacro:include filename="$(find cob_description)/urdf/lookat/lookat.urdf.xacro" />
   <!-- arm -->
   <xacro:include filename="$(find cob_description)/urdf/lbr/lbr.urdf.xacro" />
@@ -36,4 +37,8 @@
     <origin xyz="${head_x} ${head_y} ${head_z}" rpy="${head_roll} ${head_pitch} ${head_yaw}" />
   </xacro:head>
+  <xacro:lookat name="lookat" parent="torso_upper_neck_tilt_link" lower="-5.0" upper="5.0">
+    <origin xyz="${head_x} ${head_y} ${head_z}" rpy="${head_roll} ${head_pitch} ${head_yaw}" />
+    <axis xyz="-1 0 0"/>
+  </xacro:lookat>
   <xacro:schunk_sdh name="sdh" parent="arm_7_link">
     <origin xyz="${sdh_x} ${sdh_y} ${sdh_z}" rpy="${sdh_roll} ${sdh_pitch} ${sdh_yaw}" />

File: cob_hardware_config/cob3-5/urdf/cob3-5.urdf.xacro (robot description, xacro)
@@ -16,4 +16,5 @@
   <!-- head -->
   <xacro:include filename="$(find cob_description)/urdf/cob3_head/head_prosilicas_kinect.urdf.xacro" />
+  <xacro:include filename="$(find cob_description)/urdf/lookat/lookat.urdf.xacro" />
   <!-- arm -->
   <xacro:include filename="$(find schunk_description)/urdf/lwa/lwa.urdf.xacro" />
@@ -36,4 +37,8 @@
     <origin xyz="${head_x} ${head_y} ${head_z}" rpy="${head_roll} ${head_pitch} ${head_yaw}" />
   </xacro:head>
+  <xacro:lookat name="lookat" parent="torso_upper_neck_tilt_link" lower="-5.0" upper="5.0">
+    <origin xyz="${head_x} ${head_y} ${head_z}" rpy="${head_roll} ${head_pitch} ${head_yaw}" />
+    <axis xyz="-1 0 0"/>
+  </xacro:lookat>
   <xacro:schunk_sdh name="sdh" parent="arm_7_link">
     <origin xyz="${sdh_x} ${sdh_y} ${sdh_z}" rpy="${sdh_roll} ${sdh_pitch} ${sdh_yaw}" />

File: cob_hardware_config/cob3-6/urdf/cob3-6.urdf.xacro (robot description, xacro)
@@ -16,4 +16,5 @@
   <!-- head -->
   <xacro:include filename="$(find cob_description)/urdf/cob3_head/head_prosilicas_kinect.urdf.xacro" />
+  <xacro:include filename="$(find cob_description)/urdf/lookat/lookat.urdf.xacro" />
   <!-- arm -->
   <xacro:include filename="$(find schunk_description)/urdf/lwa/lwa.urdf.xacro" />
@@ -36,4 +37,8 @@
     <origin xyz="${head_x} ${head_y} ${head_z}" rpy="${head_roll} ${head_pitch} ${head_yaw}" />
   </xacro:head>
+  <xacro:lookat name="lookat" parent="torso_upper_neck_tilt_link" lower="-5.0" upper="5.0">
+    <origin xyz="${head_x} ${head_y} ${head_z}" rpy="${head_roll} ${head_pitch} ${head_yaw}" />
+    <axis xyz="-1 0 0"/>
+  </xacro:lookat>
   <xacro:schunk_sdh name="sdh" parent="arm_7_link">
     <origin xyz="${sdh_x} ${sdh_y} ${sdh_z}" rpy="${sdh_roll} ${sdh_pitch} ${sdh_yaw}" />

File: cob_hardware_config/cob3-7/urdf/cob3-7.urdf.xacro (robot description, xacro)
@@ -16,4 +16,5 @@
   <!-- head -->
   <xacro:include filename="$(find cob_description)/urdf/cob3_head/head_prosilicas_kinect.urdf.xacro" />
+  <xacro:include filename="$(find cob_description)/urdf/lookat/lookat.urdf.xacro" />
   <!-- ur_connector -->
   <xacro:include filename="$(find cob_description)/urdf/ur_connector/ur_connector.urdf.xacro" />
@@ -33,4 +34,8 @@
     <origin xyz="${head_x} ${head_y} ${head_z}" rpy="${head_roll} ${head_pitch} ${head_yaw}" />
   </xacro:head>
+  <xacro:lookat name="lookat" parent="torso_upper_neck_tilt_link" lower="-5.0" upper="5.0">
+    <origin xyz="${head_x} ${head_y} ${head_z}" rpy="${head_roll} ${head_pitch} ${head_yaw}" />
+    <axis xyz="-1 0 0"/>
+  </xacro:lookat>
   <xacro:ur_connector name="ur_connector" parent="base_link">
     <origin xyz="${ur_connector_x} ${ur_connector_y} ${ur_connector_z}" rpy="${ur_connector_roll} ${ur_connector_pitch} ${ur_connector_yaw}" />

File: cob_hardware_config/cob3-8/urdf/cob3-8.urdf.xacro (robot description, xacro)
@@ -16,4 +16,5 @@
   <!-- head -->
   <xacro:include filename="$(find cob_description)/urdf/cob3_head/head_kinect.urdf.xacro" />
+  <xacro:include filename="$(find cob_description)/urdf/lookat/lookat.urdf.xacro" />
   <!-- arm -->
   <xacro:include filename="$(find schunk_description)/urdf/lwa4d/lwa4d.urdf.xacro" />
@@ -36,5 +37,5 @@
     <origin xyz="${head_x} ${head_y} ${head_z}" rpy="${head_roll} ${head_pitch} ${head_yaw}" />
   </xacro:head>
-  <xacro:schunk_pg70 name="pg70" parent="arm_7_link" pg70_finger_left_ref="${pg70_finger_left_ref}" pg70_finger_right_ref="${pg70_finger_right_ref}" >
+  <xacro:schunk_pg70 name="pg70" parent="arm_7_link">
     <origin xyz="${pg70_x} ${pg70_y} ${pg70_z}" rpy="${pg70_roll} ${pg70_pitch} ${pg70_yaw}" />
   </xacro:schunk_pg70>

File: cob_hardware_config/cob4-1/urdf/cob4-1.urdf.xacro (robot description, xacro)
@@ -32,4 +32,5 @@
     <origin xyz="${sensorring_x} ${sensorring_y} ${sensorring_z}" rpy="${sensorring_roll} ${sensorring_pitch} ${sensorring_yaw}" />
   </xacro:sensorring>
+<!--
   <xacro:schunk_lwa4p_extended name="arm_right" parent="torso_3_link"
             arm_1_ref="${arm_right_1_ref}"
@@ -52,4 +53,5 @@
     <origin xyz="${arm_left_x} ${arm_left_y} ${arm_left_z}" rpy="${arm_left_roll} ${arm_left_pitch} ${arm_left_yaw}" />
   </xacro:schunk_lwa4p_extended>
+-->
   <xacro:lookat name="lookat" parent="torso_center_link" lower="0.0" upper="5.0">
     <origin xyz="0 0 0" rpy="0 0 0" />

File: cob_hardware_config/cob4-2/urdf/calibration_default.urdf.xacro (robot description, xacro)
@@ -51,5 +51,5 @@
 	<!-- arm right mount positions | relative to torso_3_link -->
 	<property name="def_arm_right_x" value="0.0"/>
-	<property name="def_arm_right_y" value="-0.014"/>
+	<property name="def_arm_right_y" value="-0.148"/>
 	<property name="def_arm_right_z" value="0.55"/>
 	<property name="def_arm_right_roll" value="1.57097"/>
@@ -58,5 +58,5 @@
 	<!-- arm left mount positions | relative to torso_3_link -->
 	<property name="def_arm_left_x" value="0.0"/>
-	<property name="def_arm_left_y" value="0.014"/>
+	<property name="def_arm_left_y" value="0.148"/>
 	<property name="def_arm_left_z" value="0.55"/>
 	<property name="def_arm_left_roll" value="1.57097"/>
