Commit message: new schunk description structure

File: cob_hardware_config/cob3-9/urdf/cob3-9.urdf.xacro (robot description, xacro)
@@ -15,5 +15,5 @@
   <xacro:include filename="$(find cob_description)/urdf/cob3_torso/torso_v2.urdf.xacro" />
   <!-- arm -->
-  <xacro:include filename="$(find schunk_description)/urdf/lwa4d/lwa4d_without_base.urdf.xacro" />
+  <xacro:include filename="$(find schunk_description)/urdf/lwa4d/lwa4d.urdf.xacro" />
   <!-- gripper -->
   <xacro:include filename="$(find schunk_description)/urdf/pg70/pg70.urdf.xacro" />
@@ -42,5 +42,5 @@
     </plugin>
   </gazebo>
-  <xacro:schunk_lwa4d_without_base name="arm" parent="base_link"
+  <xacro:schunk_lwa4d name="arm" parent="base_link" has_podest="false"
           arm_1_ref="${arm_1_ref}"
           arm_2_ref="${arm_2_ref}"
@@ -51,5 +51,5 @@
           arm_7_ref="${arm_7_ref}">
     <origin xyz="${arm_x} ${arm_y} ${arm_z}" rpy="${arm_roll} ${arm_pitch} ${arm_yaw}" />
-  </xacro:schunk_lwa4d_without_base>
+  </xacro:schunk_lwa4d>
   <gazebo>
     <plugin name="ros_control" filename="libmulti_hw_interface_gazebo_ros_control.so">

File: cob_hardware_config/cob4-1/urdf/cob4-1.urdf.xacro (robot description, xacro)
@@ -54,5 +54,5 @@
     </plugin>
   </gazebo>
-  <xacro:schunk_lwa4p_extended name="arm_right" parent="torso_3_link"
+  <xacro:schunk_lwa4p_extended name="arm_right" parent="torso_3_link" has_podest="false"
             arm_1_ref="${arm_right_1_ref}"
             arm_2_ref="${arm_right_2_ref}"
@@ -70,5 +70,5 @@
     </plugin>
   </gazebo>
-  <xacro:schunk_lwa4p_extended name="arm_left" parent="torso_3_link"
+  <xacro:schunk_lwa4p_extended name="arm_left" parent="torso_3_link" has_podest="false"
             arm_1_ref="${arm_left_1_ref}"
             arm_2_ref="${arm_left_2_ref}"

File: cob_hardware_config/cob4-2/urdf/cob4-2.urdf.xacro (robot description, xacro)
@@ -14,5 +14,5 @@
   <xacro:include filename="$(find cob_description)/urdf/lookat/lookat.urdf.xacro" />
   <!-- arm -->
-  <xacro:include filename="$(find schunk_description)/urdf/lwa4p_extended/lwa4p_extended_without_base.urdf.xacro" />
+  <xacro:include filename="$(find schunk_description)/urdf/lwa4p_extended/lwa4p_extended.urdf.xacro" />
   <!-- head -->
   <xacro:include filename="$(find cob_description)/urdf/cob4_head/head_static.urdf.xacro" />
@@ -42,15 +42,5 @@
     </plugin>
   </gazebo>
-  <!-- joint between torso_3_link and lwa4p_extended_connector_link -->
-  <joint name="arm_right_base_joint" type="fixed">
-    <origin xyz="${arm_right_x} ${arm_right_y} ${arm_right_z}" rpy="${arm_right_roll} ${arm_right_pitch} ${arm_right_yaw}" />
-    <parent link="torso_3_link"/>
-    <child link="arm_right_base_link"/>
-  </joint>
-  <!-- static part of PRL100 -->
-  <link name="arm_right_base_link">
-    <xacro:default_inertial/>
-  </link>
-  <xacro:schunk_lwa4p_extended_without_base name="arm_right" parent="arm_right_base_link"
+  <xacro:schunk_lwa4p_extended name="arm_right" parent="torso_3_link" has_podest="false"
             arm_1_ref="${arm_right_1_ref}"
             arm_2_ref="${arm_right_2_ref}"
@@ -60,6 +50,6 @@
             arm_6_ref="${arm_right_6_ref}"
             arm_7_ref="${arm_right_7_ref}">
-    <origin xyz="0 0 0.139" rpy="0 0 0" />
-  </xacro:schunk_lwa4p_extended_without_base>
+    <origin xyz="${arm_right_x} ${arm_right_y} ${arm_right_z}" rpy="${arm_right_roll} ${arm_right_pitch} ${arm_right_yaw}" />
+  </xacro:schunk_lwa4p_extended>
   <gazebo>
     <plugin name="ros_control" filename="libmulti_hw_interface_gazebo_ros_control.so">
@@ -68,15 +58,5 @@
     </plugin>
   </gazebo>
-  <!-- joint between torso_3_link and lwa4p_extended_connector_link -->
-  <joint name="arm_left_base_joint" type="fixed">
-    <origin xyz="${arm_left_x} ${arm_left_y} ${arm_left_z}" rpy="${arm_left_roll} ${arm_left_pitch} ${arm_left_yaw}" />
-    <parent link="torso_3_link"/>
-    <child link="arm_left_base_link"/>
-  </joint>
-  <!-- static part of PRL100 -->
-  <link name="arm_left_base_link">
-    <xacro:default_inertial/>
-  </link>
-  <xacro:schunk_lwa4p_extended_without_base name="arm_left" parent="arm_left_base_link"
+  <xacro:schunk_lwa4p_extended name="arm_left" parent="torso_3_link" has_podest="false"
             arm_1_ref="${arm_left_1_ref}"
             arm_2_ref="${arm_left_2_ref}"
@@ -86,6 +66,6 @@
             arm_6_ref="${arm_left_6_ref}"
             arm_7_ref="${arm_left_7_ref}">
-    <origin xyz="0 0 0.139" rpy="0 0 0" />
-  </xacro:schunk_lwa4p_extended_without_base>
+    <origin xyz="${arm_left_x} ${arm_left_y} ${arm_left_z}" rpy="${arm_left_roll} ${arm_left_pitch} ${arm_left_yaw}" />
+  </xacro:schunk_lwa4p_extended>
   <gazebo>
     <plugin name="ros_control" filename="libmulti_hw_interface_gazebo_ros_control.so">
