Commit message: gazebo controllers for cob4

File: cob_hardware_config/cob4-1/urdf/calibration_default.urdf.xacro (robot description, xacro)
@@ -43,10 +43,10 @@
 	<property name="def_head_yaw" value="0.0"/>
 	<!-- head sensors mount positions | relative to head_3_link -->
-	<property name="def_head_sensors_x" value="0.0"/>
-	<property name="def_head_sensors_y" value="0.0"/>
-	<property name="def_head_sensors_z" value="0.07"/>
-	<property name="def_head_sensors_roll" value="0.0"/>
-	<property name="def_head_sensors_pitch" value="0.0"/>
-	<property name="def_head_sensors_yaw" value="0.0"/>
+	<property name="def_sensorring_x" value="0.0"/>
+	<property name="def_sensorring_y" value="0.0"/>
+	<property name="def_sensorring_z" value="0.07"/>
+	<property name="def_sensorring_roll" value="0.0"/>
+	<property name="def_sensorring_pitch" value="0.0"/>
+	<property name="def_sensorring_yaw" value="0.0"/>
 	<!-- arm right mount positions | relative to torso_3_link -->
 	<property name="def_arm_right_x" value="0.0"/>
@@ -74,5 +74,5 @@
 	<property name="def_head_2_ref" value="0.0"/>
 	<property name="def_head_3_ref" value="0.0"/>
-	<property name="def_head_sensor_ref" value="0.0"/>
+	<property name="def_sensorring_ref" value="0.0"/>
 	<!-- arm right reference positions | used as calibration_rising for arm chain-->
 	<property name="def_arm_right_1_ref" value="0.0"/>

File: cob_hardware_config/cob4-1/urdf/cob4-1.urdf.xacro (robot description, xacro)
@@ -5,22 +5,22 @@
        xmlns:xacro="http://playerstage.sourceforge.net/gazebo/xmlschema/#interface"
        name="cob4-1" >
-  <!-- common stuff -->
-  <include filename="$(find cob_description)/urdf/common.xacro" />
-  <include filename="$(find cob_description)/urdf/materials.urdf.xacro" />
-  <include filename="$(find schunk_description)/urdf/materials.urdf.xacro" />
-  <!-- calibration -->
-  <include filename="$(find cob_hardware_config)/cob4-1/urdf/properties.urdf.xacro" />
-  <!-- base -->
-  <include filename="$(find cob_description)/urdf/base_cob4/base.urdf.xacro" />
-  <!-- torso -->
-  <include filename="$(find cob_description)/urdf/torso_cob4/torso.urdf.xacro" />
-  <!-- arm -->
-  <include filename="$(find schunk_description)/urdf/lwa4p_extended/lwa4p_extended.urdf.xacro" />
-  <!-- head -->
-  <include filename="$(find cob_description)/urdf/head_cob4/head.urdf.xacro" />
-  <!-- head_sensors -->
-  <include filename="$(find cob_description)/urdf/sensorring/sensorring.urdf.xacro" />
-  <!-- generic simulator_gazebo plugins for starting mechanism control, ros time, ros battery -->
-  <include filename="$(find cob_description)/gazebo/gazebo.urdf.xacro" />
+	<!-- common stuff -->
+	<include filename="$(find cob_description)/urdf/common.xacro" />
+	<include filename="$(find cob_description)/urdf/materials.urdf.xacro" />
+	<include filename="$(find schunk_description)/urdf/materials.urdf.xacro" />
+	<!-- calibration -->
+	<include filename="$(find cob_hardware_config)/cob4-1/urdf/properties.urdf.xacro" />
+	<!-- base -->
+	<include filename="$(find cob_description)/urdf/base_cob4/base.urdf.xacro" />
+	<!-- torso -->
+	<include filename="$(find cob_description)/urdf/torso_cob4/torso.urdf.xacro" />
+	<!-- arm -->
+	<include filename="$(find schunk_description)/urdf/lwa4p_extended/lwa4p_extended.urdf.xacro" />
+	<!-- head -->
+	<include filename="$(find cob_description)/urdf/head_cob4/head.urdf.xacro" />
+	<!-- sensorring -->
+	<include filename="$(find cob_description)/urdf/sensorring/sensorring.urdf.xacro" />
+	<!-- generic simulator_gazebo plugins for starting mechanism control, ros time, ros battery -->
+	<include filename="$(find cob_description)/gazebo/gazebo.urdf.xacro" />
 	<!-- composition of the robot -->
 	<xacro:cob4_base name="base"/>
@@ -28,9 +28,9 @@
 		<origin xyz="${torso_x} ${torso_y} ${torso_z}" rpy="${torso_roll} ${torso_pitch} ${torso_yaw}" />
 	</xacro:cob4_torso>
-	<!--xacro:cob4_head name="head" parent="torso_3_link">
+	<xacro:cob4_head name="head" parent="torso_3_link">
 		<origin xyz="${head_x} ${head_y} ${head_z}" rpy="${head_roll} ${head_pitch} ${head_yaw}" />
 	</xacro:cob4_head>
 	<xacro:cob_sensorring name="sensorring" parent="head_3_link">
-		<origin xyz="${head_sensors_x} ${head_sensors_y} ${head_sensors_z}" rpy="${head_sensors_roll} ${head_sensors_pitch} ${head_sensors_yaw}" />
+		<origin xyz="${sensorring_x} ${sensorring_y} ${sensorring_z}" rpy="${sensorring_roll} ${sensorring_pitch} ${sensorring_yaw}" />
 	</xacro:cob_sensorring>
 	<xacro:schunk_lwa4p_extended name="arm_right" parent="torso_3_link"
@@ -53,4 +53,4 @@
 						arm_7_ref="${arm_left_7_ref}">
 		<origin xyz="${arm_left_x} ${arm_left_y} ${arm_left_z}" rpy="${arm_left_roll} ${arm_left_pitch} ${arm_left_yaw}" />
-	</xacro:schunk_lwa4p_extended-->
+	</xacro:schunk_lwa4p_extended>
 </robot>

File: cob_hardware_config/cob4-1/urdf/properties.urdf.xacro (robot description, xacro)
@@ -46,10 +46,10 @@
 	<property name="head_yaw" value="${def_head_yaw+offset_head_yaw}"/>
 	<!-- head sensors mount positions | relative to head_3_link -->
-	<property name="head_sensors_x" value="${def_head_sensors_x+offset_head_sensors_x}"/>
-	<property name="head_sensors_y" value="${def_head_sensors_y+offset_head_sensors_y}"/>
-	<property name="head_sensors_z" value="${def_head_sensors_z+offset_head_sensors_z}"/>
-	<property name="head_sensors_roll" value="${def_head_sensors_roll+offset_head_sensors_roll}"/>
-	<property name="head_sensors_pitch" value="${def_head_sensors_pitch+offset_head_sensors_pitch}"/>
-	<property name="head_sensors_yaw" value="${def_head_sensors_yaw+offset_head_sensors_yaw}"/>
+	<property name="sensorring_x" value="${def_sensorring_x+offset_sensorring_x}"/>
+	<property name="sensorring_y" value="${def_sensorring_y+offset_sensorring_y}"/>
+	<property name="sensorring_z" value="${def_sensorring_z+offset_sensorring_z}"/>
+	<property name="sensorring_roll" value="${def_sensorring_roll+offset_sensorring_roll}"/>
+	<property name="sensorring_pitch" value="${def_sensorring_pitch+offset_sensorring_pitch}"/>
+	<property name="sensorring_yaw" value="${def_sensorring_yaw+offset_sensorring_yaw}"/>
 	<!-- arm mount positions | relative to torso_3_link -->
 	<property name="arm_right_x" value="${def_arm_right_x+offset_arm_right_x}"/>
@@ -79,5 +79,5 @@
 	<property name="head_2_ref" value="${def_head_2_ref+offset_head_2_ref}"/>
 	<property name="head_3_ref" value="${def_head_3_ref+offset_head_3_ref}"/>
-	<property name="head_sensor_ref" value="${def_head_sensor_ref+offset_head_sensor_ref}"/>
+	<property name="sensorring_ref" value="${def_sensorring_ref+offset_sensorring_ref}"/>
 	<!-- arm right reference positions | used as calibration_rising for arm chain-->
 	<property name="arm_right_1_ref" value="${def_arm_right_1_ref+offset_arm_right_1_ref}"/>

Commit message: cleanup: cob4-1 with torso and head; cob4-2 without torso and head

File: cob_hardware_config/cob4-1/urdf/calibration_default.urdf.xacro (robot description, xacro)
@@ -54,5 +54,5 @@
 	<property name="def_arm_right_z" value="0.55"/>
 	<property name="def_arm_right_roll" value="1.57097"/>
-	<property name="def_arm_right_pitch" value="3.14159"/>
+	<property name="def_arm_right_pitch" value="0"/>
 	<property name="def_arm_right_yaw" value="0.0"/>
 	<!-- arm left mount positions | relative to torso_3_link -->
@@ -61,5 +61,5 @@
 	<property name="def_arm_left_z" value="0.55"/>
 	<property name="def_arm_left_roll" value="1.57097"/>
-	<property name="def_arm_left_pitch" value="3.14159"/>
+	<property name="def_arm_left_pitch" value="0"/>
 	<property name="def_arm_left_yaw" value="3.14159"/>
 	<!-- *********************************** -->
@@ -74,4 +74,5 @@
 	<property name="def_head_2_ref" value="0.0"/>
 	<property name="def_head_3_ref" value="0.0"/>
+	<!-- sensorring reference positions | used as calibration_rising for sensorring chain -->
 	<property name="def_sensorring_ref" value="0.0"/>
 	<!-- arm right reference positions | used as calibration_rising for arm chain-->

File: cob_hardware_config/cob4-1/urdf/properties.urdf.xacro (robot description, xacro)
@@ -69,5 +69,4 @@
 	<!-- kinematic chain reference positions -->
 	<!-- *********************************** -->
-	<!-- torso chain calibration_offest! | relative to reference position (see below)-->
 	<!-- torso reference positions | used as calibration_rising for torso chain -->
 	<!-- ! set these values to make torso straight with (0, 0, 0) joint angles ! -->
@@ -79,4 +78,5 @@
 	<property name="head_2_ref" value="${def_head_2_ref+offset_head_2_ref}"/>
 	<property name="head_3_ref" value="${def_head_3_ref+offset_head_3_ref}"/>
+	<!-- sensorring reference positions | used as calibration_rising for sensorring chain -->
 	<property name="sensorring_ref" value="${def_sensorring_ref+offset_sensorring_ref}"/>
 	<!-- arm right reference positions | used as calibration_rising for arm chain-->

File: cob_hardware_config/cob4-2/urdf/calibration_default.urdf.xacro (robot description, xacro)
@@ -66,12 +66,5 @@
 	<!-- kinematic chain reference positions -->
 	<!-- *********************************** -->
-	<!-- torso chain calibration_offest! | relative to reference position (see below)-->
-	<property name="def_torso_1_ref" value="0.0"/>
-	<property name="def_torso_2_ref" value="0.0"/>
-	<property name="def_torso_3_ref" value="0.0"/>
-	<!-- head reference positions | used as calibration_rising for head axis chain -->
-	<property name="def_head_1_ref" value="0.0"/>
-	<property name="def_head_2_ref" value="0.0"/>
-	<property name="def_head_3_ref" value="0.0"/>
+	<!-- sensorring reference positions | used as calibration_rising for sensorring chain -->
 	<property name="def_sensorring_ref" value="0.0"/>
 	<!-- arm right reference positions | used as calibration_rising for arm chain-->

File: cob_hardware_config/cob4-2/urdf/cob4-2.urdf.xacro (robot description, xacro)
@@ -30,19 +30,7 @@
     <origin xyz="${torso_x} ${torso_y} ${torso_z}" rpy="${torso_roll} ${torso_pitch} ${torso_yaw}" />
   </xacro:torso>
-  <gazebo>
-    <plugin name="ros_control" filename="libmulti_hw_interface_gazebo_ros_control.so">
-      <robotNamespace>torso</robotNamespace>
-      <filterJointsParam>joint_names</filterJointsParam>
-    </plugin>
-  </gazebo>
   <xacro:head name="head" parent="torso_3_link">
     <origin xyz="${head_x} ${head_y} ${head_z}" rpy="${head_roll} ${head_pitch} ${head_yaw}" />
   </xacro:head>
-  <gazebo>
-    <plugin name="ros_control" filename="libmulti_hw_interface_gazebo_ros_control.so">
-      <robotNamespace>head</robotNamespace>
-      <filterJointsParam>joint_names</filterJointsParam>
-    </plugin>
-  </gazebo>
   <xacro:sensorring name="sensorring" parent="head_3_link">
     <origin xyz="${sensorring_x} ${sensorring_y} ${sensorring_z}" rpy="${sensorring_roll} ${sensorring_pitch} ${sensorring_yaw}" />
@@ -86,12 +74,4 @@
     </plugin>
   </gazebo>
-  <xacro:lookat name="torso_lookat" parent="torso_center_link" lower="0.0" upper="5.0">
-    <origin xyz="0 0 0" rpy="0 0 0" />
-    <axis xyz="1 0 0"/>
-  </xacro:lookat>
-  <xacro:lookat name="head_lookat" parent="head_center_link" lower="0.0" upper="5.0">
-    <origin xyz="0 0 0" rpy="0 0 0" />
-    <axis xyz="1 0 0"/>
-  </xacro:lookat>
   <!-- virtual component -->
 </robot>

File: cob_hardware_config/cob4-2/urdf/properties.urdf.xacro (robot description, xacro)
@@ -69,14 +69,5 @@
 	<!-- kinematic chain reference positions -->
 	<!-- *********************************** -->
-	<!-- torso chain calibration_offest! | relative to reference position (see below)-->
-	<!-- torso reference positions | used as calibration_rising for torso chain -->
-	<!-- ! set these values to make torso straight with (0, 0, 0) joint angles ! -->
-	<property name="torso_1_ref" value="${def_torso_1_ref+offset_torso_1_ref}"/>
-	<property name="torso_2_ref" value="${def_torso_2_ref+offset_torso_2_ref}"/>
-	<property name="torso_3_ref" value="${def_torso_3_ref+offset_torso_3_ref}"/>
-	<!-- head reference positions | used as calibration_rising for head axis chain -->
-	<property name="head_1_ref" value="${def_head_1_ref+offset_head_1_ref}"/>
-	<property name="head_2_ref" value="${def_head_2_ref+offset_head_2_ref}"/>
-	<property name="head_3_ref" value="${def_head_3_ref+offset_head_3_ref}"/>
+	<!-- sensorring reference positions | used as calibration_rising for sensorring chain -->
 	<property name="sensorring_ref" value="${def_sensorring_ref+offset_sensorring_ref}"/>
 	<!-- arm right reference positions | used as calibration_rising for arm chain-->

Commit message: add gripper for cob4-1

File: cob_hardware_config/cob4-1/urdf/calibration_default.urdf.xacro (robot description, xacro)
@@ -63,4 +63,18 @@
 	<property name="def_arm_left_pitch" value="0"/>
 	<property name="def_arm_left_yaw" value="3.14159"/>
+	<!-- gripper right mount positions | relative to arm_right_7_link -->
+	<property name="def_gripper_right_x" value="0.0"/>
+	<property name="def_gripper_right_y" value="0.0"/>
+	<property name="def_gripper_right_z" value="0.0748"/>
+	<property name="def_gripper_right_roll" value="0.0"/>
+	<property name="def_gripper_right_pitch" value="0.0"/>
+	<property name="def_gripper_right_yaw" value="3.14159"/>
+	<!-- gripper left mount positions | relative to arm_left_7_link -->
+	<property name="def_gripper_left_x" value="0.0"/>
+	<property name="def_gripper_left_y" value="0.0"/>
+	<property name="def_gripper_left_z" value="0.0748"/>
+	<property name="def_gripper_left_roll" value="0.0"/>
+	<property name="def_gripper_left_pitch" value="0.0"/>
+	<property name="def_gripper_left_yaw" value="3.14159"/>
 	<!-- *********************************** -->
 	<!-- kinematic chain reference positions -->
@@ -84,4 +98,10 @@
 	<property name="def_arm_right_6_ref" value="0.0"/>
 	<property name="def_arm_right_7_ref" value="0.0"/>
+	<!-- gripper right reference positions | used as calibration_rising for gripper chain-->
+	<property name="def_gripper_right_finger_1_ref" value="0.0"/>
+	<property name="def_gripper_right_finger_2_ref" value="0.0"/>
+	<!-- gripper left reference positions | used as calibration_rising for gripper chain-->
+	<property name="def_gripper_left_finger_1_ref" value="0.0"/>
+	<property name="def_gripper_left_finger_2_ref" value="0.0"/>
 	<!-- arm left reference positions | used as calibration_rising for arm chain-->
 	<property name="def_arm_left_1_ref" value="0.0"/>

File: cob_hardware_config/cob4-1/urdf/cob4-1.urdf.xacro (robot description, xacro)
@@ -15,4 +15,6 @@
   <!-- arm -->
   <xacro:include filename="$(find schunk_description)/urdf/lwa4p_extended/lwa4p_extended.urdf.xacro" />
+  <!-- gripper -->
+  <xacro:include filename="$(find cob_description)/urdf/cob4_gripper/gripper.urdf.xacro" />
   <!-- head -->
   <xacro:include filename="$(find cob_description)/urdf/cob4_head/head.urdf.xacro" />
@@ -86,4 +88,26 @@
     </plugin>
   </gazebo>
+  <xacro:gripper name="gripper_right" parent="arm_right_7_link"
+            finger_1_ref="${gripper_right_finger_1_ref}"
+            finger_2_ref="${gripper_right_finger_2_ref}" >
+    <origin xyz="${gripper_right_x} ${gripper_right_y} ${gripper_right_z}" rpy="${gripper_right_roll} ${gripper_right_pitch} ${gripper_right_yaw}" />
+  </xacro:gripper>
+  <gazebo>
+    <plugin name="ros_control" filename="libmulti_hw_interface_gazebo_ros_control.so">
+      <robotNamespace>gripper_right</robotNamespace>
+      <filterJointsParam>joint_names</filterJointsParam>
+    </plugin>
+  </gazebo>
+  <xacro:gripper name="gripper_left" parent="arm_left_7_link"
+            finger_1_ref="${gripper_left_finger_1_ref}"
+            finger_2_ref="${gripper_left_finger_2_ref}" >
+    <origin xyz="${gripper_left_x} ${gripper_left_y} ${gripper_left_z}" rpy="${gripper_left_roll} ${gripper_left_pitch} ${gripper_left_yaw}" />
+  </xacro:gripper>
+  <gazebo>
+    <plugin name="ros_control" filename="libmulti_hw_interface_gazebo_ros_control.so">
+      <robotNamespace>gripper_left</robotNamespace>
+      <filterJointsParam>joint_names</filterJointsParam>
+    </plugin>
+  </gazebo>
   <!-- virtual component -->
 <!--

File: cob_hardware_config/cob4-1/urdf/properties.urdf.xacro (robot description, xacro)
@@ -66,4 +66,18 @@
 	<property name="arm_left_pitch" value="${def_arm_left_pitch+offset_arm_left_pitch}"/>
 	<property name="arm_left_yaw" value="${def_arm_left_yaw+offset_arm_left_yaw}"/>
+	<!-- gripper right mount positions | relative to arm_right_7_link -->
+	<property name="gripper_right_x" value="${def_gripper_right_x+offset_gripper_right_x}"/>
+	<property name="gripper_right_y" value="${def_gripper_right_y+offset_gripper_right_y}"/>
+	<property name="gripper_right_z" value="${def_gripper_right_z+offset_gripper_right_z}"/>
+	<property name="gripper_right_roll" value="${def_gripper_right_roll+offset_gripper_right_roll}"/>
+	<property name="gripper_right_pitch" value="${def_gripper_right_pitch+offset_gripper_right_pitch}"/>
+	<property name="gripper_right_yaw" value="${def_gripper_right_yaw+offset_gripper_right_yaw}"/>
+	<!-- gripper left mount positions | relative to arm_left_7_link -->
+	<property name="gripper_left_x" value="${def_gripper_left_x+offset_gripper_left_x}"/>
+	<property name="gripper_left_y" value="${def_gripper_left_y+offset_gripper_left_y}"/>
+	<property name="gripper_left_z" value="${def_gripper_left_z+offset_gripper_left_z}"/>
+	<property name="gripper_left_roll" value="${def_gripper_left_roll+offset_gripper_left_roll}"/>
+	<property name="gripper_left_pitch" value="${def_gripper_left_pitch+offset_gripper_left_pitch}"/>
+	<property name="gripper_left_yaw" value="${def_gripper_left_yaw+offset_gripper_left_yaw}"/>
 	<!-- *********************************** -->
 	<!-- kinematic chain reference positions -->
@@ -96,4 +110,10 @@
 	<property name="arm_left_6_ref" value="${def_arm_left_6_ref+offset_arm_left_6_ref}"/>
 	<property name="arm_left_7_ref" value="${def_arm_left_7_ref+offset_arm_left_7_ref}"/>
+	<!-- gripper right reference positions | used as calibration_rising for gripper chain-->
+	<property name="gripper_right_finger_1_ref" value="${def_gripper_right_finger_1_ref+offset_gripper_right_finger_1_ref}"/>
+	<property name="gripper_right_finger_2_ref" value="${def_gripper_right_finger_2_ref+offset_gripper_right_finger_2_ref}"/>
+	<!-- gripper left reference positions | used as calibration_rising for gripper chain-->
+	<property name="gripper_left_finger_1_ref" value="${def_gripper_left_finger_1_ref+offset_gripper_left_finger_1_ref}"/>
+	<property name="gripper_left_finger_2_ref" value="${def_gripper_left_finger_2_ref+offset_gripper_left_finger_2_ref}"/>
 	<!-- cam3d left | handeye calibration | relative to torso_3_link -->
 	<property name="torso_cam3d_left_x" value="${def_torso_cam3d_left_x+offset_torso_cam3d_left_x}"/>
