Commit message: fixes while testing in simulation

File: cob_hardware_config/cob4-1/urdf/cob4-1.urdf.xacro (robot description, xacro)
@@ -2,52 +2,52 @@
 <robot xmlns:xacro="http://www.ros.org/wiki/xacro"
        name="cob4-1" >
-	<!-- common stuff -->
-	<xacro:include filename="$(find cob_description)/urdf/common.xacro" />
-	<xacro:include filename="$(find cob_description)/urdf/materials.urdf.xacro" />
-	<xacro:include filename="$(find schunk_description)/urdf/materials.urdf.xacro" />
-	<!-- calibration -->
-	<xacro:include filename="$(find cob_hardware_config)/cob4-1/urdf/properties.urdf.xacro" />
-	<!-- base -->
-	<xacro:include filename="$(find cob_description)/urdf/cob4_base/base.urdf.xacro" />
-	<!-- torso -->
-	<xacro:include filename="$(find cob_description)/urdf/cob4_torso/torso.urdf.xacro" />
-	<!-- arm -->
-	<xacro:include filename="$(find schunk_description)/urdf/lwa4p_extended/lwa4p_extended.urdf.xacro" />
-	<!-- head -->
-	<xacro:include filename="$(find cob_description)/urdf/cob4_head/head.urdf.xacro" />
-	<!-- sensorring -->
-	<xacro:include filename="$(find cob_description)/urdf/cob4_sensorring/sensorring.urdf.xacro" />
-	<!-- generic simulator_gazebo plugins for starting mechanism control, ros time, ros battery -->
-	<xacro:include filename="$(find cob_description)/gazebo/gazebo.urdf.xacro" />
-	<!-- composition of the robot -->
-	<xacro:base name="base"/>
-	<xacro:torso name="torso" parent="base_link">
-		<origin xyz="${torso_x} ${torso_y} ${torso_z}" rpy="${torso_roll} ${torso_pitch} ${torso_yaw}" />
-	</xacro:torso>
-	<xacro:head name="head" parent="torso_3_link">
-		<origin xyz="${head_x} ${head_y} ${head_z}" rpy="${head_roll} ${head_pitch} ${head_yaw}" />
-	</xacro:head>
-	<xacro:sensorring name="sensorring" parent="head_3_link">
-		<origin xyz="${sensorring_x} ${sensorring_y} ${sensorring_z}" rpy="${sensorring_roll} ${sensorring_pitch} ${sensorring_yaw}" />
-	</xacro:sensorring>
-	<xacro:schunk_lwa4p_extended name="arm_right" parent="torso_3_link"
-						arm_1_ref="${arm_right_1_ref}"
-						arm_2_ref="${arm_right_2_ref}"
-						arm_3_ref="${arm_right_3_ref}"
-						arm_4_ref="${arm_right_4_ref}"
-						arm_5_ref="${arm_right_5_ref}"
-						arm_6_ref="${arm_right_6_ref}"
-						arm_7_ref="${arm_right_7_ref}">
-		<origin xyz="${arm_right_x} ${arm_right_y} ${arm_right_z}" rpy="${arm_right_roll} ${arm_right_pitch} ${arm_right_yaw}" />
-	</xacro:schunk_lwa4p_extended>
-	<xacro:schunk_lwa4p_extended name="arm_left" parent="torso_3_link"
-						arm_1_ref="${arm_left_1_ref}"
-						arm_2_ref="${arm_left_2_ref}"
-						arm_3_ref="${arm_left_3_ref}"
-						arm_4_ref="${arm_left_4_ref}"
-						arm_5_ref="${arm_left_5_ref}"
-						arm_6_ref="${arm_left_6_ref}"
-						arm_7_ref="${arm_left_7_ref}">
-		<origin xyz="${arm_left_x} ${arm_left_y} ${arm_left_z}" rpy="${arm_left_roll} ${arm_left_pitch} ${arm_left_yaw}" />
-	</xacro:schunk_lwa4p_extended>
+  <!-- common stuff -->
+  <xacro:include filename="$(find cob_description)/urdf/common.xacro" />
+  <xacro:include filename="$(find cob_description)/urdf/materials.urdf.xacro" />
+  <xacro:include filename="$(find schunk_description)/urdf/materials.urdf.xacro" />
+  <!-- calibration -->
+  <xacro:include filename="$(find cob_hardware_config)/cob4-1/urdf/properties.urdf.xacro" />
+  <!-- base -->
+  <xacro:include filename="$(find cob_description)/urdf/cob4_base/base.urdf.xacro" />
+  <!-- torso -->
+  <xacro:include filename="$(find cob_description)/urdf/cob4_torso/torso.urdf.xacro" />
+  <!-- arm -->
+  <xacro:include filename="$(find schunk_description)/urdf/lwa4p_extended/lwa4p_extended.urdf.xacro" />
+  <!-- head -->
+  <xacro:include filename="$(find cob_description)/urdf/cob4_head/head.urdf.xacro" />
+  <!-- sensorring -->
+  <xacro:include filename="$(find cob_description)/urdf/cob4_sensorring/sensorring.urdf.xacro" />
+  <!-- generic simulator_gazebo plugins for starting mechanism control, ros time, ros battery -->
+  <xacro:include filename="$(find cob_description)/gazebo/gazebo.urdf.xacro" />
+  <!-- composition of the robot -->
+  <xacro:base name="base"/>
+  <xacro:torso name="torso" parent="base_link">
+    <origin xyz="${torso_x} ${torso_y} ${torso_z}" rpy="${torso_roll} ${torso_pitch} ${torso_yaw}" />
+  </xacro:torso>
+  <xacro:head name="head" parent="torso_3_link">
+    <origin xyz="${head_x} ${head_y} ${head_z}" rpy="${head_roll} ${head_pitch} ${head_yaw}" />
+  </xacro:head>
+  <xacro:sensorring name="sensorring" parent="head_3_link">
+    <origin xyz="${sensorring_x} ${sensorring_y} ${sensorring_z}" rpy="${sensorring_roll} ${sensorring_pitch} ${sensorring_yaw}" />
+  </xacro:sensorring>
+  <xacro:schunk_lwa4p_extended name="arm_right" parent="torso_3_link"
+            arm_1_ref="${arm_right_1_ref}"
+            arm_2_ref="${arm_right_2_ref}"
+            arm_3_ref="${arm_right_3_ref}"
+            arm_4_ref="${arm_right_4_ref}"
+            arm_5_ref="${arm_right_5_ref}"
+            arm_6_ref="${arm_right_6_ref}"
+            arm_7_ref="${arm_right_7_ref}">
+    <origin xyz="${arm_right_x} ${arm_right_y} ${arm_right_z}" rpy="${arm_right_roll} ${arm_right_pitch} ${arm_right_yaw}" />
+  </xacro:schunk_lwa4p_extended>
+  <xacro:schunk_lwa4p_extended name="arm_left" parent="torso_3_link"
+            arm_1_ref="${arm_left_1_ref}"
+            arm_2_ref="${arm_left_2_ref}"
+            arm_3_ref="${arm_left_3_ref}"
+            arm_4_ref="${arm_left_4_ref}"
+            arm_5_ref="${arm_left_5_ref}"
+            arm_6_ref="${arm_left_6_ref}"
+            arm_7_ref="${arm_left_7_ref}">
+    <origin xyz="${arm_left_x} ${arm_left_y} ${arm_left_z}" rpy="${arm_left_roll} ${arm_left_pitch} ${arm_left_yaw}" />
+  </xacro:schunk_lwa4p_extended>
 </robot>

File: cob_hardware_config/cob4-1/urdf/properties.urdf.xacro (robot description, xacro)
@@ -1,7 +1,7 @@
 <?xml version="1.0" ?>
-<robot>
+<robot xmlns:xacro="http://www.ros.org/wiki/xacro">
 	<!--reference calc-->
 	<xacro:include filename="$(find cob_calibration_data)/cob4-1/calibration/calibration_offset.urdf.xacro" />
-	<xacro:include filename="$(find cob_hardware_config)/cob4-1/urdf/calibration_default.urdf.xacro" />>
+	<xacro:include filename="$(find cob_hardware_config)/cob4-1/urdf/calibration_default.urdf.xacro" />
 	<!-- ***************** -->
 	<!-- base calibration -->

Commit message: lookat component for cob4-1

File: cob_hardware_config/cob4-1/urdf/cob4-1.urdf.xacro (robot description, xacro)
@@ -12,4 +12,5 @@
   <!-- torso -->
   <xacro:include filename="$(find cob_description)/urdf/cob4_torso/torso.urdf.xacro" />
+  <xacro:include filename="$(find cob_description)/urdf/lookat/lookat.urdf.xacro" />
   <!-- arm -->
   <xacro:include filename="$(find schunk_description)/urdf/lwa4p_extended/lwa4p_extended.urdf.xacro" />
@@ -51,3 +52,7 @@
     <origin xyz="${arm_left_x} ${arm_left_y} ${arm_left_z}" rpy="${arm_left_roll} ${arm_left_pitch} ${arm_left_yaw}" />
   </xacro:schunk_lwa4p_extended>
+  <xacro:lookat name="lookat" parent="torso_center_link" lower="0.0" upper="5.0">
+    <origin xyz="0 0 0" rpy="0 0 0" />
+    <axis xyz="1 0 0"/>
+  </xacro:lookat>
 </robot>

Commit message: remove lookat

File: cob_hardware_config/cob4-1/urdf/cob4-1.urdf.xacro (robot description, xacro)
@@ -12,5 +12,4 @@
   <!-- torso -->
   <xacro:include filename="$(find cob_description)/urdf/cob4_torso/torso_3dof.urdf.xacro" />
-  <xacro:include filename="$(find cob_description)/urdf/lookat/lookat.urdf.xacro" />
   <!-- arm -->
   <xacro:include filename="$(find schunk_description)/urdf/lwa4p_extended/lwa4p_extended.urdf.xacro" />
@@ -92,10 +91,3 @@
     </plugin>
   </gazebo>
-  <!-- virtual component -->
-<!--
-  <xacro:lookat name="lookat" parent="torso_center_link" lower="0.0" upper="5.0">
-    <origin xyz="0 0 0" rpy="0 0 0" />
-    <axis xyz="1 0 0"/>
-  </xacro:lookat>
--->
 </robot>

File: cob_hardware_config/cob4-2/urdf/cob4-2.urdf.xacro (robot description, xacro)
@@ -12,5 +12,4 @@
   <!-- torso -->
   <xacro:include filename="$(find cob_description)/urdf/cob4_torso/torso_2dof.urdf.xacro" />
-  <xacro:include filename="$(find cob_description)/urdf/lookat/lookat.urdf.xacro" />
   <!-- arm -->
   <xacro:include filename="$(find schunk_description)/urdf/lwa4p_extended/lwa4p_extended.urdf.xacro" />
@@ -86,4 +85,3 @@
     </plugin>
   </gazebo>
-  <!-- virtual component -->
 </robot>

File: cob_hardware_config/raw3-3/urdf/raw3-3.urdf.xacro (robot description, xacro)
@@ -29,10 +29,4 @@
   <!-- prace macros -->
   <xacro:prace/>
-<!--
-  <xacro:lookat name="lookat" parent="head_cam_holder_link" lower="0.0" upper="8.0">
-    <origin xyz="${head_x} ${head_y} ${head_z}" rpy="${head_roll} ${head_pitch} ${head_yaw}" />
-    <axis xyz="1 0 0"/>
-  </xacro:lookat>
--->
   <!-- scan top mount -->
     <joint name="base_laser_top_joint" type="fixed" >

Commit message: use cob4-1 as cob4-2 without arms - copying configuration files

File: cob_hardware_config/cob4-1/urdf/cob4-1.urdf.xacro (robot description, xacro)
@@ -11,13 +11,9 @@
   <xacro:include filename="$(find cob_description)/urdf/cob4_base/base.urdf.xacro" />
   <!-- torso -->
-  <xacro:include filename="$(find cob_description)/urdf/cob4_torso/torso_3dof.urdf.xacro" />
-  <!-- arm -->
-  <xacro:include filename="$(find schunk_description)/urdf/lwa4p_extended/lwa4p_extended.urdf.xacro" />
-  <!-- gripper -->
-  <xacro:include filename="$(find cob_description)/urdf/cob4_gripper/gripper.urdf.xacro" />
+  <xacro:include filename="$(find cob_description)/urdf/cob4_torso/torso_2dof.urdf.xacro" />
   <!-- head -->
-  <xacro:include filename="$(find cob_description)/urdf/cob4_head/head.urdf.xacro" />
+  <xacro:include filename="$(find cob_description)/urdf/cob4_head/head_static.urdf.xacro" />
   <!-- sensorring -->
-  <xacro:include filename="$(find cob_description)/urdf/cob4_sensorring/sensorring.urdf.xacro" />
+  <xacro:include filename="$(find cob_description)/urdf/cob4_sensorring/sensorring_asus.urdf.xacro" />
   <!-- composition of the robot -->
   <xacro:base name="base" use_old_joint_names="true"/>
@@ -40,10 +36,4 @@
     <origin xyz="${head_x} ${head_y} ${head_z}" rpy="${head_roll} ${head_pitch} ${head_yaw}" />
   </xacro:head>
-  <gazebo>
-    <plugin name="ros_control" filename="libhwi_switch_gazebo_ros_control.so">
-      <robotNamespace>head</robotNamespace>
-      <filterJointsParam>joint_names</filterJointsParam>
-    </plugin>
-  </gazebo>
   <xacro:sensorring name="sensorring" parent="head_3_link">
     <origin xyz="${sensorring_x} ${sensorring_y} ${sensorring_z}" rpy="${sensorring_roll} ${sensorring_pitch} ${sensorring_yaw}" />
@@ -55,39 +45,3 @@
     </plugin>
   </gazebo>
-  <xacro:schunk_lwa4p_extended name="arm_right" parent="torso_3_link" has_podest="false">
-    <origin xyz="${arm_right_x} ${arm_right_y} ${arm_right_z}" rpy="${arm_right_roll} ${arm_right_pitch} ${arm_right_yaw}" />
-  </xacro:schunk_lwa4p_extended>
-  <gazebo>
-    <plugin name="ros_control" filename="libhwi_switch_gazebo_ros_control.so">
-      <robotNamespace>arm_right</robotNamespace>
-      <filterJointsParam>joint_names</filterJointsParam>
-    </plugin>
-  </gazebo>
-  <xacro:schunk_lwa4p_extended name="arm_left" parent="torso_3_link" has_podest="false">
-    <origin xyz="${arm_left_x} ${arm_left_y} ${arm_left_z}" rpy="${arm_left_roll} ${arm_left_pitch} ${arm_left_yaw}" />
-  </xacro:schunk_lwa4p_extended>
-  <gazebo>
-    <plugin name="ros_control" filename="libhwi_switch_gazebo_ros_control.so">
-      <robotNamespace>arm_left</robotNamespace>
-      <filterJointsParam>joint_names</filterJointsParam>
-    </plugin>
-  </gazebo>
-  <xacro:gripper name="gripper_right" parent="arm_right_7_link">
-    <origin xyz="${gripper_right_x} ${gripper_right_y} ${gripper_right_z}" rpy="${gripper_right_roll} ${gripper_right_pitch} ${gripper_right_yaw}" />
-  </xacro:gripper>
-  <gazebo>
-    <plugin name="ros_control" filename="libhwi_switch_gazebo_ros_control.so">
-      <robotNamespace>gripper_right</robotNamespace>
-      <filterJointsParam>joint_names</filterJointsParam>
-    </plugin>
-  </gazebo>
-  <xacro:gripper name="gripper_left" parent="arm_left_7_link">
-    <origin xyz="${gripper_left_x} ${gripper_left_y} ${gripper_left_z}" rpy="${gripper_left_roll} ${gripper_left_pitch} ${gripper_left_yaw}" />
-  </xacro:gripper>
-  <gazebo>
-    <plugin name="ros_control" filename="libhwi_switch_gazebo_ros_control.so">
-      <robotNamespace>gripper_left</robotNamespace>
-      <filterJointsParam>joint_names</filterJointsParam>
-    </plugin>
-  </gazebo>
 </robot>

Commit message: move sensors from head xacro to robot xacro

File: cob_hardware_config/cob4-1/urdf/cob4-1.urdf.xacro (robot description, xacro)
@@ -14,4 +14,5 @@
   <!-- head -->
   <xacro:include filename="$(find cob_description)/urdf/cob4_head/head.urdf.xacro" />
+  <xacro:include filename="$(find cob_description)/urdf/sensors/usb_cam.urdf.xacro" />
   <!-- sensorring -->
   <xacro:include filename="$(find cob_description)/urdf/cob4_sensorring/sensorring_asus.urdf.xacro" />
@@ -36,4 +37,7 @@
     <origin xyz="${head_x} ${head_y} ${head_z}" rpy="${head_roll} ${head_pitch} ${head_yaw}" />
   </xacro:head>
+  <xacro:usb_cam name="head_cam" parent="head_3_link" ros_topic="head_cam">
+    <origin xyz="${head_cam_x} ${head_cam_y} ${head_cam_z}" rpy="${head_cam_roll} ${head_cam_pitch} ${head_cam_yaw}" />
+  </xacro:usb_cam>
   <gazebo>
     <plugin name="ros_control" filename="libhwi_switch_gazebo_ros_control.so">

File: cob_hardware_config/cob4-10/urdf/cob4-10.urdf.xacro (robot description, xacro)
@@ -14,4 +14,5 @@
   <!-- head -->
   <xacro:include filename="$(find cob_description)/urdf/cob4_head/head.urdf.xacro" />
+  <xacro:include filename="$(find cob_description)/urdf/sensors/usb_cam.urdf.xacro" />
   <!-- sensorring -->
   <xacro:include filename="$(find cob_description)/urdf/cob4_sensorring/sensorring_asus.urdf.xacro" />
@@ -36,4 +37,7 @@
     <origin xyz="${head_x} ${head_y} ${head_z}" rpy="${head_roll} ${head_pitch} ${head_yaw}" />
   </xacro:head>
+  <xacro:usb_cam name="head_cam" parent="head_3_link" ros_topic="head_cam">
+    <origin xyz="${head_cam_x} ${head_cam_y} ${head_cam_z}" rpy="${head_cam_roll} ${head_cam_pitch} ${head_cam_yaw}" />
+  </xacro:usb_cam>
   <gazebo>
     <plugin name="ros_control" filename="libhwi_switch_gazebo_ros_control.so">

File: cob_hardware_config/cob4-2/urdf/cob4-2.urdf.xacro (robot description, xacro)
@@ -18,4 +18,5 @@
   <!-- head -->
   <xacro:include filename="$(find cob_description)/urdf/cob4_head/head.urdf.xacro" />
+  <xacro:include filename="$(find cob_description)/urdf/sensors/usb_cam.urdf.xacro" />
   <!-- sensorring -->
   <xacro:include filename="$(find cob_description)/urdf/cob4_sensorring/sensorring_asus.urdf.xacro" />
@@ -40,4 +41,7 @@
     <origin xyz="${head_x} ${head_y} ${head_z}" rpy="${head_roll} ${head_pitch} ${head_yaw}" />
   </xacro:head>
+  <xacro:usb_cam name="head_cam" parent="head_3_link" ros_topic="head_cam">
+    <origin xyz="${head_cam_x} ${head_cam_y} ${head_cam_z}" rpy="${head_cam_roll} ${head_cam_pitch} ${head_cam_yaw}" />
+  </xacro:usb_cam>
   <gazebo>
     <plugin name="ros_control" filename="libhwi_switch_gazebo_ros_control.so">

File: cob_hardware_config/cob4-5/urdf/cob4-5.urdf.xacro (robot description, xacro)
@@ -18,4 +18,5 @@
   <!-- head -->
   <xacro:include filename="$(find cob_description)/urdf/cob4_head/head_static.urdf.xacro" />
+  <xacro:include filename="$(find cob_description)/urdf/sensors/usb_cam.urdf.xacro" />
   <!-- sensorring -->
   <xacro:include filename="$(find cob_description)/urdf/cob4_sensorring/sensorring_3dcs_asus.urdf.xacro" />
@@ -34,4 +35,7 @@
     <origin xyz="${head_x} ${head_y} ${head_z}" rpy="${head_roll} ${head_pitch} ${head_yaw}" />
   </xacro:head>
+  <xacro:usb_cam name="head_cam" parent="head_3_link" ros_topic="head_cam">
+    <origin xyz="${head_cam_x} ${head_cam_y} ${head_cam_z}" rpy="${head_cam_roll} ${head_cam_pitch} ${head_cam_yaw}" />
+  </xacro:usb_cam>
   <xacro:sensorring name="sensorring" parent="head_3_link">
     <origin xyz="${sensorring_x} ${sensorring_y} ${sensorring_z}" rpy="${sensorring_roll} ${sensorring_pitch} ${sensorring_yaw}" />

File: cob_hardware_config/cob4-7/urdf/cob4-7.urdf.xacro (robot description, xacro)
@@ -16,4 +16,5 @@
   <!-- head -->
   <xacro:include filename="$(find cob_description)/urdf/cob4_head/head.urdf.xacro" />
+  <xacro:include filename="$(find cob_description)/urdf/sensors/usb_cam.urdf.xacro" />
   <!-- sensorring -->
   <xacro:include filename="$(find cob_description)/urdf/cob4_sensorring/sensorring_asus.urdf.xacro" />
@@ -56,4 +57,7 @@
     <origin xyz="${head_x} ${head_y} ${head_z}" rpy="${head_roll} ${head_pitch} ${head_yaw}" />
   </xacro:head>
+  <xacro:usb_cam name="head_cam" parent="head_3_link" ros_topic="head_cam">
+    <origin xyz="${head_cam_x} ${head_cam_y} ${head_cam_z}" rpy="${head_cam_roll} ${head_cam_pitch} ${head_cam_yaw}" />
+  </xacro:usb_cam>
   <gazebo>
     <plugin name="ros_control" filename="libhwi_switch_gazebo_ros_control.so">

Commit message: move sensors from sensorring xacro to robot xacro

File: cob_hardware_config/cob4-1/urdf/cob4-1.urdf.xacro (robot description, xacro)
@@ -17,4 +17,5 @@
   <!-- sensorring -->
   <xacro:include filename="$(find cob_description)/urdf/cob4_sensorring/sensorring_asus.urdf.xacro" />
+  <xacro:include filename="$(find cob_description)/urdf/sensors/kinect.urdf.xacro" />
   <!-- composition of the robot -->
   <xacro:base name="base" use_old_joint_names="false"/>
@@ -49,4 +50,7 @@
     <origin xyz="${sensorring_x} ${sensorring_y} ${sensorring_z}" rpy="${sensorring_roll} ${sensorring_pitch} ${sensorring_yaw}" />
   </xacro:sensorring>
+  <xacro:cob_kinect_v0 name="sensorring_cam3d" ros_topic="sensorring_cam3d" parent="sensorring_link">
+    <origin xyz="${sensorring_cam3d_x} ${sensorring_cam3d_y} ${sensorring_cam3d_z}" rpy="${sensorring_cam3d_roll} ${sensorring_cam3d_pitch} ${sensorring_cam3d_yaw}" />
+  </xacro:cob_kinect_v0>
   <gazebo>
     <plugin name="ros_control" filename="libhwi_switch_gazebo_ros_control.so">

File: cob_hardware_config/cob4-10/urdf/cob4-10.urdf.xacro (robot description, xacro)
@@ -17,4 +17,5 @@
   <!-- sensorring -->
   <xacro:include filename="$(find cob_description)/urdf/cob4_sensorring/sensorring_asus.urdf.xacro" />
+  <xacro:include filename="$(find cob_description)/urdf/sensors/kinect.urdf.xacro" />
   <!-- composition of the robot -->
   <xacro:base name="base" use_old_joint_names="false"/>
@@ -49,4 +50,7 @@
     <origin xyz="${sensorring_x} ${sensorring_y} ${sensorring_z}" rpy="${sensorring_roll} ${sensorring_pitch} ${sensorring_yaw}" />
   </xacro:sensorring>
+  <xacro:cob_kinect_v0 name="sensorring_cam3d" ros_topic="sensorring_cam3d" parent="sensorring_link">
+    <origin xyz="${sensorring_cam3d_x} ${sensorring_cam3d_y} ${sensorring_cam3d_z}" rpy="${sensorring_cam3d_roll} ${sensorring_cam3d_pitch} ${sensorring_cam3d_yaw}" />
+  </xacro:cob_kinect_v0>
   <gazebo>
     <plugin name="ros_control" filename="libhwi_switch_gazebo_ros_control.so">

File: cob_hardware_config/cob4-2/urdf/cob4-2.urdf.xacro (robot description, xacro)
@@ -21,4 +21,5 @@
   <!-- sensorring -->
   <xacro:include filename="$(find cob_description)/urdf/cob4_sensorring/sensorring_asus.urdf.xacro" />
+  <xacro:include filename="$(find cob_description)/urdf/sensors/kinect.urdf.xacro" />
   <!-- composition of the robot -->
   <xacro:base name="base" use_old_joint_names="false"/>
@@ -53,4 +54,7 @@
     <origin xyz="${sensorring_x} ${sensorring_y} ${sensorring_z}" rpy="${sensorring_roll} ${sensorring_pitch} ${sensorring_yaw}" />
   </xacro:sensorring>
+  <xacro:cob_kinect_v0 name="sensorring_cam3d" ros_topic="sensorring_cam3d" parent="sensorring_link">
+    <origin xyz="${sensorring_cam3d_x} ${sensorring_cam3d_y} ${sensorring_cam3d_z}" rpy="${sensorring_cam3d_roll} ${sensorring_cam3d_pitch} ${sensorring_cam3d_yaw}" />
+  </xacro:cob_kinect_v0>
   <gazebo>
     <plugin name="ros_control" filename="libhwi_switch_gazebo_ros_control.so">

File: cob_hardware_config/cob4-5/urdf/cob4-5.urdf.xacro (robot description, xacro)
@@ -21,4 +21,6 @@
   <!-- sensorring -->
   <xacro:include filename="$(find cob_description)/urdf/cob4_sensorring/sensorring_3dcs_asus.urdf.xacro" />
+  <xacro:include filename="$(find cob_description)/urdf/sensors/sick_3dcs.urdf.xacro" />
+  <xacro:include filename="$(find cob_description)/urdf/sensors/kinect.urdf.xacro" />
   <!-- composition of the robot -->
   <xacro:base name="base" use_old_joint_names="false"/>
@@ -41,4 +43,11 @@
     <origin xyz="${sensorring_x} ${sensorring_y} ${sensorring_z}" rpy="${sensorring_roll} ${sensorring_pitch} ${sensorring_yaw}" />
   </xacro:sensorring>
+  <!-- cameras -->
+  <xacro:sick_3dcs name="sensorring_cam3d_front" ros_topic="sensorring_cam3d_front" parent="sensorring_link">
+    <origin xyz="${sensorring_cam3d_front_x} ${sensorring_cam3d_front_y} ${sensorring_cam3d_front_z}" rpy="${sensorring_cam3d_front_roll} ${sensorring_cam3d_front_pitch} ${sensorring_cam3d_front_yaw}" />
+  </xacro:sick_3dcs>
+  <xacro:cob_kinect_v0 name="sensorring_cam3d_back" ros_topic="sensorring_cam3d_back" parent="sensorring_link">
+    <origin xyz="${sensorring_cam3d_back_x} ${sensorring_cam3d_back_y} ${sensorring_cam3d_back_z}" rpy="${sensorring_cam3d_back_roll} ${sensorring_cam3d_back_pitch} ${sensorring_cam3d_back_yaw}" />
+  </xacro:cob_kinect_v0>
   <gazebo>
     <plugin name="ros_control" filename="libhwi_switch_gazebo_ros_control.so">

File: cob_hardware_config/cob4-7/urdf/cob4-7.urdf.xacro (robot description, xacro)
@@ -19,4 +19,5 @@
   <!-- sensorring -->
   <xacro:include filename="$(find cob_description)/urdf/cob4_sensorring/sensorring_asus.urdf.xacro" />
+  <xacro:include filename="$(find cob_description)/urdf/sensors/kinect.urdf.xacro" />
   <!-- composition of the robot -->
   <xacro:base name="base" use_old_joint_names="false"/>
@@ -69,4 +70,7 @@
     <origin xyz="${sensorring_x} ${sensorring_y} ${sensorring_z}" rpy="${sensorring_roll} ${sensorring_pitch} ${sensorring_yaw}" />
   </xacro:sensorring>
+  <xacro:cob_kinect_v0 name="sensorring_cam3d" ros_topic="sensorring_cam3d" parent="sensorring_link">
+    <origin xyz="${sensorring_cam3d_x} ${sensorring_cam3d_y} ${sensorring_cam3d_z}" rpy="${sensorring_cam3d_roll} ${sensorring_cam3d_pitch} ${sensorring_cam3d_yaw}" />
+  </xacro:cob_kinect_v0>
   <gazebo>
     <plugin name="ros_control" filename="libhwi_switch_gazebo_ros_control.so">
