Commit message: more consistency and harmonization changes

File: cob_hardware_config/cob3-2/urdf/cob3-2.urdf.xacro (robot description, xacro)
@@ -2,5 +2,4 @@
 <robot xmlns:xacro="http://www.ros.org/wiki/xacro"
        name="cob3-2" >
-  <xacro:arg name="robot_id" default="/"/>
   <!-- common stuff -->
   <xacro:include filename="$(find cob_description)/urdf/common.xacro" />
@@ -25,5 +24,5 @@
   <gazebo>
     <plugin name="ros_control" filename="libhwi_switch_gazebo_ros_control.so">
-      <robotNamespace>$(arg robot_id)/base</robotNamespace>
+      <robotNamespace>base</robotNamespace>
       <filterJointsParam>joint_names</filterJointsParam>
     </plugin>
@@ -34,5 +33,5 @@
   <gazebo>
     <plugin name="ros_control" filename="libhwi_switch_gazebo_ros_control.so">
-      <robotNamespace>$(arg robot_id)/tray</robotNamespace>
+      <robotNamespace>tray</robotNamespace>
       <filterJointsParam>joint_names</filterJointsParam>
     </plugin>
@@ -43,5 +42,5 @@
   <gazebo>
     <plugin name="ros_control" filename="libhwi_switch_gazebo_ros_control.so">
-      <robotNamespace>$(arg robot_id)/torso</robotNamespace>
+      <robotNamespace>torso</robotNamespace>
       <filterJointsParam>joint_names</filterJointsParam>
     </plugin>
@@ -52,5 +51,5 @@
   <gazebo>
     <plugin name="ros_control" filename="libhwi_switch_gazebo_ros_control.so">
-      <robotNamespace>$(arg robot_id)/arm</robotNamespace>
+      <robotNamespace>arm</robotNamespace>
       <filterJointsParam>joint_names</filterJointsParam>
     </plugin>
@@ -61,5 +60,5 @@
   <gazebo>
     <plugin name="ros_control" filename="libhwi_switch_gazebo_ros_control.so">
-      <robotNamespace>$(arg robot_id)/head</robotNamespace>
+      <robotNamespace>head</robotNamespace>
       <filterJointsParam>joint_names</filterJointsParam>
     </plugin>
@@ -70,5 +69,5 @@
   <gazebo>
     <plugin name="ros_control" filename="libhwi_switch_gazebo_ros_control.so">
-      <robotNamespace>$(arg robot_id)/gripper</robotNamespace>
+      <robotNamespace>gripper</robotNamespace>
       <filterJointsParam>joint_names</filterJointsParam>
     </plugin>

File: cob_hardware_config/cob3-6/urdf/cob3-6.urdf.xacro (robot description, xacro)
@@ -2,5 +2,4 @@
 <robot xmlns:xacro="http://www.ros.org/wiki/xacro"
        name="cob3-6" >
-  <xacro:arg name="robot_id" default="/"/>
   <!-- common stuff -->
   <xacro:include filename="$(find cob_description)/urdf/common.xacro" />
@@ -25,5 +24,5 @@
   <gazebo>
     <plugin name="ros_control" filename="libhwi_switch_gazebo_ros_control.so">
-      <robotNamespace>$(arg robot_id)/base</robotNamespace>
+      <robotNamespace>base</robotNamespace>
       <filterJointsParam>joint_names</filterJointsParam>
     </plugin>
@@ -34,5 +33,5 @@
   <gazebo>
     <plugin name="ros_control" filename="libhwi_switch_gazebo_ros_control.so">
-      <robotNamespace>$(arg robot_id)/tray</robotNamespace>
+      <robotNamespace>tray</robotNamespace>
       <filterJointsParam>joint_names</filterJointsParam>
     </plugin>
@@ -43,5 +42,5 @@
   <gazebo>
     <plugin name="ros_control" filename="libhwi_switch_gazebo_ros_control.so">
-      <robotNamespace>$(arg robot_id)/torso</robotNamespace>
+      <robotNamespace>torso</robotNamespace>
       <filterJointsParam>joint_names</filterJointsParam>
     </plugin>
@@ -52,5 +51,5 @@
   <gazebo>
     <plugin name="ros_control" filename="libhwi_switch_gazebo_ros_control.so">
-      <robotNamespace>$(arg robot_id)/arm</robotNamespace>
+      <robotNamespace>arm</robotNamespace>
       <filterJointsParam>joint_names</filterJointsParam>
     </plugin>
@@ -61,5 +60,5 @@
   <gazebo>
     <plugin name="ros_control" filename="libhwi_switch_gazebo_ros_control.so">
-      <robotNamespace>$(arg robot_id)/head</robotNamespace>
+      <robotNamespace>head</robotNamespace>
       <filterJointsParam>joint_names</filterJointsParam>
     </plugin>
@@ -70,5 +69,5 @@
   <gazebo>
     <plugin name="ros_control" filename="libhwi_switch_gazebo_ros_control.so">
-      <robotNamespace>$(arg robot_id)/gripper</robotNamespace>
+      <robotNamespace>gripper</robotNamespace>
       <filterJointsParam>joint_names</filterJointsParam>
     </plugin>

File: cob_hardware_config/cob3-9/urdf/cob3-9.urdf.xacro (robot description, xacro)
@@ -2,5 +2,4 @@
 <robot xmlns:xacro="http://www.ros.org/wiki/xacro"
        name="cob3-9" >
-  <xacro:arg name="robot_id" default="/"/>
   <!-- common stuff -->
   <xacro:include filename="$(find cob_description)/urdf/common.xacro" />
@@ -25,5 +24,5 @@
   <gazebo>
     <plugin name="ros_control" filename="libhwi_switch_gazebo_ros_control.so">
-      <robotNamespace>$(arg robot_id)/base</robotNamespace>
+      <robotNamespace>base</robotNamespace>
       <filterJointsParam>joint_names</filterJointsParam>
     </plugin>
@@ -34,5 +33,5 @@
   <gazebo>
     <plugin name="ros_control" filename="libhwi_switch_gazebo_ros_control.so">
-      <robotNamespace>$(arg robot_id)/tray</robotNamespace>
+      <robotNamespace>tray</robotNamespace>
       <filterJointsParam>joint_names</filterJointsParam>
     </plugin>
@@ -43,5 +42,5 @@
   <gazebo>
     <plugin name="ros_control" filename="libhwi_switch_gazebo_ros_control.so">
-      <robotNamespace>$(arg robot_id)/torso</robotNamespace>
+      <robotNamespace>torso</robotNamespace>
       <filterJointsParam>joint_names</filterJointsParam>
     </plugin>
@@ -52,5 +51,5 @@
   <gazebo>
     <plugin name="ros_control" filename="libhwi_switch_gazebo_ros_control.so">
-      <robotNamespace>$(arg robot_id)/arm</robotNamespace>
+      <robotNamespace>arm</robotNamespace>
       <filterJointsParam>joint_names</filterJointsParam>
     </plugin>
@@ -61,5 +60,5 @@
   <gazebo>
     <plugin name="ros_control" filename="libhwi_switch_gazebo_ros_control.so">
-      <robotNamespace>$(arg robot_id)/head</robotNamespace>
+      <robotNamespace>head</robotNamespace>
       <filterJointsParam>joint_names</filterJointsParam>
     </plugin>
@@ -70,5 +69,5 @@
   <gazebo>
     <plugin name="ros_control" filename="libhwi_switch_gazebo_ros_control.so">
-      <robotNamespace>$(arg robot_id)/gripper</robotNamespace>
+      <robotNamespace>gripper</robotNamespace>
       <filterJointsParam>joint_names</filterJointsParam>
     </plugin>

File: cob_hardware_config/cob4-1/urdf/cob4-1.urdf.xacro (robot description, xacro)
@@ -2,5 +2,4 @@
 <robot xmlns:xacro="http://www.ros.org/wiki/xacro"
        name="cob4-1" >
-  <xacro:arg name="robot_id" default="/"/>
   <!-- common stuff -->
   <xacro:include filename="$(find cob_description)/urdf/common.xacro" />
@@ -13,5 +12,4 @@
   <!-- torso -->
   <xacro:include filename="$(find cob_description)/urdf/cob4_torso/torso_3dof.urdf.xacro" />
-  <xacro:include filename="$(find cob_description)/urdf/lookat/lookat.urdf.xacro" />
   <!-- arm -->
   <xacro:include filename="$(find schunk_description)/urdf/lwa4p_extended/lwa4p_extended.urdf.xacro" />
@@ -26,5 +24,5 @@
   <gazebo>
     <plugin name="ros_control" filename="libhwi_switch_gazebo_ros_control.so">
-      <robotNamespace>$(arg robot_id)/base</robotNamespace>
+      <robotNamespace>base</robotNamespace>
       <filterJointsParam>joint_names</filterJointsParam>
     </plugin>
@@ -35,5 +33,5 @@
   <gazebo>
     <plugin name="ros_control" filename="libhwi_switch_gazebo_ros_control.so">
-      <robotNamespace>$(arg robot_id)/torso</robotNamespace>
+      <robotNamespace>torso</robotNamespace>
       <filterJointsParam>joint_names</filterJointsParam>
     </plugin>
@@ -44,5 +42,5 @@
   <gazebo>
     <plugin name="ros_control" filename="libhwi_switch_gazebo_ros_control.so">
-      <robotNamespace>$(arg robot_id)/head</robotNamespace>
+      <robotNamespace>head</robotNamespace>
       <filterJointsParam>joint_names</filterJointsParam>
     </plugin>
@@ -53,5 +51,5 @@
   <gazebo>
     <plugin name="ros_control" filename="libhwi_switch_gazebo_ros_control.so">
-      <robotNamespace>$(arg robot_id)/sensorring</robotNamespace>
+      <robotNamespace>sensorring</robotNamespace>
       <filterJointsParam>joint_names</filterJointsParam>
     </plugin>
@@ -62,5 +60,5 @@
   <gazebo>
     <plugin name="ros_control" filename="libhwi_switch_gazebo_ros_control.so">
-      <robotNamespace>$(arg robot_id)/arm_right</robotNamespace>
+      <robotNamespace>arm_right</robotNamespace>
       <filterJointsParam>joint_names</filterJointsParam>
     </plugin>
@@ -71,5 +69,5 @@
   <gazebo>
     <plugin name="ros_control" filename="libhwi_switch_gazebo_ros_control.so">
-      <robotNamespace>$(arg robot_id)/arm_left</robotNamespace>
+      <robotNamespace>arm_left</robotNamespace>
       <filterJointsParam>joint_names</filterJointsParam>
     </plugin>
@@ -80,5 +78,5 @@
   <gazebo>
     <plugin name="ros_control" filename="libhwi_switch_gazebo_ros_control.so">
-      <robotNamespace>$(arg robot_id)/gripper_right</robotNamespace>
+      <robotNamespace>gripper_right</robotNamespace>
       <filterJointsParam>joint_names</filterJointsParam>
     </plugin>
@@ -89,14 +87,7 @@
   <gazebo>
     <plugin name="ros_control" filename="libhwi_switch_gazebo_ros_control.so">
-      <robotNamespace>$(arg robot_id)/gripper_left</robotNamespace>
+      <robotNamespace>gripper_left</robotNamespace>
       <filterJointsParam>joint_names</filterJointsParam>
     </plugin>
   </gazebo>
-  <!-- virtual component -->
-<!--
-  <xacro:lookat name="lookat" parent="torso_center_link" lower="0.0" upper="5.0">
-    <origin xyz="0 0 0" rpy="0 0 0" />
-    <axis xyz="1 0 0"/>
-  </xacro:lookat>
--->
 </robot>

File: cob_hardware_config/cob4-2/urdf/cob4-2.urdf.xacro (robot description, xacro)
@@ -2,5 +2,4 @@
 <robot xmlns:xacro="http://www.ros.org/wiki/xacro"
        name="cob4-2" >
-  <xacro:arg name="robot_id" default="/"/>
   <!-- common stuff -->
   <xacro:include filename="$(find cob_description)/urdf/common.xacro" />
@@ -13,5 +12,4 @@
   <!-- torso -->
   <xacro:include filename="$(find cob_description)/urdf/cob4_torso/torso_2dof.urdf.xacro" />
-  <xacro:include filename="$(find cob_description)/urdf/lookat/lookat.urdf.xacro" />
   <!-- arm -->
   <xacro:include filename="$(find schunk_description)/urdf/lwa4p_extended/lwa4p_extended.urdf.xacro" />
@@ -26,5 +24,5 @@
   <gazebo>
     <plugin name="ros_control" filename="libhwi_switch_gazebo_ros_control.so">
-      <robotNamespace>$(arg robot_id)/base</robotNamespace>
+      <robotNamespace>base</robotNamespace>
       <filterJointsParam>joint_names</filterJointsParam>
     </plugin>
@@ -35,5 +33,5 @@
   <gazebo>
     <plugin name="ros_control" filename="libhwi_switch_gazebo_ros_control.so">
-      <robotNamespace>$(arg robot_id)/torso</robotNamespace>
+      <robotNamespace>torso</robotNamespace>
       <filterJointsParam>joint_names</filterJointsParam>
     </plugin>
@@ -47,5 +45,5 @@
   <gazebo>
     <plugin name="ros_control" filename="libhwi_switch_gazebo_ros_control.so">
-      <robotNamespace>$(arg robot_id)/sensorring</robotNamespace>
+      <robotNamespace>sensorring</robotNamespace>
       <filterJointsParam>joint_names</filterJointsParam>
     </plugin>
@@ -56,5 +54,5 @@
   <gazebo>
     <plugin name="ros_control" filename="libhwi_switch_gazebo_ros_control.so">
-      <robotNamespace>$(arg robot_id)/arm_right</robotNamespace>
+      <robotNamespace>arm_right</robotNamespace>
       <filterJointsParam>joint_names</filterJointsParam>
     </plugin>
@@ -65,5 +63,5 @@
   <gazebo>
     <plugin name="ros_control" filename="libhwi_switch_gazebo_ros_control.so">
-      <robotNamespace>$(arg robot_id)/arm_left</robotNamespace>
+      <robotNamespace>arm_left</robotNamespace>
       <filterJointsParam>joint_names</filterJointsParam>
     </plugin>
@@ -74,5 +72,5 @@
   <gazebo>
     <plugin name="ros_control" filename="libhwi_switch_gazebo_ros_control.so">
-      <robotNamespace>$(arg robot_id)/gripper_right</robotNamespace>
+      <robotNamespace>gripper_right</robotNamespace>
       <filterJointsParam>joint_names</filterJointsParam>
     </plugin>
@@ -83,8 +81,7 @@
   <gazebo>
     <plugin name="ros_control" filename="libhwi_switch_gazebo_ros_control.so">
-      <robotNamespace>$(arg robot_id)/gripper_left</robotNamespace>
+      <robotNamespace>gripper_left</robotNamespace>
       <filterJointsParam>joint_names</filterJointsParam>
     </plugin>
   </gazebo>
-  <!-- virtual component -->
 </robot>

File: cob_hardware_config/cob4-4/urdf/cob4-4.urdf.xacro (robot description, xacro)
@@ -2,5 +2,4 @@
 <robot xmlns:xacro="http://www.ros.org/wiki/xacro"
        name="cob4-4" >
-  <xacro:arg name="robot_id" default="/"/>
   <!-- common stuff -->
   <xacro:include filename="$(find cob_description)/urdf/common.xacro" />
@@ -14,5 +13,5 @@
   <gazebo>
     <plugin name="ros_control" filename="libhwi_switch_gazebo_ros_control.so">
-      <robotNamespace>$(arg robot_id)/base</robotNamespace>
+      <robotNamespace>base</robotNamespace>
       <filterJointsParam>joint_names</filterJointsParam>
     </plugin>

File: cob_hardware_config/cob4-6/urdf/cob4-6.urdf.xacro (robot description, xacro)
@@ -2,5 +2,4 @@
 <robot xmlns:xacro="http://www.ros.org/wiki/xacro"
        name="cob4-6" >
-  <xacro:arg name="robot_id" default="/"/>
   <!-- common stuff -->
   <xacro:include filename="$(find cob_description)/urdf/common.xacro" />
@@ -14,5 +13,5 @@
   <gazebo>
     <plugin name="ros_control" filename="libhwi_switch_gazebo_ros_control.so">
-      <robotNamespace>$(arg robot_id)/base</robotNamespace>
+      <robotNamespace>base</robotNamespace>
       <filterJointsParam>joint_names</filterJointsParam>
     </plugin>

File: cob_hardware_config/raw3-1/urdf/raw3-1.urdf.xacro (robot description, xacro)
@@ -2,5 +2,4 @@
 <robot xmlns:xacro="http://www.ros.org/wiki/xacro"
        name="raw3-1" >
-  <xacro:arg name="robot_id" default="/"/>
   <!-- common stuff -->
   <xacro:include filename="$(find cob_description)/urdf/common.xacro" />
@@ -15,5 +14,4 @@
   <!-- head -->
   <xacro:include filename="$(find raw_description)/urdf/head/head.urdf.xacro" />
-  <xacro:include filename="$(find cob_description)/urdf/lookat/lookat.urdf.xacro" />
   <!-- ur_arm -->
   <xacro:include filename="$(find cob_description)/urdf/ur_arm/ur10_arm.urdf.xacro" />
@@ -24,5 +22,5 @@
   <gazebo>
     <plugin name="ros_control" filename="libhwi_switch_gazebo_ros_control.so">
-      <robotNamespace>$(arg robot_id)/base</robotNamespace>
+      <robotNamespace>base</robotNamespace>
       <filterJointsParam>joint_names</filterJointsParam>
     </plugin>
@@ -36,5 +34,5 @@
   <gazebo>
     <plugin name="ros_control" filename="libhwi_switch_gazebo_ros_control.so">
-      <robotNamespace>$(arg robot_id)/torso</robotNamespace>
+      <robotNamespace>torso</robotNamespace>
       <filterJointsParam>joint_names</filterJointsParam>
     </plugin>
@@ -43,8 +41,4 @@
     <origin xyz="${head_x} ${head_y} ${head_z}" rpy="${head_roll} ${head_pitch} ${head_yaw}" />
   </xacro:raw_head>
-  <!--xacro:cob_lookat name="lookat" parent="torso_2_link" lower="0.0" upper="5.0">
-    <origin xyz="${head_x} ${head_y} ${head_z}" rpy="${head_roll} ${head_pitch} ${head_yaw}" />
-    <axis xyz="1 0 0"/>
-  </xacro:cob_lookat-->
 <!--
   <xacro:ur10 name="arm" parent="base_link">
@@ -53,5 +47,5 @@
   <gazebo>
     <plugin name="ros_control" filename="libhwi_switch_gazebo_ros_control.so">
-      <robotNamespace>$(arg robot_id)/arm</robotNamespace>
+      <robotNamespace>arm</robotNamespace>
       <filterJointsParam>joint_names</filterJointsParam>
     </plugin>

File: cob_hardware_config/raw3-2/urdf/raw3-2.urdf.xacro (robot description, xacro)
@@ -2,5 +2,4 @@
 <robot xmlns:xacro="http://www.ros.org/wiki/xacro"
        name="raw3-2" >
-  <xacro:arg name="robot_id" default="/"/>
   <!-- common stuff -->
   <xacro:include filename="$(find cob_description)/urdf/common.xacro" />
@@ -14,5 +13,5 @@
   <gazebo>
     <plugin name="ros_control" filename="libhwi_switch_gazebo_ros_control.so">
-      <robotNamespace>$(arg robot_id)/base</robotNamespace>
+      <robotNamespace>base</robotNamespace>
       <filterJointsParam>joint_names</filterJointsParam>
     </plugin>

File: cob_hardware_config/raw3-3/urdf/raw3-3.urdf.xacro (robot description, xacro)
@@ -2,5 +2,4 @@
 <robot xmlns:xacro="http://www.ros.org/wiki/xacro"
        name="raw3-3" >
-  <xacro:arg name="robot_id" default="/"/>
   <!-- common stuff -->
   <xacro:include filename="$(find cob_description)/urdf/common.xacro" />
@@ -19,5 +18,5 @@
   <gazebo>
     <plugin name="ros_control" filename="libhwi_switch_gazebo_ros_control.so">
-      <robotNamespace>$(arg robot_id)/base</robotNamespace>
+      <robotNamespace>base</robotNamespace>
       <filterJointsParam>joint_names</filterJointsParam>
     </plugin>
@@ -30,10 +29,4 @@
   <!-- prace macros -->
   <xacro:prace/>
-<!--
-  <xacro:lookat name="lookat" parent="head_cam_holder_link" lower="0.0" upper="8.0">
-    <origin xyz="${head_x} ${head_y} ${head_z}" rpy="${head_roll} ${head_pitch} ${head_yaw}" />
-    <axis xyz="1 0 0"/>
-  </xacro:lookat>
--->
   <!-- scan top mount -->
     <joint name="base_laser_top_joint" type="fixed" >

File: cob_hardware_config/raw3-4/urdf/raw3-4.urdf.xacro (robot description, xacro)
@@ -2,5 +2,4 @@
 <robot xmlns:xacro="http://www.ros.org/wiki/xacro"
        name="raw3-4" >
-  <xacro:arg name="robot_id" default="/"/>
   <!-- common stuff -->
   <xacro:include filename="$(find cob_description)/urdf/common.xacro" />
@@ -17,5 +16,5 @@
   <gazebo>
     <plugin name="ros_control" filename="libhwi_switch_gazebo_ros_control.so">
-      <robotNamespace>$(arg robot_id)/base</robotNamespace>
+      <robotNamespace>base</robotNamespace>
       <filterJointsParam>joint_names</filterJointsParam>
     </plugin>

File: cob_hardware_config/raw3-5/urdf/raw3-5.urdf.xacro (robot description, xacro)
@@ -2,5 +2,4 @@
 <robot xmlns:xacro="http://www.ros.org/wiki/xacro"
        name="raw3-5" >
-  <xacro:arg name="robot_id" default="/"/>
   <!-- common stuff -->
   <xacro:include filename="$(find cob_description)/urdf/common.xacro" />
@@ -13,5 +12,5 @@
   <gazebo>
     <plugin name="ros_control" filename="libhwi_switch_gazebo_ros_control.so">
-      <robotNamespace>$(arg robot_id)/base</robotNamespace>
+      <robotNamespace>base</robotNamespace>
       <filterJointsParam>joint_names</filterJointsParam>
     </plugin>

File: cob_hardware_config/raw3-6/urdf/raw3-6.urdf.xacro (robot description, xacro)
@@ -2,5 +2,4 @@
 <robot xmlns:xacro="http://www.ros.org/wiki/xacro"
        name="raw3-6" >
-  <xacro:arg name="robot_id" default="/"/>
   <!-- common stuff -->
   <xacro:include filename="$(find cob_description)/urdf/common.xacro" />
@@ -15,5 +14,5 @@
   <gazebo>
     <plugin name="ros_control" filename="libhwi_switch_gazebo_ros_control.so">
-      <robotNamespace>$(arg robot_id)/base</robotNamespace>
+      <robotNamespace>base</robotNamespace>
       <filterJointsParam>joint_names</filterJointsParam>
     </plugin>
