Commit message: removed gripper

File: cob_hardware_config/raw3-3/urdf/raw3-3.urdf.xacro (robot description, xacro)
@@ -10,7 +10,5 @@
   <include filename="$(find cob_calibration_data)/raw3-3/calibration/calibration.urdf.xacro" />
   <!-- raw base -->
-  <include filename="$(find raw_description)/urdf/base/base.urdf.xacro" />
-  <!-- torso -->
-  <!--include filename="$(find raw_description)/urdf/torso/torso.urdf.xacro" /-->
+  <include filename="$(find raw_description)/urdf/base_short/base.urdf.xacro" />
   <!-- frida -->
   <include filename="$(find frida_description)/urdf/frida.urdf.xacro" />
@@ -20,7 +18,8 @@
   <include filename="$(find cob_description)/gazebo/gazebo.urdf.xacro" />
   <xacro:raw_base name="base"/>	<!--with new collision_model, but no platform_controller available yet-->
-  <xacro:frida parent="base_tower" name="arm">
-    <origin xyz="0 -0.029 0" rpy="0 0 -3.14159265" />
+  <xacro:frida parent="base_link" name="arm">
+    <origin xyz="0.24 0.0 0.48" rpy="0 0 0" />
   </xacro:frida>
+ <!--
   <xacro:prace_gripper name="gripper_left" parent="arm_left_7_link">
     <origin xyz="0.0 0.0 0.0561" rpy="0 0 0" />
@@ -29,3 +28,4 @@
     <origin xyz="0.0 0.0 0.0561" rpy="0 0 0" />
   </xacro:prace_gripper>
+-->
 </robot>

Commit message: new tower description

File: cob_hardware_config/raw3-3/urdf/raw3-3.urdf.xacro (robot description, xacro)
@@ -11,4 +11,6 @@
   <!-- raw base -->
   <include filename="$(find raw_description)/urdf/base_short/base.urdf.xacro" />
+  <!-- raw tower -->
+  <include filename="$(find raw_description)/urdf/tower_symetric/tower.urdf.xacro" />
   <!-- frida -->
   <include filename="$(find frida_description)/urdf/frida.urdf.xacro" />
@@ -18,4 +20,7 @@
   <include filename="$(find cob_description)/gazebo/gazebo.urdf.xacro" />
   <xacro:raw_base name="base"/>	<!--with new collision_model, but no platform_controller available yet-->
+  <xacro:tower_symetric name="tower" parent="base_link">
+    <origin xyz="0.221 0.0 0.306"/>
+  </xacro:tower_symetric>
   <xacro:frida parent="base_link" name="arm">
     <origin xyz="0.24 0.0 0.48" rpy="0 0 0" />

Commit message: added adapter plate for frida

File: cob_hardware_config/raw3-3/urdf/raw3-3.urdf.xacro (robot description, xacro)
@@ -15,4 +15,6 @@
   <!-- frida -->
   <include filename="$(find frida_description)/urdf/frida.urdf.xacro" />
+  <!-- frida adapter -->
+  <include filename="$(find frida_description)/urdf/adapter.urdf.xacro" />
   <!-- prace gripper -->
   <include filename="$(find prace_gripper_description)/urdf/prace_gripper.urdf.xacro"/>
@@ -23,14 +25,15 @@
       <origin xyz="${tower_x} ${tower_y} ${tower_z}" rpy="${tower_roll} ${tower_pitch} ${tower_yaw}" />
   </xacro:tower_symetric>
+  <xacro:frida_adapter name="adapter" parent="tower_base_link">
+      <origin xyz="0.0905 0 0.2305" rpy="0 0 0" />
+  </xacro:frida_adapter>
   <xacro:frida name="arm" parent="base_link">
       <origin xyz="${arm_x} ${arm_y} ${arm_z}" rpy="${arm_roll} ${arm_pitch} ${arm_yaw}" />
   </xacro:frida>
- <!--
-  <xacro:prace_gripper name="gripper_left" parent="arm_left_7_link">
+  <xacro:prace_gripper name="gripper_left" parent="arm_left_6_link">
       <origin xyz="${gripper_left_x} ${gripper_left_y} ${gripper_left_z}" rpy="${gripper_left_roll} ${gripper_left_pitch} ${gripper_left_yaw}" />
   </xacro:prace_gripper>
-  <xacro:prace_gripper name="gripper_right" parent="arm_right_7_link">
+  <xacro:prace_gripper name="gripper_right" parent="arm_right_6_link">
       <origin xyz="${gripper_right_x} ${gripper_right_y} ${gripper_right_z}" rpy="${gripper_right_roll} ${gripper_right_pitch} ${gripper_right_yaw}" />
   </xacro:prace_gripper>
--->
 </robot>

Commit message: added teachin handle link

File: cob_hardware_config/raw3-3/urdf/raw3-3.urdf.xacro (robot description, xacro)
@@ -17,4 +17,5 @@
   <!-- frida adapter -->
   <include filename="$(find frida_description)/urdf/adapter.urdf.xacro" />
+  <include filename="$(find frida_description)/urdf/teachin_handle.urdf.xacro" />
   <!-- prace gripper -->
   <include filename="$(find prace_gripper_description)/urdf/prace_gripper.urdf.xacro"/>
@@ -37,3 +38,6 @@
       <origin xyz="${gripper_right_x} ${gripper_right_y} ${gripper_right_z}" rpy="${gripper_right_roll} ${gripper_right_pitch} ${gripper_right_yaw}" />
   </xacro:prace_gripper>
+  <xacro:teachin_handle name="teachin_handle" parent="arm_torso_link">
+      <origin xyz="-0.15 0 0.49" rpy="0 0 0" />
+  </xacro:teachin_handle>
 </robot>

Commit message: added camera holder

File: cob_hardware_config/raw3-3/urdf/raw3-3.urdf.xacro (robot description, xacro)
@@ -17,5 +17,5 @@
   <!-- frida adapter -->
   <include filename="$(find frida_description)/urdf/adapter.urdf.xacro" />
-  <include filename="$(find frida_description)/urdf/teachin_handle.urdf.xacro" />
+  <include filename="$(find frida_description)/urdf/camera_holder.urdf.xacro" />
   <!-- prace gripper -->
   <include filename="$(find prace_gripper_description)/urdf/prace_gripper.urdf.xacro"/>
@@ -38,6 +38,6 @@
       <origin xyz="${gripper_right_x} ${gripper_right_y} ${gripper_right_z}" rpy="${gripper_right_roll} ${gripper_right_pitch} ${gripper_right_yaw}" />
   </xacro:prace_gripper>
-  <xacro:teachin_handle name="teachin_handle" parent="arm_torso_link">
-      <origin xyz="-0.15 0 0.49" rpy="0 0 0" />
+  <xacro:teachin_handle name="cam_holder" parent="arm_torso_link">
+      <origin xyz="0.0 0 0.49" rpy="0.99483 0 0" />
   </xacro:teachin_handle>
 </robot>

Commit message: added laserscanners to launch file and added frida to raw3-3 urdf

File: cob_hardware_config/raw3-3/urdf/raw3-3.urdf.xacro (robot description, xacro)
@@ -17,4 +17,5 @@
   <!-- frida adapter -->
   <include filename="$(find frida_description)/urdf/adapter.urdf.xacro" />
+  <include filename="$(find frida_description)/urdf/camera_holder.urdf.xacro" />
   <!-- prace gripper -->
   <include filename="$(find prace_gripper_description)/urdf/prace_gripper.urdf.xacro"/>
@@ -37,3 +38,6 @@
       <origin xyz="${gripper_right_x} ${gripper_right_y} ${gripper_right_z}" rpy="${gripper_right_roll} ${gripper_right_pitch} ${gripper_right_yaw}" />
   </xacro:prace_gripper>
+  <xacro:teachin_handle name="cam_holder" parent="arm_torso_link">
+      <origin xyz="0.0 0 0.49" rpy="0.99483 0 0" />
+  </xacro:teachin_handle>
 </robot>

Commit message: added gazebo controller for prace head

File: cob_hardware_config/raw3-3/urdf/raw3-3.urdf.xacro (robot description, xacro)
@@ -16,8 +16,11 @@
   <include filename="$(find frida_description)/urdf/frida.urdf.xacro" />
   <!-- frida adapter -->
-  <include filename="$(find frida_description)/urdf/adapter.urdf.xacro" />
-  <include filename="$(find frida_description)/urdf/camera_holder.urdf.xacro" />
+  <include filename="$(find prace_common)/urdf/adapter/tower_frida_adapter.urdf.xacro" />
   <!-- prace gripper -->
   <include filename="$(find prace_gripper_description)/urdf/prace_gripper.urdf.xacro"/>
+  <!-- prace neck -->
+  <include filename="$(find prace_common)/urdf/neck/neck.urdf.xacro" />
+  <!-- prace head -->
+  <include filename="$(find prace_common)/urdf/head/head.urdf.xacro" />
   <!-- generic simulator_gazebo plugins for starting mechanism control, ros time, ros battery -->
   <include filename="$(find cob_description)/gazebo/gazebo.urdf.xacro" />
@@ -26,7 +29,7 @@
       <origin xyz="${tower_x} ${tower_y} ${tower_z}" rpy="${tower_roll} ${tower_pitch} ${tower_yaw}" />
   </xacro:tower_symetric>
-  <xacro:frida_adapter name="adapter" parent="tower_base_link">
+  <xacro:tower_frida_adapter name="adapter" parent="tower_base_link">
       <origin xyz="0.0905 0 0.2305" rpy="0 0 0" />
-  </xacro:frida_adapter>
+  </xacro:tower_frida_adapter>
   <xacro:frida name="arm" parent="base_link">
       <origin xyz="${arm_x} ${arm_y} ${arm_z}" rpy="${arm_roll} ${arm_pitch} ${arm_yaw}" />
@@ -38,6 +41,9 @@
       <origin xyz="${gripper_right_x} ${gripper_right_y} ${gripper_right_z}" rpy="${gripper_right_roll} ${gripper_right_pitch} ${gripper_right_yaw}" />
   </xacro:prace_gripper>
-  <xacro:teachin_handle name="cam_holder" parent="arm_torso_link">
-      <origin xyz="0.0 0 0.49" rpy="0.99483 0 0" />
-  </xacro:teachin_handle>
+  <xacro:neck name="neck" parent="arm_torso_link">
+      <origin xyz="-0.07624 0 0.47378" rpy="0 0.607514 0" />
+  </xacro:neck>
+  <xacro:head name="head" parent="neck_mount_link">
+      <origin xyz="0 0 0.074998" rpy="0 0 0" />
+  </xacro:head>
 </robot>

Commit message: added calibration data for raw3-3s head

File: cob_hardware_config/raw3-3/urdf/raw3-3.urdf.xacro (robot description, xacro)
@@ -42,8 +42,8 @@
   </xacro:prace_gripper>
   <xacro:neck name="neck" parent="arm_torso_link">
-      <origin xyz="-0.07624 0 0.47378" rpy="0 0.607514 0" />
+      <origin xyz="${neck_x} ${neck_y} ${neck_z}" rpy="${neck_roll} ${neck_pitch} ${neck_yaw}" />
   </xacro:neck>
   <xacro:head name="head" parent="neck_mount_link">
-      <origin xyz="0 0 0.074998" rpy="0 0 0" />
+      <origin xyz="${head_x} ${head_y} ${head_z}" rpy="${head_roll} ${head_pitch} ${head_yaw}" />
   </xacro:head>
 </robot>

Commit message: support powerball head axis on raw3-3

File: cob_hardware_config/raw3-3/urdf/raw3-3.urdf.xacro (robot description, xacro)
@@ -23,4 +23,5 @@
   <!-- prace head -->
   <include filename="$(find prace_common)/urdf/head/head.urdf.xacro" />
+  <include filename="$(find cob_description)/urdf/lookat/lookat.urdf.xacro" />
   <!-- generic simulator_gazebo plugins for starting mechanism control, ros time, ros battery -->
   <include filename="$(find cob_description)/gazebo/gazebo.urdf.xacro" />
@@ -47,3 +48,7 @@
       <origin xyz="${head_x} ${head_y} ${head_z}" rpy="${head_roll} ${head_pitch} ${head_yaw}" />
   </xacro:head>
+  <xacro:lookat name="lookat" parent="head_cam_holder_link" lower="-8.0" upper="8.0">
+    <origin xyz="${head_x} ${head_y} ${head_z}" rpy="${head_roll} ${head_pitch} ${head_yaw}" />
+    <axis xyz="-1 0 0"/>
+  </xacro:lookat>
 </robot>

Commit message: vel_control and lookat_control with raw3-3

File: cob_hardware_config/raw3-3/urdf/raw3-3.urdf.xacro (robot description, xacro)
@@ -45,7 +45,7 @@
       <origin xyz="${head_x} ${head_y} ${head_z}" rpy="${head_roll} ${head_pitch} ${head_yaw}" />
   </xacro:head>
-  <xacro:lookat name="lookat" parent="head_cam_holder_link" lower="-8.0" upper="8.0">
+  <xacro:lookat name="lookat" parent="head_cam_holder_link" lower="0.0" upper="8.0">
     <origin xyz="${head_x} ${head_y} ${head_z}" rpy="${head_roll} ${head_pitch} ${head_yaw}" />
-    <axis xyz="-1 0 0"/>
+    <axis xyz="1 0 0"/>
   </xacro:lookat>
 </robot>

Commit message: merged prace descriptions into one xacro makro

File: cob_hardware_config/raw3-3/urdf/raw3-3.urdf.xacro (robot description, xacro)
@@ -11,14 +11,5 @@
   <xacro:include filename="$(find raw_description)/urdf/tower_symetric/tower.urdf.xacro" />
   <!-- frida -->
-  <xacro:include filename="$(find frida_description)/urdf/frida.urdf.xacro" />
-  <!-- frida adapter -->
-  <xacro:include filename="$(find prace_common)/urdf/adapter/tower_frida_adapter.urdf.xacro" />
-  <!-- prace gripper -->
-  <xacro:include filename="$(find prace_gripper_description)/urdf/prace_gripper.urdf.xacro"/>
-  <!-- prace neck -->
-  <xacro:include filename="$(find prace_common)/urdf/neck/neck_v2.urdf.xacro" />
-  <!-- prace head -->
-  <xacro:include filename="$(find prace_common)/urdf/head/head.urdf.xacro" />
-  <xacro:include filename="$(find cob_description)/urdf/lookat/lookat.urdf.xacro" />
+  <xacro:include filename="$(find prace_common)/urdf/prace.urdf.xacro" />
   <!-- generic simulator_gazebo plugins for starting mechanism control, ros time, ros battery -->
   <xacro:include filename="$(find cob_description)/gazebo/gazebo.urdf.xacro" />
@@ -27,22 +18,6 @@
       <origin xyz="${tower_x} ${tower_y} ${tower_z}" rpy="${tower_roll} ${tower_pitch} ${tower_yaw}" />
   </xacro:tower_symetric>
-  <xacro:tower_frida_adapter name="adapter" parent="tower_base_link">
-      <origin xyz="0.0905 0 0.2305" rpy="0 0 0" />
-  </xacro:tower_frida_adapter>
-  <xacro:frida name="arm" parent="base_link">
-      <origin xyz="${arm_x} ${arm_y} ${arm_z}" rpy="${arm_roll} ${arm_pitch} ${arm_yaw}" />
-  </xacro:frida>
-  <xacro:prace_gripper name="gripper_left" parent="arm_left_6_link">
-      <origin xyz="${gripper_left_x} ${gripper_left_y} ${gripper_left_z}" rpy="${gripper_left_roll} ${gripper_left_pitch} ${gripper_left_yaw}" />
-  </xacro:prace_gripper>
-  <xacro:prace_gripper name="gripper_right" parent="arm_right_6_link">
-      <origin xyz="${gripper_right_x} ${gripper_right_y} ${gripper_right_z}" rpy="${gripper_right_roll} ${gripper_right_pitch} ${gripper_right_yaw}" />
-  </xacro:prace_gripper>
-  <xacro:neck name="neck" parent="arm_torso_link">
-      <origin xyz="${neck_x} ${neck_y} ${neck_z}" rpy="${neck_roll} ${neck_pitch} ${neck_yaw}" />
-  </xacro:neck>
-  <xacro:head name="head" parent="neck_mount_link">
-      <origin xyz="${head_x} ${head_y} ${head_z}" rpy="${head_roll} ${head_pitch} ${head_yaw}" />
-  </xacro:head>
+  <!-- prace macros -->
+  <xacro:prace/>
   <xacro:lookat name="lookat" parent="head_cam_holder_link" lower="0.0" upper="8.0">
     <origin xyz="${head_x} ${head_y} ${head_z}" rpy="${head_roll} ${head_pitch} ${head_yaw}" />

Commit message: changed rplidar orientation

File: cob_hardware_config/raw3-3/urdf/raw3-3.urdf.xacro (robot description, xacro)
@@ -31,5 +31,5 @@
   <!-- scan top mount -->
     <joint name="base_laser_top_joint" type="fixed" >
-      <origin xyz="0.28 0.0 0.885" rpy="0.0 0.0 ${M_PI}" />
+      <origin xyz="0.28 0.0 0.885" rpy="0.0 0.0 0.0" />
       <parent link="base_link" />
       <child link="base_laser_top_link" />
