Commit message: remove obsolete components and dependencies

File: cob_hardware_config/raw3-3/urdf/calibration_default.urdf.xacro (robot description, xacro)
@@ -28,66 +28,3 @@
 	<xacro:property name="def_tower_pitch" value="0.0"/>
 	<xacro:property name="def_tower_yaw" value="0.0"/>
-	<!-- arm mount positions | relative to base_link -->
-	<xacro:property name="def_arm_x" value="0.244"/>
-	<xacro:property name="def_arm_y" value="0.0"/>
-	<xacro:property name="def_arm_z" value="0.59316"/>
-	<xacro:property name="def_arm_roll" value="0.0"/>
-	<xacro:property name="def_arm_pitch" value="0.0"/>
-	<xacro:property name="def_arm_yaw" value="0.0"/>
-	<!-- gripper_left mount positions | relative to arm_left_7_link -->
-	<xacro:property name="def_gripper_left_x" value="0.0"/>
-	<xacro:property name="def_gripper_left_y" value="0.0"/>
-	<xacro:property name="def_gripper_left_z" value="0.0"/>
-	<xacro:property name="def_gripper_left_roll" value="0.0"/>
-	<xacro:property name="def_gripper_left_pitch" value="0.0"/>
-	<xacro:property name="def_gripper_left_yaw" value="0.0"/>
-	<!-- gripper_right mount positions | relative to arm_right_7_link -->
-	<xacro:property name="def_gripper_right_x" value="0.0"/>
-	<xacro:property name="def_gripper_right_y" value="0.0"/>
-	<xacro:property name="def_gripper_right_z" value="0.0"/>
-	<xacro:property name="def_gripper_right_roll" value="0.0"/>
-	<xacro:property name="def_gripper_right_pitch" value="0.0"/>
-	<xacro:property name="def_gripper_right_yaw" value="0.0"/>
-	<!-- neck mount positions | relative to arm_torso_link -->
-	<xacro:property name="def_neck_x" value="-0.07624"/>
-	<xacro:property name="def_neck_y" value="0.0"/>
-	<xacro:property name="def_neck_z" value="0.47378"/>
-	<xacro:property name="def_neck_roll" value="0.0"/>
-	<xacro:property name="def_neck_pitch" value="0.607514"/>
-	<xacro:property name="def_neck_yaw" value="0.0"/>
-	<!-- head mount positions | relative to neck_mount_link -->
-	<xacro:property name="def_head_x" value="0.0"/>
-	<xacro:property name="def_head_y" value="0.0"/>
-	<xacro:property name="def_head_z" value="0.074998"/>
-	<xacro:property name="def_head_roll" value="0.0"/>
-	<xacro:property name="def_head_pitch" value="0.0"/>
-	<xacro:property name="def_head_yaw" value="0.0"/>
-	<!-- ids_middle mount positions | relative to head_cam_holder_link -->
-	<xacro:property name="def_ids_middle_x" value="-0.002"/>
-	<xacro:property name="def_ids_middle_y" value="0.0"/>
-	<xacro:property name="def_ids_middle_z" value="0.0145"/>
-	<xacro:property name="def_ids_middle_roll" value="0.0"/>
-	<xacro:property name="def_ids_middle_pitch" value="0.0"/>
-	<xacro:property name="def_ids_middle_yaw" value="0.0"/>
-	<!-- ids_left mount positions | relative to head_cam_holder_link -->
-	<xacro:property name="def_ids_left_x" value="-0.002"/>
-	<xacro:property name="def_ids_left_y" value="0.091"/>
-	<xacro:property name="def_ids_left_z" value="0.0145"/>
-	<xacro:property name="def_ids_left_roll" value="0.0"/>
-	<xacro:property name="def_ids_left_pitch" value="0.0"/>
-	<xacro:property name="def_ids_left_yaw" value="0.0"/>
-	<!-- ids_right mount positions | relative to head_cam_holder_link -->
-	<xacro:property name="def_ids_right_x" value="-0.002"/>
-	<xacro:property name="def_ids_right_y" value="-0.091"/>
-	<xacro:property name="def_ids_right_z" value="0.0145"/>
-	<xacro:property name="def_ids_right_roll" value="0.0"/>
-	<xacro:property name="def_ids_right_pitch" value="0.0"/>
-	<xacro:property name="def_ids_right_yaw" value="0.0"/>
-	<!-- cam_holder mount positions | relative to head_cam_holder_link -->
-	<xacro:property name="def_cam_holder_x" value="0.0"/>
-	<xacro:property name="def_cam_holder_y" value="-0.065"/>
-	<xacro:property name="def_cam_holder_z" value="0.0"/>
-	<xacro:property name="def_cam_holder_roll" value="1.5708"/>
-	<xacro:property name="def_cam_holder_pitch" value="0.0"/>
-	<xacro:property name="def_cam_holder_yaw" value="0.0"/>
 </robot>

File: cob_hardware_config/raw3-3/urdf/properties.urdf.xacro (robot description, xacro)
@@ -30,66 +30,3 @@
 	<xacro:property name="tower_pitch" value="${def_tower_pitch+offset_tower_pitch}"/>
 	<xacro:property name="tower_yaw" value="${def_tower_yaw+offset_tower_yaw}"/>
-	<!-- arm mount positions | relative to base_link -->
-	<xacro:property name="arm_x" value="${def_arm_x+offset_arm_x}"/>
-	<xacro:property name="arm_y" value="${def_arm_y+offset_arm_y}"/>
-	<xacro:property name="arm_z" value="${def_arm_z+offset_arm_z}"/>
-	<xacro:property name="arm_roll" value="${def_arm_roll+offset_arm_roll}"/>
-	<xacro:property name="arm_pitch" value="${def_arm_pitch+offset_arm_pitch}"/>
-	<xacro:property name="arm_yaw" value="${def_arm_yaw+offset_arm_yaw}"/>
-	<!-- gripper_left mount positions | relative to arm_left_7_link -->
-	<xacro:property name="gripper_left_x" value="${def_gripper_left_x+offset_gripper_left_x}"/>
-	<xacro:property name="gripper_left_y" value="${def_gripper_left_y+offset_gripper_left_y}"/>
-	<xacro:property name="gripper_left_z" value="${def_gripper_left_z+offset_gripper_left_z}"/>
-	<xacro:property name="gripper_left_roll" value="${def_gripper_left_roll+offset_gripper_left_roll}"/>
-	<xacro:property name="gripper_left_pitch" value="${def_gripper_left_pitch+offset_gripper_left_pitch}"/>
-	<xacro:property name="gripper_left_yaw" value="${def_gripper_left_yaw+offset_gripper_left_yaw}"/>
-	<!-- gripper_right mount positions | relative to arm_right_7_link -->
-	<xacro:property name="gripper_right_x" value="${def_gripper_right_x+offset_gripper_right_x}"/>
-	<xacro:property name="gripper_right_y" value="${def_gripper_right_y+offset_gripper_right_y}"/>
-	<xacro:property name="gripper_right_z" value="${def_gripper_right_z+offset_gripper_right_z}"/>
-	<xacro:property name="gripper_right_roll" value="${def_gripper_right_roll+offset_gripper_right_roll}"/>
-	<xacro:property name="gripper_right_pitch" value="${def_gripper_right_pitch+offset_gripper_right_pitch}"/>
-	<xacro:property name="gripper_right_yaw" value="${def_gripper_right_yaw+offset_gripper_right_yaw}"/>
-	<!-- neck mount positions | relative to arm_torso_link -->
-	<xacro:property name="neck_x" value="${def_neck_x+offset_neck_x}"/>
-	<xacro:property name="neck_y" value="${def_neck_y+offset_neck_y}"/>
-	<xacro:property name="neck_z" value="${def_neck_z+offset_neck_z}"/>
-	<xacro:property name="neck_roll" value="${def_neck_roll+offset_neck_roll}"/>
-	<xacro:property name="neck_pitch" value="${def_neck_pitch+offset_neck_pitch}"/>
-	<xacro:property name="neck_yaw" value="${def_neck_yaw+offset_neck_yaw}"/>
-	<!-- head mount positions | relative to neck_mount_link -->
-	<xacro:property name="head_x" value="${def_head_x+offset_head_x}"/>
-	<xacro:property name="head_y" value="${def_head_y+offset_head_y}"/>
-	<xacro:property name="head_z" value="${def_head_z+offset_head_z}"/>
-	<xacro:property name="head_roll" value="${def_head_roll+offset_head_roll}"/>
-	<xacro:property name="head_pitch" value="${def_head_pitch+offset_head_pitch}"/>
-	<xacro:property name="head_yaw" value="${def_head_yaw+offset_head_yaw}"/>
-	<!-- ids_middle mount positions | relative to head_cam_holder_link -->
-	<xacro:property name="ids_middle_x" value="${def_ids_middle_x+offset_ids_middle_x}"/>
-	<xacro:property name="ids_middle_y" value="${def_ids_middle_y+offset_ids_middle_y}"/>
-	<xacro:property name="ids_middle_z" value="${def_ids_middle_z+offset_ids_middle_z}"/>
-	<xacro:property name="ids_middle_roll" value="${def_ids_middle_roll+offset_ids_middle_roll}"/>
-	<xacro:property name="ids_middle_pitch" value="${def_ids_middle_pitch+offset_ids_middle_pitch}"/>
-	<xacro:property name="ids_middle_yaw" value="${def_ids_middle_yaw+offset_ids_middle_yaw}"/>
-	<!-- ids_left mount positions | relative to head_cam_holder_link -->
-	<xacro:property name="ids_left_x" value="${def_ids_left_x+offset_ids_left_x}"/>
-	<xacro:property name="ids_left_y" value="${def_ids_left_y+offset_ids_left_y}"/>
-	<xacro:property name="ids_left_z" value="${def_ids_left_z+offset_ids_left_z}"/>
-	<xacro:property name="ids_left_roll" value="${def_ids_left_roll+offset_ids_left_roll}"/>
-	<xacro:property name="ids_left_pitch" value="${def_ids_left_pitch+offset_ids_left_pitch}"/>
-	<xacro:property name="ids_left_yaw" value="${def_ids_left_yaw+offset_ids_left_yaw}"/>
-	<!-- ids_right mount positions | relative to head_cam_holder_link -->
-	<xacro:property name="ids_right_x" value="${def_ids_right_x+offset_ids_right_x}"/>
-	<xacro:property name="ids_right_y" value="${def_ids_right_y+offset_ids_right_y}"/>
-	<xacro:property name="ids_right_z" value="${def_ids_right_z+offset_ids_right_z}"/>
-	<xacro:property name="ids_right_roll" value="${def_ids_right_roll+offset_ids_right_roll}"/>
-	<xacro:property name="ids_right_pitch" value="${def_ids_right_pitch+offset_ids_right_pitch}"/>
-	<xacro:property name="ids_right_yaw" value="${def_ids_right_yaw+offset_ids_right_yaw}"/>
-	<!-- cam_holder mount positions | relative to head_powerball_knob_link -->
-	<xacro:property name="cam_holder_x" value="${def_cam_holder_x+offset_cam_holder_x}"/>
-	<xacro:property name="cam_holder_y" value="${def_cam_holder_y+offset_cam_holder_y}"/>
-	<xacro:property name="cam_holder_z" value="${def_cam_holder_z+offset_cam_holder_z}"/>
-	<xacro:property name="cam_holder_roll" value="${def_cam_holder_roll+offset_cam_holder_roll}"/>
-	<xacro:property name="cam_holder_pitch" value="${def_cam_holder_pitch+offset_cam_holder_pitch}"/>
-	<xacro:property name="cam_holder_yaw" value="${def_cam_holder_yaw+offset_cam_holder_yaw}"/>
 </robot>

File: cob_hardware_config/raw3-3/urdf/raw3-3.urdf.xacro (robot description, xacro)
@@ -12,6 +12,4 @@
   <xacro:include filename="$(find raw_description)/urdf/tower_symetric/tower.urdf.xacro" />
 -->
-  <!-- frida -->
-  <xacro:include filename="$(find prace_common)/urdf/prace.urdf.xacro" />
   <!-- composition of the robot -->
   <xacro:raw_base name="base"/>
@@ -27,6 +25,4 @@
   </xacro:tower_symetric>
 -->
-  <!-- prace macros -->
-  <xacro:prace/>
   <!-- scan top mount -->
     <joint name="base_laser_top_joint" type="fixed" >
