Commit message: added arms, hands and cameras

File: cob_hardware_config/cob4-5/urdf/calibration_default.urdf.xacro (robot description, xacro)
@@ -49,4 +49,18 @@
 	<property name="def_sensorring_pitch" value="0.0"/>
 	<property name="def_sensorring_yaw" value="0.0"/>
+	<!-- arm right mount positions | relative to torso_3_link -->
+	<property name="def_arm_right_x" value="0.0"/>
+	<property name="def_arm_right_y" value="-0.014"/>
+	<property name="def_arm_right_z" value="0.55"/>
+	<property name="def_arm_right_roll" value="1.57097"/>
+	<property name="def_arm_right_pitch" value="0"/>
+	<property name="def_arm_right_yaw" value="0.0"/>
+	<!-- arm left mount positions | relative to torso_3_link -->
+	<property name="def_arm_left_x" value="0.0"/>
+	<property name="def_arm_left_y" value="0.014"/>
+	<property name="def_arm_left_z" value="0.55"/>
+	<property name="def_arm_left_roll" value="1.57097"/>
+	<property name="def_arm_left_pitch" value="0"/>
+	<property name="def_arm_left_yaw" value="3.14159"/>
 	<!-- *********************************** -->
 	<!-- kinematic chain reference positions -->
@@ -71,13 +85,20 @@
 	<property name="def_torso_cam3d_down_y" value="0.0"/>
 	<property name="def_torso_cam3d_down_z" value="0.14005"/>
-	<property name="def_torso_cam3d_down_roll" value="2.18166"/> <!--2.18166-->
-	<property name="def_torso_cam3d_down_pitch" value="0.0"/>
-	<property name="def_torso_cam3d_down_yaw" value="1.57079"/> <!--1.57079-->
+	<property name="def_torso_cam3d_down_roll" value="0.0"/>
+	<property name="def_torso_cam3d_down_pitch" value="0.54"/>
+	<property name="def_torso_cam3d_down_yaw" value="0.0"/>
 	<!-- cam3d | handeye calibration | relative to sensorring_link -->
-	<property name="def_sensorring_cam3d_x" value="0.096"/>
-	<property name="def_sensorring_cam3d_y" value="0.0"/>
-	<property name="def_sensorring_cam3d_z" value="0.0195"/>
-	<property name="def_sensorring_cam3d_roll" value="-1.5708"/>
-	<property name="def_sensorring_cam3d_pitch" value="0.0"/>
-	<property name="def_sensorring_cam3d_yaw" value="-1.5708"/>
+	<property name="def_sensorring_cam3d_front_x" value="0.096"/>
+	<property name="def_sensorring_cam3d_front_y" value="0.0"/>
+	<property name="def_sensorring_cam3d_front_z" value="0.0195"/>
+	<property name="def_sensorring_cam3d_front_roll" value="-1.95"/>
+	<property name="def_sensorring_cam3d_front_pitch" value="0.0"/>
+	<property name="def_sensorring_cam3d_front_yaw" value="-1.5708"/>
+	<!-- cam3d | handeye calibration | relative to sensorring_link -->
+	<property name="def_sensorring_cam3d_back_x" value="-0.096"/>
+	<property name="def_sensorring_cam3d_back_y" value="0.0"/>
+	<property name="def_sensorring_cam3d_back_z" value="0.0195"/>
+	<property name="def_sensorring_cam3d_back_roll" value="-1.5708"/>
+	<property name="def_sensorring_cam3d_back_pitch" value="0.0"/>
+	<property name="def_sensorring_cam3d_back_yaw" value="-1.5708"/>
 </robot>

File: cob_hardware_config/cob4-5/urdf/cob4-5.urdf.xacro (robot description, xacro)
@@ -11,9 +11,11 @@
   <xacro:include filename="$(find cob_description)/urdf/cob4_base/base.urdf.xacro" />
   <!-- torso -->
-  <xacro:include filename="$(find cob_description)/urdf/cob4_torso/torso_2dof.urdf.xacro" />
+  <xacro:include filename="$(find cob_description)/urdf/cob4_torso/torso_static_realsense.urdf.xacro" />
+  <!-- arm -->
+  <xacro:include filename="$(find schunk_description)/urdf/lwa4p_extended/lwa4p_extended.urdf.xacro" />
   <!-- head -->
   <xacro:include filename="$(find cob_description)/urdf/cob4_head/head_static.urdf.xacro" />
   <!-- sensorring -->
-  <xacro:include filename="$(find cob_description)/urdf/cob4_sensorring/sensorring_asus.urdf.xacro" />
+  <xacro:include filename="$(find cob_description)/urdf/cob4_sensorring/sensorring_3dcs_asus.urdf.xacro" />
   <!-- composition of the robot -->
   <xacro:base name="base" use_old_joint_names="false"/>
@@ -45,3 +47,21 @@
     </plugin>
   </gazebo>
+  <xacro:schunk_lwa4p_extended name="arm_right" parent="torso_3_link" has_podest="false">
+    <origin xyz="${arm_right_x} ${arm_right_y} ${arm_right_z}" rpy="${arm_right_roll} ${arm_right_pitch} ${arm_right_yaw}" />
+  </xacro:schunk_lwa4p_extended>
+  <gazebo>
+    <plugin name="ros_control" filename="libhwi_switch_gazebo_ros_control.so">
+      <robotNamespace>arm_right</robotNamespace>
+      <filterJointsParam>joint_names</filterJointsParam>
+    </plugin>
+  </gazebo>
+  <xacro:schunk_lwa4p_extended name="arm_left" parent="torso_3_link" has_podest="false">
+    <origin xyz="${arm_left_x} ${arm_left_y} ${arm_left_z}" rpy="${arm_left_roll} ${arm_left_pitch} ${arm_left_yaw}" />
+  </xacro:schunk_lwa4p_extended>
+  <gazebo>
+    <plugin name="ros_control" filename="libhwi_switch_gazebo_ros_control.so">
+      <robotNamespace>arm_left</robotNamespace>
+      <filterJointsParam>joint_names</filterJointsParam>
+    </plugin>
+  </gazebo>
 </robot>

File: cob_hardware_config/cob4-5/urdf/properties.urdf.xacro (robot description, xacro)
@@ -52,4 +52,18 @@
 	<property name="sensorring_pitch" value="${def_sensorring_pitch+offset_sensorring_pitch}"/>
 	<property name="sensorring_yaw" value="${def_sensorring_yaw+offset_sensorring_yaw}"/>
+	<!-- arm mount positions | relative to torso_3_link -->
+	<property name="arm_right_x" value="${def_arm_right_x+offset_arm_right_x}"/>
+	<property name="arm_right_y" value="${def_arm_right_y+offset_arm_right_y}"/>
+	<property name="arm_right_z" value="${def_arm_right_z+offset_arm_right_z}"/>
+	<property name="arm_right_roll" value="${def_arm_right_roll+offset_arm_right_roll}"/>
+	<property name="arm_right_pitch" value="${def_arm_right_pitch+offset_arm_right_pitch}"/>
+	<property name="arm_right_yaw" value="${def_arm_right_yaw+offset_arm_right_yaw}"/>
+	<!-- arm mount positions | relative to torso_3_link -->
+	<property name="arm_left_x" value="${def_arm_left_x+offset_arm_left_x}"/>
+	<property name="arm_left_y" value="${def_arm_left_y+offset_arm_left_y}"/>
+	<property name="arm_left_z" value="${def_arm_left_z+offset_arm_left_z}"/>
+	<property name="arm_left_roll" value="${def_arm_left_roll+offset_arm_left_roll}"/>
+	<property name="arm_left_pitch" value="${def_arm_left_pitch+offset_arm_left_pitch}"/>
+	<property name="arm_left_yaw" value="${def_arm_left_yaw+offset_arm_left_yaw}"/>
 	<!-- *********************************** -->
 	<!-- kinematic chain reference positions -->
@@ -78,9 +92,16 @@
 	<property name="torso_cam3d_down_yaw" value="${def_torso_cam3d_down_yaw+offset_torso_cam3d_down_yaw}"/>
 	<!-- cam3d | handeye calibration | relative to sensorring_link -->
-	<property name="sensorring_cam3d_x" value="${def_sensorring_cam3d_x+offset_sensorring_cam3d_x}"/>
-	<property name="sensorring_cam3d_y" value="${def_sensorring_cam3d_y+offset_sensorring_cam3d_y}"/>
-	<property name="sensorring_cam3d_z" value="${def_sensorring_cam3d_z+offset_sensorring_cam3d_z}"/>
-	<property name="sensorring_cam3d_roll" value="${def_sensorring_cam3d_roll+offset_sensorring_cam3d_roll}"/>
-	<property name="sensorring_cam3d_pitch" value="${def_sensorring_cam3d_pitch+offset_sensorring_cam3d_pitch}"/>
-	<property name="sensorring_cam3d_yaw" value="${def_sensorring_cam3d_yaw+offset_sensorring_cam3d_yaw}"/>
+	<property name="sensorring_cam3d_front_x" value="${def_sensorring_cam3d_front_x+offset_sensorring_cam3d_front_x}"/>
+	<property name="sensorring_cam3d_front_y" value="${def_sensorring_cam3d_front_y+offset_sensorring_cam3d_front_y}"/>
+	<property name="sensorring_cam3d_front_z" value="${def_sensorring_cam3d_front_z+offset_sensorring_cam3d_front_z}"/>
+	<property name="sensorring_cam3d_front_roll" value="${def_sensorring_cam3d_front_roll+offset_sensorring_cam3d_front_roll}"/>
+	<property name="sensorring_cam3d_front_pitch" value="${def_sensorring_cam3d_front_pitch+offset_sensorring_cam3d_front_pitch}"/>
+	<property name="sensorring_cam3d_front_yaw" value="${def_sensorring_cam3d_front_yaw+offset_sensorring_cam3d_front_yaw}"/>
+	<!-- cam3d | handeye calibration | relative to sensorring_link -->
+	<property name="sensorring_cam3d_back_x" value="${def_sensorring_cam3d_back_x+offset_sensorring_cam3d_back_x}"/>
+	<property name="sensorring_cam3d_back_y" value="${def_sensorring_cam3d_back_y+offset_sensorring_cam3d_back_y}"/>
+	<property name="sensorring_cam3d_back_z" value="${def_sensorring_cam3d_back_z+offset_sensorring_cam3d_back_z}"/>
+	<property name="sensorring_cam3d_back_roll" value="${def_sensorring_cam3d_back_roll+offset_sensorring_cam3d_back_roll}"/>
+	<property name="sensorring_cam3d_back_pitch" value="${def_sensorring_cam3d_back_pitch+offset_sensorring_cam3d_back_pitch}"/>
+	<property name="sensorring_cam3d_back_yaw" value="${def_sensorring_cam3d_back_yaw+offset_sensorring_cam3d_back_yaw}"/>
 </robot>
