Commit message: harmonize with cob structure

File: cob_hardware_config/raw3-1/urdf/calibration_default.urdf.xacro (robot description, xacro)
@@ -22,4 +22,11 @@
 	<property name="def_torso_pitch" value="0"/>
 	<property name="def_torso_yaw" value="0"/>
+	<!-- head mount positions | relative to head_cover_link -->
+	<property name="def_head_x" value="0.0"/>
+	<property name="def_head_y" value="0.0"/>
+	<property name="def_head_z" value="0.0"/>
+	<property name="def_head_roll" value="0.0"/>
+	<property name="def_head_pitch" value="0.0"/>
+	<property name="def_head_yaw" value="0.0"/>
 	<!--arm mount positions | relative to base_link-->
 	<property name="def_arm_x" value="0.324"/>
@@ -40,23 +47,30 @@
 	<!-- ***************************** -->
 	<!-- left | handeye calibration | relative to head_axis_link -->
-	<property name="def_cam_l_x" value="-0.0171250371"/>
-	<property name="def_cam_l_y" value="-0.0389120491"/>
-	<property name="def_cam_l_z" value="-0.12027305"/>
-	<property name="def_cam_l_roll" value="2.149627771"/>
-	<property name="def_cam_l_pitch" value="-1.5608998734"/>
-	<property name="def_cam_l_yaw" value="-2.2074792588"/>
+	<property name="def_cam_reference_x" value="0.044"/>
+	<property name="def_cam_reference_y" value="0.06"/>
+	<property name="def_cam_reference_z" value="0.092"/>
+	<property name="def_cam_reference_roll" value="-1.57"/>
+	<property name="def_cam_reference_pitch" value="0.0"/>
+	<property name="def_cam_reference_yaw" value="-1.57"/>
+	<!-- left | handeye calibration | relative to head_axis_link -->
+	<property name="def_cam_l_x" value="0.0"/>
+	<property name="def_cam_l_y" value="0.0"/>
+	<property name="def_cam_l_z" value="0.0"/>
+	<property name="def_cam_l_roll" value="0.0"/>
+	<property name="def_cam_l_pitch" value="0.0"/>
+	<property name="def_cam_l_yaw" value="0.0"/>
 	<!-- right | stereo baseline calibration | relative to left camera -->
-	<property name="def_cam_r_x" value="0.044"/>
-	<property name="def_cam_r_y" value="-0.06"/>
-	<property name="def_cam_r_z" value="0.092"/>
-	<property name="def_cam_r_roll" value="-1.57"/>
+	<property name="def_cam_r_x" value="0.12"/>
+	<property name="def_cam_r_y" value="0.0"/>
+	<property name="def_cam_r_z" value="0.0"/>
+	<property name="def_cam_r_roll" value="0.0"/>
 	<property name="def_cam_r_pitch" value="0.0"/>
-	<property name="def_cam_r_yaw" value="-1.57"/>
+	<property name="def_cam_r_yaw" value="0.0"/>
 	<!-- cam3d | handeye calibration | relative to head_axis_link -->
-	<property name="def_cam3d_x" value="0.015"/>
+	<property name="def_cam3d_x" value="0.06"/>
 	<property name="def_cam3d_y" value="0.0"/>
-	<property name="def_cam3d_z" value="0.12"/>
-	<property name="def_cam3d_roll" value="-1.57"/>
+	<property name="def_cam3d_z" value="0.0"/>
+	<property name="def_cam3d_roll" value="0.0"/>
 	<property name="def_cam3d_pitch" value="0.0"/>
-	<property name="def_cam3d_yaw" value="-1.57"/>
+	<property name="def_cam3d_yaw" value="0.0"/>
 </robot>

File: cob_hardware_config/raw3-1/urdf/properties.urdf.xacro (robot description, xacro)
@@ -20,4 +20,11 @@
 	<property name="torso_pitch" value="${def_torso_pitch+offset_torso_pitch}"/>
 	<property name="torso_yaw" value="${def_torso_yaw+offset_torso_yaw}"/>
+	<!-- head mount positions | relative to head_cover_link -->
+	<property name="head_x" value="${def_head_x+offset_head_x}"/>
+	<property name="head_y" value="${def_head_y+offset_head_y}"/>
+	<property name="head_z" value="${def_head_z+offset_head_z}"/>
+	<property name="head_roll" value="${def_head_roll+offset_head_roll}"/>
+	<property name="head_pitch" value="${def_head_pitch+offset_head_pitch}"/>
+	<property name="head_yaw" value="${def_head_yaw+offset_head_yaw}"/>
 	<!-- arm mount positions | relative to base_link -->
 	<property name="arm_x" value="${def_arm_x+offset_arm_x}"/>
@@ -37,11 +44,17 @@
 	<!-- camera calibration properties -->
 	<!-- ***************************** -->
+	<property name="cam_reference_x" value="${def_cam_reference_x+offset_cam_reference_x}"/>
+	<property name="cam_reference_y" value="${def_cam_reference_y+offset_cam_reference_y}"/>
+	<property name="cam_reference_z" value="${def_cam_reference_z+offset_cam_reference_z}"/>
+	<property name="cam_reference_roll" value="${def_cam_reference_roll+offset_cam_reference_roll}"/>
+	<property name="cam_reference_pitch" value="${def_cam_reference_pitch+offset_cam_reference_pitch}"/>
+	<property name="cam_reference_yaw" value="${def_cam_reference_yaw+offset_cam_reference_yaw}"/>
 	<!-- left | handeye calibration | relative to head_axis_link -->
-	<property name="cam_ref_x" value="${def_cam_ref_x+offset_cam_ref_x}"/>
-	<property name="cam_ref_y" value="${def_cam_ref_y+offset_cam_ref_y}"/>
-	<property name="cam_ref_z" value="${def_cam_ref_z+offset_cam_ref_z}"/>
-	<property name="cam_ref_roll" value="${def_cam_ref_roll+offset_cam_ref_roll}"/>
-	<property name="cam_ref_pitch" value="${def_cam_ref_pitch+offset_cam_ref_pitch}"/>
-	<property name="cam_ref_yaw" value="${def_cam_ref_yaw+offset_cam_ref_yaw}"/>
+	<property name="cam_l_x" value="${def_cam_l_x+offset_cam_l_x}"/>
+	<property name="cam_l_y" value="${def_cam_l_y+offset_cam_l_y}"/>
+	<property name="cam_l_z" value="${def_cam_l_z+offset_cam_l_z}"/>
+	<property name="cam_l_roll" value="${def_cam_l_roll+offset_cam_l_roll}"/>
+	<property name="cam_l_pitch" value="${def_cam_l_pitch+offset_cam_l_pitch}"/>
+	<property name="cam_l_yaw" value="${def_cam_l_yaw+offset_cam_l_yaw}"/>
 	<!-- right | stereo baseline calibration | relative to left camera -->
 	<property name="cam_r_x" value="${def_cam_r_x+offset_cam_r_x}"/>

File: cob_hardware_config/raw3-1/urdf/raw3-1.urdf.xacro (robot description, xacro)
@@ -13,16 +13,29 @@
   <!-- raw tower -->
   <include filename="$(find raw_description)/urdf/tower_asymetric/tower.urdf.xacro" />
+  <!-- torso -->
+  <include filename="$(find raw_description)/urdf/torso/torso.urdf.xacro" />
+  <!-- head -->
+  <include filename="$(find raw_description)/urdf/head/head.urdf.xacro" />
+  <include filename="$(find cob_description)/urdf/lookat/lookat.urdf.xacro" />
+  <!-- ur_arm -->
+  <include filename="$(find raw_description)/urdf/ur_arm/ur10_arm.urdf.xacro" />
   <!-- raw boxgripper -->
   <include filename="$(find raw_description)/urdf/boxgripper/boxgripper.urdf.xacro" />
   <!-- generic simulator_gazebo plugins for starting mechanism control, ros time, ros battery -->
   <include filename="$(find cob_description)/gazebo/gazebo.urdf.xacro" />
-  <!-- torso -->
-  <include filename="$(find raw_description)/urdf/torso/torso.urdf.xacro" />
-  <!-- ur_arm -->
-  <include filename="$(find raw_description)/urdf/ur_arm/ur10_arm.urdf.xacro" />
   <xacro:raw_base name="base"/>
   <xacro:tower_asymetric name="tower" parent="base_link">
       <origin xyz="${tower_x} ${tower_y} ${tower_z}" rpy="${tower_roll} ${tower_pitch} ${tower_yaw}" />
   </xacro:tower_asymetric>
+  <xacro:raw_torso name="torso" parent="base_link">
+      <origin xyz="${torso_x} ${torso_y} ${torso_z}" rpy="${torso_roll} ${torso_pitch} ${torso_yaw}" />
+  </xacro:raw_torso>
+  <xacro:raw_head name="head" parent="torso_2_link">
+    <origin xyz="${head_x} ${head_y} ${head_z}" rpy="${head_roll} ${head_pitch} ${head_yaw}" />
+  </xacro:raw_head>
+  <xacro:cob_lookat name="lookat" parent="torso_2_link">
+    <origin xyz="${head_x} ${head_y} ${head_z}" rpy="${head_roll} ${head_pitch} ${head_yaw}" />
+    <axis xyz="1 0 0"/>
+  </xacro:cob_lookat>
   <xacro:cob_ur10 name="arm" parent="base_link">
       <origin xyz="${arm_x} ${arm_y} ${arm_z}" rpy="${arm_roll} ${arm_pitch} ${arm_yaw}" />
@@ -35,7 +48,4 @@
   </joint>
   <xacro:ur10_robot prefix="arm_"/>-->
-  <xacro:raw_torso name="torso" parent="base_link">
-      <origin xyz="${torso_x} ${torso_y} ${torso_z}" rpy="${torso_roll} ${torso_pitch} ${torso_yaw}" />
-  </xacro:raw_torso>
   <xacro:raw_boxgripper name="gripper" parent="arm_ee_link">
       <origin xyz="${gripper_x} ${gripper_y} ${gripper_z}" rpy="${gripper_roll} ${gripper_pitch} ${gripper_yaw}" />

Commit message: added arm in bringup, corrected torso mounting angle

File: cob_hardware_config/raw3-1/urdf/calibration_default.urdf.xacro (robot description, xacro)
@@ -34,5 +34,5 @@
 	<xacro:property name="def_torso_roll" value="0"/>
 	<xacro:property name="def_torso_pitch" value="0"/>
-	<xacro:property name="def_torso_yaw" value="0"/>
+	<xacro:property name="def_torso_yaw" value="-0.445"/>
 	<!-- head mount positions | relative to head_cover_link -->
 	<xacro:property name="def_head_x" value="0.0"/>

Commit message: adaptations to current configuration for order-picking

File: cob_hardware_config/raw3-1/urdf/calibration_default.urdf.xacro (robot description, xacro)
@@ -45,5 +45,5 @@
 	<property name="def_arm_x" value="0.324"/>
 	<property name="def_arm_y" value="-0.191"/>
-	<property name="def_arm_z" value="0.565"/>
+	<property name="def_arm_z" value="0.585"/>  <!-- 0.565 -->
 	<property name="def_arm_roll" value="0.0"/>
 	<property name="def_arm_pitch" value="0.0"/>

File: cob_hardware_config/raw3-1/urdf/raw3-1.urdf.xacro (robot description, xacro)
@@ -9,5 +9,6 @@
   <xacro:include filename="$(find raw_description)/urdf/base_long/base.urdf.xacro" />
   <!-- raw tower -->
-  <xacro:include filename="$(find raw_description)/urdf/tower_asymetric/tower.urdf.xacro" />
+  <!--xacro:include filename="$(find raw_description)/urdf/tower_asymetric/tower.urdf.xacro" /-->
+  <xacro:include filename="$(find raw_description)/urdf/tower_symetric/tower.urdf.xacro" />
   <!-- torso -->
   <xacro:include filename="$(find raw_description)/urdf/torso/torso.urdf.xacro" />
@@ -26,7 +27,10 @@
     </plugin>
   </gazebo>
-  <xacro:tower_asymetric name="tower" parent="base_link">
+  <!--xacro:tower_asymetric name="tower" parent="base_link">
     <origin xyz="${tower_x} ${tower_y} ${tower_z}" rpy="${tower_roll} ${tower_pitch} ${tower_yaw}" />
-  </xacro:tower_asymetric>
+  </xacro:tower_asymetric-->
+  <xacro:tower_symetric name="tower" parent="base_link">
+    <origin xyz="${tower_x} ${tower_y} ${tower_z}" rpy="${tower_roll} ${tower_pitch} ${tower_yaw}" />
+  </xacro:tower_symetric>
   <xacro:raw_torso name="torso" parent="base_link">
     <origin xyz="${torso_x} ${torso_y} ${torso_z}" rpy="${torso_roll} ${torso_pitch} ${torso_yaw}" />
@@ -71,5 +75,5 @@
   <!-- END: IMU brick  mount -->
   <!-- rfid_front mount on raw3-1 -->
-  <joint name="rfid_front_joint" type="fixed" >
+  <!--joint name="rfid_front_joint" type="fixed" >
     <origin xyz="0.55128 0.0 0.09" rpy="0 0 0" />
     <parent link="base_link" />
@@ -87,8 +91,8 @@
       </material>
     </visual>
-  </link>
+  </link-->
   <!-- END: rfid front mount -->
   <!-- rfid_rear mount on raw3-1 -->
-  <joint name="rfid_rear_joint" type="fixed" >
+  <!--joint name="rfid_rear_joint" type="fixed" >
     <origin xyz="-0.55128 0.0 0.09" rpy="0 0 ${M_PI}" />
     <parent link="base_link" />
@@ -106,8 +110,8 @@
       </material>
     </visual>
-  </link>
+  </link-->
   <!-- END: rfid rear mount -->
   <!-- rfid_right mount on raw3-1 -->
-  <joint name="rfid_right_joint" type="fixed" >
+  <!--joint name="rfid_right_joint" type="fixed" >
     <origin xyz="0.0 -0.30850 0.09" rpy="0 0 ${-0.5*M_PI}" />
     <parent link="base_link" />
@@ -125,8 +129,8 @@
       </material>
     </visual>
-  </link>
+  </link-->
   <!-- END: rfid right mount -->
   <!-- Camera pillar -->
-  <joint name="camera_pillar_joint" type="fixed" >
+  <!--joint name="camera_pillar_joint" type="fixed" >
     <origin xyz="0.4925 0.0825 0.48" rpy="0 0 0" />
     <parent link="base_link" />
@@ -142,8 +146,8 @@
       <material name="IPA/LightGrey" />
     </visual>
-  </link>
+  </link-->
   <!-- END: camera_pillar -->
   <!-- Softkinetic 'left' mount on raw3-1 -->
-  <joint name="softkinetic_left_joint" type="fixed" >
+  <!--joint name="softkinetic_left_joint" type="fixed" >
     <origin xyz="0.015 0.06 0.215" rpy="0.0 ${M_PI/2} 0.0" />
     <parent link="camera_pillar_link" />
@@ -159,8 +163,8 @@
       <material name="IPA/Black" />
     </visual>
-  </link>
+  </link-->
   <!-- END: Softkinetic 'left' mount -->
   <!-- Softkinetic 'right' mount on raw3-1 -->
-  <joint name="softkinetic_right_joint" type="fixed" >
+  <!--joint name="softkinetic_right_joint" type="fixed" >
     <origin xyz="0.015 -0.06 0.215" rpy="${M_PI} -${M_PI/2} 0.0" />
     <parent link="camera_pillar_link" />
@@ -176,8 +180,8 @@
       <material name="IPA/Black" />
     </visual>
-  </link>
+  </link-->
   <!-- END: Softkinetic 'right' mount -->
   <!-- Kinect mount on raw3-1 -->
-  <joint name="kinect_joint" type="fixed" >
+  <!--joint name="kinect_joint" type="fixed" >
     <origin xyz="0.015 0.0 0.25" rpy="${M_PI/2} 0 ${M_PI/2}" />
     <parent link="camera_pillar_link" />
@@ -193,5 +197,5 @@
       <material name="IPA/Black" />
     </visual>
-  </link>
+  </link-->
   <!-- END: Kinect mount -->
 </robot>

Commit message: adaptations to current configuration for order-picking

File: cob_hardware_config/raw3-1/urdf/calibration_default.urdf.xacro (robot description, xacro)
@@ -45,5 +45,5 @@
 	<xacro:property name="def_arm_x" value="0.324"/>
 	<xacro:property name="def_arm_y" value="-0.191"/>
-	<xacro:property name="def_arm_z" value="0.565"/>
+	<xacro:property name="def_arm_z" value="0.585"/>
 	<xacro:property name="def_arm_roll" value="0.0"/>
 	<xacro:property name="def_arm_pitch" value="0.0"/>

File: cob_hardware_config/raw3-1/urdf/raw3-1.urdf.xacro (robot description, xacro)
@@ -9,5 +9,6 @@
   <xacro:include filename="$(find raw_description)/urdf/base_long/base.urdf.xacro" />
   <!-- raw tower -->
-  <xacro:include filename="$(find raw_description)/urdf/tower_asymetric/tower.urdf.xacro" />
+  <!--xacro:include filename="$(find raw_description)/urdf/tower_asymetric/tower.urdf.xacro" /-->
+  <xacro:include filename="$(find raw_description)/urdf/tower_symetric/tower.urdf.xacro" />
   <!-- torso -->
   <xacro:include filename="$(find raw_description)/urdf/torso/torso.urdf.xacro" />
@@ -20,7 +21,10 @@
   <!-- composition of the robot -->
   <xacro:raw_base name="base"/>
-  <xacro:tower_asymetric name="tower" parent="base_link">
+  <!--xacro:tower_asymetric name="tower" parent="base_link">
     <origin xyz="${tower_x} ${tower_y} ${tower_z}" rpy="${tower_roll} ${tower_pitch} ${tower_yaw}" />
-  </xacro:tower_asymetric>
+  </xacro:tower_asymetric-->
+  <xacro:tower_symetric name="tower" parent="base_link">
+    <origin xyz="${tower_x} ${tower_y} ${tower_z}" rpy="${tower_roll} ${tower_pitch} ${tower_yaw}" />
+  </xacro:tower_symetric>
   <xacro:raw_torso name="torso" parent="base_link">
     <origin xyz="${torso_x} ${torso_y} ${torso_z}" rpy="${torso_roll} ${torso_pitch} ${torso_yaw}" />
@@ -53,5 +57,5 @@
   <!-- END: IMU brick  mount -->
   <!-- rfid_front mount on raw3-1 -->
-  <joint name="rfid_front_joint" type="fixed" >
+  <!--joint name="rfid_front_joint" type="fixed" >
     <origin xyz="0.55128 0.0 0.09" rpy="0 0 0" />
     <parent link="base_link" />
@@ -69,8 +73,8 @@
       </material>
     </visual>
-  </link>
+  </link-->
   <!-- END: rfid front mount -->
   <!-- rfid_rear mount on raw3-1 -->
-  <joint name="rfid_rear_joint" type="fixed" >
+  <!--joint name="rfid_rear_joint" type="fixed" >
     <origin xyz="-0.55128 0.0 0.09" rpy="0 0 ${M_PI}" />
     <parent link="base_link" />
@@ -88,8 +92,8 @@
       </material>
     </visual>
-  </link>
+  </link-->
   <!-- END: rfid rear mount -->
   <!-- rfid_right mount on raw3-1 -->
-  <joint name="rfid_right_joint" type="fixed" >
+  <!--joint name="rfid_right_joint" type="fixed" >
     <origin xyz="0.0 -0.30850 0.09" rpy="0 0 ${-0.5*M_PI}" />
     <parent link="base_link" />
@@ -107,8 +111,8 @@
       </material>
     </visual>
-  </link>
+  </link-->
   <!-- END: rfid right mount -->
   <!-- Camera pillar -->
-  <joint name="camera_pillar_joint" type="fixed" >
+  <!--joint name="camera_pillar_joint" type="fixed" >
     <origin xyz="0.4925 0.0825 0.48" rpy="0 0 0" />
     <parent link="base_link" />
@@ -124,8 +128,8 @@
       <material name="IPA/LightGrey" />
     </visual>
-  </link>
+  </link-->
   <!-- END: camera_pillar -->
   <!-- Softkinetic 'left' mount on raw3-1 -->
-  <joint name="softkinetic_left_joint" type="fixed" >
+  <!--joint name="softkinetic_left_joint" type="fixed" >
     <origin xyz="0.015 0.06 0.215" rpy="0.0 ${M_PI/2} 0.0" />
     <parent link="camera_pillar_link" />
@@ -141,8 +145,8 @@
       <material name="IPA/Black" />
     </visual>
-  </link>
+  </link-->
   <!-- END: Softkinetic 'left' mount -->
   <!-- Softkinetic 'right' mount on raw3-1 -->
-  <joint name="softkinetic_right_joint" type="fixed" >
+  <!--joint name="softkinetic_right_joint" type="fixed" >
     <origin xyz="0.015 -0.06 0.215" rpy="${M_PI} -${M_PI/2} 0.0" />
     <parent link="camera_pillar_link" />
@@ -158,8 +162,8 @@
       <material name="IPA/Black" />
     </visual>
-  </link>
+  </link-->
   <!-- END: Softkinetic 'right' mount -->
   <!-- Kinect mount on raw3-1 -->
-  <joint name="kinect_joint" type="fixed" >
+  <!--joint name="kinect_joint" type="fixed" >
     <origin xyz="0.015 0.0 0.25" rpy="${M_PI/2} 0 ${M_PI/2}" />
     <parent link="camera_pillar_link" />
@@ -175,5 +179,5 @@
       <material name="IPA/Black" />
     </visual>
-  </link>
+  </link-->
   <!-- END: Kinect mount -->
 </robot>
