Commit message: renamed icob to raw and merged and cleaned up lots of things

File: cob_hardware_config/raw3-1/urdf/raw3-1.urdf.xacro (robot description, xacro)
@@ -8,9 +8,15 @@
   <include filename="$(find cob_description)/urdf/common.xacro" />
   <include filename="$(find cob_description)/urdf/materials.urdf.xacro" />
+  <include filename="$(find cob_hardware_config)/raw3-1/calibration/calibration.urdf.xacro" />
   <!-- icob base -->
   <!--include filename="$(find icob_description)/ros/urdf/base_v1/base.urdf.xacro" /-->	<!-- fxm: old	-->
-  <include filename="$(find icob_description)/urdf/base/base.urdf.xacro" />
+  <include filename="$(find raw_description)/urdf/base/base.urdf.xacro" />
   <!-- generic simulator_gazebo plugins for starting mechanism control, ros time, ros battery -->
   <include filename="$(find cob_description)/gazebo/gazebo.urdf.xacro" />
+  <!-- ur_arm -->
+ <include filename="$(find raw_description)/urdf/arm_ur/arm.urdf.xacro" />
   <xacro:icob_base name="base"/>	<!--with new collision_model, but no platform_controller available yet-->
+  <xacro:cob_arm_ur name="arm" parent="base_link">
+    <origin xyz="-0.33 0.16 0.6" rpy="0 1.57 0" />
+  </xacro:cob_arm_ur>
 </robot>

Commit message: modifications on robot with ur5 arm

File: cob_hardware_config/raw3-1/urdf/raw3-1.urdf.xacro (robot description, xacro)
@@ -15,8 +15,9 @@
   <include filename="$(find cob_description)/gazebo/gazebo.urdf.xacro" />
   <!-- ur_arm -->
- <include filename="$(find raw_description)/urdf/arm_ur/arm.urdf.xacro" />
+ <!--include filename="$(find raw_description)/urdf/arm_ur/arm.urdf.xacro" /-->
+ <include filename="$(find ur5_description)/urdf/model.urdf.xacro" />
   <xacro:icob_base name="base"/>	<!--with new collision_model, but no platform_controller available yet-->
-  <xacro:cob_arm_ur name="arm" parent="base_link">
-    <origin xyz="-0.33 0.16 0.6" rpy="0 1.57 0" />
-  </xacro:cob_arm_ur>
+  <xacro:ur5 name="arm" parent="base_link">
+    <origin xyz="-0.32 -0.03 0.48" rpy="0 0 2.35" />
+  </xacro:ur5>
 </robot>

Commit message: changed direction of urdf model to new convention

File: cob_hardware_config/raw3-1/urdf/raw3-1.urdf.xacro (robot description, xacro)
@@ -19,5 +19,5 @@
   <xacro:icob_base name="base"/>	<!--with new collision_model, but no platform_controller available yet-->
   <xacro:ur5 name="arm" parent="base_link">
-    <origin xyz="-0.32 -0.03 0.48" rpy="0 0 2.35" />
+    <origin xyz="0.32 0.03 0.48" rpy="0 0 -0.79" />
   </xacro:ur5>
 </robot>

Commit message: modifications for upstream ur5_description

File: cob_hardware_config/raw3-1/urdf/raw3-1.urdf.xacro (robot description, xacro)
@@ -17,7 +17,14 @@
  <!--include filename="$(find raw_description)/urdf/arm_ur/arm.urdf.xacro" /-->
  <include filename="$(find ur5_description)/urdf/model.urdf.xacro" />
+ <!--include filename="$(find frida_description)/urdf/frida/frida.urdf.xacro" /-->
   <xacro:icob_base name="base"/>
-  <xacro:ur5 name="arm" parent="base_link">
-    <origin xyz="0.32 0.03 0.48" rpy="0 0 -0.79" />
-  </xacro:ur5>
+  <!--xacro:frida name="arm" parent="base_link">
+    <origin xyz="0.62 0.00 0.88" rpy="0 0 0" />
+  </xacro:frida-->
+  <xacro:ur5_robot prefix="arm_"/>
+  <joint name="arm_base_joint" type="fixed" >
+		 <origin xyz="0.32 0.03 0.48" rpy="0 0 -0.79" />
+		<parent link="base_link" />
+		<child link="arm_base_link" />
+  </joint>
 </robot>

Commit message: modifications for raw3-1

File: cob_hardware_config/raw3-1/urdf/raw3-1.urdf.xacro (robot description, xacro)
@@ -15,8 +15,10 @@
   <include filename="$(find cob_description)/gazebo/gazebo.urdf.xacro" />
   <!-- ur_arm -->
- <include filename="$(find raw_description)/urdf/arm_ur/arm.urdf.xacro" />
-  <xacro:icob_base name="base"/>	<!--with new collision_model, but no platform_controller available yet-->
+  <include filename="$(find raw_description)/urdf/arm_ur/arm.urdf.xacro" />
+  <!-- frida -->
+  <!--include filename="$(find frida_description)/urdf/frida/frida.urdf.xacro" /-->
+  <xacro:raw_base name="base"/>	<!--with new collision_model, but no platform_controller available yet-->
   <xacro:cob_arm_ur name="arm" parent="base_link">
-    <origin xyz="-0.33 0.16 0.6" rpy="0 1.57 0" />
+    <origin xyz="-0.33 0.16 0.6" rpy="0 ${M_PI/2} 0" />
   </xacro:cob_arm_ur>
 </robot>

Commit message: use old arm model

File: cob_hardware_config/raw3-1/urdf/raw3-1.urdf.xacro (robot description, xacro)
@@ -17,6 +17,6 @@
   <include filename="$(find raw_description)/urdf/torso/torso.urdf.xacro" />
   <!-- ur_arm -->
- <!--include filename="$(find raw_description)/urdf/arm_ur/arm.urdf.xacro" /-->
- <include filename="$(find ur5_description)/urdf/model.urdf.xacro" />
+ <include filename="$(find raw_description)/urdf/arm_ur/arm.urdf.xacro" />
+ <!--include filename="$(find ur5_description)/urdf/model.urdf.xacro" /-->
   <!-- frida -->
   <!--include filename="$(find frida_description)/urdf/frida/frida.urdf.xacro" /-->
@@ -25,13 +25,13 @@
     <origin xyz="0.166 0.2175 0.5405" rpy="0 0 0" />
   </xacro:cob_torso_v1>
-  <!--xacro:cob_arm_ur name="arm" parent="base_link">
+  <xacro:cob_arm_ur name="arm" parent="base_link">
     <origin xyz="-0.33 0.16 0.6" rpy="0 ${M_PI/2} 0" />
-  </xacro:cob_arm_ur-->
-  <xacro:ur5_robot prefix="arm_"/>
+  </xacro:cob_arm_ur>
+  <!--xacro:ur5_robot prefix="arm_"/>
   <joint name="arm_base_joint" type="fixed" >
 		 <origin xyz="0.3235 -0.191 0.58" rpy="0 0 -0.79" />
 		<parent link="base_link" />
 		<child link="arm_base_link" />
-  </joint>
+  </joint-->
   <!--xacro:frida name="arm" parent="base_link">
     <origin xyz="0.62 0.00 0.88" rpy="0 0 0" />

Commit message: finished raw3-1 model --- V1

File: cob_hardware_config/raw3-1/urdf/raw3-1.urdf.xacro (robot description, xacro)
@@ -22,9 +22,12 @@
   <!--include filename="$(find frida_description)/urdf/frida/frida.urdf.xacro" /-->
   <xacro:raw_base name="base"/>	<!--with new collision_model, but no platform_controller available yet-->
+ <!--origin xyz="0.166 0.2175 0.5405" rpy="0 0 0" /-->
   <xacro:cob_torso_v1 name="torso" parent="base_link">
-    <origin xyz="0.166 0.2175 0.5405" rpy="0 0 0" />
+    <origin xyz="-0.36 -0.099 0.488" rpy="${M_PI} 0 0" />
   </xacro:cob_torso_v1>
   <xacro:cob_arm_ur name="arm" parent="base_link">
-    <origin xyz="-0.33 0.16 0.6" rpy="0 ${M_PI/2} 0" />
+    <!--origin xyz="-0.33 0.16 0.6" rpy="0 ${M_PI/2} 0" /-->
+    <origin xyz="-0.324 0.22 0.565" rpy="0 ${M_PI/2} 0" />
+	<!--in cad model z = 0.587  - fxmlc-->
   </xacro:cob_arm_ur>
   <!--xacro:ur5_robot prefix="arm_"/>

Commit message: final raw-model

File: cob_hardware_config/raw3-1/urdf/raw3-1.urdf.xacro (robot description, xacro)
@@ -18,25 +18,35 @@
   <!-- ur_arm -->
  <include filename="$(find raw_description)/urdf/arm_ur/arm.urdf.xacro" />
- <!--include filename="$(find ur5_description)/urdf/model.urdf.xacro" /-->
+ <include filename="$(find ur5_description)/urdf/model.urdf.xacro" />
   <!-- frida -->
-  <!--include filename="$(find frida_description)/urdf/frida/frida.urdf.xacro" /-->
+  <include filename="$(find frida_description)/urdf/frida/frida.urdf.xacro" />
   <xacro:raw_base name="base"/>	<!--with new collision_model, but no platform_controller available yet-->
- <!--origin xyz="0.166 0.2175 0.5405" rpy="0 0 0" /-->
+  <!-- baer base-->
+  <!--include filename="$(find raw_description)/urdf/base/baer_base.urdf.xacro" />
+  <xacro:baer_base name="base"/-->
+  <!--
   <xacro:cob_torso_v1 name="torso" parent="base_link">
     <origin xyz="-0.36 -0.099 0.488" rpy="${M_PI} 0 0" />
   </xacro:cob_torso_v1>
-  <xacro:cob_arm_ur name="arm" parent="base_link">
-    <!--origin xyz="-0.33 0.16 0.6" rpy="0 ${M_PI/2} 0" /-->
+  -->
+  <!--origin xyz="-0.33 0.16 0.6" rpy="0 ${M_PI/2} 0" /-->
+  <!--in cad model z = 0.587  - fxmlc-->
+  <!--xacro:cob_arm_ur name="arm" parent="base_link">
     <origin xyz="-0.324 0.22 0.565" rpy="0 ${M_PI/2} 0" />
-	<!--in cad model z = 0.587  - fxmlc-->
-  </xacro:cob_arm_ur>
-  <!--xacro:ur5_robot prefix="arm_"/>
+  </xacro:cob_arm_ur-->
+  <xacro:ur5_robot prefix="arm_"/>
   <joint name="arm_base_joint" type="fixed" >
-		 <origin xyz="0.3235 -0.191 0.58" rpy="0 0 -0.79" />
+		<origin xyz="-0.324 0.22 0.565" rpy="0 0 0" />
 		<parent link="base_link" />
 		<child link="arm_base_link" />
-  </joint-->
-  <!--xacro:frida name="arm" parent="base_link">
-    <origin xyz="0.62 0.00 0.88" rpy="0 0 0" />
-  </xacro:frida-->
+  </joint>
+  <!--xacro:frida_torso parent="base_link">
+    <origin xyz="0 0 0.88" rpy="0 0 0" />
+  </xacro:frida_torso>
+  <xacro:frida_arm name="arm" suffix ="left" reflect = "0">
+    <origin xyz="0 0 0" rpy="0 0 0" />
+  </xacro:frida_arm-->
+  <!--xacro:frida_arm name="arm" suffix= "right" reflect = "1">
+    <origin xyz="0 -0.15 0" rpy="0 0 ${-M_PI/4}" />
+  </xacro:frida_arm-->
 </robot>

Commit message: clean raw3-1 hardware_config

File: cob_hardware_config/raw3-1/urdf/raw3-1.urdf.xacro (robot description, xacro)
@@ -9,6 +9,5 @@
   <include filename="$(find cob_description)/urdf/materials.urdf.xacro" />
   <include filename="$(find cob_hardware_config)/raw3-1/calibration/calibration.urdf.xacro" />
-  <!-- icob base -->
-  <!--include filename="$(find icob_description)/ros/urdf/base_v1/base.urdf.xacro" /-->	<!-- fxm: old	-->
+  <!-- raw base -->
   <include filename="$(find raw_description)/urdf/base/base.urdf.xacro" />
   <!-- generic simulator_gazebo plugins for starting mechanism control, ros time, ros battery -->
@@ -19,15 +18,5 @@
  <include filename="$(find raw_description)/urdf/arm_ur/arm.urdf.xacro" />
  <include filename="$(find ur5_description)/urdf/model.urdf.xacro" />
-  <!-- frida -->
-  <include filename="$(find frida_description)/urdf/frida/frida.urdf.xacro" />
   <xacro:raw_base name="base"/>	<!--with new collision_model, but no platform_controller available yet-->
-  <!-- baer base-->
-  <!--include filename="$(find raw_description)/urdf/base/baer_base.urdf.xacro" />
-  <xacro:baer_base name="base"/-->
-  <!--
-  <xacro:cob_torso_v1 name="torso" parent="base_link">
-    <origin xyz="-0.36 -0.099 0.488" rpy="${M_PI} 0 0" />
-  </xacro:cob_torso_v1>
-  -->
   <!--origin xyz="-0.33 0.16 0.6" rpy="0 ${M_PI/2} 0" /-->
   <!--in cad model z = 0.587  - fxmlc-->
@@ -41,12 +30,3 @@
 		<child link="arm_base_link" />
   </joint>
-  <!--xacro:frida_torso parent="base_link">
-    <origin xyz="0 0 0.88" rpy="0 0 0" />
-  </xacro:frida_torso>
-  <xacro:frida_arm name="arm" suffix ="left" reflect = "0">
-    <origin xyz="0 0 0" rpy="0 0 0" />
-  </xacro:frida_arm-->
-  <!--xacro:frida_arm name="arm" suffix= "right" reflect = "1">
-    <origin xyz="0 -0.15 0" rpy="0 0 ${-M_PI/4}" />
-  </xacro:frida_arm-->
 </robot>

Commit message: final raw-model V2

File: cob_hardware_config/raw3-1/urdf/raw3-1.urdf.xacro (robot description, xacro)
@@ -26,5 +26,5 @@
   <xacro:ur5_robot prefix="arm_"/>
   <joint name="arm_base_joint" type="fixed" >
-		<origin xyz="-0.324 0.22 0.565" rpy="0 0 0" />
+		<origin xyz="-0.324 0.191 0.565" rpy="0 0 0" />
 		<parent link="base_link" />
 		<child link="arm_base_link" />

Commit message: adapted raw_torso files

File: cob_hardware_config/raw3-1/urdf/raw3-1.urdf.xacro (robot description, xacro)
@@ -30,3 +30,7 @@
 		<child link="arm_base_link" />
   </joint>
+  <!--ToDo: find correct transformation-->
+  <!--xacro:raw_torso name="torso" parent="base_tower">
+    <origin xyz="0 0 0.7" rpy="0 0 0"/>
+  </xacro:raw_torso-->
 </robot>

Commit message: removed old arm_ur model

File: cob_hardware_config/raw3-1/urdf/raw3-1.urdf.xacro (robot description, xacro)
@@ -16,12 +16,6 @@
   <include filename="$(find raw_description)/urdf/torso/torso.urdf.xacro" />
   <!-- ur_arm -->
- <include filename="$(find raw_description)/urdf/arm_ur/arm.urdf.xacro" />
  <include filename="$(find ur5_description)/urdf/model.urdf.xacro" />
   <xacro:raw_base name="base"/>	<!--with new collision_model, but no platform_controller available yet-->
-  <!--origin xyz="-0.33 0.16 0.6" rpy="0 ${M_PI/2} 0" /-->
-  <!--in cad model z = 0.587  - fxmlc-->
-  <!--xacro:cob_arm_ur name="arm" parent="base_link">
-    <origin xyz="-0.324 0.22 0.565" rpy="0 ${M_PI/2} 0" />
-  </xacro:cob_arm_ur-->
   <xacro:ur5_robot prefix="arm_"/>
   <joint name="arm_base_joint" type="fixed" >

Commit message: new pc names on raw3-1 and working torso config for new urdf

File: cob_hardware_config/raw3-1/urdf/raw3-1.urdf.xacro (robot description, xacro)
@@ -24,7 +24,6 @@
 		<child link="arm_base_link" />
   </joint>
-  <!--ToDo: find correct transformation-->
-  <xacro:raw_torso name="torso" parent="base_tower">
-    <origin xyz="0 0 0.7" rpy="0 0 0"/>
-  </xacro:raw_torso>
+  <xacro:cob_torso_v1 name="torso" parent="base_link">
+    <origin xyz="0.166 0.2175 0.5405" rpy="0 0 0" />
+  </xacro:cob_torso_v1>
 </robot>

Commit message: changed position of manipulator from back to front

File: cob_hardware_config/raw3-1/urdf/raw3-1.urdf.xacro (robot description, xacro)
@@ -20,5 +20,5 @@
   <xacro:ur5_robot prefix="arm_"/>
   <joint name="arm_base_joint" type="fixed" >
-		<origin xyz="-0.324 0.191 0.565" rpy="0 0 0" />
+		<origin xyz="0.324 -0.191 0.565" rpy="0 0 3.14" />
 		<parent link="base_link" />
 		<child link="arm_base_link" />

Commit message: added amadeus box gripper to raw3-1 urdf description

File: cob_hardware_config/raw3-1/urdf/raw3-1.urdf.xacro (robot description, xacro)
@@ -11,4 +11,6 @@
   <!-- raw base -->
   <include filename="$(find raw_description)/urdf/base/base.urdf.xacro" />
+  <!-- raw boxgripper -->
+  <include filename="$(find raw_description)/urdf/boxgripper/boxgripper.urdf.xacro" />
   <!-- generic simulator_gazebo plugins for starting mechanism control, ros time, ros battery -->
   <include filename="$(find cob_description)/gazebo/gazebo.urdf.xacro" />
@@ -27,3 +29,6 @@
     <origin xyz="0.166 0.2175 0.5405" rpy="0 0 0" />
   </xacro:raw_torso>
+  <xacro:raw_boxgripper name="gripper" parent="arm_ee_link">
+    <origin xyz="0.025 0 -0.08" rpy="0 0 0" />
+  </xacro:raw_boxgripper>
 </robot>

Commit message: modified/corrected raw3-1 urdf description

File: cob_hardware_config/raw3-1/urdf/raw3-1.urdf.xacro (robot description, xacro)
@@ -22,5 +22,5 @@
   <xacro:ur5_robot prefix="arm_"/>
   <joint name="arm_base_joint" type="fixed" >
-		<origin xyz="0.324 -0.191 0.565" rpy="0 0 3.14" />
+		<origin xyz="0.324 -0.191 0.565" rpy="0 0 -0.79" />
 		<parent link="base_link" />
 		<child link="arm_base_link" />
@@ -30,5 +30,5 @@
   </xacro:raw_torso>
   <xacro:raw_boxgripper name="gripper" parent="arm_ee_link">
-    <origin xyz="0.025 0 -0.08" rpy="0 0 0" />
+    <origin xyz="0.04 0.122 0" rpy="1.570796 0 0.12" />
   </xacro:raw_boxgripper>
 </robot>

Commit message: calibration data for arm mount position

File: cob_hardware_config/raw3-1/urdf/raw3-1.urdf.xacro (robot description, xacro)
@@ -21,5 +21,5 @@
   <xacro:raw_base name="base"/>	<!--with new collision_model, but no platform_controller available yet-->
   <xacro:ur10_robot name="arm" parent="base_link">
-	<origin xyz="0.324 -0.191 0.565" rpy="0 0 3.14" />
+      <origin xyz="${arm_x} ${arm_y} ${arm_z}" rpy="${arm_roll} ${arm_pitch} ${arm_yaw}" />
   </xacro:ur10_robot>
   <xacro:raw_torso name="torso" parent="base_link">

Commit message: fixed gripper position

File: cob_hardware_config/raw3-1/urdf/raw3-1.urdf.xacro (robot description, xacro)
@@ -26,6 +26,12 @@
     <origin xyz="0.166 0.2175 0.5405" rpy="0 0 0" />
   </xacro:raw_torso>
+  <link name="arm_ee_link"/>
+  <joint name ="arm_ee_joint" type="fixed">
+	  <origin xyz="0.0 0.090 0" rpy="-1.570796 0 0" />
+	  <parent link="arm_wrist_3_link" />
+	  <child link="arm_ee_link" />
+  </joint>
   <xacro:raw_boxgripper name="gripper" parent="arm_ee_link">
-    <origin xyz="0 0 0" rpy="1.570796 0 0" />
+	  <origin xyz="-0.1 0.0 0.05" rpy="0 0 0" />
   </xacro:raw_boxgripper>
-</robot>
+  </robot>

Commit message: torso mount position can now be parameterized within calibration_data

File: cob_hardware_config/raw3-1/urdf/raw3-1.urdf.xacro (robot description, xacro)
@@ -24,5 +24,6 @@
   </xacro:ur10_robot>
   <xacro:raw_torso name="torso" parent="base_link">
-    <origin xyz="0.166 0.2175 0.5405" rpy="0 0 0" />
+    <!--origin xyz="0.166 0.2175 0.5405" rpy="0 0 0" /-->
+      <origin xyz="${torso_x} ${torso_y} ${torso_z}" rpy="${torso_roll} ${torso_pitch} ${torso_yaw}" />
   </xacro:raw_torso>
   <link name="arm_ee_link"/>

Commit message: changes for icra

File: cob_hardware_config/raw3-1/urdf/raw3-1.urdf.xacro (robot description, xacro)
@@ -11,4 +11,5 @@
   <!-- raw base -->
   <include filename="$(find raw_description)/urdf/base/base.urdf.xacro" />
+rm_x} ${arm_y} ${arm_z}" rpy="${arm_roll} ${arm_roll} ${arm_yaw}"
   <!-- raw boxgripper -->
   <include filename="$(find raw_description)/urdf/boxgripper/boxgripper.urdf.xacro" />
@@ -18,21 +19,28 @@
   <include filename="$(find raw_description)/urdf/torso/torso.urdf.xacro" />
   <!-- ur_arm -->
- <include filename="$(find ur_description)/urdf/ur10.urdf.xacro" />
+  <include filename="$(find ur10_description)/urdf/gazebo.urdf.xacro" />
+  <include filename="$(find ur10_description)/urdf/model.urdf.xacro" />
   <xacro:raw_base name="base"/>	<!--with new collision_model, but no platform_controller available yet-->
-  <xacro:ur10_robot name="arm" parent="base_link">
-      <origin xyz="${arm_x} ${arm_y} ${arm_z}" rpy="${arm_roll} ${arm_pitch} ${arm_yaw}" />
-  </xacro:ur10_robot>
+  <xacro:macro name="ur_arm_base_joint" >
+  <joint name="arm_base_joint" type="fixed" >
+    <origin xyz="${arm_x} ${arm_y} ${arm_z}" rpy="${arm_roll} ${arm_roll} ${arm_yaw}" />
+    <parent link="base_link" />
+    <child link="arm_base_link" />
+  </joint>
+  </xacro:macro>
+ <xacro:ur_arm_base_joint/>
+ <xacro:ur10_robot prefix="arm_"/>
   <xacro:raw_torso name="torso" parent="base_link">
     <!--origin xyz="0.166 0.2175 0.5405" rpy="0 0 0" /-->
       <origin xyz="${torso_x} ${torso_y} ${torso_z}" rpy="${torso_roll} ${torso_pitch} ${torso_yaw}" />
   </xacro:raw_torso>
-  <link name="arm_ee_link"/>
-  <joint name ="arm_ee_joint" type="fixed">
+  <!--link name="arm_ee_link"/-->
+  <!--joint name ="arm_ee_joint" type="fixed">
 	  <origin xyz="0.0 0.090 0" rpy="-1.570796 0 0" />
 	  <parent link="arm_wrist_3_link" />
 	  <child link="arm_ee_link" />
-  </joint>
+  </joint-->
   <xacro:raw_boxgripper name="gripper" parent="arm_ee_link">
-	  <origin xyz="-0.1 0.0 0.05" rpy="0 0 0" />
+	<origin xyz="0.00 0.0 0.0" rpy="0 0 0" />
   </xacro:raw_boxgripper>
   </robot>

Commit message: some fixes in urdf.xacro for raw3-1

File: cob_hardware_config/raw3-1/urdf/raw3-1.urdf.xacro (robot description, xacro)
@@ -11,5 +11,4 @@
   <!-- raw base -->
   <include filename="$(find raw_description)/urdf/base/base.urdf.xacro" />
-rm_x} ${arm_y} ${arm_z}" rpy="${arm_roll} ${arm_roll} ${arm_yaw}"
   <!-- raw boxgripper -->
   <include filename="$(find raw_description)/urdf/boxgripper/boxgripper.urdf.xacro" />
@@ -19,18 +18,16 @@
   <include filename="$(find raw_description)/urdf/torso/torso.urdf.xacro" />
   <!-- ur_arm -->
-  <include filename="$(find ur10_description)/urdf/gazebo.urdf.xacro" />
   <include filename="$(find ur10_description)/urdf/model.urdf.xacro" />
   <xacro:raw_base name="base"/>	<!--with new collision_model, but no platform_controller available yet-->
   <xacro:macro name="ur_arm_base_joint" >
-  <joint name="arm_base_joint" type="fixed" >
-    <origin xyz="${arm_x} ${arm_y} ${arm_z}" rpy="${arm_roll} ${arm_roll} ${arm_yaw}" />
-    <parent link="base_link" />
-    <child link="arm_base_link" />
-  </joint>
+	<joint name="arm_base_joint" type="fixed" >
+		<origin xyz="${arm_x} ${arm_y} ${arm_z}" rpy="${arm_roll} ${arm_roll} ${arm_yaw}" />
+		<parent link="base_link" />
+		<child link="arm_base_link" />
+	</joint>
   </xacro:macro>
  <xacro:ur_arm_base_joint/>
  <xacro:ur10_robot prefix="arm_"/>
   <xacro:raw_torso name="torso" parent="base_link">
-    <!--origin xyz="0.166 0.2175 0.5405" rpy="0 0 0" /-->
       <origin xyz="${torso_x} ${torso_y} ${torso_z}" rpy="${torso_roll} ${torso_pitch} ${torso_yaw}" />
   </xacro:raw_torso>
