Commit message: changed urdfs to new base_long and base_short structure, cleaned up all raw's

File: cob_hardware_config/raw3-1/urdf/raw3-1.urdf.xacro (robot description, xacro)
@@ -10,5 +10,7 @@
   <include filename="$(find cob_calibration_data)/raw3-1/calibration/calibration.urdf.xacro" />
   <!-- raw base -->
-  <include filename="$(find raw_description)/urdf/base/base.urdf.xacro" />
+  <include filename="$(find raw_description)/urdf/base_long/base.urdf.xacro" />
+  <!-- raw tower -->
+  <include filename="$(find raw_description)/urdf/tower_asymetric/tower.urdf.xacro" />
   <!-- raw boxgripper -->
   <include filename="$(find raw_description)/urdf/boxgripper/boxgripper.urdf.xacro" />
@@ -19,13 +21,17 @@
   <!-- ur_arm -->
   <include filename="$(find ur_description)/urdf/ur10.urdf.xacro" />
-  <xacro:raw_base name="base"/>	<!--with new collision_model, but no platform_controller available yet-->
-  <xacro:ur10_robot name="arm" parent="base_link">
+  <xacro:raw_base name="base"/>
+  <xacro:tower_asymetric name="tower" parent="base_link">
+      <origin xyz="${tower_x} ${tower_y} ${tower_z}" rpy="${tower_roll} ${tower_pitch} ${tower_yaw}" />
+  </xacro:tower_asymetric>
+  <!-- comment out ur10 as this is not working now -->
+  <!--xacro:ur10_robot name="arm" parent="base_link">
       <origin xyz="${arm_x} ${arm_y} ${arm_z}" rpy="${arm_roll} ${arm_pitch} ${arm_yaw}" />
-  </xacro:ur10_robot>
+  </xacro:ur10_robot-->
   <xacro:raw_torso name="torso" parent="base_link">
       <origin xyz="${torso_x} ${torso_y} ${torso_z}" rpy="${torso_roll} ${torso_pitch} ${torso_yaw}" />
   </xacro:raw_torso>
-  <xacro:raw_boxgripper name="gripper" parent="arm_wrist_3_link">
+  <!--xacro:raw_boxgripper name="gripper" parent="arm_wrist_3_link">
       <origin xyz="${gripper_x} ${gripper_y} ${gripper_z}" rpy="${gripper_roll} ${gripper_pitch} ${gripper_yaw}" />
-  </xacro:raw_boxgripper>
+  </xacro:raw_boxgripper-->
   </robot>

File: cob_hardware_config/raw3-2/urdf/raw3-2.urdf.xacro (robot description, xacro)
@@ -9,7 +9,12 @@
   <include filename="$(find cob_description)/urdf/materials.urdf.xacro" />
   <include filename="$(find cob_calibration_data)/raw3-2/calibration/calibration.urdf.xacro" />
-  <include filename="$(find raw_description)/urdf/base/base.urdf.xacro" />
+  <include filename="$(find raw_description)/urdf/base_long/base.urdf.xacro" />
+  <!-- raw tower -->
+  <include filename="$(find raw_description)/urdf/tower_asymetric/tower.urdf.xacro" />
   <!-- generic simulator_gazebo plugins for starting mechanism control, ros time, ros battery -->
   <include filename="$(find cob_description)/gazebo/gazebo.urdf.xacro" />
-  <xacro:raw_base name="base"/>	<!--with new collision_model, but no platform_controller available yet-->
+  <xacro:raw_base name="base"/>
+  <xacro:tower_asymetric name="tower" parent="base_link">
+      <origin xyz="${tower_x} ${tower_y} ${tower_z}" rpy="${tower_roll} ${tower_pitch} ${tower_yaw}" />
+  </xacro:tower_asymetric>
 </robot>

File: cob_hardware_config/raw3-3/urdf/raw3-3.urdf.xacro (robot description, xacro)
@@ -21,5 +21,5 @@
   <!-- generic simulator_gazebo plugins for starting mechanism control, ros time, ros battery -->
   <include filename="$(find cob_description)/gazebo/gazebo.urdf.xacro" />
-  <xacro:raw_base name="base"/>	<!--with new collision_model, but no platform_controller available yet-->
+  <xacro:raw_base name="base"/>
   <xacro:tower_symetric name="tower" parent="base_link">
       <origin xyz="${tower_x} ${tower_y} ${tower_z}" rpy="${tower_roll} ${tower_pitch} ${tower_yaw}" />

File: cob_hardware_config/raw3-4/urdf/raw3-4.urdf.xacro (robot description, xacro)
@@ -9,7 +9,13 @@
   <include filename="$(find cob_description)/urdf/materials.urdf.xacro" />
   <include filename="$(find cob_calibration_data)/raw3-4/calibration/calibration.urdf.xacro" />
-  <include filename="$(find raw_description)/urdf/base/base.urdf.xacro" />
+  <!-- raw base -->
+  <include filename="$(find raw_description)/urdf/base_long/base.urdf.xacro" />
+  <!-- raw tower -->
+  <include filename="$(find raw_description)/urdf/tower_asymetric/tower.urdf.xacro" />
   <!-- generic simulator_gazebo plugins for starting mechanism control, ros time, ros battery -->
   <include filename="$(find cob_description)/gazebo/gazebo.urdf.xacro" />
-  <xacro:raw_base name="base"/>	<!--with new collision_model, but no platform_controller available yet-->
+  <xacro:raw_base name="base"/>
+  <xacro:tower_asymetric name="tower" parent="base_link">
+      <origin xyz="${tower_x} ${tower_y} ${tower_z}" rpy="${tower_roll} ${tower_pitch} ${tower_yaw}" />
+  </xacro:tower_asymetric>
 </robot>

Commit message: removed wifi monitor and mounted ur10 on robot again, not tested in gazebo yet

File: cob_hardware_config/raw3-1/urdf/raw3-1.urdf.xacro (robot description, xacro)
@@ -20,18 +20,24 @@
   <include filename="$(find raw_description)/urdf/torso/torso.urdf.xacro" />
   <!-- ur_arm -->
-  <include filename="$(find ur_description)/urdf/ur10.urdf.xacro" />
+  <include filename="$(find raw_description)/urdf/ur_arm/ur10_arm.urdf.xacro" />
   <xacro:raw_base name="base"/>
   <xacro:tower_asymetric name="tower" parent="base_link">
       <origin xyz="${tower_x} ${tower_y} ${tower_z}" rpy="${tower_roll} ${tower_pitch} ${tower_yaw}" />
   </xacro:tower_asymetric>
-  <!-- comment out ur10 as this is not working now -->
-  <!--xacro:ur10_robot name="arm" parent="base_link">
+  <xacro:cob_ur10 name="arm" parent="base_link">
       <origin xyz="${arm_x} ${arm_y} ${arm_z}" rpy="${arm_roll} ${arm_pitch} ${arm_yaw}" />
-  </xacro:ur10_robot-->
+  </xacro:cob_ur10>
+  <!-- mount the arm to the robot
+  <joint name="arm_base_joint" type="fixed" >
+      <origin xyz="${arm_x} ${arm_y} ${arm_z}" rpy="${arm_roll} ${arm_pitch} ${arm_yaw}" />
+      <parent link="base_link" />
+      <child link="arm_base_link" />
+  </joint>
+  <xacro:ur10_robot prefix="arm_"/>-->
   <xacro:raw_torso name="torso" parent="base_link">
       <origin xyz="${torso_x} ${torso_y} ${torso_z}" rpy="${torso_roll} ${torso_pitch} ${torso_yaw}" />
   </xacro:raw_torso>
-  <!--xacro:raw_boxgripper name="gripper" parent="arm_wrist_3_link">
+  <xacro:raw_boxgripper name="gripper" parent="arm_wrist_3_link">
       <origin xyz="${gripper_x} ${gripper_y} ${gripper_z}" rpy="${gripper_roll} ${gripper_pitch} ${gripper_yaw}" />
-  </xacro:raw_boxgripper-->
+  </xacro:raw_boxgripper>
   </robot>

Commit message: Updated urdf of raw3-1 in cob_hardware_config regarding latest IMU-brick mount on raw3-1

File: cob_hardware_config/raw3-1/urdf/raw3-1.urdf.xacro (robot description, xacro)
@@ -51,3 +51,24 @@
       <origin xyz="${gripper_x} ${gripper_y} ${gripper_z}" rpy="${gripper_roll} ${gripper_pitch} ${gripper_yaw}" />
   </xacro:raw_boxgripper>
+   <!-- IMU brick mount on raw3-1 -->
+   <joint name="imu_brick_joint" type="fixed" >
+      <origin xyz="0.402 -0.0811 0.335" rpy="0 0 0" />
+      <parent link="base_link" />
+      <child link="imu_brick_link" />
+    </joint>
+    <link name="imu_brick_link">
+       <inertial>
+            <mass value="0.0001" />
+            <origin xyz="0 0 0" rpy="0 0 0" />
+            <inertia ixx="0.00001" ixy="0" ixz="0" iyy="0.00001" iyz="0" izz="0.00001" />
+       </inertial>
+       <visual>
+   	    <origin xyz="0 0 -0.02" rpy="0 0 0" />
+	    <geometry>
+    	       <box size="0.04 0.04 0.02" />
+	    </geometry>
+	    <material name="IPA/LightGrey" />
+       </visual>
+    </link>
+    <!-- END: IMU brick	mount -->
   </robot>

Commit message: added rfid reader on raw31 in raw3-1.urdf.xacro

File: cob_hardware_config/raw3-1/urdf/raw3-1.urdf.xacro (robot description, xacro)
@@ -72,3 +72,71 @@
     </link>
     <!-- END: IMU brick	mount -->
+       <!-- rfid_front mount on raw3-1 -->
+   <joint name="rfid_front_joint" type="fixed" >
+      <origin xyz="0.55128 0.0 0.09" rpy="0 0 0" />
+      <parent link="base_link" />
+      <child link="rfid_front_link" />
+    </joint>
+    <link name="rfid_front_link">
+       <inertial>
+            <mass value="0.2" />
+            <origin xyz="0 0 0" rpy="0 0 0" />
+            <inertia ixx="0.2" ixy="0" ixz="0" iyy="0.2" iyz="0" izz="0.2" />
+       </inertial>
+       <visual>
+   	    <origin xyz="0 0 0" rpy="0 0 0" />
+	    <geometry>
+    	       <box size="0.16 0.36 0.09" />
+	    </geometry>
+	    <material name="blue">
+        <color rgba="0 0 .8 1"/>
+      </material>
+       </visual>
+    </link>
+        <!-- rfid_rear mount on raw3-1 -->
+   <joint name="rfid_rear_joint" type="fixed" >
+      <origin xyz="-0.55128 0.0 0.09" rpy="0 0 ${M_PI}" />
+      <parent link="base_link" />
+      <child link="rfid_rear_link" />
+    </joint>
+    <link name="rfid_rear_link">
+       <inertial>
+            <mass value="0.2" />
+            <origin xyz="0 0 0" rpy="0 0 0" />
+            <inertia ixx="0.2" ixy="0" ixz="0" iyy="0.2" iyz="0" izz="0.2" />
+       </inertial>
+       <visual>
+   	    <origin xyz="0 0 0" rpy="0 0 0" />
+	    <geometry>
+    	       <box size="0.16 0.36 0.09" />
+	    </geometry>
+	    <material name="blue">
+        <color rgba="0 0 .8 1"/>
+      </material>
+       </visual>
+    </link>
+    <!-- END: rfid rear	mount -->
+            <!-- rfid_right mount on raw3-1 -->
+   <joint name="rfid_right_joint" type="fixed" >
+      <origin xyz="0.0 -0.30850 0.09" rpy="0 0 ${-0.5*M_PI}" />
+      <parent link="base_link" />
+      <child link="rfid_right_link" />
+    </joint>
+    <link name="rfid_right_link">
+       <inertial>
+            <mass value="0.2" />
+            <origin xyz="0 0 0" rpy="0 0 0" />
+            <inertia ixx="0.2" ixy="0" ixz="0" iyy="0.2" iyz="0" izz="0.2" />
+       </inertial>
+       <visual>
+   	    <origin xyz="0 0 0" rpy="0 0 0" />
+	    <geometry>
+    	       <box size="0.16 0.36 0.09" />
+	    </geometry>
+	    <material name="blue">
+        <color rgba="0 0 .8 1"/>
+      </material>
+       </visual>
+    </link>
+    <!-- END: rfid right	mount -->
   </robot>

Commit message: added rfid urdf in hydro

File: cob_hardware_config/raw3-1/urdf/raw3-1.urdf.xacro (robot description, xacro)
@@ -69,3 +69,72 @@
     </link>
     <!-- END: IMU brick	mount -->
+    <!-- rfid_front mount on raw3-1 -->
+   <joint name="rfid_front_joint" type="fixed" >
+      <origin xyz="0.55128 0.0 0.09" rpy="0 0 0" />
+      <parent link="base_link" />
+      <child link="rfid_front_link" />
+    </joint>
+    <link name="rfid_front_link">
+       <inertial>
+            <mass value="0.2" />
+            <origin xyz="0 0 0" rpy="0 0 0" />
+            <inertia ixx="0.2" ixy="0" ixz="0" iyy="0.2" iyz="0" izz="0.2" />
+       </inertial>
+       <visual>
+   	    <origin xyz="0 0 0" rpy="0 0 0" />
+	    <geometry>
+    	       <box size="0.16 0.36 0.09" />
+	    </geometry>
+	    <material name="blue">
+        <color rgba="0 0 .8 1"/>
+      </material>
+       </visual>
+    </link>
+    <!-- END: rfid front mount -->
+   <!-- rfid_rear mount on raw3-1 -->
+   <joint name="rfid_rear_joint" type="fixed" >
+      <origin xyz="-0.55128 0.0 0.09" rpy="0 0 ${M_PI}" />
+      <parent link="base_link" />
+      <child link="rfid_rear_link" />
+    </joint>
+    <link name="rfid_rear_link">
+       <inertial>
+            <mass value="0.2" />
+            <origin xyz="0 0 0" rpy="0 0 0" />
+            <inertia ixx="0.2" ixy="0" ixz="0" iyy="0.2" iyz="0" izz="0.2" />
+       </inertial>
+       <visual>
+   	    <origin xyz="0 0 0" rpy="0 0 0" />
+	    <geometry>
+    	       <box size="0.16 0.36 0.09" />
+	    </geometry>
+	    <material name="blue">
+        <color rgba="0 0 .8 1"/>
+      </material>
+       </visual>
+    </link>
+    <!-- END: rfid rear mount -->
+   <!-- rfid_right mount on raw3-1 -->
+   <joint name="rfid_right_joint" type="fixed" >
+      <origin xyz="0.0 -0.30850 0.09" rpy="0 0 ${-0.5*M_PI}" />
+      <parent link="base_link" />
+      <child link="rfid_right_link" />
+    </joint>
+    <link name="rfid_right_link">
+       <inertial>
+            <mass value="0.2" />
+            <origin xyz="0 0 0" rpy="0 0 0" />
+            <inertia ixx="0.2" ixy="0" ixz="0" iyy="0.2" iyz="0" izz="0.2" />
+       </inertial>
+       <visual>
+   	    <origin xyz="0 0 0" rpy="0 0 0" />
+	    <geometry>
+    	       <box size="0.16 0.36 0.09" />
+	    </geometry>
+	    <material name="blue">
+        <color rgba="0 0 .8 1"/>
+      </material>
+       </visual>
+    </link>
+    <!-- END: rfid right mount -->
   </robot>

Commit message: softkinetic cameras mount (including camera pillar) on raw3-1

File: cob_hardware_config/raw3-1/urdf/raw3-1.urdf.xacro (robot description, xacro)
@@ -138,3 +138,66 @@
     </link>
     <!-- END: rfid right mount -->
+    <!-- Camera pillar -->
+    <joint name="camera_pillar_joint" type="fixed" >
+      <origin xyz="0.4925 0.0825 0.48" rpy="0 0 0" />
+      <parent link="base_link" />
+      <child link="camera_pillar_link" />
+    </joint>
+    <link name="camera_pillar_link">
+       <inertial>
+            <mass value="0.0001" />
+            <origin xyz="0 0 0" rpy="0 0 0" />
+            <inertia ixx="0.00001" ixy="0" ixz="0" iyy="0.00001" iyz="0" izz="0.00001" />
+       </inertial>
+       <visual>
+   	    <origin xyz="0 0 0.123" rpy="0 0 0" />
+	    <geometry>
+    	       <box size="0.045 0.045 0.246" />
+	    </geometry>
+	    <material name="IPA/LightGrey" />
+       </visual>
+    </link>
+    <!-- END: camera_pillar -->
+    <!-- Softkinetic 'left' mount on raw3-1 -->
+    <joint name="softkinetic_left_joint" type="fixed" >
+      <origin xyz="0.015 0.06 0.215" rpy="0.0 ${M_PI/2} 0.0" />
+      <parent link="camera_pillar_link" />
+      <child link="softkinetic_left_link" />
+    </joint>
+    <link name="softkinetic_left_link">
+       <inertial>
+            <mass value="0.0001" />
+            <origin xyz="0 0 0" rpy="0.0 0.0 0.0" />
+            <inertia ixx="0.00001" ixy="0" ixz="0" iyy="0.00001" iyz="0" izz="0.00001" />
+       </inertial>
+       <visual>
+   	    <origin xyz="0.0 0.0 0.0" rpy="0.0 0.0 0.0" />
+            <geometry>
+    	       <box size="0.10 0.03 0.03" />
+            </geometry>
+            <material name="IPA/Black" />
+       </visual>
+    </link>
+    <!-- END: Softkinetic 'left' mount -->
+    <!-- Softkinetic 'right' mount on raw3-1 -->
+    <joint name="softkinetic_right_joint" type="fixed" >
+      <origin xyz="0.015 -0.06 0.215" rpy="${M_PI} -${M_PI/2} 0.0" />
+      <parent link="camera_pillar_link" />
+      <child link="softkinetic_right_link" />
+    </joint>
+    <link name="softkinetic_right_link">
+       <inertial>
+            <mass value="0.0001" />
+            <origin xyz="0 0 0" rpy="0 0 0" />
+            <inertia ixx="0.00001" ixy="0" ixz="0" iyy="0.00001" iyz="0" izz="0.00001" />
+       </inertial>
+       <visual>
+   	    <origin xyz="0.0 0.0 0.0" rpy="0.0 0.0 0.0" />
+	    <geometry>
+    	       <box size="0.10 0.03 0.03" />
+	    </geometry>
+	    <material name="IPA/Black" />
+       </visual>
+    </link>
+    <!-- END: Softkinetic 'right' mount -->
   </robot>
