Commit message: cleaning up

File: cob_hardware_config/raw3-1/urdf/raw3-1.urdf.xacro (robot description, xacro)
@@ -23,8 +23,8 @@
   <xacro:raw_base name="base"/>
   <xacro:tower_asymetric name="tower" parent="base_link">
-      <origin xyz="${tower_x} ${tower_y} ${tower_z}" rpy="${tower_roll} ${tower_pitch} ${tower_yaw}" />
+    <origin xyz="${tower_x} ${tower_y} ${tower_z}" rpy="${tower_roll} ${tower_pitch} ${tower_yaw}" />
   </xacro:tower_asymetric>
   <xacro:raw_torso name="torso" parent="base_link">
-      <origin xyz="${torso_x} ${torso_y} ${torso_z}" rpy="${torso_roll} ${torso_pitch} ${torso_yaw}" />
+    <origin xyz="${torso_x} ${torso_y} ${torso_z}" rpy="${torso_roll} ${torso_pitch} ${torso_yaw}" />
   </xacro:raw_torso>
   <xacro:raw_head name="head" parent="torso_2_link">
@@ -36,237 +36,133 @@
   </xacro:cob_lookat>
   <xacro:ur10 name="arm" parent="base_link">
-      <origin xyz="${arm_x} ${arm_y} ${arm_z}" rpy="${arm_roll} ${arm_pitch} ${arm_yaw}" />
+    <origin xyz="${arm_x} ${arm_y} ${arm_z}" rpy="${arm_roll} ${arm_pitch} ${arm_yaw}" />
   </xacro:ur10>
-  <!-- mount the arm to the robot
-  <joint name="arm_base_joint" type="fixed" >
-      <origin xyz="${arm_x} ${arm_y} ${arm_z}" rpy="${arm_roll} ${arm_pitch} ${arm_yaw}" />
-      <parent link="base_link" />
-      <child link="arm_base_link" />
+  <xacro:raw_boxgripper name="gripper" parent="arm_ee_link">
+    <origin xyz="${gripper_x} ${gripper_y} ${gripper_z}" rpy="${gripper_roll} ${gripper_pitch} ${gripper_yaw}" />
+  </xacro:raw_boxgripper>
+  <!-- IMU brick mount on raw3-1 -->
+  <joint name="imu_brick_joint" type="fixed" >
+    <origin xyz="0.402 -0.0811 0.335" rpy="0 0 0" />
+    <parent link="base_link" />
+    <child link="imu_brick_link" />
   </joint>
-  <xacro:ur10_robot prefix="arm_"/>-->
-  <xacro:raw_boxgripper name="gripper" parent="arm_ee_link">
-      <origin xyz="${gripper_x} ${gripper_y} ${gripper_z}" rpy="${gripper_roll} ${gripper_pitch} ${gripper_yaw}" />
-  </xacro:raw_boxgripper>
-   <!-- IMU brick mount on raw3-1 -->
-   <joint name="imu_brick_joint" type="fixed" >
-      <origin xyz="0.402 -0.0811 0.335" rpy="0 0 0" />
-      <parent link="base_link" />
-      <child link="imu_brick_link" />
-    </joint>
-    <link name="imu_brick_link">
-       <inertial>
-            <mass value="0.0001" />
-            <origin xyz="0 0 0" rpy="0 0 0" />
-            <inertia ixx="0.00001" ixy="0" ixz="0" iyy="0.00001" iyz="0" izz="0.00001" />
-       </inertial>
-       <visual>
-   	    <origin xyz="0 0 -0.02" rpy="0 0 0" />
-	    <geometry>
-    	       <box size="0.04 0.04 0.02" />
-	    </geometry>
-	    <material name="IPA/LightGrey" />
-       </visual>
-    </link>
-    <!-- END: IMU brick	mount -->
-   <!-- rfid_front mount on raw3-1 -->
-   <joint name="rfid_front_joint" type="fixed" >
-      <origin xyz="0.55128 0.0 0.09" rpy="0 0 0" />
-      <parent link="base_link" />
-      <child link="rfid_front_link" />
-    </joint>
-    <link name="rfid_front_link">
-       <inertial>
-            <mass value="0.2" />
-            <origin xyz="0 0 0" rpy="0 0 0" />
-            <inertia ixx="0.2" ixy="0" ixz="0" iyy="0.2" iyz="0" izz="0.2" />
-       </inertial>
-       <visual>
-   	    <origin xyz="0 0 0" rpy="0 0 0" />
-	    <geometry>
-    	       <box size="0.16 0.36 0.09" />
-	    </geometry>
-	    <material name="blue">
+  <link name="imu_brick_link">
+    <xacro:default_inertial />
+    <visual>
+      <origin xyz="0 0 -0.02" rpy="0 0 0" />
+      <geometry>
+        <box size="0.04 0.04 0.02" />
+      </geometry>
+      <material name="IPA/LightGrey" />
+    </visual>
+  </link>
+  <!-- END: IMU brick  mount -->
+  <!-- rfid_front mount on raw3-1 -->
+  <joint name="rfid_front_joint" type="fixed" >
+    <origin xyz="0.55128 0.0 0.09" rpy="0 0 0" />
+    <parent link="base_link" />
+    <child link="rfid_front_link" />
+  </joint>
+  <link name="rfid_front_link">
+    <xacro:default_inertial />
+    <visual>
+      <origin xyz="0 0 0" rpy="0 0 0" />
+      <geometry>
+        <box size="0.16 0.36 0.09" />
+      </geometry>
+      <material name="blue">
         <color rgba="0 0 .8 1"/>
       </material>
-       </visual>
-    </link>
-    <!-- END: rfid front mount -->
-   <!-- rfid_rear mount on raw3-1 -->
-   <joint name="rfid_rear_joint" type="fixed" >
-      <origin xyz="-0.55128 0.0 0.09" rpy="0 0 ${M_PI}" />
-      <parent link="base_link" />
-      <child link="rfid_rear_link" />
-    </joint>
-    <link name="rfid_rear_link">
-       <inertial>
-            <mass value="0.2" />
-            <origin xyz="0 0 0" rpy="0 0 0" />
-            <inertia ixx="0.2" ixy="0" ixz="0" iyy="0.2" iyz="0" izz="0.2" />
-       </inertial>
-       <visual>
-   	    <origin xyz="0 0 0" rpy="0 0 0" />
-	    <geometry>
-    	       <box size="0.16 0.36 0.09" />
-	    </geometry>
-	    <material name="blue">
+    </visual>
+  </link>
+  <!-- END: rfid front mount -->
+  <!-- rfid_rear mount on raw3-1 -->
+  <joint name="rfid_rear_joint" type="fixed" >
+    <origin xyz="-0.55128 0.0 0.09" rpy="0 0 ${M_PI}" />
+    <parent link="base_link" />
+    <child link="rfid_rear_link" />
+  </joint>
+  <link name="rfid_rear_link">
+    <xacro:default_inertial />
+    <visual>
+      <origin xyz="0 0 0" rpy="0 0 0" />
+      <geometry>
+        <box size="0.16 0.36 0.09" />
+      </geometry>
+      <material name="blue">
         <color rgba="0 0 .8 1"/>
       </material>
-       </visual>
-    </link>
-    <!-- END: rfid rear mount -->
-   <!-- rfid_right mount on raw3-1 -->
-   <joint name="rfid_right_joint" type="fixed" >
-      <origin xyz="0.0 -0.30850 0.09" rpy="0 0 ${-0.5*M_PI}" />
-      <parent link="base_link" />
-      <child link="rfid_right_link" />
-    </joint>
-    <link name="rfid_right_link">
-       <inertial>
-            <mass value="0.2" />
-            <origin xyz="0 0 0" rpy="0 0 0" />
-            <inertia ixx="0.2" ixy="0" ixz="0" iyy="0.2" iyz="0" izz="0.2" />
-       </inertial>
-       <visual>
-   	    <origin xyz="0 0 0" rpy="0 0 0" />
-	    <geometry>
-    	       <box size="0.16 0.36 0.09" />
-	    </geometry>
-	    <material name="blue">
+    </visual>
+  </link>
+  <!-- END: rfid rear mount -->
+  <!-- rfid_right mount on raw3-1 -->
+  <joint name="rfid_right_joint" type="fixed" >
+    <origin xyz="0.0 -0.30850 0.09" rpy="0 0 ${-0.5*M_PI}" />
+    <parent link="base_link" />
+    <child link="rfid_right_link" />
+  </joint>
+  <link name="rfid_right_link">
+    <xacro:default_inertial />
+    <visual>
+      <origin xyz="0 0 0" rpy="0 0 0" />
+      <geometry>
+        <box size="0.16 0.36 0.09" />
+      </geometry>
+      <material name="blue">
         <color rgba="0 0 .8 1"/>
       </material>
-       </visual>
-    </link>
-    <!-- END: rfid right mount -->
-    <!-- rfid_front mount on raw3-1 -->
-   <joint name="rfid_front_joint" type="fixed" >
-      <origin xyz="0.55128 0.0 0.09" rpy="0 0 0" />
-      <parent link="base_link" />
-      <child link="rfid_front_link" />
-    </joint>
-    <link name="rfid_front_link">
-       <inertial>
-            <mass value="0.2" />
-            <origin xyz="0 0 0" rpy="0 0 0" />
-            <inertia ixx="0.2" ixy="0" ixz="0" iyy="0.2" iyz="0" izz="0.2" />
-       </inertial>
-       <visual>
-   	    <origin xyz="0 0 0" rpy="0 0 0" />
-	    <geometry>
-    	       <box size="0.16 0.36 0.09" />
-	    </geometry>
-	    <material name="blue">
-        <color rgba="0 0 .8 1"/>
-      </material>
-       </visual>
-    </link>
-    <!-- END: rfid front mount -->
-   <!-- rfid_rear mount on raw3-1 -->
-   <joint name="rfid_rear_joint" type="fixed" >
-      <origin xyz="-0.55128 0.0 0.09" rpy="0 0 ${M_PI}" />
-      <parent link="base_link" />
-      <child link="rfid_rear_link" />
-    </joint>
-    <link name="rfid_rear_link">
-       <inertial>
-            <mass value="0.2" />
-            <origin xyz="0 0 0" rpy="0 0 0" />
-            <inertia ixx="0.2" ixy="0" ixz="0" iyy="0.2" iyz="0" izz="0.2" />
-       </inertial>
-       <visual>
-   	    <origin xyz="0 0 0" rpy="0 0 0" />
-	    <geometry>
-    	       <box size="0.16 0.36 0.09" />
-	    </geometry>
-	    <material name="blue">
-        <color rgba="0 0 .8 1"/>
-      </material>
-       </visual>
-    </link>
-    <!-- END: rfid rear mount -->
-   <!-- rfid_right mount on raw3-1 -->
-   <joint name="rfid_right_joint" type="fixed" >
-      <origin xyz="0.0 -0.30850 0.09" rpy="0 0 ${-0.5*M_PI}" />
-      <parent link="base_link" />
-      <child link="rfid_right_link" />
-    </joint>
-    <link name="rfid_right_link">
-       <inertial>
-            <mass value="0.2" />
-            <origin xyz="0 0 0" rpy="0 0 0" />
-            <inertia ixx="0.2" ixy="0" ixz="0" iyy="0.2" iyz="0" izz="0.2" />
-       </inertial>
-       <visual>
-   	    <origin xyz="0 0 0" rpy="0 0 0" />
-	    <geometry>
-    	       <box size="0.16 0.36 0.09" />
-	    </geometry>
-	    <material name="blue">
-        <color rgba="0 0 .8 1"/>
-      </material>
-       </visual>
-    </link>
-    <!-- END: rfid right mount -->
-    <!-- Camera pillar -->
-    <joint name="camera_pillar_joint" type="fixed" >
-      <origin xyz="0.4925 0.0825 0.48" rpy="0 0 0" />
-      <parent link="base_link" />
-      <child link="camera_pillar_link" />
-    </joint>
-    <link name="camera_pillar_link">
-       <inertial>
-            <mass value="0.0001" />
-            <origin xyz="0 0 0" rpy="0 0 0" />
-            <inertia ixx="0.00001" ixy="0" ixz="0" iyy="0.00001" iyz="0" izz="0.00001" />
-       </inertial>
-       <visual>
-   	    <origin xyz="0 0 0.123" rpy="0 0 0" />
-	    <geometry>
-    	       <box size="0.045 0.045 0.246" />
-	    </geometry>
-	    <material name="IPA/LightGrey" />
-       </visual>
-    </link>
-    <!-- END: camera_pillar -->
-    <!-- Softkinetic 'left' mount on raw3-1 -->
-    <joint name="softkinetic_left_joint" type="fixed" >
-      <origin xyz="0.015 0.06 0.215" rpy="0.0 ${M_PI/2} 0.0" />
-      <parent link="camera_pillar_link" />
-      <child link="softkinetic_left_link" />
-    </joint>
-    <link name="softkinetic_left_link">
-       <inertial>
-            <mass value="0.0001" />
-            <origin xyz="0 0 0" rpy="0.0 0.0 0.0" />
-            <inertia ixx="0.00001" ixy="0" ixz="0" iyy="0.00001" iyz="0" izz="0.00001" />
-       </inertial>
-       <visual>
-   	    <origin xyz="0.0 0.0 0.0" rpy="0.0 0.0 0.0" />
-            <geometry>
-    	       <box size="0.10 0.03 0.03" />
-            </geometry>
-            <material name="IPA/Black" />
-       </visual>
-    </link>
-    <!-- END: Softkinetic 'left' mount -->
-    <!-- Softkinetic 'right' mount on raw3-1 -->
-    <joint name="softkinetic_right_joint" type="fixed" >
-      <origin xyz="0.015 -0.06 0.215" rpy="${M_PI} -${M_PI/2} 0.0" />
-      <parent link="camera_pillar_link" />
-      <child link="softkinetic_right_link" />
-    </joint>
-    <link name="softkinetic_right_link">
-       <inertial>
-            <mass value="0.0001" />
-            <origin xyz="0 0 0" rpy="0 0 0" />
-            <inertia ixx="0.00001" ixy="0" ixz="0" iyy="0.00001" iyz="0" izz="0.00001" />
-       </inertial>
-       <visual>
-   	    <origin xyz="0.0 0.0 0.0" rpy="0.0 0.0 0.0" />
-	    <geometry>
-    	       <box size="0.10 0.03 0.03" />
-	    </geometry>
-	    <material name="IPA/Black" />
-       </visual>
-    </link>
-    <!-- END: Softkinetic 'right' mount -->
-  </robot>
+    </visual>
+  </link>
+  <!-- END: rfid right mount -->
+  <!-- Camera pillar -->
+  <joint name="camera_pillar_joint" type="fixed" >
+    <origin xyz="0.4925 0.0825 0.48" rpy="0 0 0" />
+    <parent link="base_link" />
+    <child link="camera_pillar_link" />
+  </joint>
+  <link name="camera_pillar_link">
+    <xacro:default_inertial />
+    <visual>
+      <origin xyz="0 0 0.123" rpy="0 0 0" />
+      <geometry>
+        <box size="0.045 0.045 0.246" />
+      </geometry>
+      <material name="IPA/LightGrey" />
+    </visual>
+  </link>
+  <!-- END: camera_pillar -->
+  <!-- Softkinetic 'left' mount on raw3-1 -->
+  <joint name="softkinetic_left_joint" type="fixed" >
+    <origin xyz="0.015 0.06 0.215" rpy="0.0 ${M_PI/2} 0.0" />
+    <parent link="camera_pillar_link" />
+    <child link="softkinetic_left_link" />
+  </joint>
+  <link name="softkinetic_left_link">
+    <xacro:default_inertial />
+    <visual>
+      <origin xyz="0.0 0.0 0.0" rpy="0.0 0.0 0.0" />
+      <geometry>
+        <box size="0.10 0.03 0.03" />
+      </geometry>
+      <material name="IPA/Black" />
+    </visual>
+  </link>
+  <!-- END: Softkinetic 'left' mount -->
+  <!-- Softkinetic 'right' mount on raw3-1 -->
+  <joint name="softkinetic_right_joint" type="fixed" >
+    <origin xyz="0.015 -0.06 0.215" rpy="${M_PI} -${M_PI/2} 0.0" />
+    <parent link="camera_pillar_link" />
+    <child link="softkinetic_right_link" />
+  </joint>
+  <link name="softkinetic_right_link">
+    <xacro:default_inertial />
+    <visual>
+      <origin xyz="0.0 0.0 0.0" rpy="0.0 0.0 0.0" />
+      <geometry>
+        <box size="0.10 0.03 0.03" />
+      </geometry>
+      <material name="IPA/Black" />
+    </visual>
+  </link>
+  <!-- END: Softkinetic 'right' mount -->
+</robot>

Commit message: cob_hardware_config: adapted raw3-1 urdf concerning rfid-frame-names to match those in rfid-manager

File: cob_hardware_config/raw3-1/urdf/raw3-1.urdf.xacro (robot description, xacro)
@@ -62,7 +62,7 @@
     <origin xyz="0.55128 0.0 0.09" rpy="0 0 0" />
     <parent link="base_link" />
-    <child link="rfid_front_link" />
+    <child link="base_rfid_front_link" />
   </joint>
-  <link name="rfid_front_link">
+  <link name="base_rfid_front_link">
     <xacro:default_inertial />
     <visual>
@@ -81,7 +81,7 @@
     <origin xyz="-0.55128 0.0 0.09" rpy="0 0 ${M_PI}" />
     <parent link="base_link" />
-    <child link="rfid_rear_link" />
+    <child link="base_rfid_rear_link" />
   </joint>
-  <link name="rfid_rear_link">
+  <link name="base_rfid_rear_link">
     <xacro:default_inertial />
     <visual>
@@ -100,7 +100,7 @@
     <origin xyz="0.0 -0.30850 0.09" rpy="0 0 ${-0.5*M_PI}" />
     <parent link="base_link" />
-    <child link="rfid_right_link" />
+    <child link="base_rfid_side_link" />
   </joint>
-  <link name="rfid_right_link">
+  <link name="base_rfid_side_link">
     <xacro:default_inertial />
     <visual>

Commit message: updates from raw3-1 robot user

File: cob_hardware_config/raw3-1/urdf/raw3-1.urdf.xacro (robot description, xacro)
@@ -185,3 +185,20 @@
   </link>
   <!-- END: Softkinetic 'right' mount -->
+  <!-- Kinect mount on raw3-1 -->
+  <joint name="kinect_joint" type="fixed" >
+    <origin xyz="0.015 0.0 0.25" rpy="${M_PI/2} 0 ${M_PI/2}" />
+    <parent link="camera_pillar_link" />
+    <child link="kinect_link" />
+  </joint>
+  <link name="kinect_link">
+    <xacro:default_inertial />
+    <visual>
+      <origin xyz="0.0 0.0 0.0" rpy="0.0 0.0 0.0" />
+      <geometry>
+        <box size="0.10 0.03 0.03" />
+      </geometry>
+      <material name="IPA/Black" />
+    </visual>
+  </link>
+  <!-- END: Kinect mount -->
 </robot>

Commit message: added vacuum gripper

File: cob_hardware_config/raw3-1/urdf/raw3-1.urdf.xacro (robot description, xacro)
@@ -18,5 +18,8 @@
   <xacro:include filename="$(find cob_description)/urdf/ur_arm/ur10_arm.urdf.xacro" />
   <!-- raw boxgripper
-  <xacro:include filename="$(find raw_description)/urdf/boxgripper/boxgripper.urdf.xacro" />-->
+  <xacro:include filename="$(find raw_description)/urdf/boxgripper/boxgripper.urdf.xacro" /> -->
+  <!-- gripper -->
+  <xacro:include filename="$(find raw_description)/urdf/vacuum_gripper/gripper.urdf.xacro"/>
+  <xacro:property name="arm_prefix" value="arm_"/>
   <!-- composition of the robot -->
   <xacro:raw_base name="base"/>
@@ -56,5 +59,14 @@
   <!--xacro:raw_boxgripper name="gripper" parent="arm_ee_link">
     <origin xyz="${gripper_x} ${gripper_y} ${gripper_z}" rpy="${gripper_roll} ${gripper_pitch} ${gripper_yaw}" />
-  </xacro:raw_boxgripper-->
+  </xacro:raw_boxgripper> -->
+	<!-- arm-gripper coupling joint definitions
+	<joint name="${arm_prefix}to_gripper" type="fixed">
+		<parent link="arm_ee_link"/>
+		<child link="${arm_prefix}gripper_frame"/>
+		<origin xyz="0 0 0" rpy="-1.57 0 -1.57"/>
+	</joint>-->
+  <xacro:vacuum_gripper_definition name="gripper" parent="arm_ee_link" prefix="arm_">
+    <origin xyz="${gripper_x} ${gripper_y} ${gripper_z}" rpy="0 0 0" />
+  </xacro:vacuum_gripper_definition>
   <!-- IMU brick mount on raw3-1 -->
   <joint name="imu_brick_joint" type="fixed" >

Commit message: added vacuum gripper

File: cob_hardware_config/raw3-1/urdf/raw3-1.urdf.xacro (robot description, xacro)
@@ -18,5 +18,8 @@
   <xacro:include filename="$(find cob_description)/urdf/ur_arm/ur10_arm.urdf.xacro" />
   <!-- raw boxgripper
-  <xacro:include filename="$(find raw_description)/urdf/boxgripper/boxgripper.urdf.xacro" />-->
+  <xacro:include filename="$(find raw_description)/urdf/boxgripper/boxgripper.urdf.xacro" /> -->
+  <!-- gripper -->
+  <xacro:include filename="$(find raw_description)/urdf/vacuum_gripper/gripper.urdf.xacro"/>
+  <xacro:property name="arm_prefix" value="arm_"/>
   <!-- composition of the robot -->
   <xacro:raw_base name="base"/>
@@ -38,5 +41,14 @@
   <!--xacro:raw_boxgripper name="gripper" parent="arm_ee_link">
     <origin xyz="${gripper_x} ${gripper_y} ${gripper_z}" rpy="${gripper_roll} ${gripper_pitch} ${gripper_yaw}" />
-  </xacro:raw_boxgripper-->
+  </xacro:raw_boxgripper> -->
+	<!-- arm-gripper coupling joint definitions
+	<joint name="${arm_prefix}to_gripper" type="fixed">
+		<parent link="arm_ee_link"/>
+		<child link="${arm_prefix}gripper_frame"/>
+		<origin xyz="0 0 0" rpy="-1.57 0 -1.57"/>
+	</joint>-->
+  <xacro:vacuum_gripper_definition name="gripper" parent="arm_ee_link" prefix="arm_">
+    <origin xyz="${gripper_x} ${gripper_y} ${gripper_z}" rpy="0 0 0" />
+  </xacro:vacuum_gripper_definition>
   <!-- IMU brick mount on raw3-1 -->
   <joint name="imu_brick_joint" type="fixed" >
