Commit message: make simulation work preliminarily

File: cob_hardware_config/raw3-1/urdf/raw3-1.urdf.xacro (robot description, xacro)
@@ -9,6 +9,5 @@
   <xacro:include filename="$(find raw_description)/urdf/base_long/base.urdf.xacro" />
   <!-- raw tower -->
-  <!--xacro:include filename="$(find raw_description)/urdf/tower_asymetric/tower.urdf.xacro" /-->
-  <xacro:include filename="$(find raw_description)/urdf/tower_symetric/tower.urdf.xacro" />
+  <xacro:include filename="$(find raw_description)/urdf/tower_asymetric/tower.urdf.xacro" />
   <!-- torso -->
   <xacro:include filename="$(find raw_description)/urdf/torso/torso.urdf.xacro" />
@@ -17,17 +16,12 @@
   <!-- ur_arm -->
   <xacro:include filename="$(find cob_description)/urdf/ur_arm/ur10_arm.urdf.xacro" />
-  <!-- raw boxgripper
-  <xacro:include filename="$(find raw_description)/urdf/boxgripper/boxgripper.urdf.xacro" /> -->
-  <!-- gripper -->
-  <xacro:include filename="$(find raw_description)/urdf/vacuum_gripper/gripper.urdf.xacro"/>
+  <!-- vacuum gripper -->
+  <xacro:include filename="$(find raw_description)/urdf/vacuum_gripper/gripper.urdf.xacro" />
   <xacro:property name="arm_prefix" value="arm_"/>
   <!-- composition of the robot -->
   <xacro:raw_base name="base"/>
-  <!--xacro:tower_asymetric name="tower" parent="base_link">
+  <xacro:tower_asymetric name="tower" parent="base_link">
     <origin xyz="${tower_x} ${tower_y} ${tower_z}" rpy="${tower_roll} ${tower_pitch} ${tower_yaw}" />
-  </xacro:tower_asymetric-->
-  <xacro:tower_symetric name="tower" parent="base_link">
-    <origin xyz="${tower_x} ${tower_y} ${tower_z}" rpy="${tower_roll} ${tower_pitch} ${tower_yaw}" />
-  </xacro:tower_symetric>
+  </xacro:tower_asymetric>
   <xacro:raw_torso name="torso" parent="base_link">
     <origin xyz="${torso_x} ${torso_y} ${torso_z}" rpy="${torso_roll} ${torso_pitch} ${torso_yaw}" />
@@ -39,157 +33,6 @@
     <origin xyz="${arm_x} ${arm_y} ${arm_z}" rpy="${arm_roll} ${arm_pitch} ${arm_yaw}" />
   </xacro:ur10>
-  <!--xacro:raw_boxgripper name="gripper" parent="arm_ee_link">
+  <xacro:vacuum_gripper_definition name="gripper" parent="arm_ee_link" prefix="${arm_prefix}">
     <origin xyz="${gripper_x} ${gripper_y} ${gripper_z}" rpy="${gripper_roll} ${gripper_pitch} ${gripper_yaw}" />
-  </xacro:raw_boxgripper> -->
-	<!-- arm-gripper coupling joint definitions
-	<joint name="${arm_prefix}to_gripper" type="fixed">
-		<parent link="arm_ee_link"/>
-		<child link="${arm_prefix}gripper_frame"/>
-		<origin xyz="0 0 0" rpy="-1.57 0 -1.57"/>
-	</joint>-->
-  <xacro:vacuum_gripper_definition name="gripper" parent="arm_ee_link" prefix="arm_">
-    <origin xyz="${gripper_x} ${gripper_y} ${gripper_z}" rpy="0 0 0" />
   </xacro:vacuum_gripper_definition>
-  <!-- IMU brick mount on raw3-1 -->
-  <joint name="imu_brick_joint" type="fixed" >
-    <origin xyz="0.402 -0.0811 0.335" rpy="0 0 0" />
-    <parent link="base_link" />
-    <child link="imu_brick_link" />
-  </joint>
-  <link name="imu_brick_link">
-    <xacro:default_inertial />
-    <visual>
-      <origin xyz="0 0 -0.02" rpy="0 0 0" />
-      <geometry>
-        <box size="0.04 0.04 0.02" />
-      </geometry>
-      <material name="IPA/LightGrey" />
-    </visual>
-  </link>
-  <!-- END: IMU brick  mount -->
-  <!-- rfid_front mount on raw3-1 -->
-  <!--joint name="rfid_front_joint" type="fixed" >
-    <origin xyz="0.55128 0.0 0.09" rpy="0 0 0" />
-    <parent link="base_link" />
-    <child link="rfid_front_link" />
-  </joint>
-  <link name="rfid_front_link">
-    <xacro:default_inertial />
-    <visual>
-      <origin xyz="0 0 0" rpy="0 0 0" />
-      <geometry>
-        <box size="0.16 0.36 0.09" />
-      </geometry>
-      <material name="blue">
-        <color rgba="0 0 .8 1"/>
-      </material>
-    </visual>
-  </link-->
-  <!-- END: rfid front mount -->
-  <!-- rfid_rear mount on raw3-1 -->
-  <!--joint name="rfid_rear_joint" type="fixed" >
-    <origin xyz="-0.55128 0.0 0.09" rpy="0 0 ${M_PI}" />
-    <parent link="base_link" />
-    <child link="rfid_rear_link" />
-  </joint>
-  <link name="rfid_rear_link">
-    <xacro:default_inertial />
-    <visual>
-      <origin xyz="0 0 0" rpy="0 0 0" />
-      <geometry>
-        <box size="0.16 0.36 0.09" />
-      </geometry>
-      <material name="blue">
-        <color rgba="0 0 .8 1"/>
-      </material>
-    </visual>
-  </link-->
-  <!-- END: rfid rear mount -->
-  <!-- rfid_right mount on raw3-1 -->
-  <!--joint name="rfid_right_joint" type="fixed" >
-    <origin xyz="0.0 -0.30850 0.09" rpy="0 0 ${-0.5*M_PI}" />
-    <parent link="base_link" />
-    <child link="rfid_right_link" />
-  </joint>
-  <link name="rfid_right_link">
-    <xacro:default_inertial />
-    <visual>
-      <origin xyz="0 0 0" rpy="0 0 0" />
-      <geometry>
-        <box size="0.16 0.36 0.09" />
-      </geometry>
-      <material name="blue">
-        <color rgba="0 0 .8 1"/>
-      </material>
-    </visual>
-  </link-->
-  <!-- END: rfid right mount -->
-  <!-- Camera pillar -->
-  <!--joint name="camera_pillar_joint" type="fixed" >
-    <origin xyz="0.4925 0.0825 0.48" rpy="0 0 0" />
-    <parent link="base_link" />
-    <child link="camera_pillar_link" />
-  </joint>
-  <link name="camera_pillar_link">
-    <xacro:default_inertial />
-    <visual>
-      <origin xyz="0 0 0.123" rpy="0 0 0" />
-      <geometry>
-        <box size="0.045 0.045 0.246" />
-      </geometry>
-      <material name="IPA/LightGrey" />
-    </visual>
-  </link-->
-  <!-- END: camera_pillar -->
-  <!-- Softkinetic 'left' mount on raw3-1 -->
-  <!--joint name="softkinetic_left_joint" type="fixed" >
-    <origin xyz="0.015 0.06 0.215" rpy="0.0 ${M_PI/2} 0.0" />
-    <parent link="camera_pillar_link" />
-    <child link="softkinetic_left_link" />
-  </joint>
-  <link name="softkinetic_left_link">
-    <xacro:default_inertial />
-    <visual>
-      <origin xyz="0.0 0.0 0.0" rpy="0.0 0.0 0.0" />
-      <geometry>
-        <box size="0.10 0.03 0.03" />
-      </geometry>
-      <material name="IPA/Black" />
-    </visual>
-  </link-->
-  <!-- END: Softkinetic 'left' mount -->
-  <!-- Softkinetic 'right' mount on raw3-1 -->
-  <!--joint name="softkinetic_right_joint" type="fixed" >
-    <origin xyz="0.015 -0.06 0.215" rpy="${M_PI} -${M_PI/2} 0.0" />
-    <parent link="camera_pillar_link" />
-    <child link="softkinetic_right_link" />
-  </joint>
-  <link name="softkinetic_right_link">
-    <xacro:default_inertial />
-    <visual>
-      <origin xyz="0.0 0.0 0.0" rpy="0.0 0.0 0.0" />
-      <geometry>
-        <box size="0.10 0.03 0.03" />
-      </geometry>
-      <material name="IPA/Black" />
-    </visual>
-  </link-->
-  <!-- END: Softkinetic 'right' mount -->
-  <!-- Kinect mount on raw3-1 -->
-  <!--joint name="kinect_joint" type="fixed" >
-    <origin xyz="0.015 0.0 0.25" rpy="${M_PI/2} 0 ${M_PI/2}" />
-    <parent link="camera_pillar_link" />
-    <child link="kinect_link" />
-  </joint>
-  <link name="kinect_link">
-    <xacro:default_inertial />
-    <visual>
-      <origin xyz="0.0 0.0 0.0" rpy="0.0 0.0 0.0" />
-      <geometry>
-        <box size="0.10 0.03 0.03" />
-      </geometry>
-      <material name="IPA/Black" />
-    </visual>
-  </link-->
-  <!-- END: Kinect mount -->
 </robot>

Commit message: Update raw3-1.urdf.xacro

File: cob_hardware_config/raw3-1/urdf/raw3-1.urdf.xacro (robot description, xacro)
@@ -18,5 +18,4 @@
   <!-- vacuum gripper -->
   <xacro:include filename="$(find raw_description)/urdf/vacuum_gripper/gripper.urdf.xacro" />
-  <xacro:property name="arm_prefix" value="arm_"/>
   <!-- composition of the robot -->
   <xacro:raw_base name="base"/>
