Commit message: add lookat components to cob4-2

File: cob_hardware_config/cob4-2/urdf/cob4-2.urdf.xacro (robot description, xacro)
@@ -86,10 +86,12 @@
     </plugin>
   </gazebo>
-<!--
-  <xacro:lookat name="lookat" parent="torso_center_link" lower="0.0" upper="5.0">
+  <xacro:lookat name="torso_lookat" parent="torso_center_link" lower="0.0" upper="5.0">
     <origin xyz="0 0 0" rpy="0 0 0" />
     <axis xyz="1 0 0"/>
   </xacro:lookat>
--->
+  <xacro:lookat name="head_lookat" parent="head_center_link" lower="0.0" upper="5.0">
+    <origin xyz="0 0 0" rpy="0 0 0" />
+    <axis xyz="1 0 0"/>
+  </xacro:lookat>
   <!-- virtual component -->
 </robot>

Commit message: new structure, lwa4p_extended_withour_base

File: cob_hardware_config/cob4-2/urdf/cob4-2.urdf.xacro (robot description, xacro)
@@ -14,5 +14,5 @@
   <xacro:include filename="$(find cob_description)/urdf/lookat/lookat.urdf.xacro" />
   <!-- arm -->
-  <xacro:include filename="$(find schunk_description)/urdf/lwa4p_extended/lwa4p_extended.urdf.xacro" />
+  <xacro:include filename="$(find schunk_description)/urdf/lwa4p_extended/lwa4p_extended_without_base.urdf.xacro" />
   <!-- head -->
   <xacro:include filename="$(find cob_description)/urdf/cob4_head/head_static.urdf.xacro" />
@@ -42,5 +42,15 @@
     </plugin>
   </gazebo>
-  <xacro:schunk_lwa4p_extended name="arm_right" parent="torso_3_link"
+  <!-- joint between torso_3_link and lwa4p_extended_connector_link -->
+  <joint name="arm_right_base_joint" type="fixed">
+    <origin xyz="${arm_right_x} ${arm_right_y} ${arm_right_z}" rpy="${arm_right_roll} ${arm_right_pitch} ${arm_right_yaw}" />
+    <parent link="torso_3_link"/>
+    <child link="arm_right_base_link"/>
+  </joint>
+  <!-- static part of PRL100 -->
+  <link name="arm_right_base_link">
+    <xacro:default_inertial/>
+  </link>
+  <xacro:schunk_lwa4p_extended_without_base name="arm_right" parent="arm_right_base_link"
             arm_1_ref="${arm_right_1_ref}"
             arm_2_ref="${arm_right_2_ref}"
@@ -50,6 +60,6 @@
             arm_6_ref="${arm_right_6_ref}"
             arm_7_ref="${arm_right_7_ref}">
-    <origin xyz="${arm_right_x} ${arm_right_y} ${arm_right_z}" rpy="${arm_right_roll} ${arm_right_pitch} ${arm_right_yaw}" />
-  </xacro:schunk_lwa4p_extended>
+    <origin xyz="0 0 0.139" rpy="0 0 0" />
+  </xacro:schunk_lwa4p_extended_without_base>
   <gazebo>
     <plugin name="ros_control" filename="libmulti_hw_interface_gazebo_ros_control.so">
@@ -58,5 +68,15 @@
     </plugin>
   </gazebo>
-  <xacro:schunk_lwa4p_extended name="arm_left" parent="torso_3_link"
+  <!-- joint between torso_3_link and lwa4p_extended_connector_link -->
+  <joint name="arm_left_base_joint" type="fixed">
+    <origin xyz="${arm_left_x} ${arm_left_y} ${arm_left_z}" rpy="${arm_left_roll} ${arm_left_pitch} ${arm_left_yaw}" />
+    <parent link="torso_3_link"/>
+    <child link="arm_left_base_link"/>
+  </joint>
+  <!-- static part of PRL100 -->
+  <link name="arm_left_base_link">
+    <xacro:default_inertial/>
+  </link>
+  <xacro:schunk_lwa4p_extended_without_base name="arm_left" parent="arm_left_base_link"
             arm_1_ref="${arm_left_1_ref}"
             arm_2_ref="${arm_left_2_ref}"
@@ -66,6 +86,6 @@
             arm_6_ref="${arm_left_6_ref}"
             arm_7_ref="${arm_left_7_ref}">
-    <origin xyz="${arm_left_x} ${arm_left_y} ${arm_left_z}" rpy="${arm_left_roll} ${arm_left_pitch} ${arm_left_yaw}" />
-  </xacro:schunk_lwa4p_extended>
+    <origin xyz="0 0 0.139" rpy="0 0 0" />
+  </xacro:schunk_lwa4p_extended_without_base>
   <gazebo>
     <plugin name="ros_control" filename="libmulti_hw_interface_gazebo_ros_control.so">

Commit message: upgrade cob4-2

File: cob_hardware_config/cob4-2/urdf/cob4-2.urdf.xacro (robot description, xacro)
@@ -12,8 +12,4 @@
   <!-- torso -->
   <xacro:include filename="$(find cob_description)/urdf/cob4_torso/torso.urdf.xacro" />
-  <!-- arm -->
-  <xacro:include filename="$(find schunk_description)/urdf/lwa4p_extended/lwa4p_extended.urdf.xacro" />
-  <!-- gripper -->
-  <xacro:include filename="$(find cob_description)/urdf/cob4_gripper/gripper.urdf.xacro" />
   <!-- head -->
   <xacro:include filename="$(find cob_description)/urdf/cob4_head/head.urdf.xacro" />
@@ -53,7 +49,5 @@
     </plugin>
   </gazebo>
-  <!-- not yet active on cob4-2 hardware -->
-  <!--xacro:head name="head" parent="torso_3_link" dof1="true" dof2="true" dof3="true"-->
-  <xacro:head name="head" parent="torso_3_link" dof1="false" dof2="false" dof3="false">
+  <xacro:head name="head" parent="torso_3_link" dof1="true" dof2="true" dof3="true">
     <origin xyz="${head_x} ${head_y} ${head_z}" rpy="${head_roll} ${head_pitch} ${head_yaw}" />
   </xacro:head>
@@ -61,13 +55,11 @@
     <origin xyz="${head_cam_x} ${head_cam_y} ${head_cam_z}" rpy="${head_cam_roll} ${head_cam_pitch} ${head_cam_yaw}" />
   </xacro:usb_cam>
-  <!--gazebo>
+  <gazebo>
     <plugin name="ros_control" filename="libhwi_switch_gazebo_ros_control.so">
       <robotNamespace>head</robotNamespace>
       <filterJointsParam>joint_names</filterJointsParam>
     </plugin>
-  </gazebo-->
-  <!-- not yet active on cob4-2 hardware -->
-  <!--xacro:sensorring name="sensorring" parent="head_3_link" active="true" -->
-  <xacro:sensorring name="sensorring" parent="head_3_link" active="false" >
+  </gazebo>
+  <xacro:sensorring name="sensorring" parent="head_3_link" active="true">
     <origin xyz="${sensorring_x} ${sensorring_y} ${sensorring_z}" rpy="${sensorring_roll} ${sensorring_pitch} ${sensorring_yaw}" />
   </xacro:sensorring>
@@ -75,45 +67,9 @@
     <origin xyz="${sensorring_cam3d_x} ${sensorring_cam3d_y} ${sensorring_cam3d_z}" rpy="${sensorring_cam3d_roll} ${sensorring_cam3d_pitch} ${sensorring_cam3d_yaw}" />
   </xacro:cob_kinect_v0>
-  <!--gazebo>
+  <gazebo>
     <plugin name="ros_control" filename="libhwi_switch_gazebo_ros_control.so">
       <robotNamespace>sensorring</robotNamespace>
       <filterJointsParam>joint_names</filterJointsParam>
     </plugin>
-  </gazebo-->
-  <xacro:schunk_lwa4p_extended name="arm_right" parent="torso_3_link" has_podest="false">
-    <origin xyz="${arm_right_x} ${arm_right_y} ${arm_right_z}" rpy="${arm_right_roll} ${arm_right_pitch} ${arm_right_yaw}" />
-  </xacro:schunk_lwa4p_extended>
-  <gazebo>
-    <plugin name="ros_control" filename="libhwi_switch_gazebo_ros_control.so">
-      <robotNamespace>arm_right</robotNamespace>
-      <filterJointsParam>joint_names</filterJointsParam>
-    </plugin>
-  </gazebo>
-  <xacro:schunk_lwa4p_extended name="arm_left" parent="torso_3_link" has_podest="false">
-    <origin xyz="${arm_left_x} ${arm_left_y} ${arm_left_z}" rpy="${arm_left_roll} ${arm_left_pitch} ${arm_left_yaw}" />
-  </xacro:schunk_lwa4p_extended>
-  <gazebo>
-    <plugin name="ros_control" filename="libhwi_switch_gazebo_ros_control.so">
-      <robotNamespace>arm_left</robotNamespace>
-      <filterJointsParam>joint_names</filterJointsParam>
-    </plugin>
-  </gazebo>
-  <xacro:gripper name="gripper_right" parent="arm_right_7_link">
-    <origin xyz="${gripper_right_x} ${gripper_right_y} ${gripper_right_z}" rpy="${gripper_right_roll} ${gripper_right_pitch} ${gripper_right_yaw}" />
-  </xacro:gripper>
-  <gazebo>
-    <plugin name="ros_control" filename="libhwi_switch_gazebo_ros_control.so">
-      <robotNamespace>gripper_right</robotNamespace>
-      <filterJointsParam>joint_names</filterJointsParam>
-    </plugin>
-  </gazebo>
-  <xacro:gripper name="gripper_left" parent="arm_left_7_link">
-    <origin xyz="${gripper_left_x} ${gripper_left_y} ${gripper_left_z}" rpy="${gripper_left_roll} ${gripper_left_pitch} ${gripper_left_yaw}" />
-  </xacro:gripper>
-  <gazebo>
-    <plugin name="ros_control" filename="libhwi_switch_gazebo_ros_control.so">
-      <robotNamespace>gripper_left</robotNamespace>
-      <filterJointsParam>joint_names</filterJointsParam>
-    </plugin>
   </gazebo>
 </robot>
