Commit message: cob4_gripper

File: cob_hardware_config/cob4-2/urdf/calibration_default.urdf.xacro (robot description, xacro)
@@ -63,4 +63,18 @@
 	<property name="def_arm_left_pitch" value="0"/>
 	<property name="def_arm_left_yaw" value="3.14159"/>
+	<!-- gripper right mount positions | relative to arm_right_7_link -->
+	<property name="def_gripper_right_x" value="0.0"/>
+	<property name="def_gripper_right_y" value="0.0"/>
+	<property name="def_gripper_right_z" value="0.0"/>
+	<property name="def_gripper_right_roll" value="0.0"/>
+	<property name="def_gripper_right_pitch" value="0.0"/>
+	<property name="def_gripper_right_yaw" value="0.0"/>
+	<!-- gripper left mount positions | relative to arm_left_7_link -->
+	<property name="def_gripper_left_x" value="0.0"/>
+	<property name="def_gripper_left_y" value="0.0"/>
+	<property name="def_gripper_left_z" value="0.0"/>
+	<property name="def_gripper_left_roll" value="0.0"/>
+	<property name="def_gripper_left_pitch" value="0.0"/>
+	<property name="def_gripper_left_yaw" value="0.0"/>
 	<!-- *********************************** -->
 	<!-- kinematic chain reference positions -->
@@ -84,4 +98,10 @@
 	<property name="def_arm_left_6_ref" value="0.0"/>
 	<property name="def_arm_left_7_ref" value="0.0"/>
+	<!-- gripper right reference positions | used as calibration_rising for gripper chain-->
+	<property name="def_gripper_right_finger_1_ref" value="0.0"/>
+	<property name="def_gripper_right_finger_2_ref" value="0.0"/>
+	<!-- gripper left reference positions | used as calibration_rising for gripper chain-->
+	<property name="def_gripper_left_finger_1_ref" value="0.0"/>
+	<property name="def_gripper_left_finger_2_ref" value="0.0"/>
 	<!-- cam3d left | handeye calibration | relative to torso_3_link -->
 	<property name="def_torso_cam3d_left_x" value="0.12839"/>

File: cob_hardware_config/cob4-2/urdf/cob4-2.urdf.xacro (robot description, xacro)
@@ -15,4 +15,6 @@
   <!-- arm -->
   <xacro:include filename="$(find schunk_description)/urdf/lwa4p_extended/lwa4p_extended.urdf.xacro" />
+  <!-- gripper -->
+  <xacro:include filename="$(find cob_description)/urdf/cob4_gripper/gripper.urdf.xacro" />
   <!-- head -->
   <xacro:include filename="$(find cob_description)/urdf/cob4_head/head_static.urdf.xacro" />
@@ -74,4 +76,26 @@
     </plugin>
   </gazebo>
+  <xacro:gripper name="gripper_right" parent="arm_right_7_link"
+            finger_1_ref="${gripper_right_finger_1_ref}"
+            finger_2_ref="${gripper_right_finger_2_ref}" >
+    <origin xyz="${gripper_right_x} ${gripper_right_y} ${gripper_right_z}" rpy="${gripper_right_roll} ${gripper_right_pitch} ${gripper_right_yaw}" />
+  </xacro:gripper>
+  <gazebo>
+    <plugin name="ros_control" filename="libmulti_hw_interface_gazebo_ros_control.so">
+      <robotNamespace>gripper_right</robotNamespace>
+      <filterJointsParam>joint_names</filterJointsParam>
+    </plugin>
+  </gazebo>
+  <xacro:gripper name="gripper_left" parent="arm_left_7_link"
+            finger_1_ref="${gripper_left_finger_1_ref}"
+            finger_2_ref="${gripper_left_finger_2_ref}" >
+    <origin xyz="${gripper_left_x} ${gripper_left_y} ${gripper_left_z}" rpy="${gripper_left_roll} ${gripper_left_pitch} ${gripper_left_yaw}" />
+  </xacro:gripper>
+  <gazebo>
+    <plugin name="ros_control" filename="libmulti_hw_interface_gazebo_ros_control.so">
+      <robotNamespace>gripper_left</robotNamespace>
+      <filterJointsParam>joint_names</filterJointsParam>
+    </plugin>
+  </gazebo>
   <!-- virtual component -->
 </robot>

File: cob_hardware_config/cob4-2/urdf/properties.urdf.xacro (robot description, xacro)
@@ -66,4 +66,18 @@
 	<property name="arm_left_pitch" value="${def_arm_left_pitch+offset_arm_left_pitch}"/>
 	<property name="arm_left_yaw" value="${def_arm_left_yaw+offset_arm_left_yaw}"/>
+	<!-- gripper right mount positions | relative to arm_right_7_link -->
+	<property name="gripper_right_x" value="${def_gripper_right_x+offset_gripper_right_x}"/>
+	<property name="gripper_right_y" value="${def_gripper_right_y+offset_gripper_right_y}"/>
+	<property name="gripper_right_z" value="${def_gripper_right_z+offset_gripper_right_z}"/>
+	<property name="gripper_right_roll" value="${def_gripper_right_roll+offset_gripper_right_roll}"/>
+	<property name="gripper_right_pitch" value="${def_gripper_right_pitch+offset_gripper_right_pitch}"/>
+	<property name="gripper_right_yaw" value="${def_gripper_right_yaw+offset_gripper_right_yaw}"/>
+	<!-- gripper left mount positions | relative to arm_left_7_link -->
+	<property name="gripper_left_x" value="${def_gripper_left_x+offset_gripper_left_x}"/>
+	<property name="gripper_left_y" value="${def_gripper_left_y+offset_gripper_left_y}"/>
+	<property name="gripper_left_z" value="${def_gripper_left_z+offset_gripper_left_z}"/>
+	<property name="gripper_left_roll" value="${def_gripper_left_roll+offset_gripper_left_roll}"/>
+	<property name="gripper_left_pitch" value="${def_gripper_left_pitch+offset_gripper_left_pitch}"/>
+	<property name="gripper_left_yaw" value="${def_gripper_left_yaw+offset_gripper_left_yaw}"/>
 	<!-- *********************************** -->
 	<!-- kinematic chain reference positions -->
@@ -87,4 +101,10 @@
 	<property name="arm_left_6_ref" value="${def_arm_left_6_ref+offset_arm_left_6_ref}"/>
 	<property name="arm_left_7_ref" value="${def_arm_left_7_ref+offset_arm_left_7_ref}"/>
+	<!-- gripper right reference positions | used as calibration_rising for gripper chain-->
+	<property name="gripper_right_finger_1_ref" value="${def_gripper_right_finger_1_ref+offset_gripper_right_finger_1_ref}"/>
+	<property name="gripper_right_finger_2_ref" value="${def_gripper_right_finger_2_ref+offset_gripper_right_finger_2_ref}"/>
+	<!-- gripper left reference positions | used as calibration_rising for gripper chain-->
+	<property name="gripper_left_finger_1_ref" value="${def_gripper_left_finger_1_ref+offset_gripper_left_finger_1_ref}"/>
+	<property name="gripper_left_finger_2_ref" value="${def_gripper_left_finger_2_ref+offset_gripper_left_finger_2_ref}"/>
 	<!-- cam3d left | handeye calibration | relative to torso_3_link -->
 	<property name="torso_cam3d_left_x" value="${def_torso_cam3d_left_x+offset_torso_cam3d_left_x}"/>

Commit message: cob4_gripper

File: cob_hardware_config/cob4-2/urdf/calibration_default.urdf.xacro (robot description, xacro)
@@ -63,4 +63,18 @@
 	<property name="def_arm_left_pitch" value="0"/>
 	<property name="def_arm_left_yaw" value="3.14159"/>
+	<!-- gripper right mount positions | relative to arm_right_7_link -->
+	<property name="def_gripper_right_x" value="0.0"/>
+	<property name="def_gripper_right_y" value="0.0"/>
+	<property name="def_gripper_right_z" value="0.0748"/>
+	<property name="def_gripper_right_roll" value="0.0"/>
+	<property name="def_gripper_right_pitch" value="0.0"/>
+	<property name="def_gripper_right_yaw" value="0.0"/>
+	<!-- gripper left mount positions | relative to arm_left_7_link -->
+	<property name="def_gripper_left_x" value="0.0"/>
+	<property name="def_gripper_left_y" value="0.0"/>
+	<property name="def_gripper_left_z" value="0.0748"/>
+	<property name="def_gripper_left_roll" value="0.0"/>
+	<property name="def_gripper_left_pitch" value="0.0"/>
+	<property name="def_gripper_left_yaw" value="0.0"/>
 	<!-- *********************************** -->
 	<!-- kinematic chain reference positions -->
@@ -84,4 +98,10 @@
 	<property name="def_arm_left_6_ref" value="0.0"/>
 	<property name="def_arm_left_7_ref" value="0.0"/>
+	<!-- gripper right reference positions | used as calibration_rising for gripper chain-->
+	<property name="def_gripper_right_finger_1_ref" value="0.0"/>
+	<property name="def_gripper_right_finger_2_ref" value="0.0"/>
+	<!-- gripper left reference positions | used as calibration_rising for gripper chain-->
+	<property name="def_gripper_left_finger_1_ref" value="0.0"/>
+	<property name="def_gripper_left_finger_2_ref" value="0.0"/>
 	<!-- cam3d left | handeye calibration | relative to torso_3_link -->
 	<property name="def_torso_cam3d_left_x" value="0.12839"/>

File: cob_hardware_config/cob4-2/urdf/cob4-2.urdf.xacro (robot description, xacro)
@@ -15,4 +15,6 @@
   <!-- arm -->
   <xacro:include filename="$(find schunk_description)/urdf/lwa4p_extended/lwa4p_extended.urdf.xacro" />
+  <!-- gripper -->
+  <xacro:include filename="$(find cob_description)/urdf/cob4_gripper/gripper.urdf.xacro" />
   <!-- head -->
   <xacro:include filename="$(find cob_description)/urdf/cob4_head/head_static.urdf.xacro" />
@@ -74,4 +76,26 @@
     </plugin>
   </gazebo>
+  <xacro:gripper name="gripper_right" parent="arm_right_7_link"
+            finger_1_ref="${gripper_right_finger_1_ref}"
+            finger_2_ref="${gripper_right_finger_2_ref}" >
+    <origin xyz="${gripper_right_x} ${gripper_right_y} ${gripper_right_z}" rpy="${gripper_right_roll} ${gripper_right_pitch} ${gripper_right_yaw}" />
+  </xacro:gripper>
+  <gazebo>
+    <plugin name="ros_control" filename="libmulti_hw_interface_gazebo_ros_control.so">
+      <robotNamespace>gripper_right</robotNamespace>
+      <filterJointsParam>joint_names</filterJointsParam>
+    </plugin>
+  </gazebo>
+  <xacro:gripper name="gripper_left" parent="arm_left_7_link"
+            finger_1_ref="${gripper_left_finger_1_ref}"
+            finger_2_ref="${gripper_left_finger_2_ref}" >
+    <origin xyz="${gripper_left_x} ${gripper_left_y} ${gripper_left_z}" rpy="${gripper_left_roll} ${gripper_left_pitch} ${gripper_left_yaw}" />
+  </xacro:gripper>
+  <gazebo>
+    <plugin name="ros_control" filename="libmulti_hw_interface_gazebo_ros_control.so">
+      <robotNamespace>gripper_left</robotNamespace>
+      <filterJointsParam>joint_names</filterJointsParam>
+    </plugin>
+  </gazebo>
   <!-- virtual component -->
 </robot>

Commit message: remove cob4-2 leftover

File: cob_hardware_config/cob4-2/urdf/calibration_default.urdf.xacro (robot description, xacro)
@@ -49,32 +49,4 @@
 	<xacro:property name="def_sensorring_pitch" value="0.0"/>
 	<xacro:property name="def_sensorring_yaw" value="0.0"/>
-	<!-- arm right mount positions | relative to torso_3_link -->
-	<xacro:property name="def_arm_right_x" value="0.0"/>
-	<xacro:property name="def_arm_right_y" value="-0.014"/>
-	<xacro:property name="def_arm_right_z" value="0.55"/>
-	<xacro:property name="def_arm_right_roll" value="1.57097"/>
-	<xacro:property name="def_arm_right_pitch" value="0"/>
-	<xacro:property name="def_arm_right_yaw" value="0.0"/>
-	<!-- arm left mount positions | relative to torso_3_link -->
-	<xacro:property name="def_arm_left_x" value="0.0"/>
-	<xacro:property name="def_arm_left_y" value="0.014"/>
-	<xacro:property name="def_arm_left_z" value="0.55"/>
-	<xacro:property name="def_arm_left_roll" value="1.57097"/>
-	<xacro:property name="def_arm_left_pitch" value="0"/>
-	<xacro:property name="def_arm_left_yaw" value="3.14159"/>
-	<!-- gripper right mount positions | relative to arm_right_7_link -->
-	<xacro:property name="def_gripper_right_x" value="0.0"/>
-	<xacro:property name="def_gripper_right_y" value="0.0"/>
-	<xacro:property name="def_gripper_right_z" value="0.0748"/>
-	<xacro:property name="def_gripper_right_roll" value="0.0"/>
-	<xacro:property name="def_gripper_right_pitch" value="0.0"/>
-	<xacro:property name="def_gripper_right_yaw" value="3.14159"/>
-	<!-- gripper left mount positions | relative to arm_left_7_link -->
-	<xacro:property name="def_gripper_left_x" value="0.0"/>
-	<xacro:property name="def_gripper_left_y" value="0.0"/>
-	<xacro:property name="def_gripper_left_z" value="0.0748"/>
-	<xacro:property name="def_gripper_left_roll" value="0.0"/>
-	<xacro:property name="def_gripper_left_pitch" value="0.0"/>
-	<xacro:property name="def_gripper_left_yaw" value="3.14159"/>
 	<!-- *********************************** -->
 	<!-- kinematic chain reference positions -->

File: cob_hardware_config/cob4-2/urdf/properties.urdf.xacro (robot description, xacro)
@@ -52,32 +52,4 @@
 	<xacro:property name="sensorring_pitch" value="${def_sensorring_pitch+offset_sensorring_pitch}"/>
 	<xacro:property name="sensorring_yaw" value="${def_sensorring_yaw+offset_sensorring_yaw}"/>
-	<!-- arm mount positions | relative to torso_3_link -->
-	<xacro:property name="arm_right_x" value="${def_arm_right_x+offset_arm_right_x}"/>
-	<xacro:property name="arm_right_y" value="${def_arm_right_y+offset_arm_right_y}"/>
-	<xacro:property name="arm_right_z" value="${def_arm_right_z+offset_arm_right_z}"/>
-	<xacro:property name="arm_right_roll" value="${def_arm_right_roll+offset_arm_right_roll}"/>
-	<xacro:property name="arm_right_pitch" value="${def_arm_right_pitch+offset_arm_right_pitch}"/>
-	<xacro:property name="arm_right_yaw" value="${def_arm_right_yaw+offset_arm_right_yaw}"/>
-	<!-- arm mount positions | relative to torso_3_link -->
-	<xacro:property name="arm_left_x" value="${def_arm_left_x+offset_arm_left_x}"/>
-	<xacro:property name="arm_left_y" value="${def_arm_left_y+offset_arm_left_y}"/>
-	<xacro:property name="arm_left_z" value="${def_arm_left_z+offset_arm_left_z}"/>
-	<xacro:property name="arm_left_roll" value="${def_arm_left_roll+offset_arm_left_roll}"/>
-	<xacro:property name="arm_left_pitch" value="${def_arm_left_pitch+offset_arm_left_pitch}"/>
-	<xacro:property name="arm_left_yaw" value="${def_arm_left_yaw+offset_arm_left_yaw}"/>
-	<!-- gripper right mount positions | relative to arm_right_7_link -->
-	<xacro:property name="gripper_right_x" value="${def_gripper_right_x+offset_gripper_right_x}"/>
-	<xacro:property name="gripper_right_y" value="${def_gripper_right_y+offset_gripper_right_y}"/>
-	<xacro:property name="gripper_right_z" value="${def_gripper_right_z+offset_gripper_right_z}"/>
-	<xacro:property name="gripper_right_roll" value="${def_gripper_right_roll+offset_gripper_right_roll}"/>
-	<xacro:property name="gripper_right_pitch" value="${def_gripper_right_pitch+offset_gripper_right_pitch}"/>
-	<xacro:property name="gripper_right_yaw" value="${def_gripper_right_yaw+offset_gripper_right_yaw}"/>
-	<!-- gripper left mount positions | relative to arm_left_7_link -->
-	<xacro:property name="gripper_left_x" value="${def_gripper_left_x+offset_gripper_left_x}"/>
-	<xacro:property name="gripper_left_y" value="${def_gripper_left_y+offset_gripper_left_y}"/>
-	<xacro:property name="gripper_left_z" value="${def_gripper_left_z+offset_gripper_left_z}"/>
-	<xacro:property name="gripper_left_roll" value="${def_gripper_left_roll+offset_gripper_left_roll}"/>
-	<xacro:property name="gripper_left_pitch" value="${def_gripper_left_pitch+offset_gripper_left_pitch}"/>
-	<xacro:property name="gripper_left_yaw" value="${def_gripper_left_yaw+offset_gripper_left_yaw}"/>
 	<!-- *********************************** -->
 	<!-- kinematic chain reference positions -->

Commit message: fixed camera down camera calibration

File: cob_hardware_config/cob4-2/urdf/calibration_default.urdf.xacro (robot description, xacro)
@@ -71,7 +71,7 @@
 	<xacro:property name="def_torso_cam3d_down_y" value="0.0"/>
 	<xacro:property name="def_torso_cam3d_down_z" value="0.14005"/>
-	<xacro:property name="def_torso_cam3d_down_roll" value="2.18166"/> <!--2.18166-->
-	<xacro:property name="def_torso_cam3d_down_pitch" value="0.0"/>
-	<xacro:property name="def_torso_cam3d_down_yaw" value="1.57079"/> <!--1.57079-->
+	<xacro:property name="def_torso_cam3d_down_roll" value="0.0"/> <!--2.18166-->
+	<xacro:property name="def_torso_cam3d_down_pitch" value="0.61086"/>
+	<xacro:property name="def_torso_cam3d_down_yaw" value="0.0"/> <!--1.57079-->
 	<!-- cam3d | handeye calibration | relative to sensorring_link -->
 	<xacro:property name="def_sensorring_cam3d_x" value="0.096"/>
