Commit message: fixed camera down camera calibration for all robots

File: cob_hardware_config/cob4-10/urdf/calibration_default.urdf.xacro (robot description, xacro)
@@ -71,7 +71,7 @@
 	<xacro:property name="def_torso_cam3d_down_y" value="0.0"/>
 	<xacro:property name="def_torso_cam3d_down_z" value="0.14005"/>
-	<xacro:property name="def_torso_cam3d_down_roll" value="2.18166"/> <!--2.18166-->
-	<xacro:property name="def_torso_cam3d_down_pitch" value="0.0"/>
-	<xacro:property name="def_torso_cam3d_down_yaw" value="1.57079"/> <!--1.57079-->
+	<xacro:property name="def_torso_cam3d_down_roll" value="0.0"/>
+	<xacro:property name="def_torso_cam3d_down_pitch" value="0.61086"/>
+	<xacro:property name="def_torso_cam3d_down_yaw" value="0.0"/>
 	<!-- cam3d | handeye calibration | relative to sensorring_link -->
 	<xacro:property name="def_sensorring_cam3d_x" value="0.096"/>

File: cob_hardware_config/cob4-2/urdf/calibration_default.urdf.xacro (robot description, xacro)
@@ -71,7 +71,7 @@
 	<xacro:property name="def_torso_cam3d_down_y" value="0.0"/>
 	<xacro:property name="def_torso_cam3d_down_z" value="0.14005"/>
-	<xacro:property name="def_torso_cam3d_down_roll" value="0.0"/> <!--2.18166-->
+	<xacro:property name="def_torso_cam3d_down_roll" value="0.0"/>
 	<xacro:property name="def_torso_cam3d_down_pitch" value="0.61086"/>
-	<xacro:property name="def_torso_cam3d_down_yaw" value="0.0"/> <!--1.57079-->
+	<xacro:property name="def_torso_cam3d_down_yaw" value="0.0"/>
 	<!-- cam3d | handeye calibration | relative to sensorring_link -->
 	<xacro:property name="def_sensorring_cam3d_x" value="0.096"/>

File: cob_hardware_config/cob4-5/urdf/calibration_default.urdf.xacro (robot description, xacro)
@@ -100,5 +100,5 @@
 	<xacro:property name="def_torso_cam3d_down_z" value="0.14005"/>
 	<xacro:property name="def_torso_cam3d_down_roll" value="0.0"/>
-	<xacro:property name="def_torso_cam3d_down_pitch" value="0.54"/>
+	<xacro:property name="def_torso_cam3d_down_pitch" value="0.61086"/>
 	<xacro:property name="def_torso_cam3d_down_yaw" value="0.0"/>
 	<!-- cam3d | handeye calibration | relative to sensorring_link -->

File: cob_hardware_config/cob4-7/urdf/calibration_default.urdf.xacro (robot description, xacro)
@@ -85,7 +85,7 @@
 	<xacro:property name="def_torso_cam3d_down_y" value="0.0"/>
 	<xacro:property name="def_torso_cam3d_down_z" value="0.14005"/>
-	<xacro:property name="def_torso_cam3d_down_roll" value="2.18166"/> <!--2.18166-->
-	<xacro:property name="def_torso_cam3d_down_pitch" value="0.0"/>
-	<xacro:property name="def_torso_cam3d_down_yaw" value="1.57079"/> <!--1.57079-->
+	<xacro:property name="def_torso_cam3d_down_roll" value="0.0"/>
+	<xacro:property name="def_torso_cam3d_down_pitch" value="0.61086"/>
+	<xacro:property name="def_torso_cam3d_down_yaw" value="0.0"/>
 	<!-- cam3d | handeye calibration | relative to sensorring_link -->
 	<xacro:property name="def_sensorring_cam3d_x" value="0.096"/>
