Commit message: build torso with arms

File: cob_hardware_config/cob4-7/urdf/calibration_default.urdf.xacro (robot description, xacro)
@@ -49,4 +49,18 @@
 	<property name="def_sensorring_pitch" value="0.0"/>
 	<property name="def_sensorring_yaw" value="0.0"/>
+	<!-- arm right mount positions | relative to torso_3_link -->
+	<property name="def_arm_right_x" value="0.0"/>
+	<property name="def_arm_right_y" value="-0.014"/>
+	<property name="def_arm_right_z" value="0.55"/>
+	<property name="def_arm_right_roll" value="1.57097"/>
+	<property name="def_arm_right_pitch" value="0"/>
+	<property name="def_arm_right_yaw" value="0.0"/>
+	<!-- arm left mount positions | relative to torso_3_link -->
+	<property name="def_arm_left_x" value="0.0"/>
+	<property name="def_arm_left_y" value="0.014"/>
+	<property name="def_arm_left_z" value="0.55"/>
+	<property name="def_arm_left_roll" value="1.57097"/>
+	<property name="def_arm_left_pitch" value="0"/>
+	<property name="def_arm_left_yaw" value="3.14159"/>
 	<!-- *********************************** -->
 	<!-- kinematic chain reference positions -->
@@ -81,3 +95,10 @@
 	<property name="def_sensorring_cam3d_pitch" value="0.0"/>
 	<property name="def_sensorring_cam3d_yaw" value="-1.5708"/>
+	<!-- cam | handeye calibration | relative to head_3_link -->
+	<property name="def_head_cam_x" value="-0.181"/>
+	<property name="def_head_cam_y" value="0.0"/>
+	<property name="def_head_cam_z" value="0.325"/>
+	<property name="def_head_cam_roll" value="0.0"/>
+	<property name="def_head_cam_pitch" value="-0.73"/>
+	<property name="def_head_cam_yaw" value="3.14"/>
 </robot>

File: cob_hardware_config/cob4-7/urdf/cob4-7.urdf.xacro (robot description, xacro)
@@ -12,4 +12,6 @@
   <!-- torso -->
   <xacro:include filename="$(find cob_description)/urdf/cob4_torso/torso_2dof.urdf.xacro" />
+  <!-- arm -->
+  <xacro:include filename="$(find schunk_description)/urdf/lwa4p_extended/lwa4p_extended.urdf.xacro" />
   <!-- head -->
   <xacro:include filename="$(find cob_description)/urdf/cob4_head/head_static.urdf.xacro" />
@@ -33,4 +35,22 @@
     </plugin>
   </gazebo>
+  <xacro:schunk_lwa4p_extended name="arm_right" parent="torso_3_link" has_podest="false">
+    <origin xyz="${arm_right_x} ${arm_right_y} ${arm_right_z}" rpy="${arm_right_roll} ${arm_right_pitch} ${arm_right_yaw}" />
+  </xacro:schunk_lwa4p_extended>
+  <gazebo>
+    <plugin name="ros_control" filename="libhwi_switch_gazebo_ros_control.so">
+      <robotNamespace>arm_right</robotNamespace>
+      <filterJointsParam>joint_names</filterJointsParam>
+    </plugin>
+  </gazebo>
+  <xacro:schunk_lwa4p_extended name="arm_left" parent="torso_3_link" has_podest="false">
+    <origin xyz="${arm_left_x} ${arm_left_y} ${arm_left_z}" rpy="${arm_left_roll} ${arm_left_pitch} ${arm_left_yaw}" />
+  </xacro:schunk_lwa4p_extended>
+  <gazebo>
+    <plugin name="ros_control" filename="libhwi_switch_gazebo_ros_control.so">
+      <robotNamespace>arm_left</robotNamespace>
+      <filterJointsParam>joint_names</filterJointsParam>
+    </plugin>
+  </gazebo>
   <xacro:head name="head" parent="torso_3_link">
     <origin xyz="${head_x} ${head_y} ${head_z}" rpy="${head_roll} ${head_pitch} ${head_yaw}" />

File: cob_hardware_config/cob4-7/urdf/properties.urdf.xacro (robot description, xacro)
@@ -52,4 +52,18 @@
 	<property name="sensorring_pitch" value="${def_sensorring_pitch+offset_sensorring_pitch}"/>
 	<property name="sensorring_yaw" value="${def_sensorring_yaw+offset_sensorring_yaw}"/>
+	<!-- arm mount positions | relative to torso_3_link -->
+	<property name="arm_right_x" value="${def_arm_right_x+offset_arm_right_x}"/>
+	<property name="arm_right_y" value="${def_arm_right_y+offset_arm_right_y}"/>
+	<property name="arm_right_z" value="${def_arm_right_z+offset_arm_right_z}"/>
+	<property name="arm_right_roll" value="${def_arm_right_roll+offset_arm_right_roll}"/>
+	<property name="arm_right_pitch" value="${def_arm_right_pitch+offset_arm_right_pitch}"/>
+	<property name="arm_right_yaw" value="${def_arm_right_yaw+offset_arm_right_yaw}"/>
+	<!-- arm mount positions | relative to torso_3_link -->
+	<property name="arm_left_x" value="${def_arm_left_x+offset_arm_left_x}"/>
+	<property name="arm_left_y" value="${def_arm_left_y+offset_arm_left_y}"/>
+	<property name="arm_left_z" value="${def_arm_left_z+offset_arm_left_z}"/>
+	<property name="arm_left_roll" value="${def_arm_left_roll+offset_arm_left_roll}"/>
+	<property name="arm_left_pitch" value="${def_arm_left_pitch+offset_arm_left_pitch}"/>
+	<property name="arm_left_yaw" value="${def_arm_left_yaw+offset_arm_left_yaw}"/>
 	<!-- *********************************** -->
 	<!-- kinematic chain reference positions -->
@@ -84,3 +98,10 @@
 	<property name="sensorring_cam3d_pitch" value="${def_sensorring_cam3d_pitch+offset_sensorring_cam3d_pitch}"/>
 	<property name="sensorring_cam3d_yaw" value="${def_sensorring_cam3d_yaw+offset_sensorring_cam3d_yaw}"/>
+	<!-- cam | handeye calibration | relative to head_3_link -->
+	<property name="head_cam_x" value="${def_head_cam_x+offset_head_cam_x}"/>
+	<property name="head_cam_y" value="${def_head_cam_y+offset_head_cam_y}"/>
+	<property name="head_cam_z" value="${def_head_cam_z+offset_head_cam_z}"/>
+	<property name="head_cam_roll" value="${def_head_cam_roll+offset_head_cam_roll}"/>
+	<property name="head_cam_pitch" value="${def_head_cam_pitch+offset_head_cam_pitch}"/>
+	<property name="head_cam_yaw" value="${def_head_cam_yaw+offset_head_cam_yaw}"/>
 </robot>

Commit message: update cob4-7 setup , cob4-paul-stuttgart

File: cob_hardware_config/cob4-7/urdf/calibration_default.urdf.xacro (robot description, xacro)
@@ -49,18 +49,4 @@
 	<xacro:property name="def_sensorring_pitch" value="0.0"/>
 	<xacro:property name="def_sensorring_yaw" value="0.0"/>
-	<!-- arm right mount positions | relative to torso_3_link -->
-	<xacro:property name="def_arm_right_x" value="0.0"/>
-	<xacro:property name="def_arm_right_y" value="-0.014"/>
-	<xacro:property name="def_arm_right_z" value="0.55"/>
-	<xacro:property name="def_arm_right_roll" value="1.57097"/>
-	<xacro:property name="def_arm_right_pitch" value="0"/>
-	<xacro:property name="def_arm_right_yaw" value="0.0"/>
-	<!-- arm left mount positions | relative to torso_3_link -->
-	<xacro:property name="def_arm_left_x" value="0.0"/>
-	<xacro:property name="def_arm_left_y" value="0.014"/>
-	<xacro:property name="def_arm_left_z" value="0.55"/>
-	<xacro:property name="def_arm_left_roll" value="1.57097"/>
-	<xacro:property name="def_arm_left_pitch" value="0"/>
-	<xacro:property name="def_arm_left_yaw" value="3.14159"/>
 	<!-- *********************************** -->
 	<!-- kinematic chain reference positions -->

File: cob_hardware_config/cob4-7/urdf/cob4-7.urdf.xacro (robot description, xacro)
@@ -12,6 +12,4 @@
   <!-- torso -->
   <xacro:include filename="$(find cob_description)/urdf/cob4_torso/torso.urdf.xacro" />
-  <!-- arm -->
-  <xacro:include filename="$(find schunk_description)/urdf/lwa4p_extended/lwa4p_extended.urdf.xacro" />
   <!-- head -->
   <xacro:include filename="$(find cob_description)/urdf/cob4_head/head.urdf.xacro" />
@@ -39,10 +37,4 @@
     <origin xyz="${torso_cam3d_down_x} ${torso_cam3d_down_y} ${torso_cam3d_down_z}" rpy="${torso_cam3d_down_roll} ${torso_cam3d_down_pitch} ${torso_cam3d_down_yaw}" />
   </xacro:realsense>
-  <xacro:schunk_lwa4p_extended name="arm_right" parent="torso_3_link" has_podest="false">
-    <origin xyz="${arm_right_x} ${arm_right_y} ${arm_right_z}" rpy="${arm_right_roll} ${arm_right_pitch} ${arm_right_yaw}" />
-  </xacro:schunk_lwa4p_extended>
-  <xacro:schunk_lwa4p_extended name="arm_left" parent="torso_3_link" has_podest="false">
-    <origin xyz="${arm_left_x} ${arm_left_y} ${arm_left_z}" rpy="${arm_left_roll} ${arm_left_pitch} ${arm_left_yaw}" />
-  </xacro:schunk_lwa4p_extended>
   <xacro:head name="head" parent="torso_3_link" dof1="true" dof2="true" dof3="true">
     <origin xyz="${head_x} ${head_y} ${head_z}" rpy="${head_roll} ${head_pitch} ${head_yaw}" />

File: cob_hardware_config/cob4-7/urdf/properties.urdf.xacro (robot description, xacro)
@@ -52,18 +52,4 @@
 	<xacro:property name="sensorring_pitch" value="${def_sensorring_pitch+offset_sensorring_pitch}"/>
 	<xacro:property name="sensorring_yaw" value="${def_sensorring_yaw+offset_sensorring_yaw}"/>
-	<!-- arm mount positions | relative to torso_3_link -->
-	<xacro:property name="arm_right_x" value="${def_arm_right_x+offset_arm_right_x}"/>
-	<xacro:property name="arm_right_y" value="${def_arm_right_y+offset_arm_right_y}"/>
-	<xacro:property name="arm_right_z" value="${def_arm_right_z+offset_arm_right_z}"/>
-	<xacro:property name="arm_right_roll" value="${def_arm_right_roll+offset_arm_right_roll}"/>
-	<xacro:property name="arm_right_pitch" value="${def_arm_right_pitch+offset_arm_right_pitch}"/>
-	<xacro:property name="arm_right_yaw" value="${def_arm_right_yaw+offset_arm_right_yaw}"/>
-	<!-- arm mount positions | relative to torso_3_link -->
-	<xacro:property name="arm_left_x" value="${def_arm_left_x+offset_arm_left_x}"/>
-	<xacro:property name="arm_left_y" value="${def_arm_left_y+offset_arm_left_y}"/>
-	<xacro:property name="arm_left_z" value="${def_arm_left_z+offset_arm_left_z}"/>
-	<xacro:property name="arm_left_roll" value="${def_arm_left_roll+offset_arm_left_roll}"/>
-	<xacro:property name="arm_left_pitch" value="${def_arm_left_pitch+offset_arm_left_pitch}"/>
-	<xacro:property name="arm_left_yaw" value="${def_arm_left_yaw+offset_arm_left_yaw}"/>
 	<!-- *********************************** -->
 	<!-- kinematic chain reference positions -->
