Commit message: separate laser scanner from base

File: cob_hardware_config/robots/cob4-2/urdf/cob4-2.urdf.xacro (robot description, xacro)
@@ -20,6 +20,17 @@
   <xacro:include filename="$(find cob_description)/urdf/sensors/kinect.urdf.xacro" />
   <xacro:include filename="$(find cob_description)/urdf/sensors/usb_cam.urdf.xacro" />
+  <xacro:include filename="$(find cob_description)/urdf/sensors/sick_s300_laser.urdf.xacro"/>
   <!-- composition of the robot -->
   <xacro:base name="base" use_old_joint_names="false"/>
+  <!-- laser scanners -->
+  <xacro:sick_s300_laser_v0 name="base_laser_front" parent="base">
+    <origin xyz="${laser_front_x} ${laser_front_y} ${laser_front_z}" rpy="${laser_front_roll} ${laser_front_pitch} ${laser_front_yaw}" />
+  </xacro:sick_s300_laser_v0>
+  <xacro:sick_s300_laser_v0 name="base_laser_left" parent="base">
+    <origin xyz="${laser_left_x} ${laser_left_y} ${laser_left_z}" rpy="${laser_left_roll} ${laser_left_pitch} ${laser_left_yaw}" />
+  </xacro:sick_s300_laser_v0>
+  <xacro:sick_s300_laser_v0 name="base_laser_right" parent="base">
+    <origin xyz="${laser_right_x} ${laser_right_y} ${laser_right_z}" rpy="${laser_right_roll} ${laser_right_pitch} ${laser_right_yaw}" />
+  </xacro:sick_s300_laser_v0>
   <xacro:torso name="torso" parent="base_link" dof1="false" dof2="true" dof3="true">
     <origin xyz="${torso_x} ${torso_y} ${torso_z}" rpy="${torso_roll} ${torso_pitch} ${torso_yaw}" />

File: cob_hardware_config/robots/cob4-5/urdf/cob4-5.urdf.xacro (robot description, xacro)
@@ -25,6 +25,17 @@
   <xacro:include filename="$(find cob_description)/urdf/sensors/usb_cam.urdf.xacro" />
   <xacro:include filename="$(find cob_description)/urdf/sensors/sick_3dcs.urdf.xacro" />
+  <xacro:include filename="$(find cob_description)/urdf/sensors/sick_s300_laser.urdf.xacro"/>
   <!-- composition of the robot -->
   <xacro:base name="base" use_old_joint_names="false"/>
+  <!-- laser scanners -->
+  <xacro:sick_s300_laser_v0 name="base_laser_front" parent="base">
+    <origin xyz="${laser_front_x} ${laser_front_y} ${laser_front_z}" rpy="${laser_front_roll} ${laser_front_pitch} ${laser_front_yaw}" />
+  </xacro:sick_s300_laser_v0>
+  <xacro:sick_s300_laser_v0 name="base_laser_left" parent="base">
+    <origin xyz="${laser_left_x} ${laser_left_y} ${laser_left_z}" rpy="${laser_left_roll} ${laser_left_pitch} ${laser_left_yaw}" />
+  </xacro:sick_s300_laser_v0>
+  <xacro:sick_s300_laser_v0 name="base_laser_right" parent="base">
+    <origin xyz="${laser_right_x} ${laser_right_y} ${laser_right_z}" rpy="${laser_right_roll} ${laser_right_pitch} ${laser_right_yaw}" />
+  </xacro:sick_s300_laser_v0>
   <xacro:torso name="torso" parent="base_link" dof1="false" dof2="false" dof3="false">
     <origin xyz="${torso_x} ${torso_y} ${torso_z}" rpy="${torso_roll} ${torso_pitch} ${torso_yaw}" />

File: cob_hardware_config/robots/cob4-7/urdf/cob4-7.urdf.xacro (robot description, xacro)
@@ -20,6 +20,17 @@
   <xacro:include filename="$(find cob_description)/urdf/sensors/kinect.urdf.xacro" />
   <xacro:include filename="$(find cob_description)/urdf/sensors/usb_cam.urdf.xacro" />
+  <xacro:include filename="$(find cob_description)/urdf/sensors/sick_s300_laser.urdf.xacro"/>
   <!-- composition of the robot -->
   <xacro:base name="base" use_old_joint_names="false"/>
+  <!-- laser scanners -->
+  <xacro:sick_s300_laser_v0 name="base_laser_front" parent="base">
+    <origin xyz="${laser_front_x} ${laser_front_y} ${laser_front_z}" rpy="${laser_front_roll} ${laser_front_pitch} ${laser_front_yaw}" />
+  </xacro:sick_s300_laser_v0>
+  <xacro:sick_s300_laser_v0 name="base_laser_left" parent="base">
+    <origin xyz="${laser_left_x} ${laser_left_y} ${laser_left_z}" rpy="${laser_left_roll} ${laser_left_pitch} ${laser_left_yaw}" />
+  </xacro:sick_s300_laser_v0>
+  <xacro:sick_s300_laser_v0 name="base_laser_right" parent="base">
+    <origin xyz="${laser_right_x} ${laser_right_y} ${laser_right_z}" rpy="${laser_right_roll} ${laser_right_pitch} ${laser_right_yaw}" />
+  </xacro:sick_s300_laser_v0>
   <xacro:torso name="torso" parent="base_link" dof1="false" dof2="true" dof3="true">
     <origin xyz="${torso_x} ${torso_y} ${torso_z}" rpy="${torso_roll} ${torso_pitch} ${torso_yaw}" />

File: cob_hardware_config/robots/raw3-1/urdf/raw3-1.urdf.xacro (robot description, xacro)
@@ -18,6 +18,16 @@
   <!-- vacuum gripper -->
   <xacro:include filename="$(find raw_description)/urdf/vacuum_gripper/gripper.urdf.xacro" />
+  <!-- sensors -->
+  <xacro:include filename="$(find cob_description)/urdf/sensors/sick_s300_laser.urdf.xacro"/>
   <!-- composition of the robot -->
   <xacro:raw_base name="base"/>
+  <!-- base laser front -->
+  <xacro:sick_s300_laser_v0 name="base_laser_front" parent="base">
+    <origin xyz="${laser_front_x} ${laser_front_y} ${laser_front_z}" rpy="${laser_front_roll} ${laser_front_pitch} ${laser_front_yaw}" />
+  </xacro:sick_s300_laser_v0>
+  <!-- base laser rear -->
+  <xacro:sick_s300_laser_v0 name="base_laser_rear" parent="base">
+    <origin xyz="${laser_rear_x} ${laser_rear_y} ${laser_rear_z}" rpy="${laser_rear_roll} ${laser_rear_pitch} ${laser_rear_yaw}" />
+  </xacro:sick_s300_laser_v0>
   <xacro:tower_asymetric name="tower" parent="base_link">
     <origin xyz="${tower_x} ${tower_y} ${tower_z}" rpy="${tower_roll} ${tower_pitch} ${tower_yaw}" />

File: cob_hardware_config/robots/raw3-3/urdf/raw3-3.urdf.xacro (robot description, xacro)
@@ -9,9 +9,17 @@
   <xacro:include filename="$(find raw_description)/urdf/base_short/base.urdf.xacro" />
   <!-- raw tower -->
-<!--
-  <xacro:include filename="$(find raw_description)/urdf/tower_symetric/tower.urdf.xacro" />
--->
+  <!--xacro:include filename="$(find raw_description)/urdf/tower_symetric/tower.urdf.xacro" /-->
+  <!-- sensors -->
+  <xacro:include filename="$(find cob_description)/urdf/sensors/sick_s300_laser.urdf.xacro"/>
   <!-- composition of the robot -->
   <xacro:raw_base name="base"/>
+  <!-- base laser front -->
+  <xacro:sick_s300_laser_v0 name="base_laser_front" parent="base">
+    <origin xyz="${laser_front_x} ${laser_front_y} ${laser_front_z}" rpy="${laser_front_roll} ${laser_front_pitch} ${laser_front_yaw}" />
+  </xacro:sick_s300_laser_v0>
+  <!-- base laser rear -->
+  <xacro:sick_s300_laser_v0 name="base_laser_rear" parent="base">
+    <origin xyz="${laser_rear_x} ${laser_rear_y} ${laser_rear_z}" rpy="${laser_rear_roll} ${laser_rear_pitch} ${laser_rear_yaw}" />
+  </xacro:sick_s300_laser_v0>
 <!--
   <xacro:tower_symetric name="tower" parent="base_link">
