Commit message: consistency for all robots

File: cob_hardware_config/robots/cob4-2/urdf/calibration_default.urdf.xacro (robot description, xacro)
@@ -57,6 +57,6 @@
 	<xacro:property name="def_torso_cam3d_left_y" value="0.01802"/>
 	<xacro:property name="def_torso_cam3d_left_z" value="0.24214"/>
-	<xacro:property name="def_torso_cam3d_left_roll" value="0"/>
-	<xacro:property name="def_torso_cam3d_left_pitch" value="1.57079"/>
+	<xacro:property name="def_torso_cam3d_left_roll" value="1.57079"/>
+	<xacro:property name="def_torso_cam3d_left_pitch" value="0.0"/>
 	<xacro:property name="def_torso_cam3d_left_yaw" value="0.418879"/>
 	<!-- cam3d right | handeye calibration | relative to torso_3_link -->
@@ -64,6 +64,6 @@
 	<xacro:property name="def_torso_cam3d_right_y" value="-0.01802"/>
 	<xacro:property name="def_torso_cam3d_right_z" value="0.24214"/>
-	<xacro:property name="def_torso_cam3d_right_roll" value="0"/>
-	<xacro:property name="def_torso_cam3d_right_pitch" value="1.57079"/>
+	<xacro:property name="def_torso_cam3d_right_roll" value="1.57079"/>
+	<xacro:property name="def_torso_cam3d_right_pitch" value="0.0"/>
 	<xacro:property name="def_torso_cam3d_right_yaw" value="-0.418879"/>
 	<!-- cam3d down | handeye calibration | relative to torso_3_link -->
@@ -78,7 +78,7 @@
 	<xacro:property name="def_sensorring_cam3d_y" value="0.0"/>
 	<xacro:property name="def_sensorring_cam3d_z" value="0.0195"/>
-	<xacro:property name="def_sensorring_cam3d_roll" value="-1.5708"/>
+	<xacro:property name="def_sensorring_cam3d_roll" value="0.0"/>
 	<xacro:property name="def_sensorring_cam3d_pitch" value="0.0"/>
-	<xacro:property name="def_sensorring_cam3d_yaw" value="-1.5708"/>
+	<xacro:property name="def_sensorring_cam3d_yaw" value="0.0"/>
 	<!-- cam | handeye calibration | relative to head_3_link -->
 	<xacro:property name="def_head_cam_x" value="-0.181"/>
@@ -87,4 +87,4 @@
 	<xacro:property name="def_head_cam_roll" value="0.0"/>
 	<xacro:property name="def_head_cam_pitch" value="-0.73"/>
-	<xacro:property name="def_head_cam_yaw" value="3.14"/>
+	<xacro:property name="def_head_cam_yaw" value="0.0"/>
 </robot>

File: cob_hardware_config/robots/cob4-8/urdf/calibration_default.urdf.xacro (robot description, xacro)
@@ -85,6 +85,6 @@
 	<xacro:property name="def_torso_cam3d_left_y" value="0.01802"/>
 	<xacro:property name="def_torso_cam3d_left_z" value="0.24214"/>
-	<xacro:property name="def_torso_cam3d_left_roll" value="0"/>
-	<xacro:property name="def_torso_cam3d_left_pitch" value="1.57079"/>
+	<xacro:property name="def_torso_cam3d_left_roll" value="1.57079"/>
+	<xacro:property name="def_torso_cam3d_left_pitch" value="0.0"/>
 	<xacro:property name="def_torso_cam3d_left_yaw" value="0.418879"/>
 	<!-- cam3d right | handeye calibration | relative to torso_3_link -->
@@ -92,6 +92,6 @@
 	<xacro:property name="def_torso_cam3d_right_y" value="-0.01802"/>
 	<xacro:property name="def_torso_cam3d_right_z" value="0.24214"/>
-	<xacro:property name="def_torso_cam3d_right_roll" value="0"/>
-	<xacro:property name="def_torso_cam3d_right_pitch" value="1.57079"/>
+	<xacro:property name="def_torso_cam3d_right_roll" value="1.57079"/>
+	<xacro:property name="def_torso_cam3d_right_pitch" value="0.0"/>
 	<xacro:property name="def_torso_cam3d_right_yaw" value="-0.418879"/>
 	<!-- cam3d down | handeye calibration | relative to torso_3_link -->
@@ -106,7 +106,7 @@
 	<xacro:property name="def_sensorring_cam3d_y" value="0.0"/>
 	<xacro:property name="def_sensorring_cam3d_z" value="0.0195"/>
-	<xacro:property name="def_sensorring_cam3d_roll" value="-1.5708"/>
+	<xacro:property name="def_sensorring_cam3d_roll" value="0.0"/>
 	<xacro:property name="def_sensorring_cam3d_pitch" value="0.0"/>
-	<xacro:property name="def_sensorring_cam3d_yaw" value="-1.5708"/>
+	<xacro:property name="def_sensorring_cam3d_yaw" value="0.0"/>
 	<!-- cam | handeye calibration | relative to head_3_link -->
 	<xacro:property name="def_head_cam_x" value="-0.181"/>
@@ -115,4 +115,4 @@
 	<xacro:property name="def_head_cam_roll" value="0.0"/>
 	<xacro:property name="def_head_cam_pitch" value="-0.73"/>
-	<xacro:property name="def_head_cam_yaw" value="3.14"/>
+	<xacro:property name="def_head_cam_yaw" value="0.0"/>
 </robot>
