Commit message: use zr300 for torso_right camera

File: cob_hardware_config/robots/cob4-7/urdf/cob4-7.urdf.xacro (robot description, xacro)
@@ -17,4 +17,5 @@
   <!-- sensors -->
   <xacro:include filename="$(find cob_description)/urdf/sensors/realsense.urdf.xacro" />
+  <xacro:include filename="$(find cob_description)/urdf/sensors/realsense_zr300.urdf.xacro" />
   <xacro:include filename="$(find cob_description)/urdf/sensors/kinect.urdf.xacro" />
   <xacro:include filename="$(find cob_description)/urdf/sensors/usb_cam.urdf.xacro" />
@@ -47,4 +48,7 @@
     <origin xyz="${torso_cam3d_down_x} ${torso_cam3d_down_y} ${torso_cam3d_down_z}" rpy="${torso_cam3d_down_roll} ${torso_cam3d_down_pitch} ${torso_cam3d_down_yaw}" />
   </xacro:realsense>
+  <xacro:realsense_zr300 name="torso_cam3d_zr300" ros_topic="torso_cam3d_zr300" parent="torso_3_link">
+    <origin xyz="${torso_cam3d_zr300_x} ${torso_cam3d_zr300_y} ${torso_cam3d_zr300_z}" rpy="${torso_cam3d_zr300_roll} ${torso_cam3d_zr300_pitch} ${torso_cam3d_zr300_yaw}" />
+  </xacro:realsense_zr300>
   <xacro:head name="head" parent="torso_3_link" dof1="true" dof2="true" dof3="true">
     <origin xyz="${head_x} ${head_y} ${head_z}" rpy="${head_roll} ${head_pitch} ${head_yaw}" />

Commit message: finalize zr300 transformations

File: cob_hardware_config/robots/cob4-7/urdf/cob4-7.urdf.xacro (robot description, xacro)
@@ -37,18 +37,15 @@
   </xacro:torso>
   <!-- left camera -->
-  <xacro:cob_kinect_v0 name="torso_cam3d_left" ros_topic="torso_cam3d_left" parent="torso_3_link"  update_rate="30" data_skip="9">
+  <xacro:realsense_zr300 name="torso_cam3d_left" ros_topic="torso_cam3d_left" parent="torso_3_link">
     <origin xyz="${torso_cam3d_left_x} ${torso_cam3d_left_y} ${torso_cam3d_left_z}" rpy="${torso_cam3d_left_roll} ${torso_cam3d_left_pitch} ${torso_cam3d_left_yaw}" />
-  </xacro:cob_kinect_v0>
+  </xacro:realsense_zr300>
   <!-- right camera -->
-  <xacro:cob_kinect_v0 name="torso_cam3d_right" ros_topic="torso_cam3d_right" parent="torso_3_link" update_rate="30" data_skip="9">
+  <xacro:realsense_zr300 name="torso_cam3d_right" ros_topic="torso_cam3d_right" parent="torso_3_link">
     <origin xyz="${torso_cam3d_right_x} ${torso_cam3d_right_y} ${torso_cam3d_right_z}" rpy="${torso_cam3d_right_roll} ${torso_cam3d_right_pitch} ${torso_cam3d_right_yaw}" />
-  </xacro:cob_kinect_v0>
+  </xacro:realsense_zr300>
   <!-- down camera -->
   <xacro:realsense name="torso_cam3d_down" ros_topic="torso_cam3d_down" parent="torso_3_link">
     <origin xyz="${torso_cam3d_down_x} ${torso_cam3d_down_y} ${torso_cam3d_down_z}" rpy="${torso_cam3d_down_roll} ${torso_cam3d_down_pitch} ${torso_cam3d_down_yaw}" />
   </xacro:realsense>
-  <xacro:realsense_zr300 name="torso_cam3d_zr300" ros_topic="torso_cam3d_zr300" parent="torso_3_link">
-    <origin xyz="${torso_cam3d_zr300_x} ${torso_cam3d_zr300_y} ${torso_cam3d_zr300_z}" rpy="${torso_cam3d_zr300_roll} ${torso_cam3d_zr300_pitch} ${torso_cam3d_zr300_yaw}" />
-  </xacro:realsense_zr300>
   <xacro:head name="head" parent="torso_3_link" dof1="true" dof2="true" dof3="true">
     <origin xyz="${head_x} ${head_y} ${head_z}" rpy="${head_roll} ${head_pitch} ${head_yaw}" />
