Commit message: use zr300 for torso_right camera

File: cob_hardware_config/robots/cob4-7/urdf/calibration_default.urdf.xacro (robot description, xacro)
@@ -74,4 +74,11 @@
 	<xacro:property name="def_torso_cam3d_down_pitch" value="0.61086"/>
 	<xacro:property name="def_torso_cam3d_down_yaw" value="0.0"/>
+	<!-- cam3d zr300 | handeye calibration | relative to torso_3_link -->
+	<xacro:property name="def_torso_cam3d_zr300_x" value="0.12"/>
+	<xacro:property name="def_torso_cam3d_zr300_y" value="-0.06"/>
+	<xacro:property name="def_torso_cam3d_zr300_z" value="0.24214"/>
+	<xacro:property name="def_torso_cam3d_zr300_roll" value="-1.5908"/>
+	<xacro:property name="def_torso_cam3d_zr300_pitch" value="0.0"/>
+	<xacro:property name="def_torso_cam3d_zr300_yaw" value="-0.418879"/>
 	<!-- cam3d | handeye calibration | relative to sensorring_link -->
 	<xacro:property name="def_sensorring_cam3d_x" value="0.096"/>

File: cob_hardware_config/robots/cob4-7/urdf/cob4-7.urdf.xacro (robot description, xacro)
@@ -18,4 +18,5 @@
   <!-- sensors -->
   <xacro:include filename="$(find cob_description)/urdf/sensors/realsense.urdf.xacro" />
+  <xacro:include filename="$(find cob_description)/urdf/sensors/realsense_zr300.urdf.xacro" />
   <xacro:include filename="$(find cob_description)/urdf/sensors/kinect.urdf.xacro" />
   <xacro:include filename="$(find cob_description)/urdf/sensors/usb_cam.urdf.xacro" />
@@ -48,4 +49,7 @@
     <origin xyz="${torso_cam3d_down_x} ${torso_cam3d_down_y} ${torso_cam3d_down_z}" rpy="${torso_cam3d_down_roll} ${torso_cam3d_down_pitch} ${torso_cam3d_down_yaw}" />
   </xacro:realsense>
+  <xacro:realsense_zr300 name="torso_cam3d_zr300" ros_topic="torso_cam3d_zr300" parent="torso_3_link">
+    <origin xyz="${torso_cam3d_zr300_x} ${torso_cam3d_zr300_y} ${torso_cam3d_zr300_z}" rpy="${torso_cam3d_zr300_roll} ${torso_cam3d_zr300_pitch} ${torso_cam3d_zr300_yaw}" />
+  </xacro:realsense_zr300>
   <xacro:head name="head" parent="torso_3_link" dof1="true" dof2="true" dof3="true">
     <origin xyz="${head_x} ${head_y} ${head_z}" rpy="${head_roll} ${head_pitch} ${head_yaw}" />

File: cob_hardware_config/robots/cob4-7/urdf/properties.urdf.xacro (robot description, xacro)
@@ -77,4 +77,11 @@
 	<xacro:property name="torso_cam3d_down_pitch" value="${def_torso_cam3d_down_pitch+offset_torso_cam3d_down_pitch}"/>
 	<xacro:property name="torso_cam3d_down_yaw" value="${def_torso_cam3d_down_yaw+offset_torso_cam3d_down_yaw}"/>
+	<!-- cam3d zr300 | handeye calibration | relative to torso_3_link -->
+	<xacro:property name="torso_cam3d_zr300_x" value="${def_torso_cam3d_zr300_x+offset_torso_cam3d_zr300_x}"/>
+	<xacro:property name="torso_cam3d_zr300_y" value="${def_torso_cam3d_zr300_y+offset_torso_cam3d_zr300_y}"/>
+	<xacro:property name="torso_cam3d_zr300_z" value="${def_torso_cam3d_zr300_z+offset_torso_cam3d_zr300_z}"/>
+	<xacro:property name="torso_cam3d_zr300_roll" value="${def_torso_cam3d_zr300_roll+offset_torso_cam3d_zr300_roll}"/>
+	<xacro:property name="torso_cam3d_zr300_pitch" value="${def_torso_cam3d_zr300_pitch+offset_torso_cam3d_zr300_pitch}"/>
+	<xacro:property name="torso_cam3d_zr300_yaw" value="${def_torso_cam3d_zr300_yaw+offset_torso_cam3d_zr300_yaw}"/>
 	<!-- cam3d | handeye calibration | relative to sensorring_link -->
 	<xacro:property name="sensorring_cam3d_x" value="${def_sensorring_cam3d_x+offset_sensorring_cam3d_x}"/>

Commit message: finalize zr300 transformations

File: cob_hardware_config/robots/cob4-7/urdf/calibration_default.urdf.xacro (robot description, xacro)
@@ -57,6 +57,6 @@
 	<xacro:property name="def_torso_cam3d_left_y" value="0.01802"/>
 	<xacro:property name="def_torso_cam3d_left_z" value="0.24214"/>
-	<xacro:property name="def_torso_cam3d_left_roll" value="0"/>
-	<xacro:property name="def_torso_cam3d_left_pitch" value="1.57079"/>
+	<xacro:property name="def_torso_cam3d_left_roll" value="-1.57079"/>
+	<xacro:property name="def_torso_cam3d_left_pitch" value="0.0"/>
 	<xacro:property name="def_torso_cam3d_left_yaw" value="0.418879"/>
 	<!-- cam3d right | handeye calibration | relative to torso_3_link -->
@@ -64,6 +64,6 @@
 	<xacro:property name="def_torso_cam3d_right_y" value="-0.01802"/>
 	<xacro:property name="def_torso_cam3d_right_z" value="0.24214"/>
-	<xacro:property name="def_torso_cam3d_right_roll" value="0"/>
-	<xacro:property name="def_torso_cam3d_right_pitch" value="1.57079"/>
+	<xacro:property name="def_torso_cam3d_right_roll" value="-1.57079"/>
+	<xacro:property name="def_torso_cam3d_right_pitch" value="0.0"/>
 	<xacro:property name="def_torso_cam3d_right_yaw" value="-0.418879"/>
 	<!-- cam3d down | handeye calibration | relative to torso_3_link -->
@@ -74,11 +74,4 @@
 	<xacro:property name="def_torso_cam3d_down_pitch" value="0.61086"/>
 	<xacro:property name="def_torso_cam3d_down_yaw" value="0.0"/>
-	<!-- cam3d zr300 | handeye calibration | relative to torso_3_link -->
-	<xacro:property name="def_torso_cam3d_zr300_x" value="0.12"/>
-	<xacro:property name="def_torso_cam3d_zr300_y" value="-0.06"/>
-	<xacro:property name="def_torso_cam3d_zr300_z" value="0.24214"/>
-	<xacro:property name="def_torso_cam3d_zr300_roll" value="-1.5908"/>
-	<xacro:property name="def_torso_cam3d_zr300_pitch" value="0.0"/>
-	<xacro:property name="def_torso_cam3d_zr300_yaw" value="-0.418879"/>
 	<!-- cam3d | handeye calibration | relative to sensorring_link -->
 	<xacro:property name="def_sensorring_cam3d_x" value="0.096"/>

File: cob_hardware_config/robots/cob4-7/urdf/cob4-7.urdf.xacro (robot description, xacro)
@@ -38,18 +38,15 @@
   </xacro:torso>
   <!-- left camera -->
-  <xacro:cob_kinect_v0 name="torso_cam3d_left" ros_topic="torso_cam3d_left" parent="torso_3_link"  update_rate="30" data_skip="9">
+  <xacro:realsense_zr300 name="torso_cam3d_left" ros_topic="torso_cam3d_left" parent="torso_3_link">
     <origin xyz="${torso_cam3d_left_x} ${torso_cam3d_left_y} ${torso_cam3d_left_z}" rpy="${torso_cam3d_left_roll} ${torso_cam3d_left_pitch} ${torso_cam3d_left_yaw}" />
-  </xacro:cob_kinect_v0>
+  </xacro:realsense_zr300>
   <!-- right camera -->
-  <xacro:cob_kinect_v0 name="torso_cam3d_right" ros_topic="torso_cam3d_right" parent="torso_3_link" update_rate="30" data_skip="9">
+  <xacro:realsense_zr300 name="torso_cam3d_right" ros_topic="torso_cam3d_right" parent="torso_3_link">
     <origin xyz="${torso_cam3d_right_x} ${torso_cam3d_right_y} ${torso_cam3d_right_z}" rpy="${torso_cam3d_right_roll} ${torso_cam3d_right_pitch} ${torso_cam3d_right_yaw}" />
-  </xacro:cob_kinect_v0>
+  </xacro:realsense_zr300>
   <!-- down camera -->
   <xacro:realsense name="torso_cam3d_down" ros_topic="torso_cam3d_down" parent="torso_3_link">
     <origin xyz="${torso_cam3d_down_x} ${torso_cam3d_down_y} ${torso_cam3d_down_z}" rpy="${torso_cam3d_down_roll} ${torso_cam3d_down_pitch} ${torso_cam3d_down_yaw}" />
   </xacro:realsense>
-  <xacro:realsense_zr300 name="torso_cam3d_zr300" ros_topic="torso_cam3d_zr300" parent="torso_3_link">
-    <origin xyz="${torso_cam3d_zr300_x} ${torso_cam3d_zr300_y} ${torso_cam3d_zr300_z}" rpy="${torso_cam3d_zr300_roll} ${torso_cam3d_zr300_pitch} ${torso_cam3d_zr300_yaw}" />
-  </xacro:realsense_zr300>
   <xacro:head name="head" parent="torso_3_link" dof1="true" dof2="true" dof3="true">
     <origin xyz="${head_x} ${head_y} ${head_z}" rpy="${head_roll} ${head_pitch} ${head_yaw}" />

File: cob_hardware_config/robots/cob4-7/urdf/properties.urdf.xacro (robot description, xacro)
@@ -77,11 +77,4 @@
 	<xacro:property name="torso_cam3d_down_pitch" value="${def_torso_cam3d_down_pitch+offset_torso_cam3d_down_pitch}"/>
 	<xacro:property name="torso_cam3d_down_yaw" value="${def_torso_cam3d_down_yaw+offset_torso_cam3d_down_yaw}"/>
-	<!-- cam3d zr300 | handeye calibration | relative to torso_3_link -->
-	<xacro:property name="torso_cam3d_zr300_x" value="${def_torso_cam3d_zr300_x+offset_torso_cam3d_zr300_x}"/>
-	<xacro:property name="torso_cam3d_zr300_y" value="${def_torso_cam3d_zr300_y+offset_torso_cam3d_zr300_y}"/>
-	<xacro:property name="torso_cam3d_zr300_z" value="${def_torso_cam3d_zr300_z+offset_torso_cam3d_zr300_z}"/>
-	<xacro:property name="torso_cam3d_zr300_roll" value="${def_torso_cam3d_zr300_roll+offset_torso_cam3d_zr300_roll}"/>
-	<xacro:property name="torso_cam3d_zr300_pitch" value="${def_torso_cam3d_zr300_pitch+offset_torso_cam3d_zr300_pitch}"/>
-	<xacro:property name="torso_cam3d_zr300_yaw" value="${def_torso_cam3d_zr300_yaw+offset_torso_cam3d_zr300_yaw}"/>
 	<!-- cam3d | handeye calibration | relative to sensorring_link -->
 	<xacro:property name="sensorring_cam3d_x" value="${def_sensorring_cam3d_x+offset_sensorring_cam3d_x}"/>

Commit message: fix camera coord frames for asus and zr300 on cob4-7

File: cob_hardware_config/robots/cob4-7/urdf/calibration_default.urdf.xacro (robot description, xacro)
@@ -57,5 +57,5 @@
 	<xacro:property name="def_torso_cam3d_left_y" value="0.01802"/>
 	<xacro:property name="def_torso_cam3d_left_z" value="0.24214"/>
-	<xacro:property name="def_torso_cam3d_left_roll" value="-1.57079"/>
+	<xacro:property name="def_torso_cam3d_left_roll" value="1.57079"/>
 	<xacro:property name="def_torso_cam3d_left_pitch" value="0.0"/>
 	<xacro:property name="def_torso_cam3d_left_yaw" value="0.418879"/>
@@ -64,5 +64,5 @@
 	<xacro:property name="def_torso_cam3d_right_y" value="-0.01802"/>
 	<xacro:property name="def_torso_cam3d_right_z" value="0.24214"/>
-	<xacro:property name="def_torso_cam3d_right_roll" value="-1.57079"/>
+	<xacro:property name="def_torso_cam3d_right_roll" value="1.57079"/>
 	<xacro:property name="def_torso_cam3d_right_pitch" value="0.0"/>
 	<xacro:property name="def_torso_cam3d_right_yaw" value="-0.418879"/>
@@ -78,7 +78,7 @@
 	<xacro:property name="def_sensorring_cam3d_y" value="0.0"/>
 	<xacro:property name="def_sensorring_cam3d_z" value="0.0195"/>
-	<xacro:property name="def_sensorring_cam3d_roll" value="-1.5708"/>
+	<xacro:property name="def_sensorring_cam3d_roll" value="0.0"/>
 	<xacro:property name="def_sensorring_cam3d_pitch" value="0.0"/>
-	<xacro:property name="def_sensorring_cam3d_yaw" value="-1.5708"/>
+	<xacro:property name="def_sensorring_cam3d_yaw" value="0.0"/>
 	<!-- cam | handeye calibration | relative to head_3_link -->
 	<xacro:property name="def_head_cam_x" value="-0.181"/>

Commit message: setup cob4-7

File: cob_hardware_config/robots/cob4-7/urdf/calibration_default.urdf.xacro (robot description, xacro)
@@ -49,4 +49,18 @@
 	<xacro:property name="def_sensorring_pitch" value="0.0"/>
 	<xacro:property name="def_sensorring_yaw" value="0.0"/>
+	<!-- arm right mount positions | relative to torso_3_link -->
+	<xacro:property name="def_arm_right_x" value="0.0"/>
+	<xacro:property name="def_arm_right_y" value="-0.014"/>
+	<xacro:property name="def_arm_right_z" value="0.55"/>
+	<xacro:property name="def_arm_right_roll" value="1.57097"/>
+	<xacro:property name="def_arm_right_pitch" value="0"/>
+	<xacro:property name="def_arm_right_yaw" value="0.0"/>
+	<!-- arm left mount positions | relative to torso_3_link -->
+	<xacro:property name="def_arm_left_x" value="0.0"/>
+	<xacro:property name="def_arm_left_y" value="0.014"/>
+	<xacro:property name="def_arm_left_z" value="0.55"/>
+	<xacro:property name="def_arm_left_roll" value="1.57097"/>
+	<xacro:property name="def_arm_left_pitch" value="0"/>
+	<xacro:property name="def_arm_left_yaw" value="3.14159"/>
 	<!-- *********************************** -->
 	<!-- kinematic chain reference positions -->

File: cob_hardware_config/robots/cob4-7/urdf/cob4-7.urdf.xacro (robot description, xacro)
@@ -11,4 +11,8 @@
   <!-- torso -->
   <xacro:include filename="$(find cob_description)/urdf/cob4_torso/torso.urdf.xacro" />
+  <!-- arm -->
+  <xacro:include filename="$(find cob_description)/urdf/cob4_arm/cob4_arm.urdf.xacro" />
+  <!-- hand -->
+  <xacro:include filename="$(find cob_description)/urdf/cob4_gripper/gripper.urdf.xacro" />
   <!-- head -->
   <xacro:include filename="$(find cob_description)/urdf/cob4_head/head.urdf.xacro" />
@@ -54,4 +58,10 @@
     <origin xyz="${head_cam_x} ${head_cam_y} ${head_cam_z}" rpy="${head_cam_roll} ${head_cam_pitch} ${head_cam_yaw}" />
   </xacro:usb_cam>
+  <xacro:cob4_arm name="arm_right" parent="torso_3_link" has_podest="false">
+    <origin xyz="${arm_right_x} ${arm_right_y} ${arm_right_z}" rpy="${arm_right_roll} ${arm_right_pitch} ${arm_right_yaw}" />
+  </xacro:cob4_arm>
+  <xacro:cob4_arm name="arm_left" parent="torso_3_link" has_podest="false">
+    <origin xyz="${arm_left_x} ${arm_left_y} ${arm_left_z}" rpy="${arm_left_roll} ${arm_left_pitch} ${arm_left_yaw}" />
+  </xacro:cob4_arm>
   <xacro:sensorring name="sensorring" parent="head_3_link" active="true">
     <origin xyz="${sensorring_x} ${sensorring_y} ${sensorring_z}" rpy="${sensorring_roll} ${sensorring_pitch} ${sensorring_yaw}" />

File: cob_hardware_config/robots/cob4-7/urdf/properties.urdf.xacro (robot description, xacro)
@@ -52,4 +52,18 @@
 	<xacro:property name="sensorring_pitch" value="${def_sensorring_pitch+offset_sensorring_pitch}"/>
 	<xacro:property name="sensorring_yaw" value="${def_sensorring_yaw+offset_sensorring_yaw}"/>
+	<!-- arm mount positions | relative to torso_3_link -->
+	<xacro:property name="arm_right_x" value="${def_arm_right_x+offset_arm_right_x}"/>
+	<xacro:property name="arm_right_y" value="${def_arm_right_y+offset_arm_right_y}"/>
+	<xacro:property name="arm_right_z" value="${def_arm_right_z+offset_arm_right_z}"/>
+	<xacro:property name="arm_right_roll" value="${def_arm_right_roll+offset_arm_right_roll}"/>
+	<xacro:property name="arm_right_pitch" value="${def_arm_right_pitch+offset_arm_right_pitch}"/>
+	<xacro:property name="arm_right_yaw" value="${def_arm_right_yaw+offset_arm_right_yaw}"/>
+	<!-- arm mount positions | relative to torso_3_link -->
+	<xacro:property name="arm_left_x" value="${def_arm_left_x+offset_arm_left_x}"/>
+	<xacro:property name="arm_left_y" value="${def_arm_left_y+offset_arm_left_y}"/>
+	<xacro:property name="arm_left_z" value="${def_arm_left_z+offset_arm_left_z}"/>
+	<xacro:property name="arm_left_roll" value="${def_arm_left_roll+offset_arm_left_roll}"/>
+	<xacro:property name="arm_left_pitch" value="${def_arm_left_pitch+offset_arm_left_pitch}"/>
+	<xacro:property name="arm_left_yaw" value="${def_arm_left_yaw+offset_arm_left_yaw}"/>
 	<!-- *********************************** -->
 	<!-- kinematic chain reference positions -->
