Commit message: full config for cob4-10 tlabs

File: cob_hardware_config/robots/cob4-10/urdf/calibration_default.urdf.xacro (robot description, xacro)
@@ -25,3 +25,94 @@
 	<xacro:property name="def_laser_right_pitch" value="0.0"/>
 	<xacro:property name="def_laser_right_yaw" value="-2.094"/>
+	<!-- *********************** -->
+	<!-- upper robot calibration -->
+	<!-- *********************** -->
+	<!-- torso mount positions | relative to base_link -->
+	<xacro:property name="def_torso_x" value="0.0"/>
+	<xacro:property name="def_torso_y" value="0.0"/>
+	<xacro:property name="def_torso_z" value="0.26411"/>
+	<xacro:property name="def_torso_roll" value="0.0"/>
+	<xacro:property name="def_torso_pitch" value="0.0"/>
+	<xacro:property name="def_torso_yaw" value="0.0"/>
+	<!-- head mount positions | relative to torso_3_link -->
+	<xacro:property name="def_head_x" value="0.0"/>
+	<xacro:property name="def_head_y" value="0.0"/>
+	<xacro:property name="def_head_z" value="0.610"/>
+	<xacro:property name="def_head_roll" value="0.0"/>
+	<xacro:property name="def_head_pitch" value="0.0"/>
+	<xacro:property name="def_head_yaw" value="0.0"/>
+	<!-- head sensors mount positions | relative to head_3_link -->
+	<xacro:property name="def_sensorring_x" value="0.0"/>
+	<xacro:property name="def_sensorring_y" value="0.0"/>
+	<xacro:property name="def_sensorring_z" value="0.006"/>
+	<xacro:property name="def_sensorring_roll" value="0.0"/>
+	<xacro:property name="def_sensorring_pitch" value="0.0"/>
+	<xacro:property name="def_sensorring_yaw" value="0.0"/>
+	<!-- arm right mount positions | relative to torso_3_link -->
+	<xacro:property name="def_arm_right_x" value="0.0"/>
+	<xacro:property name="def_arm_right_y" value="-0.014"/>
+	<xacro:property name="def_arm_right_z" value="0.55"/>
+	<xacro:property name="def_arm_right_roll" value="1.57097"/>
+	<xacro:property name="def_arm_right_pitch" value="0"/>
+	<xacro:property name="def_arm_right_yaw" value="0.0"/>
+	<!-- arm left mount positions | relative to torso_3_link -->
+	<xacro:property name="def_arm_left_x" value="0.0"/>
+	<xacro:property name="def_arm_left_y" value="0.014"/>
+	<xacro:property name="def_arm_left_z" value="0.55"/>
+	<xacro:property name="def_arm_left_roll" value="1.57097"/>
+	<xacro:property name="def_arm_left_pitch" value="0"/>
+	<xacro:property name="def_arm_left_yaw" value="3.14159"/>
+	<!-- gripper right mount positions | relative to arm_right_7_link -->
+	<xacro:property name="def_gripper_right_x" value="0.0"/>
+	<xacro:property name="def_gripper_right_y" value="0.0"/>
+	<xacro:property name="def_gripper_right_z" value="0.0748"/>
+	<xacro:property name="def_gripper_right_roll" value="0.0"/>
+	<xacro:property name="def_gripper_right_pitch" value="0.0"/>
+	<xacro:property name="def_gripper_right_yaw" value="3.14159"/>
+	<!-- gripper left mount positions | relative to arm_left_7_link -->
+	<xacro:property name="def_gripper_left_x" value="0.0"/>
+	<xacro:property name="def_gripper_left_y" value="0.0"/>
+	<xacro:property name="def_gripper_left_z" value="0.0748"/>
+	<xacro:property name="def_gripper_left_roll" value="0.0"/>
+	<xacro:property name="def_gripper_left_pitch" value="0.0"/>
+	<xacro:property name="def_gripper_left_yaw" value="3.14159"/>
+	<!-- *********************************** -->
+	<!-- kinematic chain reference positions -->
+	<!-- *********************************** -->
+	<!-- this feature is no longer supported as urdfdom does not parse the according 'calibration_rising' tag -->
+	<!-- cam3d left | handeye calibration | relative to torso_3_link -->
+	<xacro:property name="def_torso_cam3d_left_x" value="0.125"/>
+	<xacro:property name="def_torso_cam3d_left_y" value="0.01802"/>
+	<xacro:property name="def_torso_cam3d_left_z" value="0.24214"/>
+	<xacro:property name="def_torso_cam3d_left_roll" value="0"/>
+	<xacro:property name="def_torso_cam3d_left_pitch" value="1.57079"/>
+	<xacro:property name="def_torso_cam3d_left_yaw" value="0.418879"/>
+	<!-- cam3d right | handeye calibration | relative to torso_3_link -->
+	<xacro:property name="def_torso_cam3d_right_x" value="0.12839"/>
+	<xacro:property name="def_torso_cam3d_right_y" value="-0.01802"/>
+	<xacro:property name="def_torso_cam3d_right_z" value="0.24214"/>
+	<xacro:property name="def_torso_cam3d_right_roll" value="0"/>
+	<xacro:property name="def_torso_cam3d_right_pitch" value="1.57079"/>
+	<xacro:property name="def_torso_cam3d_right_yaw" value="-0.418879"/>
+	<!-- cam3d down | handeye calibration | relative to torso_3_link -->
+	<xacro:property name="def_torso_cam3d_down_x" value="0.15908"/>
+	<xacro:property name="def_torso_cam3d_down_y" value="0.0"/>
+	<xacro:property name="def_torso_cam3d_down_z" value="0.14005"/>
+	<xacro:property name="def_torso_cam3d_down_roll" value="0.0"/>
+	<xacro:property name="def_torso_cam3d_down_pitch" value="0.61086"/>
+	<xacro:property name="def_torso_cam3d_down_yaw" value="0.0"/>
+	<!-- cam3d | handeye calibration | relative to sensorring_link -->
+	<xacro:property name="def_sensorring_cam3d_x" value="0.096"/>
+	<xacro:property name="def_sensorring_cam3d_y" value="0.0"/>
+	<xacro:property name="def_sensorring_cam3d_z" value="0.0195"/>
+	<xacro:property name="def_sensorring_cam3d_roll" value="-1.5708"/>
+	<xacro:property name="def_sensorring_cam3d_pitch" value="0.0"/>
+	<xacro:property name="def_sensorring_cam3d_yaw" value="-1.5708"/>
+	<!-- cam | handeye calibration | relative to head_3_link -->
+	<xacro:property name="def_head_cam_x" value="-0.181"/>
+	<xacro:property name="def_head_cam_y" value="0.0"/>
+	<xacro:property name="def_head_cam_z" value="0.325"/>
+	<xacro:property name="def_head_cam_roll" value="0.0"/>
+	<xacro:property name="def_head_cam_pitch" value="-0.73"/>
+	<xacro:property name="def_head_cam_yaw" value="3.14"/>
 </robot>

File: cob_hardware_config/robots/cob4-10/urdf/cob4-10.urdf.xacro (robot description, xacro)
@@ -5,10 +5,22 @@
   <xacro:include filename="$(find cob_description)/urdf/common.xacro" />
   <xacro:include filename="$(find cob_description)/urdf/materials.urdf.xacro" />
-  <xacro:include filename="$(find schunk_description)/urdf/materials.urdf.xacro" />
   <!-- calibration -->
   <xacro:include filename="$(find cob_hardware_config)/robots/cob4-10/urdf/properties.urdf.xacro" />
   <!-- base -->
   <xacro:include filename="$(find cob_description)/urdf/cob4_base/base.urdf.xacro" />
+  <!-- torso -->
+  <xacro:include filename="$(find cob_description)/urdf/cob4_torso/torso.urdf.xacro" />
+  <!-- arm -->
+  <xacro:include filename="$(find cob_description)/urdf/cob4_arm/cob4_arm.urdf.xacro" />
+  <!-- hand -->
+  <xacro:include filename="$(find cob_description)/urdf/cob4_gripper/gripper.urdf.xacro" />
+  <!-- head -->
+  <xacro:include filename="$(find cob_description)/urdf/cob4_head/head.urdf.xacro" />
+  <!-- sensorring -->
+  <xacro:include filename="$(find cob_description)/urdf/cob4_sensorring/sensorring.urdf.xacro" />
   <!-- sensors -->
+  <xacro:include filename="$(find cob_description)/urdf/sensors/realsense.urdf.xacro" />
+  <xacro:include filename="$(find cob_description)/urdf/sensors/kinect.urdf.xacro" />
+  <xacro:include filename="$(find cob_description)/urdf/sensors/usb_cam.urdf.xacro" />
   <xacro:include filename="$(find cob_description)/urdf/sensors/sick_s300_laser.urdf.xacro"/>
   <!-- composition of the robot -->
@@ -24,3 +36,43 @@
     <origin xyz="${laser_right_x} ${laser_right_y} ${laser_right_z}" rpy="${laser_right_roll} ${laser_right_pitch} ${laser_right_yaw}" />
   </xacro:sick_s300_laser_v0>
+  <xacro:torso name="torso" parent="base_link" dof1="false" dof2="false" dof3="false">
+    <origin xyz="${torso_x} ${torso_y} ${torso_z}" rpy="${torso_roll} ${torso_pitch} ${torso_yaw}" />
+  </xacro:torso>
+  <!-- left camera -->
+  <xacro:cob_kinect_v0 name="torso_cam3d_left" ros_topic="torso_cam3d_left" parent="torso_3_link" update_rate="30" data_skip="9">
+    <origin xyz="${torso_cam3d_left_x} ${torso_cam3d_left_y} ${torso_cam3d_left_z}" rpy="${torso_cam3d_left_roll} ${torso_cam3d_left_pitch} ${torso_cam3d_left_yaw}" />
+  </xacro:cob_kinect_v0>
+  <!-- right camera -->
+  <xacro:cob_kinect_v0 name="torso_cam3d_right" ros_topic="torso_cam3d_right" parent="torso_3_link" update_rate="30" data_skip="9">
+    <origin xyz="${torso_cam3d_right_x} ${torso_cam3d_right_y} ${torso_cam3d_right_z}" rpy="${torso_cam3d_right_roll} ${torso_cam3d_right_pitch} ${torso_cam3d_right_yaw}" />
+  </xacro:cob_kinect_v0>
+  <!-- down camera -->
+  <xacro:realsense name="torso_cam3d_down" ros_topic="torso_cam3d_down" parent="torso_3_link">
+    <origin xyz="${torso_cam3d_down_x} ${torso_cam3d_down_y} ${torso_cam3d_down_z}" rpy="${torso_cam3d_down_roll} ${torso_cam3d_down_pitch} ${torso_cam3d_down_yaw}" />
+  </xacro:realsense>
+  <xacro:head name="head" parent="torso_3_link" dof1="false" dof2="false" dof3="false">
+    <origin xyz="${head_x} ${head_y} ${head_z}" rpy="${head_roll} ${head_pitch} ${head_yaw}" />
+  </xacro:head>
+  <xacro:usb_cam name="head_cam" parent="head_3_link" ros_topic="head_cam" update_rate="3.5" height="1536" width="2048" > <!-- get this from config/head_cam.yaml -->
+    <origin xyz="${head_cam_x} ${head_cam_y} ${head_cam_z}" rpy="${head_cam_roll} ${head_cam_pitch} ${head_cam_yaw}" />
+  </xacro:usb_cam>
+  <xacro:sensorring name="sensorring" parent="head_3_link" active="true">
+    <origin xyz="${sensorring_x} ${sensorring_y} ${sensorring_z}" rpy="${sensorring_roll} ${sensorring_pitch} ${sensorring_yaw}" />
+  </xacro:sensorring>
+  <!-- cameras -->
+  <xacro:cob_kinect_v0 name="sensorring_cam3d" ros_topic="sensorring_cam3d" parent="sensorring_link" update_rate="30" data_skip="9">
+    <origin xyz="${sensorring_cam3d_x} ${sensorring_cam3d_y} ${sensorring_cam3d_z}" rpy="${sensorring_cam3d_roll} ${sensorring_cam3d_pitch} ${sensorring_cam3d_yaw}" />
+  </xacro:cob_kinect_v0>
+  <xacro:cob4_arm name="arm_right" parent="torso_3_link" has_podest="false">
+    <origin xyz="${arm_right_x} ${arm_right_y} ${arm_right_z}" rpy="${arm_right_roll} ${arm_right_pitch} ${arm_right_yaw}" />
+  </xacro:cob4_arm>
+  <xacro:cob4_arm name="arm_left" parent="torso_3_link" has_podest="false">
+    <origin xyz="${arm_left_x} ${arm_left_y} ${arm_left_z}" rpy="${arm_left_roll} ${arm_left_pitch} ${arm_left_yaw}" />
+  </xacro:cob4_arm>
+  <xacro:gripper name="gripper_right" parent="arm_right_7_link">
+    <origin xyz="${gripper_right_x} ${gripper_right_y} ${gripper_right_z}" rpy="${gripper_right_roll} ${gripper_right_pitch} ${gripper_right_yaw}" />
+  </xacro:gripper>
+  <xacro:gripper name="gripper_left" parent="arm_left_7_link">
+    <origin xyz="${gripper_left_x} ${gripper_left_y} ${gripper_left_z}" rpy="${gripper_left_roll} ${gripper_left_pitch} ${gripper_left_yaw}" />
+  </xacro:gripper>
 </robot>

File: cob_hardware_config/robots/cob4-10/urdf/properties.urdf.xacro (robot description, xacro)
@@ -28,3 +28,94 @@
 	<xacro:property name="laser_right_pitch" value="${def_laser_right_pitch+offset_laser_right_pitch}"/>
 	<xacro:property name="laser_right_yaw" value="${def_laser_right_yaw+offset_laser_right_yaw}"/>
+	<!-- *********************** -->
+	<!-- upper robot calibration -->
+	<!-- *********************** -->
+	<!-- torso mount positions | relative to base_link -->
+	<xacro:property name="torso_x" value="${def_torso_x+offset_torso_x}"/>
+	<xacro:property name="torso_y" value="${def_torso_y+offset_torso_y}"/>
+	<xacro:property name="torso_z" value="${def_torso_z+offset_torso_z}"/>
+	<xacro:property name="torso_roll" value="${def_torso_roll+offset_torso_roll}"/>
+	<xacro:property name="torso_pitch" value="${def_torso_pitch+offset_torso_pitch}"/>
+	<xacro:property name="torso_yaw" value="${def_torso_yaw+offset_torso_yaw}"/>
+	<!-- head mount positions | relative to torso_3_link -->
+	<xacro:property name="head_x" value="${def_head_x+offset_head_x}"/>
+	<xacro:property name="head_y" value="${def_head_y+offset_head_y}"/>
+	<xacro:property name="head_z" value="${def_head_z+offset_head_z}"/>
+	<xacro:property name="head_roll" value="${def_head_roll+offset_head_roll}"/>
+	<xacro:property name="head_pitch" value="${def_head_pitch+offset_head_pitch}"/>
+	<xacro:property name="head_yaw" value="${def_head_yaw+offset_head_yaw}"/>
+	<!-- head sensors mount positions | relative to head_3_link -->
+	<xacro:property name="sensorring_x" value="${def_sensorring_x+offset_sensorring_x}"/>
+	<xacro:property name="sensorring_y" value="${def_sensorring_y+offset_sensorring_y}"/>
+	<xacro:property name="sensorring_z" value="${def_sensorring_z+offset_sensorring_z}"/>
+	<xacro:property name="sensorring_roll" value="${def_sensorring_roll+offset_sensorring_roll}"/>
+	<xacro:property name="sensorring_pitch" value="${def_sensorring_pitch+offset_sensorring_pitch}"/>
+	<xacro:property name="sensorring_yaw" value="${def_sensorring_yaw+offset_sensorring_yaw}"/>
+	<!-- arm mount positions | relative to torso_3_link -->
+	<xacro:property name="arm_right_x" value="${def_arm_right_x+offset_arm_right_x}"/>
+	<xacro:property name="arm_right_y" value="${def_arm_right_y+offset_arm_right_y}"/>
+	<xacro:property name="arm_right_z" value="${def_arm_right_z+offset_arm_right_z}"/>
+	<xacro:property name="arm_right_roll" value="${def_arm_right_roll+offset_arm_right_roll}"/>
+	<xacro:property name="arm_right_pitch" value="${def_arm_right_pitch+offset_arm_right_pitch}"/>
+	<xacro:property name="arm_right_yaw" value="${def_arm_right_yaw+offset_arm_right_yaw}"/>
+	<!-- arm mount positions | relative to torso_3_link -->
+	<xacro:property name="arm_left_x" value="${def_arm_left_x+offset_arm_left_x}"/>
+	<xacro:property name="arm_left_y" value="${def_arm_left_y+offset_arm_left_y}"/>
+	<xacro:property name="arm_left_z" value="${def_arm_left_z+offset_arm_left_z}"/>
+	<xacro:property name="arm_left_roll" value="${def_arm_left_roll+offset_arm_left_roll}"/>
+	<xacro:property name="arm_left_pitch" value="${def_arm_left_pitch+offset_arm_left_pitch}"/>
+	<xacro:property name="arm_left_yaw" value="${def_arm_left_yaw+offset_arm_left_yaw}"/>
+	<!-- gripper mount positions | relative to arm_7_link -->
+	<xacro:property name="gripper_right_x" value="${def_gripper_right_x+offset_gripper_right_x}"/>
+	<xacro:property name="gripper_right_y" value="${def_gripper_right_y+offset_gripper_right_y}"/>
+	<xacro:property name="gripper_right_z" value="${def_gripper_right_z+offset_gripper_right_z}"/>
+	<xacro:property name="gripper_right_roll" value="${def_gripper_right_roll+offset_gripper_right_roll}"/>
+	<xacro:property name="gripper_right_pitch" value="${def_gripper_right_pitch+offset_gripper_right_pitch}"/>
+	<xacro:property name="gripper_right_yaw" value="${def_gripper_right_yaw+offset_gripper_right_yaw}"/>
+	<!-- gripper mount positions | relative to arm_7_link -->
+	<xacro:property name="gripper_left_x" value="${def_gripper_left_x+offset_gripper_left_x}"/>
+	<xacro:property name="gripper_left_y" value="${def_gripper_left_y+offset_gripper_left_y}"/>
+	<xacro:property name="gripper_left_z" value="${def_gripper_left_z+offset_gripper_left_z}"/>
+	<xacro:property name="gripper_left_roll" value="${def_gripper_left_roll+offset_gripper_left_roll}"/>
+	<xacro:property name="gripper_left_pitch" value="${def_gripper_left_pitch+offset_gripper_left_pitch}"/>
+	<xacro:property name="gripper_left_yaw" value="${def_gripper_left_yaw+offset_gripper_left_yaw}"/>
+	<!-- *********************************** -->
+	<!-- kinematic chain reference positions -->
+	<!-- *********************************** -->
+	<!-- this feature is no longer supported as urdfdom does not parse the according 'calibration_rising' tag -->
+	<!-- cam3d left | handeye calibration | relative to torso_3_link -->
+	<xacro:property name="torso_cam3d_left_x" value="${def_torso_cam3d_left_x+offset_torso_cam3d_left_x}"/>
+	<xacro:property name="torso_cam3d_left_y" value="${def_torso_cam3d_left_y+offset_torso_cam3d_left_y}"/>
+	<xacro:property name="torso_cam3d_left_z" value="${def_torso_cam3d_left_z+offset_torso_cam3d_left_z}"/>
+	<xacro:property name="torso_cam3d_left_roll" value="${def_torso_cam3d_left_roll+offset_torso_cam3d_left_roll}"/>
+	<xacro:property name="torso_cam3d_left_pitch" value="${def_torso_cam3d_left_pitch+offset_torso_cam3d_left_pitch}"/>
+	<xacro:property name="torso_cam3d_left_yaw" value="${def_torso_cam3d_left_yaw+offset_torso_cam3d_left_yaw}"/>
+	<!-- cam3d right | handeye calibration | relative to torso_3_link -->
+	<xacro:property name="torso_cam3d_right_x" value="${def_torso_cam3d_right_x+offset_torso_cam3d_right_x}"/>
+	<xacro:property name="torso_cam3d_right_y" value="${def_torso_cam3d_right_y+offset_torso_cam3d_right_y}"/>
+	<xacro:property name="torso_cam3d_right_z" value="${def_torso_cam3d_right_z+offset_torso_cam3d_right_z}"/>
+	<xacro:property name="torso_cam3d_right_roll" value="${def_torso_cam3d_right_roll+offset_torso_cam3d_right_roll}"/>
+	<xacro:property name="torso_cam3d_right_pitch" value="${def_torso_cam3d_right_pitch+offset_torso_cam3d_right_pitch}"/>
+	<xacro:property name="torso_cam3d_right_yaw" value="${def_torso_cam3d_right_yaw+offset_torso_cam3d_right_yaw}"/>
+	<!-- cam3d down | handeye calibration | relative to torso_3_link -->
+	<xacro:property name="torso_cam3d_down_x" value="${def_torso_cam3d_down_x+offset_torso_cam3d_down_x}"/>
+	<xacro:property name="torso_cam3d_down_y" value="${def_torso_cam3d_down_y+offset_torso_cam3d_down_y}"/>
+	<xacro:property name="torso_cam3d_down_z" value="${def_torso_cam3d_down_z+offset_torso_cam3d_down_z}"/>
+	<xacro:property name="torso_cam3d_down_roll" value="${def_torso_cam3d_down_roll+offset_torso_cam3d_down_roll}"/>
+	<xacro:property name="torso_cam3d_down_pitch" value="${def_torso_cam3d_down_pitch+offset_torso_cam3d_down_pitch}"/>
+	<xacro:property name="torso_cam3d_down_yaw" value="${def_torso_cam3d_down_yaw+offset_torso_cam3d_down_yaw}"/>
+	<!-- cam3d | handeye calibration | relative to sensorring_link -->
+	<xacro:property name="sensorring_cam3d_x" value="${def_sensorring_cam3d_x+offset_sensorring_cam3d_x}"/>
+	<xacro:property name="sensorring_cam3d_y" value="${def_sensorring_cam3d_y+offset_sensorring_cam3d_y}"/>
+	<xacro:property name="sensorring_cam3d_z" value="${def_sensorring_cam3d_z+offset_sensorring_cam3d_z}"/>
+	<xacro:property name="sensorring_cam3d_roll" value="${def_sensorring_cam3d_roll+offset_sensorring_cam3d_roll}"/>
+	<xacro:property name="sensorring_cam3d_pitch" value="${def_sensorring_cam3d_pitch+offset_sensorring_cam3d_pitch}"/>
+	<xacro:property name="sensorring_cam3d_yaw" value="${def_sensorring_cam3d_yaw+offset_sensorring_cam3d_yaw}"/>
+	<!-- cam | handeye calibration | relative to head_3_link -->
+	<xacro:property name="head_cam_x" value="${def_head_cam_x+offset_head_cam_x}"/>
+	<xacro:property name="head_cam_y" value="${def_head_cam_y+offset_head_cam_y}"/>
+	<xacro:property name="head_cam_z" value="${def_head_cam_z+offset_head_cam_z}"/>
+	<xacro:property name="head_cam_roll" value="${def_head_cam_roll+offset_head_cam_roll}"/>
+	<xacro:property name="head_cam_pitch" value="${def_head_cam_pitch+offset_head_cam_pitch}"/>
+	<xacro:property name="head_cam_yaw" value="${def_head_cam_yaw+offset_head_cam_yaw}"/>
 </robot>
