Commit message: setup cob4-10

File: cob_hardware_config/robots/cob4-10/urdf/calibration_default.urdf.xacro (robot description, xacro)
@@ -103,10 +103,17 @@
 	<xacro:property name="def_torso_cam3d_down_yaw" value="0.0"/>
 	<!-- cam3d | handeye calibration | relative to sensorring_link -->
-	<xacro:property name="def_sensorring_cam3d_x" value="0.096"/>
-	<xacro:property name="def_sensorring_cam3d_y" value="0.0"/>
-	<xacro:property name="def_sensorring_cam3d_z" value="0.0195"/>
-	<xacro:property name="def_sensorring_cam3d_roll" value="-1.5708"/>
-	<xacro:property name="def_sensorring_cam3d_pitch" value="0.0"/>
-	<xacro:property name="def_sensorring_cam3d_yaw" value="-1.5708"/>
+	<xacro:property name="def_sensorring_cam3d_front_x" value="0.096"/>
+	<xacro:property name="def_sensorring_cam3d_front_y" value="0.0"/>
+	<xacro:property name="def_sensorring_cam3d_front_z" value="0.0195"/>
+	<xacro:property name="def_sensorring_cam3d_front_roll" value="-1.95"/>
+	<xacro:property name="def_sensorring_cam3d_front_pitch" value="0.0"/>
+	<xacro:property name="def_sensorring_cam3d_front_yaw" value="-1.5708"/>
+	<!-- cam3d | handeye calibration | relative to sensorring_link -->
+	<xacro:property name="def_sensorring_cam3d_back_x" value="-0.096"/>
+	<xacro:property name="def_sensorring_cam3d_back_y" value="0.0"/>
+	<xacro:property name="def_sensorring_cam3d_back_z" value="0.0195"/>
+	<xacro:property name="def_sensorring_cam3d_back_roll" value="-1.5708"/>
+	<xacro:property name="def_sensorring_cam3d_back_pitch" value="0.0"/>
+	<xacro:property name="def_sensorring_cam3d_back_yaw" value="1.5708"/>
 	<!-- cam | handeye calibration | relative to head_3_link -->
 	<xacro:property name="def_head_cam_x" value="-0.181"/>

File: cob_hardware_config/robots/cob4-10/urdf/cob4-10.urdf.xacro (robot description, xacro)
@@ -23,4 +23,5 @@
   <xacro:include filename="$(find cob_description)/urdf/sensors/kinect.urdf.xacro" />
   <xacro:include filename="$(find cob_description)/urdf/sensors/usb_cam.urdf.xacro" />
+  <xacro:include filename="$(find cob_description)/urdf/sensors/sick_3dcs.urdf.xacro" />
   <xacro:include filename="$(find cob_description)/urdf/sensors/sick_s300_laser.urdf.xacro"/>
   <!-- composition of the robot -->
@@ -61,6 +62,9 @@
   </xacro:sensorring>
   <!-- cameras -->
-  <xacro:cob_kinect_v0 name="sensorring_cam3d" ros_topic="sensorring_cam3d" parent="sensorring_link" update_rate="30" data_skip="9">
-    <origin xyz="${sensorring_cam3d_x} ${sensorring_cam3d_y} ${sensorring_cam3d_z}" rpy="${sensorring_cam3d_roll} ${sensorring_cam3d_pitch} ${sensorring_cam3d_yaw}" />
+  <xacro:sick_3dcs name="sensorring_cam3d_front" ros_topic="sensorring_cam3d_front" parent="sensorring_link">
+    <origin xyz="${sensorring_cam3d_front_x} ${sensorring_cam3d_front_y} ${sensorring_cam3d_front_z}" rpy="${sensorring_cam3d_front_roll} ${sensorring_cam3d_front_pitch} ${sensorring_cam3d_front_yaw}" />
+  </xacro:sick_3dcs>
+  <xacro:cob_kinect_v0 name="sensorring_cam3d_back" ros_topic="sensorring_cam3d_back" parent="sensorring_link" update_rate="30" data_skip="9">
+    <origin xyz="${sensorring_cam3d_back_x} ${sensorring_cam3d_back_y} ${sensorring_cam3d_back_z}" rpy="${sensorring_cam3d_back_roll} ${sensorring_cam3d_back_pitch} ${sensorring_cam3d_back_yaw}" />
   </xacro:cob_kinect_v0>
   <xacro:cob4_arm name="arm_right" parent="torso_3_link" has_podest="false">

File: cob_hardware_config/robots/cob4-10/urdf/properties.urdf.xacro (robot description, xacro)
@@ -106,10 +106,17 @@
 	<xacro:property name="torso_cam3d_down_yaw" value="${def_torso_cam3d_down_yaw+offset_torso_cam3d_down_yaw}"/>
 	<!-- cam3d | handeye calibration | relative to sensorring_link -->
-	<xacro:property name="sensorring_cam3d_x" value="${def_sensorring_cam3d_x+offset_sensorring_cam3d_x}"/>
-	<xacro:property name="sensorring_cam3d_y" value="${def_sensorring_cam3d_y+offset_sensorring_cam3d_y}"/>
-	<xacro:property name="sensorring_cam3d_z" value="${def_sensorring_cam3d_z+offset_sensorring_cam3d_z}"/>
-	<xacro:property name="sensorring_cam3d_roll" value="${def_sensorring_cam3d_roll+offset_sensorring_cam3d_roll}"/>
-	<xacro:property name="sensorring_cam3d_pitch" value="${def_sensorring_cam3d_pitch+offset_sensorring_cam3d_pitch}"/>
-	<xacro:property name="sensorring_cam3d_yaw" value="${def_sensorring_cam3d_yaw+offset_sensorring_cam3d_yaw}"/>
+	<xacro:property name="sensorring_cam3d_front_x" value="${def_sensorring_cam3d_front_x+offset_sensorring_cam3d_front_x}"/>
+	<xacro:property name="sensorring_cam3d_front_y" value="${def_sensorring_cam3d_front_y+offset_sensorring_cam3d_front_y}"/>
+	<xacro:property name="sensorring_cam3d_front_z" value="${def_sensorring_cam3d_front_z+offset_sensorring_cam3d_front_z}"/>
+	<xacro:property name="sensorring_cam3d_front_roll" value="${def_sensorring_cam3d_front_roll+offset_sensorring_cam3d_front_roll}"/>
+	<xacro:property name="sensorring_cam3d_front_pitch" value="${def_sensorring_cam3d_front_pitch+offset_sensorring_cam3d_front_pitch}"/>
+	<xacro:property name="sensorring_cam3d_front_yaw" value="${def_sensorring_cam3d_front_yaw+offset_sensorring_cam3d_front_yaw}"/>
+	<!-- cam3d | handeye calibration | relative to sensorring_link -->
+	<xacro:property name="sensorring_cam3d_back_x" value="${def_sensorring_cam3d_back_x+offset_sensorring_cam3d_back_x}"/>
+	<xacro:property name="sensorring_cam3d_back_y" value="${def_sensorring_cam3d_back_y+offset_sensorring_cam3d_back_y}"/>
+	<xacro:property name="sensorring_cam3d_back_z" value="${def_sensorring_cam3d_back_z+offset_sensorring_cam3d_back_z}"/>
+	<xacro:property name="sensorring_cam3d_back_roll" value="${def_sensorring_cam3d_back_roll+offset_sensorring_cam3d_back_roll}"/>
+	<xacro:property name="sensorring_cam3d_back_pitch" value="${def_sensorring_cam3d_back_pitch+offset_sensorring_cam3d_back_pitch}"/>
+	<xacro:property name="sensorring_cam3d_back_yaw" value="${def_sensorring_cam3d_back_yaw+offset_sensorring_cam3d_back_yaw}"/>
 	<!-- cam | handeye calibration | relative to head_3_link -->
 	<xacro:property name="head_cam_x" value="${def_head_cam_x+offset_head_cam_x}"/>

Commit message: fix frames for usb_camera and sick_3dcs

File: cob_hardware_config/robots/cob4-10/urdf/calibration_default.urdf.xacro (robot description, xacro)
@@ -85,6 +85,6 @@
 	<xacro:property name="def_torso_cam3d_left_y" value="0.01802"/>
 	<xacro:property name="def_torso_cam3d_left_z" value="0.24214"/>
-	<xacro:property name="def_torso_cam3d_left_roll" value="0"/>
-	<xacro:property name="def_torso_cam3d_left_pitch" value="1.57079"/>
+	<xacro:property name="def_torso_cam3d_left_roll" value="1.57079"/>
+	<xacro:property name="def_torso_cam3d_left_pitch" value="0.0"/>
 	<xacro:property name="def_torso_cam3d_left_yaw" value="0.418879"/>
 	<!-- cam3d right | handeye calibration | relative to torso_3_link -->
@@ -92,6 +92,6 @@
 	<xacro:property name="def_torso_cam3d_right_y" value="-0.01802"/>
 	<xacro:property name="def_torso_cam3d_right_z" value="0.24214"/>
-	<xacro:property name="def_torso_cam3d_right_roll" value="0"/>
-	<xacro:property name="def_torso_cam3d_right_pitch" value="1.57079"/>
+	<xacro:property name="def_torso_cam3d_right_roll" value="1.57079"/>
+	<xacro:property name="def_torso_cam3d_right_pitch" value="0.0"/>
 	<xacro:property name="def_torso_cam3d_right_yaw" value="-0.418879"/>
 	<!-- cam3d down | handeye calibration | relative to torso_3_link -->
@@ -106,14 +106,14 @@
 	<xacro:property name="def_sensorring_cam3d_front_y" value="0.0"/>
 	<xacro:property name="def_sensorring_cam3d_front_z" value="0.0195"/>
-	<xacro:property name="def_sensorring_cam3d_front_roll" value="-1.95"/>
-	<xacro:property name="def_sensorring_cam3d_front_pitch" value="0.0"/>
-	<xacro:property name="def_sensorring_cam3d_front_yaw" value="-1.5708"/>
+	<xacro:property name="def_sensorring_cam3d_front_roll" value="3.14"/>
+	<xacro:property name="def_sensorring_cam3d_front_pitch" value="0.38"/>
+	<xacro:property name="def_sensorring_cam3d_front_yaw" value="0.0"/>
 	<!-- cam3d | handeye calibration | relative to sensorring_link -->
 	<xacro:property name="def_sensorring_cam3d_back_x" value="-0.096"/>
 	<xacro:property name="def_sensorring_cam3d_back_y" value="0.0"/>
 	<xacro:property name="def_sensorring_cam3d_back_z" value="0.0195"/>
-	<xacro:property name="def_sensorring_cam3d_back_roll" value="-1.5708"/>
+	<xacro:property name="def_sensorring_cam3d_back_roll" value="0.0"/>
 	<xacro:property name="def_sensorring_cam3d_back_pitch" value="0.0"/>
-	<xacro:property name="def_sensorring_cam3d_back_yaw" value="1.5708"/>
+	<xacro:property name="def_sensorring_cam3d_back_yaw" value="3.14"/>
 	<!-- cam | handeye calibration | relative to head_3_link -->
 	<xacro:property name="def_head_cam_x" value="-0.181"/>
@@ -122,4 +122,4 @@
 	<xacro:property name="def_head_cam_roll" value="0.0"/>
 	<xacro:property name="def_head_cam_pitch" value="-0.73"/>
-	<xacro:property name="def_head_cam_yaw" value="3.14"/>
+	<xacro:property name="def_head_cam_yaw" value="0.0"/>
 </robot>

File: cob_hardware_config/robots/cob4-7/urdf/calibration_default.urdf.xacro (robot description, xacro)
@@ -87,4 +87,4 @@
 	<xacro:property name="def_head_cam_roll" value="0.0"/>
 	<xacro:property name="def_head_cam_pitch" value="-0.73"/>
-	<xacro:property name="def_head_cam_yaw" value="3.14"/>
+	<xacro:property name="def_head_cam_yaw" value="0.0"/>
 </robot>

Commit message: fix head_cam mount position

File: cob_hardware_config/robots/cob4-10/urdf/calibration_default.urdf.xacro (robot description, xacro)
@@ -120,5 +120,5 @@
 	<xacro:property name="def_head_cam_y" value="0.0"/>
 	<xacro:property name="def_head_cam_z" value="0.325"/>
-	<xacro:property name="def_head_cam_roll" value="0.0"/>
+	<xacro:property name="def_head_cam_roll" value="-1.57079"/>
 	<xacro:property name="def_head_cam_pitch" value="-0.73"/>
 	<xacro:property name="def_head_cam_yaw" value="0.0"/>

File: cob_hardware_config/robots/cob4-2/urdf/calibration_default.urdf.xacro (robot description, xacro)
@@ -85,5 +85,5 @@
 	<xacro:property name="def_head_cam_y" value="0.0"/>
 	<xacro:property name="def_head_cam_z" value="0.325"/>
-	<xacro:property name="def_head_cam_roll" value="0.0"/>
+	<xacro:property name="def_head_cam_roll" value="-1.57079"/>
 	<xacro:property name="def_head_cam_pitch" value="-0.73"/>
 	<xacro:property name="def_head_cam_yaw" value="0.0"/>

File: cob_hardware_config/robots/cob4-8/urdf/calibration_default.urdf.xacro (robot description, xacro)
@@ -113,5 +113,5 @@
 	<xacro:property name="def_head_cam_y" value="0.0"/>
 	<xacro:property name="def_head_cam_z" value="0.325"/>
-	<xacro:property name="def_head_cam_roll" value="0.0"/>
+	<xacro:property name="def_head_cam_roll" value="-1.57079"/>
 	<xacro:property name="def_head_cam_pitch" value="-0.73"/>
 	<xacro:property name="def_head_cam_yaw" value="0.0"/>
