Commit message: cob4-13 config fixes

File: cob_hardware_config/robots/cob4-13/urdf/calibration_default.urdf.xacro (robot description, xacro)
@@ -11,5 +11,5 @@
 	<xacro:property name="def_laser_front_pitch" value="0.0"/>
 	<xacro:property name="def_laser_front_yaw" value="0.0"/>
-	<!-- laser rear mount positions | relative to base_link -->
+	<!-- laser left mount positions | relative to base_link -->
 	<xacro:property name="def_laser_left_x" value="-0.122"/>
 	<xacro:property name="def_laser_left_y" value="0.21131"/>
@@ -18,5 +18,5 @@
 	<xacro:property name="def_laser_left_pitch" value="0.0"/>
 	<xacro:property name="def_laser_left_yaw" value="2.094"/>
-	<!-- laser top mount positions | relative to base_link -->
+	<!-- laser right mount positions | relative to base_link -->
 	<xacro:property name="def_laser_right_x" value="-0.122"/>
 	<xacro:property name="def_laser_right_y" value="-0.21131"/>
@@ -105,9 +105,9 @@
 	<xacro:property name="def_torso_cam3d_down_pitch" value="0.61086"/>
 	<xacro:property name="def_torso_cam3d_down_yaw" value="0.0"/>
-	<!-- sensorring cam3d | handeye calibration | relative to sensorring_link -->
+	<!-- sensorring cam3d mount positions | relative to sensorring_link -->
 	<xacro:property name="def_sensorring_cam3d_x" value="0.096"/>
 	<xacro:property name="def_sensorring_cam3d_y" value="0.0"/>
 	<xacro:property name="def_sensorring_cam3d_z" value="0.0195"/>
-	<xacro:property name="def_sensorring_cam3d_roll" value="0.0"/>
+	<xacro:property name="def_sensorring_cam3d_roll" value="3.14159"/>
 	<xacro:property name="def_sensorring_cam3d_pitch" value="0.0"/>
 	<xacro:property name="def_sensorring_cam3d_yaw" value="0.0"/>

File: cob_hardware_config/robots/cob4-13/urdf/cob4-13.urdf.xacro (robot description, xacro)
@@ -12,7 +12,7 @@
   <xacro:include filename="$(find cob_description)/urdf/cob4_torso/torso.urdf.xacro" />
   <!-- arm -->
-  <xacro:include filename="$(find cob_description)/urdf/cob4_arm/cob4_arm.urdf.xacro" />
+  <!-- xacro:include filename="$(find cob_description)/urdf/cob4_arm/cob4_arm.urdf.xacro" /-->
   <!-- hand -->
-  <xacro:include filename="$(find cob_description)/urdf/cob4_gripper/gripper.urdf.xacro" />
+  <!-- xacro:include filename="$(find cob_description)/urdf/cob4_gripper/gripper.urdf.xacro" /-->
   <!-- head -->
   <xacro:include filename="$(find cob_description)/urdf/cob4_head/head.urdf.xacro" />
@@ -22,5 +22,4 @@
   <xacro:include filename="$(find cob_description)/urdf/sensors/realsense.urdf.xacro" />
   <xacro:include filename="$(find cob_description)/urdf/sensors/realsense_zr300.urdf.xacro" />
-  <xacro:include filename="$(find cob_description)/urdf/sensors/kinect.urdf.xacro" />
   <xacro:include filename="$(find cob_description)/urdf/sensors/usb_cam.urdf.xacro" />
   <xacro:include filename="$(find cob_description)/urdf/sensors/sick_s300_laser.urdf.xacro"/>
@@ -52,5 +51,5 @@
     <origin xyz="${torso_cam3d_down_x} ${torso_cam3d_down_y} ${torso_cam3d_down_z}" rpy="${torso_cam3d_down_roll} ${torso_cam3d_down_pitch} ${torso_cam3d_down_yaw}" />
   </xacro:realsense>
-  <xacro:head name="head" parent="torso_3_link" dof1="true" dof2="true" dof3="true">
+  <xacro:head name="head" parent="torso_3_link" dof1="false" dof2="false" dof3="false">
     <origin xyz="${head_x} ${head_y} ${head_z}" rpy="${head_roll} ${head_pitch} ${head_yaw}" />
   </xacro:head>
@@ -61,19 +60,6 @@
     <origin xyz="${sensorring_x} ${sensorring_y} ${sensorring_z}" rpy="${sensorring_roll} ${sensorring_pitch} ${sensorring_yaw}" />
   </xacro:sensorring>
-  <!-- cameras -->
-  <xacro:cob_kinect_v0 name="sensorring_cam3d" ros_topic="sensorring_cam3d" parent="sensorring_link" update_rate="30" data_skip="9">
+  <xacro:realsense_zr300 name="sensorring_cam3d" ros_topic="sensorring_cam3d" parent="sensorring_link">
     <origin xyz="${sensorring_cam3d_x} ${sensorring_cam3d_y} ${sensorring_cam3d_z}" rpy="${sensorring_cam3d_roll} ${sensorring_cam3d_pitch} ${sensorring_cam3d_yaw}" />
-  </xacro:cob_kinect_v0>
-  <xacro:cob4_arm name="arm_right" parent="torso_3_link" has_podest="false">
-    <origin xyz="${arm_right_x} ${arm_right_y} ${arm_right_z}" rpy="${arm_right_roll} ${arm_right_pitch} ${arm_right_yaw}" />
-  </xacro:cob4_arm>
-  <xacro:cob4_arm name="arm_left" parent="torso_3_link" has_podest="false">
-    <origin xyz="${arm_left_x} ${arm_left_y} ${arm_left_z}" rpy="${arm_left_roll} ${arm_left_pitch} ${arm_left_yaw}" />
-  </xacro:cob4_arm>
-  <!--xacro:gripper name="gripper_right" parent="arm_right_7_link">
-    <origin xyz="${gripper_right_x} ${gripper_right_y} ${gripper_right_z}" rpy="${gripper_right_roll} ${gripper_right_pitch} ${gripper_right_yaw}" />
-  </xacro:gripper>
-  <xacro:gripper name="gripper_left" parent="arm_left_7_link">
-    <origin xyz="${gripper_left_x} ${gripper_left_y} ${gripper_left_z}" rpy="${gripper_left_roll} ${gripper_left_pitch} ${gripper_left_yaw}" />
-  </xacro:gripper-->
+  </xacro:realsense_zr300>
 </robot>

File: cob_hardware_config/robots/cob4-13/urdf/properties.urdf.xacro (robot description, xacro)
@@ -14,5 +14,5 @@
 	<xacro:property name="laser_front_pitch" value="${def_laser_front_pitch+offset_laser_front_pitch}"/>
 	<xacro:property name="laser_front_yaw" value="${def_laser_front_yaw+offset_laser_front_yaw}"/>
-	<!-- laser rear mount positions | relative to base_link -->
+	<!-- laser left mount positions | relative to base_link -->
 	<xacro:property name="laser_left_x" value="${def_laser_left_x+offset_laser_left_x}"/>
 	<xacro:property name="laser_left_y" value="${def_laser_left_y+offset_laser_left_y}"/>
@@ -21,5 +21,5 @@
 	<xacro:property name="laser_left_pitch" value="${def_laser_left_pitch+offset_laser_left_pitch}"/>
 	<xacro:property name="laser_left_yaw" value="${def_laser_left_yaw+offset_laser_left_yaw}"/>
-	<!-- laser top mount positions | relative to base_link -->
+	<!-- laser right mount positions | relative to base_link -->
 	<xacro:property name="laser_right_x" value="${def_laser_right_x+offset_laser_right_x}"/>
 	<xacro:property name="laser_right_y" value="${def_laser_right_y+offset_laser_right_y}"/>
@@ -45,5 +45,5 @@
 	<xacro:property name="head_pitch" value="${def_head_pitch+offset_head_pitch}"/>
 	<xacro:property name="head_yaw" value="${def_head_yaw+offset_head_yaw}"/>
-	<!-- head sensors mount positions | relative to head_3_link -->
+	<!-- sensorring mount positions | relative to head_3_link -->
 	<xacro:property name="sensorring_x" value="${def_sensorring_x+offset_sensorring_x}"/>
 	<xacro:property name="sensorring_y" value="${def_sensorring_y+offset_sensorring_y}"/>
@@ -80,9 +80,8 @@
 	<xacro:property name="gripper_left_pitch" value="${def_gripper_left_pitch+offset_gripper_left_pitch}"/>
 	<xacro:property name="gripper_left_yaw" value="${def_gripper_left_yaw+offset_gripper_left_yaw}"/>
-	<!-- *********************************** -->
-	<!-- kinematic chain reference positions -->
-	<!-- *********************************** -->
-	<!-- this feature is no longer supported as urdfdom does not parse the according 'calibration_rising' tag -->
-	<!-- cam3d left | handeye calibration | relative to torso_3_link -->
+	<!-- ***************************** -->
+	<!-- extrinsic camera calibration  -->
+	<!-- ***************************** -->
+	<!-- torso cam3d left mount positions | relative to torso_3_link -->
 	<xacro:property name="torso_cam3d_left_x" value="${def_torso_cam3d_left_x+offset_torso_cam3d_left_x}"/>
 	<xacro:property name="torso_cam3d_left_y" value="${def_torso_cam3d_left_y+offset_torso_cam3d_left_y}"/>
@@ -91,5 +90,5 @@
 	<xacro:property name="torso_cam3d_left_pitch" value="${def_torso_cam3d_left_pitch+offset_torso_cam3d_left_pitch}"/>
 	<xacro:property name="torso_cam3d_left_yaw" value="${def_torso_cam3d_left_yaw+offset_torso_cam3d_left_yaw}"/>
-	<!-- cam3d right | handeye calibration | relative to torso_3_link -->
+	<!-- torso cam3d right mount positions | relative to torso_3_link -->
 	<xacro:property name="torso_cam3d_right_x" value="${def_torso_cam3d_right_x+offset_torso_cam3d_right_x}"/>
 	<xacro:property name="torso_cam3d_right_y" value="${def_torso_cam3d_right_y+offset_torso_cam3d_right_y}"/>
@@ -98,5 +97,5 @@
 	<xacro:property name="torso_cam3d_right_pitch" value="${def_torso_cam3d_right_pitch+offset_torso_cam3d_right_pitch}"/>
 	<xacro:property name="torso_cam3d_right_yaw" value="${def_torso_cam3d_right_yaw+offset_torso_cam3d_right_yaw}"/>
-	<!-- cam3d down | handeye calibration | relative to torso_3_link -->
+	<!-- torso cam3d down mount positions | relative to torso_3_link -->
 	<xacro:property name="torso_cam3d_down_x" value="${def_torso_cam3d_down_x+offset_torso_cam3d_down_x}"/>
 	<xacro:property name="torso_cam3d_down_y" value="${def_torso_cam3d_down_y+offset_torso_cam3d_down_y}"/>
@@ -105,5 +104,5 @@
 	<xacro:property name="torso_cam3d_down_pitch" value="${def_torso_cam3d_down_pitch+offset_torso_cam3d_down_pitch}"/>
 	<xacro:property name="torso_cam3d_down_yaw" value="${def_torso_cam3d_down_yaw+offset_torso_cam3d_down_yaw}"/>
-	<!-- cam3d | handeye calibration | relative to sensorring_link -->
+	<!-- sensorring cam3d mount positions | relative to sensorring_link -->
 	<xacro:property name="sensorring_cam3d_x" value="${def_sensorring_cam3d_x+offset_sensorring_cam3d_x}"/>
 	<xacro:property name="sensorring_cam3d_y" value="${def_sensorring_cam3d_y+offset_sensorring_cam3d_y}"/>
@@ -112,5 +111,5 @@
 	<xacro:property name="sensorring_cam3d_pitch" value="${def_sensorring_cam3d_pitch+offset_sensorring_cam3d_pitch}"/>
 	<xacro:property name="sensorring_cam3d_yaw" value="${def_sensorring_cam3d_yaw+offset_sensorring_cam3d_yaw}"/>
-	<!-- cam | handeye calibration | relative to head_3_link -->
+	<!-- head cam mount positions | relative to head_3_link -->
 	<xacro:property name="head_cam_x" value="${def_head_cam_x+offset_head_cam_x}"/>
 	<xacro:property name="head_cam_y" value="${def_head_cam_y+offset_head_cam_y}"/>
