Commit message: Changed height of laser scanner for raw3-3.

File: cob_hardware_config/robots/raw3-3/urdf/calibration_default.urdf.xacro (robot description, xacro)
@@ -7,5 +7,5 @@
 	<xacro:property name="def_laser_front_x" value="0.32501"/>
 	<xacro:property name="def_laser_front_y" value="-0.232"/>
-	<xacro:property name="def_laser_front_z" value="0.178"/>
+	<xacro:property name="def_laser_front_z" value="0.188"/>
 	<xacro:property name="def_laser_front_roll" value="${M_PI}"/>
 	<xacro:property name="def_laser_front_pitch" value="0.0"/>
@@ -14,5 +14,5 @@
 	<xacro:property name="def_laser_rear_x" value="-0.32501"/>
 	<xacro:property name="def_laser_rear_y" value="0.232"/>
-	<xacro:property name="def_laser_rear_z" value="0.178"/>
+	<xacro:property name="def_laser_rear_z" value="0.188"/>
 	<xacro:property name="def_laser_rear_roll" value="${M_PI}"/>
 	<xacro:property name="def_laser_rear_pitch" value="0.0"/>
