Commit message: remove unavailable components

File: cob_hardware_config/robots/raw3-1/urdf/raw3-1.urdf.xacro (robot description, xacro)
@@ -12,6 +12,4 @@
   <!-- torso -->
   <xacro:include filename="$(find raw_description)/urdf/torso/torso.urdf.xacro" />
-  <!-- head -->
-  <xacro:include filename="$(find raw_description)/urdf/head/head.urdf.xacro" />
   <!-- ur_arm -->
   <xacro:include filename="$(find raw_description)/urdf/ur_arm/ur10_arm.urdf.xacro" />
@@ -36,12 +34,9 @@
     <origin xyz="${torso_x} ${torso_y} ${torso_z}" rpy="${torso_roll} ${torso_pitch} ${torso_yaw}" />
   </xacro:raw_torso>
-  <xacro:raw_head name="head" parent="torso_2_link">
-    <origin xyz="${head_x} ${head_y} ${head_z}" rpy="${head_roll} ${head_pitch} ${head_yaw}" />
-  </xacro:raw_head>
-  <xacro:ur10 name="arm" parent="base_link">
+  <!--xacro:ur10 name="arm" parent="base_link">
     <origin xyz="${arm_x} ${arm_y} ${arm_z}" rpy="${arm_roll} ${arm_pitch} ${arm_yaw}" />
-  </xacro:ur10>
-  <xacro:vacuum_gripper name="gripper" parent="arm_ee_link">
+  </xacro:ur10-->
+  <!--xacro:vacuum_gripper name="gripper" parent="arm_ee_link">
     <origin xyz="${gripper_x} ${gripper_y} ${gripper_z}" rpy="${gripper_roll} ${gripper_pitch} ${gripper_yaw}" />
-  </xacro:vacuum_gripper>
+  </xacro:vacuum_gripper-->
 </robot>

Commit message: add schmaltz gripper

File: cob_hardware_config/robots/raw3-1/urdf/raw3-1.urdf.xacro (robot description, xacro)
@@ -14,6 +14,8 @@
   <!-- ur_arm -->
   <xacro:include filename="$(find raw_description)/urdf/ur_arm/ur10_arm.urdf.xacro" />
-  <!-- vacuum gripper -->
-  <xacro:include filename="$(find raw_description)/urdf/vacuum_gripper/gripper.urdf.xacro" />
+  <!-- schmaltz vacuum gripper -->
+  <xacro:include filename="$(find raw_description)/urdf/schmaltz_gripper/gripper.urdf.xacro" />
+  <!-- arm camera -->
+  <xacro:include filename="$(find raw_description)/urdf/arm_camera/arm_camera.urdf.xacro" />
   <!-- sensors -->
   <xacro:include filename="$(find cob_description)/urdf/sensors/sick_s300_laser.urdf.xacro"/>
@@ -40,3 +42,6 @@
     <origin xyz="${gripper_x} ${gripper_y} ${gripper_z}" rpy="${gripper_roll} ${gripper_pitch} ${gripper_yaw}" />
   </xacro:vacuum_gripper>
+  <xacro:arm_camera name="arm_camera" parent="gripper_coupling_link">
+    <origin xyz="${arm_camera_x} ${arm_camera_y} ${arm_camera_z}" rpy="${arm_camera_roll} ${arm_camera_pitch} ${arm_camera_yaw}" />
+  </xacro:arm_camera>
 </robot>
