Commit message: corrected torso definition

File: cob_hardware_config/robots/raw3-1/urdf/calibration_default.urdf.xacro (robot description, xacro)
@@ -28,11 +28,11 @@
 	<xacro:property name="def_tower_pitch" value="0.0"/>
 	<xacro:property name="def_tower_yaw" value="3.14159265359"/>
-	<!--torso mount positions | relative to base_link-->
-	<xacro:property name="def_torso_x" value="0.166"/>
-	<xacro:property name="def_torso_y" value="0.2175"/>
-	<xacro:property name="def_torso_z" value="0.5405"/>
+	<!--torso mount positions (torso_0_link) | relative to base_link-->
+	<xacro:property name="def_torso_x" value="0.166"/> #0.100
+	<xacro:property name="def_torso_y" value="0.2175"/> #0.2425
+	<xacro:property name="def_torso_z" value="0.302"/> #0.59
 	<xacro:property name="def_torso_roll" value="0.0"/>
 	<xacro:property name="def_torso_pitch" value="0.0"/>
-	<xacro:property name="def_torso_yaw" value="0.0"/>
+	<xacro:property name="def_torso_yaw" value="1.57079632679"/>
 	<!-- head mount positions | relative to head_cover_link -->
 	<xacro:property name="def_head_x" value="0.0"/>

Commit message: corrected torso definition

File: cob_hardware_config/robots/raw3-1/urdf/calibration_default.urdf.xacro (robot description, xacro)
@@ -29,7 +29,7 @@
 	<xacro:property name="def_tower_yaw" value="3.14159265359"/>
 	<!--torso mount positions | relative to base_link-->
-	<xacro:property name="def_torso_x" value="0.100"/>
-	<xacro:property name="def_torso_y" value="0.2425"/>
-	<xacro:property name="def_torso_z" value="0.57"/>
+	<xacro:property name="def_torso_x" value="0.166"/>
+	<xacro:property name="def_torso_y" value="0.2175"/>
+	<xacro:property name="def_torso_z" value="0.302"/>
 	<xacro:property name="def_torso_roll" value="0.0"/>
 	<xacro:property name="def_torso_pitch" value="0.0"/>

Commit message: Updated stuff for raw3-1 and ipp.

File: cob_hardware_config/robots/raw3-1/urdf/calibration_default.urdf.xacro (robot description, xacro)
@@ -7,5 +7,5 @@
 	<xacro:property name="def_laser_front_x" value="0.465"/>
 	<xacro:property name="def_laser_front_y" value="-0.232"/>
-	<xacro:property name="def_laser_front_z" value="0.178"/>
+	<xacro:property name="def_laser_front_z" value="0.188"/>
 	<xacro:property name="def_laser_front_roll" value="${M_PI}"/>
 	<xacro:property name="def_laser_front_pitch" value="0.0"/>
@@ -14,5 +14,5 @@
 	<xacro:property name="def_laser_rear_x" value="-0.465"/>
 	<xacro:property name="def_laser_rear_y" value="0.232"/>
-	<xacro:property name="def_laser_rear_z" value="0.178"/>
+	<xacro:property name="def_laser_rear_z" value="0.188"/>
 	<xacro:property name="def_laser_rear_roll" value="${M_PI}"/>
 	<xacro:property name="def_laser_rear_pitch" value="0.0"/>

File: cob_hardware_config/robots/raw3-1/urdf/raw3-1.urdf.xacro (robot description, xacro)
@@ -28,15 +28,15 @@
     <origin xyz="${laser_rear_x} ${laser_rear_y} ${laser_rear_z}" rpy="${laser_rear_roll} ${laser_rear_pitch} ${laser_rear_yaw}" />
   </xacro:sick_s300_laser_v0>
-  <xacro:tower_asymetric name="tower" parent="base_link">
-    <origin xyz="${tower_x} ${tower_y} ${tower_z}" rpy="${tower_roll} ${tower_pitch} ${tower_yaw}" />
-  </xacro:tower_asymetric>
-  <xacro:raw_torso_v2 name="torso" parent="base_link">
-    <origin xyz="${torso_x} ${torso_y} ${torso_z}" rpy="${torso_roll} ${torso_pitch} ${torso_yaw}" />
-  </xacro:raw_torso_v2>
-  <xacro:ur10 name="arm" parent="base_link">
-    <origin xyz="${arm_x} ${arm_y} ${arm_z}" rpy="${arm_roll} ${arm_pitch} ${arm_yaw}" />
-  </xacro:ur10>
-  <xacro:vacuum_gripper name="gripper" parent="arm_ee_link">
-    <origin xyz="${gripper_x} ${gripper_y} ${gripper_z}" rpy="${gripper_roll} ${gripper_pitch} ${gripper_yaw}" />
-  </xacro:vacuum_gripper>
+  <!--<xacro:tower_asymetric name="tower" parent="base_link">-->
+    <!--<origin xyz="${tower_x} ${tower_y} ${tower_z}" rpy="${tower_roll} ${tower_pitch} ${tower_yaw}" />-->
+  <!--</xacro:tower_asymetric>-->
+  <!--<xacro:raw_torso_v2 name="torso" parent="base_link">-->
+    <!--<origin xyz="${torso_x} ${torso_y} ${torso_z}" rpy="${torso_roll} ${torso_pitch} ${torso_yaw}" />-->
+  <!--</xacro:raw_torso_v2>-->
+  <!--<xacro:ur10 name="arm" parent="base_link">-->
+    <!--<origin xyz="${arm_x} ${arm_y} ${arm_z}" rpy="${arm_roll} ${arm_pitch} ${arm_yaw}" />-->
+  <!--</xacro:ur10>-->
+  <!--<xacro:vacuum_gripper name="gripper" parent="arm_ee_link">-->
+    <!--<origin xyz="${gripper_x} ${gripper_y} ${gripper_z}" rpy="${gripper_roll} ${gripper_pitch} ${gripper_yaw}" />-->
+  <!--</xacro:vacuum_gripper>-->
 </robot>

Commit message: add kinematic camera plugin

File: cob_hardware_config/robots/raw3-1/urdf/calibration_default.urdf.xacro (robot description, xacro)
@@ -88,9 +88,9 @@
 	<xacro:property name="def_cam3d_yaw" value="0.0"/>
         <!-- arm camera | handeye calibration | relative to cam_reference_link -->
-        <xacro:property name="def_arm_camera_x" value="0.00"/>
+        <xacro:property name="def_arm_camera_x" value="0.083"/>
         <xacro:property name="def_arm_camera_y" value="0.0"/>
         <xacro:property name="def_arm_camera_z" value="0.0"/>
         <xacro:property name="def_arm_camera_roll" value="0.0"/>
-        <xacro:property name="def_arm_camera_pitch" value="0.0"/>
-        <xacro:property name="def_arm_camera_yaw" value="0.0"/>
+        <xacro:property name="def_arm_camera_pitch" value="-1.57"/>
+        <xacro:property name="def_arm_camera_yaw" value="-3.1415"/>
 </robot>

File: cob_hardware_config/robots/raw3-1/urdf/raw3-1.urdf.xacro (robot description, xacro)
@@ -17,5 +17,5 @@
   <xacro:include filename="$(find raw_description)/urdf/schmaltz_gripper/gripper.urdf.xacro" />
   <!-- arm camera -->
-  <xacro:include filename="$(find raw_description)/urdf/arm_camera/arm_camera.urdf.xacro" />
+  <xacro:include filename="$(find raw_description)/urdf/kinect_camera/kinect_camera.urdf.xacro" />
   <!-- sensors -->
   <xacro:include filename="$(find cob_description)/urdf/sensors/sick_s300_laser.urdf.xacro"/>
@@ -42,6 +42,6 @@
     <origin xyz="${gripper_x} ${gripper_y} ${gripper_z}" rpy="${gripper_roll} ${gripper_pitch} ${gripper_yaw}" />
   </xacro:vacuum_gripper>
-  <xacro:arm_camera name="arm_camera" parent="gripper_coupling_link">
+  <xacro:kinect_camera name="arm_camera" ros_topic="arm_kinect_camera" parent="gripper_coupling_link" update_rate="30" data_skip="9">
     <origin xyz="${arm_camera_x} ${arm_camera_y} ${arm_camera_z}" rpy="${arm_camera_roll} ${arm_camera_pitch} ${arm_camera_yaw}" />
-  </xacro:arm_camera>
+  </xacro:kinect_camera>
 </robot>

Commit message: Removed personal changes,

File: cob_hardware_config/robots/raw3-1/urdf/calibration_default.urdf.xacro (robot description, xacro)
@@ -7,5 +7,5 @@
 	<xacro:property name="def_laser_front_x" value="0.465"/>
 	<xacro:property name="def_laser_front_y" value="-0.232"/>
-	<xacro:property name="def_laser_front_z" value="0.188"/>
+	<xacro:property name="def_laser_front_z" value="0.178"/>
 	<xacro:property name="def_laser_front_roll" value="${M_PI}"/>
 	<xacro:property name="def_laser_front_pitch" value="0.0"/>
@@ -14,5 +14,5 @@
 	<xacro:property name="def_laser_rear_x" value="-0.465"/>
 	<xacro:property name="def_laser_rear_y" value="0.232"/>
-	<xacro:property name="def_laser_rear_z" value="0.188"/>
+	<xacro:property name="def_laser_rear_z" value="0.178"/>
 	<xacro:property name="def_laser_rear_roll" value="${M_PI}"/>
 	<xacro:property name="def_laser_rear_pitch" value="0.0"/>

File: cob_hardware_config/robots/raw3-1/urdf/raw3-1.urdf.xacro (robot description, xacro)
@@ -28,15 +28,15 @@
     <origin xyz="${laser_rear_x} ${laser_rear_y} ${laser_rear_z}" rpy="${laser_rear_roll} ${laser_rear_pitch} ${laser_rear_yaw}" />
   </xacro:sick_s300_laser_v0>
-  <!--<xacro:tower_asymetric name="tower" parent="base_link">-->
-    <!--<origin xyz="${tower_x} ${tower_y} ${tower_z}" rpy="${tower_roll} ${tower_pitch} ${tower_yaw}" />-->
-  <!--</xacro:tower_asymetric>-->
-  <!--<xacro:raw_torso_v2 name="torso" parent="base_link">-->
-    <!--<origin xyz="${torso_x} ${torso_y} ${torso_z}" rpy="${torso_roll} ${torso_pitch} ${torso_yaw}" />-->
-  <!--</xacro:raw_torso_v2>-->
-  <!--<xacro:ur10 name="arm" parent="base_link">-->
-    <!--<origin xyz="${arm_x} ${arm_y} ${arm_z}" rpy="${arm_roll} ${arm_pitch} ${arm_yaw}" />-->
-  <!--</xacro:ur10>-->
-  <!--<xacro:vacuum_gripper name="gripper" parent="arm_ee_link">-->
-    <!--<origin xyz="${gripper_x} ${gripper_y} ${gripper_z}" rpy="${gripper_roll} ${gripper_pitch} ${gripper_yaw}" />-->
-  <!--</xacro:vacuum_gripper>-->
+  <xacro:tower_asymetric name="tower" parent="base_link">
+    <origin xyz="${tower_x} ${tower_y} ${tower_z}" rpy="${tower_roll} ${tower_pitch} ${tower_yaw}" />
+  </xacro:tower_asymetric>
+  <xacro:raw_torso_v2 name="torso" parent="base_link">
+    <origin xyz="${torso_x} ${torso_y} ${torso_z}" rpy="${torso_roll} ${torso_pitch} ${torso_yaw}" />
+  </xacro:raw_torso_v2>
+  <xacro:ur10 name="arm" parent="base_link">
+    <origin xyz="${arm_x} ${arm_y} ${arm_z}" rpy="${arm_roll} ${arm_pitch} ${arm_yaw}" />
+  </xacro:ur10>
+  <xacro:vacuum_gripper name="gripper" parent="arm_ee_link">
+    <origin xyz="${gripper_x} ${gripper_y} ${gripper_z}" rpy="${gripper_roll} ${gripper_pitch} ${gripper_yaw}" />
+  </xacro:vacuum_gripper>
 </robot>

File: cob_hardware_config/robots/raw3-3/urdf/calibration_default.urdf.xacro (robot description, xacro)
@@ -7,5 +7,5 @@
 	<xacro:property name="def_laser_front_x" value="0.32501"/>
 	<xacro:property name="def_laser_front_y" value="-0.232"/>
-	<xacro:property name="def_laser_front_z" value="0.188"/>
+	<xacro:property name="def_laser_front_z" value="0.178"/>
 	<xacro:property name="def_laser_front_roll" value="${M_PI}"/>
 	<xacro:property name="def_laser_front_pitch" value="0.0"/>
@@ -14,5 +14,5 @@
 	<xacro:property name="def_laser_rear_x" value="-0.32501"/>
 	<xacro:property name="def_laser_rear_y" value="0.232"/>
-	<xacro:property name="def_laser_rear_z" value="0.188"/>
+	<xacro:property name="def_laser_rear_z" value="0.178"/>
 	<xacro:property name="def_laser_rear_roll" value="${M_PI}"/>
 	<xacro:property name="def_laser_rear_pitch" value="0.0"/>
