Commit message: adjusted laser height

File: cob_hardware_config/robots/raw4-1/urdf/calibration_default.urdf.xacro (robot description, xacro)
@@ -7,5 +7,5 @@
 	<xacro:property name="def_laser_front_x" value="0.5075"/>
 	<xacro:property name="def_laser_front_y" value="0.240"/>
-	<xacro:property name="def_laser_front_z" value="0.10"/> <!-- 0,05 from ground to bottom of scan-->
+	<xacro:property name="def_laser_front_z" value="0.093"/> <!-- 0,0529 from ground to bottom of scan-->
 	<xacro:property name="def_laser_front_roll" value="${M_PI}"/>
 	<xacro:property name="def_laser_front_pitch" value="0.0"/>
@@ -14,5 +14,5 @@
 	<xacro:property name="def_laser_rear_x" value="-0.5075"/>
 	<xacro:property name="def_laser_rear_y" value="-0.240"/>
-	<xacro:property name="def_laser_rear_z" value="0.10"/>
+	<xacro:property name="def_laser_rear_z" value="0.093"/>
 	<xacro:property name="def_laser_rear_roll" value="${M_PI}"/>
 	<xacro:property name="def_laser_rear_pitch" value="0.0"/>
