Commit message: Modified files for raw-mini

File: cob_hardware_config/robots/raw-mini/urdf/properties.urdf.xacro (robot description, xacro)
@@ -1,15 +1,13 @@
 <?xml version="1.0"?>
 <robot xmlns:xacro="http://www.ros.org/wiki/xacro">
-	<xacro:include filename="$(find cob_hardware_config)/robots/raw-mini/urdf/calibration_default.urdf.xacro" />
-	<xacro:include filename="$(find cob_calibration_data)/raw-mini/calibration/calibration_offset.urdf.xacro" />>
 	<!-- ***************** -->
 	<!-- base calibration -->
 	<!-- ***************** -->
 	<!-- laser front mount positions | relative to base_link -->
-	<xacro:property name="laser_front_x" value="${def_laser_front_x+offset_laser_front_x}"/>
-	<xacro:property name="laser_front_y" value="${def_laser_front_y+offset_laser_front_y}"/>
-	<xacro:property name="laser_front_z" value="${def_laser_front_z+offset_laser_front_z}"/>
-	<xacro:property name="laser_front_roll" value="${def_laser_front_roll+offset_laser_front_roll}"/>
-	<xacro:property name="laser_front_pitch" value="${def_laser_front_pitch+offset_laser_front_pitch}"/>
-	<xacro:property name="laser_front_yaw" value="${def_laser_front_yaw+offset_laser_front_yaw}"/>
+	<xacro:property name="laser_front_x" value="-0.1"/>
+	<xacro:property name="laser_front_y" value="0.0"/>
+	<xacro:property name="laser_front_z" value="0.05"/>
+	<xacro:property name="laser_front_roll" value="0.0"/>
+	<xacro:property name="laser_front_pitch" value="0.0"/>
+	<xacro:property name="laser_front_yaw" value="0.0"/>
 </robot>

File: cob_hardware_config/robots/raw-mini/urdf/raw-mini.urdf.xacro (robot description, xacro)
@@ -2,3 +2,17 @@
 <robot xmlns:xacro="http://www.ros.org/wiki/xacro"
        name="raw-mini" >
+  <!-- common stuff -->
+  <xacro:include filename="$(find cob_description)/urdf/common.xacro" />
+  <xacro:include filename="$(find cob_description)/urdf/materials.urdf.xacro" />
+  <xacro:include filename="$(find cob_hardware_config)/robots/raw-mini/urdf/properties.urdf.xacro" />
+  <!-- raw base -->
+  <xacro:include filename="$(find raw_description)/urdf/base-mini/base.urdf.xacro" />
+  <!-- sensors -->
+  <xacro:include filename="$(find cob_description)/urdf/sensors/rplidar.urdf.xacro"/>
+  <!-- composition of the robot -->
+  <xacro:raw_base name="base"/>
+  <!-- base laser front -->
+  <xacro:sick_s300_laser_v0 name="base_laser" parent="base">
+    <origin xyz="${laser_front_x} ${laser_front_y} ${laser_front_z}" rpy="${laser_front_roll} ${laser_front_pitch} ${laser_front_yaw}" />
+  </xacro:sick_s300_laser_v0>
 </robot>

Commit message: Fixed bugs

File: cob_hardware_config/robots/raw-mini/urdf/properties.urdf.xacro (robot description, xacro)
@@ -7,5 +7,5 @@
 	<xacro:property name="laser_front_x" value="-0.1"/>
 	<xacro:property name="laser_front_y" value="0.0"/>
-	<xacro:property name="laser_front_z" value="0.05"/>
+	<xacro:property name="laser_front_z" value="0.15"/>
 	<xacro:property name="laser_front_roll" value="0.0"/>
 	<xacro:property name="laser_front_pitch" value="0.0"/>

File: cob_hardware_config/robots/raw-mini/urdf/raw-mini.urdf.xacro (robot description, xacro)
@@ -7,5 +7,5 @@
   <xacro:include filename="$(find cob_hardware_config)/robots/raw-mini/urdf/properties.urdf.xacro" />
   <!-- raw base -->
-  <xacro:include filename="$(find raw_description)/urdf/base-mini/base.urdf.xacro" />
+  <xacro:include filename="$(find raw_description)/urdf/base_mini/base.urdf.xacro" />
   <!-- sensors -->
   <xacro:include filename="$(find cob_description)/urdf/sensors/rplidar.urdf.xacro"/>
@@ -13,6 +13,6 @@
   <xacro:raw_base name="base"/>
   <!-- base laser front -->
-  <xacro:sick_s300_laser_v0 name="base_laser" parent="base">
+  <xacro:rplidar name="base_laser" parent="base">
     <origin xyz="${laser_front_x} ${laser_front_y} ${laser_front_z}" rpy="${laser_front_roll} ${laser_front_pitch} ${laser_front_yaw}" />
-  </xacro:sick_s300_laser_v0>
+  </xacro:rplidar>
 </robot>

Commit message: fixed laser height

File: cob_hardware_config/robots/raw-mini/urdf/properties.urdf.xacro (robot description, xacro)
@@ -7,5 +7,5 @@
 	<xacro:property name="laser_front_x" value="-0.1"/>
 	<xacro:property name="laser_front_y" value="0.0"/>
-	<xacro:property name="laser_front_z" value="0.15"/>
+	<xacro:property name="laser_front_z" value="0.11"/>
 	<xacro:property name="laser_front_roll" value="0.0"/>
 	<xacro:property name="laser_front_pitch" value="0.0"/>
