Commit message: 添加kfr分支仿真文件

File: cob_hardware_config/robots/cob4-3/urdf/cob4-3.urdf.xacro (robot description, xacro)
@@ -1,13 +1,404 @@
-<?xml version="1.0"?>
-<robot xmlns:xacro="http://www.ros.org/wiki/xacro"
-       name="cob4-3" >
-  <!-- common stuff -->
-  <xacro:include filename="$(find cob_description)/urdf/common.xacro" />
-  <xacro:include filename="$(find cob_description)/urdf/materials.urdf.xacro" />
-  <!-- calibration -->
-  <xacro:include filename="$(find cob_hardware_config)/robots/cob4-3/urdf/properties.urdf.xacro" />
-  <!-- base -->
-  <xacro:include filename="$(find cob_description)/urdf/cob4_base/base.urdf.xacro" />
-  <!-- composition of the robot -->
-  <xacro:base name="base"/>
+<?xml version="1.0" ?>
+<!-- =================================================================================== -->
+<!-- |    This document was autogenerated by xacro from cob4-3.urdf.xacro              | -->
+<!-- |    EDITING THIS FILE BY HAND IS NOT RECOMMENDED                                 | -->
+<!-- =================================================================================== -->
+<robot name="cob4-3" xmlns:xacro="http://www.ros.org/wiki/xacro">
+  <material name="IPA/LightGrey">
+    <color rgba="0.7 0.7 0.7 1.0"/>
+  </material>
+  <material name="IPA/DarkGrey">
+    <color rgba="0.4 0.4 0.4 1.0"/>
+  </material>
+  <material name="IPA/Black">
+    <color rgba="0.0 0.0 0.0 1.0"/>
+  </material>
+  <material name="IPA/Metall">
+    <color rgba="0.7 0.7 0.7 1.0"/>
+  </material>
+  <material name="IPA/YellowRubber">
+    <color rgba="0.4 0.27 0.16 1.0"/>
+  </material>
+  <material name="IPA/Orange">
+    <color rgba="1.0 0.4 0.0 1.0"/>
+  </material>
+  <material name="IPA/Blue">
+    <color rgba="0.0 0.0 0.5 1.0"/>
+  </material>
+  <link name="base_footprint"/>
+  <joint name="base_footprint_joint" type="fixed">
+    <origin rpy="0 0 0" xyz="0 0 0"/>
+    <parent link="base_footprint"/>
+    <child link="base_link"/>
+  </joint>
+  <link name="base_link">
+    <inertial>
+      <origin xyz="0 0 0"/>
+      <mass value="100"/>
+      <inertia ixx="5.652232699207" ixy="-0.009719934438" ixz="1.293988226423" iyy="5.669473158652" iyz="-0.007379583694" izz="3.683196351726"/>
+    </inertial>
+    <visual>
+      <origin rpy="0 0 0" xyz="0 0 0"/>
+      <geometry>
+        <mesh filename="package://cob_description/meshes/cob4_base/base.dae"/>
+        <!--box size="0.01 0.01 0.01" /-->
+      </geometry>
+    </visual>
+    <collision>
+      <origin rpy="0 0 0" xyz="0 0 0"/>
+      <geometry>
+        <mesh filename="package://cob_description/meshes/cob4_base/base_collision.stl"/>
+        <!--box size="0.01 0.01 0.01" /-->
+      </geometry>
+    </collision>
+  </link>
+<!--________________________________________________________________________________________-->
+  <joint name="fl_caster_rotation_joint" type="continuous">
+    <origin rpy="0 0 0" xyz="0.12422 0.21515 0.08"/>
+    <parent link="base_link"/>
+    <child link="fl_caster_rotation_link"/>
+    <axis xyz="0 0 1"/>
+    <safety_controller k_velocity="10"/>
+    <limit effort="100" velocity="117.81"/>
+    <dynamics damping="0.0" friction="0.0"/>
+  </joint>
+  <link name="fl_caster_rotation_link">
+    <inertial>
+      <origin xyz="0 0 0"/>
+      <mass value="5.9"/>
+      <inertia ixx="0.04" ixy="-0.0007" ixz="0.0" iyy="0.02" iyz="-0.000004" izz="0.05"/>
+    </inertial>
+    <visual>
+      <geometry>
+        <mesh filename="package://cob_description/meshes/drive_wheel/caster.stl"/>
+      </geometry>
+      <material name="IPA/LightGrey"/>
+    </visual>
+    <collision>
+      <geometry>
+        <box size="0.001 0.001 0.001"/>
+      </geometry>
+    </collision>
+  </link>
+  <transmission name="fl_caster_rotation_trans">
+    <type>transmission_interface/SimpleTransmission</type>
+    <joint name="fl_caster_rotation_joint">
+      <hardwareInterface>VelocityJointInterface</hardwareInterface>
+    </joint>
+    <actuator name="fl_caster_rotation_motor">
+      <mechanicalReduction>-79.2380952381</mechanicalReduction>
+    </actuator>
+  </transmission>
+  <joint name="fl_caster_r_wheel_joint" type="continuous">
+    <origin rpy="0 0 0" xyz="0 -0.0 0"/>
+    <parent link="fl_caster_rotation_link"/>
+    <child link="fl_caster_r_wheel_link"/>
+    <axis xyz="0 1 0"/>
+    <safety_controller k_velocity="10"/>
+    <limit effort="100" velocity="19.95"/>
+    <dynamics damping="0.0" friction="0.0"/>
+  </joint>
+  <link name="fl_caster_r_wheel_link">
+    <inertial>
+      <origin xyz="0 0 0"/>
+      <mass value="0.44036"/>
+      <inertia ixx="0.012411765597" ixy="-0.000711733678" ixz="0.00050272983" iyy="0.015218160428" iyz="-0.000004273467" izz="0.011763977943"/>
+    </inertial>
+    <visual>
+      <geometry>
+        <mesh filename="package://cob_description/meshes/drive_wheel/wheel.dae"/>
+      </geometry>
+    </visual>
+    <collision>
+      <geometry>
+        <mesh filename="package://cob_description/meshes/drive_wheel/wheel.stl"/>
+      </geometry>
+    </collision>
+  </link>
+  <gazebo reference="fl_caster_r_wheel_link">
+    <gravity>true</gravity>
+    <self_collide>false</self_collide>
+  </gazebo>
+  <transmission name="fl_caster_r_wheel_trans">
+    <type>transmission_interface/SimpleTransmission</type>
+    <joint name="fl_caster_r_wheel_joint">
+      <hardwareInterface>VelocityJointInterface</hardwareInterface>
+    </joint>
+    <actuator name="fl_caster_r_wheel_motor">
+      <mechanicalReduction>-79.2380952381</mechanicalReduction>
+    </actuator>
+  </transmission>
+  <gazebo reference="fl_caster_rotation_link">
+    <gravity>true</gravity>
+    <self_collide>false</self_collide>
+    <material value="IPA/Metal"/>
+  </gazebo>
+<!--________________________________________________________________________________________-->
+  <joint name="b_caster_rotation_joint" type="continuous">
+    <origin rpy="0 0 0" xyz="-0.24844 0.0 0.08"/>
+    <parent link="base_link"/>
+    <child link="b_caster_rotation_link"/>
+    <axis xyz="0 0 1"/>
+    <safety_controller k_velocity="10"/>
+    <limit effort="100" velocity="117.81"/>
+    <dynamics damping="0.0" friction="0.0"/>
+  </joint>
+  <link name="b_caster_rotation_link">
+    <inertial>
+      <origin xyz="0 0 0"/>
+      <mass value="5.9"/>
+      <inertia ixx="0.04" ixy="-0.0007" ixz="0.0" iyy="0.02" iyz="-0.000004" izz="0.05"/>
+    </inertial>
+    <visual>
+      <geometry>
+        <mesh filename="package://cob_description/meshes/drive_wheel/caster.stl"/>
+      </geometry>
+      <material name="IPA/LightGrey"/>
+    </visual>
+    <collision>
+      <geometry>
+        <box size="0.001 0.001 0.001"/>
+      </geometry>
+    </collision>
+  </link>
+  <transmission name="b_caster_rotation_trans">
+    <type>transmission_interface/SimpleTransmission</type>
+    <joint name="b_caster_rotation_joint">
+      <hardwareInterface>VelocityJointInterface</hardwareInterface>
+    </joint>
+    <actuator name="b_caster_rotation_motor">
+      <mechanicalReduction>-79.2380952381</mechanicalReduction>
+    </actuator>
+  </transmission>
+  <joint name="b_caster_r_wheel_joint" type="continuous">
+    <origin rpy="0 0 0" xyz="0 -0.0 0"/>
+    <parent link="b_caster_rotation_link"/>
+    <child link="b_caster_r_wheel_link"/>
+    <axis xyz="0 1 0"/>
+    <safety_controller k_velocity="10"/>
+    <limit effort="100" velocity="19.95"/>
+    <dynamics damping="0.0" friction="0.0"/>
+  </joint>
+  <link name="b_caster_r_wheel_link">
+    <inertial>
+      <origin xyz="0 0 0"/>
+      <mass value="0.44036"/>
+      <inertia ixx="0.012411765597" ixy="-0.000711733678" ixz="0.00050272983" iyy="0.015218160428" iyz="-0.000004273467" izz="0.011763977943"/>
+    </inertial>
+    <visual>
+      <geometry>
+        <mesh filename="package://cob_description/meshes/drive_wheel/wheel.dae"/>
+      </geometry>
+    </visual>
+    <collision>
+      <geometry>
+        <mesh filename="package://cob_description/meshes/drive_wheel/wheel.stl"/>
+      </geometry>
+    </collision>
+  </link>
+  <gazebo reference="b_caster_r_wheel_link">
+    <gravity>true</gravity>
+    <self_collide>false</self_collide>
+  </gazebo>
+  <transmission name="b_caster_r_wheel_trans">
+    <type>transmission_interface/SimpleTransmission</type>
+    <joint name="b_caster_r_wheel_joint">
+      <hardwareInterface>VelocityJointInterface</hardwareInterface>
+    </joint>
+    <actuator name="b_caster_r_wheel_motor">
+      <mechanicalReduction>-79.2380952381</mechanicalReduction>
+    </actuator>
+  </transmission>
+  <gazebo reference="b_caster_rotation_link">
+    <gravity>true</gravity>
+    <self_collide>false</self_collide>
+    <material value="IPA/Metal"/>
+  </gazebo>
+<!--________________________________________________________________________________________-->
+  <joint name="fr_caster_rotation_joint" type="continuous">
+    <origin rpy="0 0 0" xyz="0.12422 -0.21515 0.08"/>
+    <parent link="base_link"/>
+    <child link="fr_caster_rotation_link"/>
+    <axis xyz="0 0 1"/>
+    <safety_controller k_velocity="10"/>
+    <limit effort="100" velocity="117.81"/>
+    <dynamics damping="0.0" friction="0.0"/>
+  </joint>
+  <link name="fr_caster_rotation_link">
+    <inertial>
+      <origin xyz="0 0 0"/>
+      <mass value="5.9"/>
+      <inertia ixx="0.04" ixy="-0.0007" ixz="0.0" iyy="0.02" iyz="-0.000004" izz="0.05"/>
+    </inertial>
+    <visual>
+      <geometry>
+        <mesh filename="package://cob_description/meshes/drive_wheel/caster.stl"/>
+      </geometry>
+      <material name="IPA/LightGrey"/>
+    </visual>
+    <collision>
+      <geometry>
+        <box size="0.001 0.001 0.001"/>
+      </geometry>
+    </collision>
+  </link>
+  <transmission name="fr_caster_rotation_trans">
+    <type>transmission_interface/SimpleTransmission</type>
+    <joint name="fr_caster_rotation_joint">
+      <hardwareInterface>VelocityJointInterface</hardwareInterface>
+    </joint>
+    <actuator name="fr_caster_rotation_motor">
+      <mechanicalReduction>-79.2380952381</mechanicalReduction>
+    </actuator>
+  </transmission>
+  <joint name="fr_caster_r_wheel_joint" type="continuous">
+    <origin rpy="0 0 0" xyz="0 -0.0 0"/>
+    <parent link="fr_caster_rotation_link"/>
+    <child link="fr_caster_r_wheel_link"/>
+    <axis xyz="0 1 0"/>
+    <safety_controller k_velocity="10"/>
+    <limit effort="100" velocity="19.95"/>
+    <dynamics damping="0.0" friction="0.0"/>
+  </joint>
+  <link name="fr_caster_r_wheel_link">
+    <inertial>
+      <origin xyz="0 0 0"/>
+      <mass value="0.44036"/>
+      <inertia ixx="0.012411765597" ixy="-0.000711733678" ixz="0.00050272983" iyy="0.015218160428" iyz="-0.000004273467" izz="0.011763977943"/>
+    </inertial>
+    <visual>
+      <geometry>
+        <mesh filename="package://cob_description/meshes/drive_wheel/wheel.dae"/>
+      </geometry>
+    </visual>
+    <collision>
+      <geometry>
+        <mesh filename="package://cob_description/meshes/drive_wheel/wheel.stl"/>
+      </geometry>
+    </collision>
+  </link>
+  <gazebo reference="fr_caster_r_wheel_link">
+    <gravity>true</gravity>
+    <self_collide>false</self_collide>
+  </gazebo>
+  <transmission name="fr_caster_r_wheel_trans">
+    <type>transmission_interface/SimpleTransmission</type>
+    <joint name="fr_caster_r_wheel_joint">
+      <hardwareInterface>VelocityJointInterface</hardwareInterface>
+    </joint>
+    <actuator name="fr_caster_r_wheel_motor">
+      <mechanicalReduction>-79.2380952381</mechanicalReduction>
+    </actuator>
+  </transmission>
+  <gazebo reference="fr_caster_rotation_link">
+    <gravity>true</gravity>
+    <self_collide>false</self_collide>
+    <material value="IPA/Metal"/>
+  </gazebo>
+  <!-- laser_link -->
+  <gazebo reference="hokuyo_link">
+    <mu1>0.2</mu1>
+    <mu2>0.2</mu2>
+    <material>Gazebo/Orange</material>
+  </gazebo>
+  <joint name="hokuyo_joint" type="fixed">
+    <axis xyz="0 1 0" />
+    <origin xyz="0.539 0 0.5" rpy="0 0 0"/>		<!-- laser position -->
+    <parent link="base_link"/>
+    <child link="hokuyo_link"/>
+  </joint>
+  <!-- laser_scan -->
+  <link name="hokuyo_link">
+    <collision>
+      <origin xyz="0 0 0" rpy="0 0 0"/>
+      <geometry>
+			<box size="0.05 0.05 0.05"/>
+      </geometry>
+    </collision>
+    <visual>
+      <origin xyz="0 0 0" rpy="0 0 0"/>
+      <geometry>
+			<box size="0.05 0.05 0.05"/>
+      </geometry>
+    </visual>
+    <inertial>
+      <mass value="1e-5" />
+      <origin xyz="0 0 0" rpy="0 0 0"/>
+      <inertia ixx="1e-6" ixy="0" ixz="0" iyy="1e-6" iyz="0" izz="1e-6" />
+    </inertial>
+  </link>
+  <gazebo reference="hokuyo_link">
+    <sensor type="ray" name="head_hokuyo_sensor">
+      <pose>0 0 0 0 0 0</pose>
+      <visualize>true</visualize>
+      <update_rate>40</update_rate>
+      <ray>
+        <scan>
+          <horizontal>
+            <samples>720</samples>
+            <resolution>1</resolution>
+            <min_angle>-1.570796</min_angle>
+            <max_angle>1.570796</max_angle>
+          </horizontal>
+        </scan>
+        <range>
+          <min>0.10</min>
+          <max>30.0</max>
+          <resolution>0.01</resolution>
+        </range>
+        <noise>
+          <type>gaussian</type>
+          <!-- Noise parameters based on published spec for Hokuyo laser
+               achieving "+-30mm" accuracy at range < 10m.  A mean of 0.0m and
+               stddev of 0.01m will put 99.7% of samples within 0.03m of the true
+               reading. -->
+          <mean>0.0</mean>
+          <stddev>0.01</stddev>
+        </noise>
+      </ray>
+      <plugin name="gazebo_ros_head_hokuyo_controller" filename="libgazebo_ros_laser.so">
+        <topicName>/kfr1/laser/scan</topicName>
+        <frameName>hokuyo_link</frameName>
+      </plugin>
+    </sensor>
+  </gazebo>
+<!--________________________________________________________________________________________-->
+<!--________________________________________________________________________________________-->
+  <gazebo reference="base_link">
+    <gravity>true</gravity>
+    <self_collide>false</self_collide>
+    <sensor name="base_contact_sensor" type="contact">
+      <always_on>true</always_on>
+      <update_rate>100.0</update_rate>
+      <contact>
+        <collision>base_link_collision</collision>
+        <topic>base_bumper</topic>
+      </contact>
+      <plugin filename="libgazebo_ros_bumper.so" name="base_gazebo_ros_bumper_controller">
+        <frameName>world</frameName>
+        <bumperTopicName>base_bumper</bumperTopicName>
+      </plugin>
+    </sensor>
+  </gazebo>
+  <gazebo>
+    <plugin filename="libgazebo_ros_p3d.so" name="p3d_base_controller">
+      <alwaysOn>true</alwaysOn>
+      <updateRate>100.0</updateRate>
+      <bodyName>base_link</bodyName>
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