Commit message: renamed sensorring camera

File: cob_hardware_config/robots/cob4-8/urdf/calibration_default.urdf.xacro (robot description, xacro)
@@ -103,17 +103,10 @@
 	<xacro:property name="def_torso_cam3d_down_yaw" value="0.0"/>
 	<!-- cam3d | handeye calibration | relative to sensorring_link -->
-	<xacro:property name="def_sensorring_cam3d_front_x" value="0.096"/>
-	<xacro:property name="def_sensorring_cam3d_front_y" value="0.0"/>
-	<xacro:property name="def_sensorring_cam3d_front_z" value="0.0195"/>
-	<xacro:property name="def_sensorring_cam3d_front_roll" value="-1.95"/>
-	<xacro:property name="def_sensorring_cam3d_front_pitch" value="0.0"/>
-	<xacro:property name="def_sensorring_cam3d_front_yaw" value="-1.5708"/>
-	<!-- cam3d | handeye calibration | relative to sensorring_link -->
-	<xacro:property name="def_sensorring_cam3d_back_x" value="-0.096"/>
-	<xacro:property name="def_sensorring_cam3d_back_y" value="0.0"/>
-	<xacro:property name="def_sensorring_cam3d_back_z" value="0.0195"/>
-	<xacro:property name="def_sensorring_cam3d_back_roll" value="-1.5708"/>
-	<xacro:property name="def_sensorring_cam3d_back_pitch" value="0.0"/>
-	<xacro:property name="def_sensorring_cam3d_back_yaw" value="1.5708"/>
+	<xacro:property name="def_sensorring_cam3d_x" value="0.096"/>
+	<xacro:property name="def_sensorring_cam3d_y" value="0.0"/>
+	<xacro:property name="def_sensorring_cam3d_z" value="0.0195"/>
+	<xacro:property name="def_sensorring_cam3d_roll" value="-1.5708"/>
+	<xacro:property name="def_sensorring_cam3d_pitch" value="0.0"/>
+	<xacro:property name="def_sensorring_cam3d_yaw" value="-1.5708"/>
 	<!-- cam | handeye calibration | relative to head_3_link -->
 	<xacro:property name="def_head_cam_x" value="-0.181"/>

File: cob_hardware_config/robots/cob4-8/urdf/cob4-8.urdf.xacro (robot description, xacro)
@@ -63,9 +63,6 @@
   </xacro:sensorring>
   <!-- cameras -->
-  <xacro:sick_3dcs name="sensorring_cam3d_front" ros_topic="sensorring_cam3d_front" parent="sensorring_link">
-    <origin xyz="${sensorring_cam3d_front_x} ${sensorring_cam3d_front_y} ${sensorring_cam3d_front_z}" rpy="${sensorring_cam3d_front_roll} ${sensorring_cam3d_front_pitch} ${sensorring_cam3d_front_yaw}" />
-  </xacro:sick_3dcs>
-  <xacro:cob_kinect_v0 name="sensorring_cam3d_back" ros_topic="sensorring_cam3d_back" parent="sensorring_link" update_rate="30" data_skip="9">
-    <origin xyz="${sensorring_cam3d_back_x} ${sensorring_cam3d_back_y} ${sensorring_cam3d_back_z}" rpy="${sensorring_cam3d_back_roll} ${sensorring_cam3d_back_pitch} ${sensorring_cam3d_back_yaw}" />
+  <xacro:cob_kinect_v0 name="sensorring_cam3d" ros_topic="sensorring_cam3d" parent="sensorring_link" update_rate="30" data_skip="9">
+    <origin xyz="${sensorring_cam3d_x} ${sensorring_cam3d_y} ${sensorring_cam3d_z}" rpy="${sensorring_cam3d_roll} ${sensorring_cam3d_pitch} ${sensorring_cam3d_yaw}" />
   </xacro:cob_kinect_v0>
   <xacro:schunk_lwa4p_extended name="arm_right" parent="torso_3_link" has_podest="false">

File: cob_hardware_config/robots/cob4-8/urdf/properties.urdf.xacro (robot description, xacro)
@@ -106,17 +106,10 @@
 	<xacro:property name="torso_cam3d_down_yaw" value="${def_torso_cam3d_down_yaw+offset_torso_cam3d_down_yaw}"/>
 	<!-- cam3d | handeye calibration | relative to sensorring_link -->
-	<xacro:property name="sensorring_cam3d_front_x" value="${def_sensorring_cam3d_front_x+offset_sensorring_cam3d_front_x}"/>
-	<xacro:property name="sensorring_cam3d_front_y" value="${def_sensorring_cam3d_front_y+offset_sensorring_cam3d_front_y}"/>
-	<xacro:property name="sensorring_cam3d_front_z" value="${def_sensorring_cam3d_front_z+offset_sensorring_cam3d_front_z}"/>
-	<xacro:property name="sensorring_cam3d_front_roll" value="${def_sensorring_cam3d_front_roll+offset_sensorring_cam3d_front_roll}"/>
-	<xacro:property name="sensorring_cam3d_front_pitch" value="${def_sensorring_cam3d_front_pitch+offset_sensorring_cam3d_front_pitch}"/>
-	<xacro:property name="sensorring_cam3d_front_yaw" value="${def_sensorring_cam3d_front_yaw+offset_sensorring_cam3d_front_yaw}"/>
-	<!-- cam3d | handeye calibration | relative to sensorring_link -->
-	<xacro:property name="sensorring_cam3d_back_x" value="${def_sensorring_cam3d_back_x+offset_sensorring_cam3d_back_x}"/>
-	<xacro:property name="sensorring_cam3d_back_y" value="${def_sensorring_cam3d_back_y+offset_sensorring_cam3d_back_y}"/>
-	<xacro:property name="sensorring_cam3d_back_z" value="${def_sensorring_cam3d_back_z+offset_sensorring_cam3d_back_z}"/>
-	<xacro:property name="sensorring_cam3d_back_roll" value="${def_sensorring_cam3d_back_roll+offset_sensorring_cam3d_back_roll}"/>
-	<xacro:property name="sensorring_cam3d_back_pitch" value="${def_sensorring_cam3d_back_pitch+offset_sensorring_cam3d_back_pitch}"/>
-	<xacro:property name="sensorring_cam3d_back_yaw" value="${def_sensorring_cam3d_back_yaw+offset_sensorring_cam3d_back_yaw}"/>
+	<xacro:property name="sensorring_cam3d_x" value="${def_sensorring_cam3d_x+offset_sensorring_cam3d_x}"/>
+	<xacro:property name="sensorring_cam3d_y" value="${def_sensorring_cam3d_y+offset_sensorring_cam3d_y}"/>
+	<xacro:property name="sensorring_cam3d_z" value="${def_sensorring_cam3d_z+offset_sensorring_cam3d_z}"/>
+	<xacro:property name="sensorring_cam3d_roll" value="${def_sensorring_cam3d_roll+offset_sensorring_cam3d_roll}"/>
+	<xacro:property name="sensorring_cam3d_pitch" value="${def_sensorring_cam3d_pitch+offset_sensorring_cam3d_pitch}"/>
+	<xacro:property name="sensorring_cam3d_yaw" value="${def_sensorring_cam3d_yaw+offset_sensorring_cam3d_yaw}"/>
 	<!-- cam | handeye calibration | relative to head_3_link -->
 	<xacro:property name="head_cam_x" value="${def_head_cam_x+offset_head_cam_x}"/>

Commit message: Fix on the urdf: sensorring's parent link moved to head_2_link (previously on head_3_link, which is not how the hardware works)

File: cob_hardware_config/robots/cob4-8/urdf/calibration_default.urdf.xacro (robot description, xacro)
@@ -42,9 +42,16 @@
 	<xacro:property name="def_head_pitch" value="0.0"/>
 	<xacro:property name="def_head_yaw" value="0.0"/>
-	<!-- head sensors mount positions | relative to head_3_link -->
+	<!-- head sensors mount positions | relative to head_3_link
 	<xacro:property name="def_sensorring_x" value="0.0"/>
 	<xacro:property name="def_sensorring_y" value="0.0"/>
 	<xacro:property name="def_sensorring_z" value="0.006"/>
 	<xacro:property name="def_sensorring_roll" value="0.0"/>
+	<xacro:property name="def_sensorring_pitch" value="0.0"/>
+	<xacro:property name="def_sensorring_yaw" value="0.0"/>
+	-->
+	<xacro:property name="def_sensorring_x" value="0.0"/>
+	<xacro:property name="def_sensorring_y" value="-0.098"/>
+	<xacro:property name="def_sensorring_z" value="0.045"/>
+	<xacro:property name="def_sensorring_roll" value="0.349"/>
 	<xacro:property name="def_sensorring_pitch" value="0.0"/>
 	<xacro:property name="def_sensorring_yaw" value="0.0"/>

File: cob_hardware_config/robots/cob4-8/urdf/cob4-8.urdf.xacro (robot description, xacro)
@@ -20,5 +20,5 @@
   <xacro:include filename="$(find cob_description)/urdf/cob4_sensorring/sensorring.urdf.xacro" />
   <!-- sensors -->
-  <xacro:include filename="$(find cob_description)/urdf/sensors/realsense_d435.urdf.xacro" />
+  <xacro:include filename="$(find cob_description)/urdf/sensors/realsense.urdf.xacro" />
   <xacro:include filename="$(find cob_description)/urdf/sensors/kinect.urdf.xacro" />
   <xacro:include filename="$(find cob_description)/urdf/sensors/usb_cam.urdf.xacro" />
@@ -36,17 +36,20 @@
     <origin xyz="${laser_right_x} ${laser_right_y} ${laser_right_z}" rpy="${laser_right_roll} ${laser_right_pitch} ${laser_right_yaw}" />
   </xacro:sick_s300_laser_v0>
-  <xacro:torso name="torso" parent="base_link" dof1="${False}" dof2="${False}" dof3="${False}">
+  <xacro:torso name="torso" parent="base_link" dof1="false" dof2="false" dof3="false">
     <origin xyz="${torso_x} ${torso_y} ${torso_z}" rpy="${torso_roll} ${torso_pitch} ${torso_yaw}" />
   </xacro:torso>
-  <xacro:realsense_d435 name="torso_cam3d_left" parent="torso_3_link">
+  <!-- left camera -->
+  <xacro:cob_kinect_v0 name="torso_cam3d_left" ros_topic="torso_cam3d_left" parent="torso_3_link" update_rate="30" data_skip="9">
     <origin xyz="${torso_cam3d_left_x} ${torso_cam3d_left_y} ${torso_cam3d_left_z}" rpy="${torso_cam3d_left_roll} ${torso_cam3d_left_pitch} ${torso_cam3d_left_yaw}" />
-  </xacro:realsense_d435>
-  <xacro:realsense_d435 name="torso_cam3d_right" parent="torso_3_link">
+  </xacro:cob_kinect_v0>
+  <!-- right camera -->
+  <xacro:cob_kinect_v0 name="torso_cam3d_right" ros_topic="torso_cam3d_right" parent="torso_3_link" update_rate="30" data_skip="9">
     <origin xyz="${torso_cam3d_right_x} ${torso_cam3d_right_y} ${torso_cam3d_right_z}" rpy="${torso_cam3d_right_roll} ${torso_cam3d_right_pitch} ${torso_cam3d_right_yaw}" />
-  </xacro:realsense_d435>
-  <xacro:realsense_d435 name="torso_cam3d_down" parent="torso_3_link">
+  </xacro:cob_kinect_v0>
+  <!-- down camera -->
+  <xacro:realsense name="torso_cam3d_down" ros_topic="torso_cam3d_down" parent="torso_3_link">
     <origin xyz="${torso_cam3d_down_x} ${torso_cam3d_down_y} ${torso_cam3d_down_z}" rpy="${torso_cam3d_down_roll} ${torso_cam3d_down_pitch} ${torso_cam3d_down_yaw}" />
-  </xacro:realsense_d435>
-  <xacro:head name="head" parent="torso_3_link" dof1="${True}" dof2="${True}" dof3="${True}">
+  </xacro:realsense>
+  <xacro:head name="head" parent="torso_3_link" dof1="true" dof2="true" dof3="true">
     <origin xyz="${head_x} ${head_y} ${head_z}" rpy="${head_roll} ${head_pitch} ${head_yaw}" />
   </xacro:head>
@@ -54,7 +57,8 @@
     <origin xyz="${head_cam_x} ${head_cam_y} ${head_cam_z}" rpy="${head_cam_roll} ${head_cam_pitch} ${head_cam_yaw}" />
   </xacro:usb_cam>
-  <xacro:sensorring name="sensorring" parent="head_3_link" active="${True}">
+  <xacro:sensorring name="sensorring" parent="head_2_link" active="true">
     <origin xyz="${sensorring_x} ${sensorring_y} ${sensorring_z}" rpy="${sensorring_roll} ${sensorring_pitch} ${sensorring_yaw}" />
   </xacro:sensorring>
+  <!-- cameras -->
   <xacro:cob_kinect_v0 name="sensorring_cam3d" ros_topic="sensorring_cam3d" parent="sensorring_link" update_rate="30" data_skip="9">
     <origin xyz="${sensorring_cam3d_x} ${sensorring_cam3d_y} ${sensorring_cam3d_z}" rpy="${sensorring_cam3d_roll} ${sensorring_cam3d_pitch} ${sensorring_cam3d_yaw}" />

Commit message: Fix on the urdf: sensorring's parent link moved to head_2_link (previously on head_3_link, which is not how the hardware works)

File: cob_hardware_config/robots/cob4-8/urdf/calibration_default.urdf.xacro (robot description, xacro)
@@ -42,9 +42,16 @@
 	<xacro:property name="def_head_pitch" value="0.0"/>
 	<xacro:property name="def_head_yaw" value="0.0"/>
-	<!-- head sensors mount positions | relative to head_3_link -->
+	<!-- head sensors mount positions | relative to head_3_link
 	<xacro:property name="def_sensorring_x" value="0.0"/>
 	<xacro:property name="def_sensorring_y" value="0.0"/>
 	<xacro:property name="def_sensorring_z" value="0.006"/>
 	<xacro:property name="def_sensorring_roll" value="0.0"/>
+	<xacro:property name="def_sensorring_pitch" value="0.0"/>
+	<xacro:property name="def_sensorring_yaw" value="0.0"/>
+	-->
+	<xacro:property name="def_sensorring_x" value="0.0"/>
+	<xacro:property name="def_sensorring_y" value="-0.098"/>
+	<xacro:property name="def_sensorring_z" value="0.045"/>
+	<xacro:property name="def_sensorring_roll" value="0.349"/>
 	<xacro:property name="def_sensorring_pitch" value="0.0"/>
 	<xacro:property name="def_sensorring_yaw" value="0.0"/>

File: cob_hardware_config/robots/cob4-8/urdf/cob4-8.urdf.xacro (robot description, xacro)
@@ -57,5 +57,5 @@
     <origin xyz="${head_cam_x} ${head_cam_y} ${head_cam_z}" rpy="${head_cam_roll} ${head_cam_pitch} ${head_cam_yaw}" />
   </xacro:usb_cam>
-  <xacro:sensorring name="sensorring" parent="head_3_link" active="true">
+  <xacro:sensorring name="sensorring" parent="head_2_link" active="true">
     <origin xyz="${sensorring_x} ${sensorring_y} ${sensorring_z}" rpy="${sensorring_roll} ${sensorring_pitch} ${sensorring_yaw}" />
   </xacro:sensorring>

Commit message: Better comment plus 6 mm fix (from doing the math)

File: cob_hardware_config/robots/cob4-8/urdf/calibration_default.urdf.xacro (robot description, xacro)
@@ -42,5 +42,7 @@
 	<xacro:property name="def_head_pitch" value="0.0"/>
 	<xacro:property name="def_head_yaw" value="0.0"/>
-	<!-- head sensors mount positions | relative to head_3_link
+    <!-- Legacy transformation, following from WRONG urdf-->
+	<!-- head sensors mount positions | relative to head_3_link -->
+	<!--
 	<xacro:property name="def_sensorring_x" value="0.0"/>
 	<xacro:property name="def_sensorring_y" value="0.0"/>
@@ -50,7 +52,8 @@
 	<xacro:property name="def_sensorring_yaw" value="0.0"/>
 	-->
+	<!-- head sensors mount positions | relative to head_2_link -->
 	<xacro:property name="def_sensorring_x" value="0.0"/>
 	<xacro:property name="def_sensorring_y" value="-0.098"/>
-	<xacro:property name="def_sensorring_z" value="0.045"/>
+	<xacro:property name="def_sensorring_z" value="0.051"/>
 	<xacro:property name="def_sensorring_roll" value="0.349"/>
 	<xacro:property name="def_sensorring_pitch" value="0.0"/>

Commit message: remove legacy transformation and fix indent

File: cob_hardware_config/robots/cob4-8/urdf/calibration_default.urdf.xacro (robot description, xacro)
@@ -42,14 +42,4 @@
 	<xacro:property name="def_head_pitch" value="0.0"/>
 	<xacro:property name="def_head_yaw" value="0.0"/>
-    <!-- Legacy transformation, following from WRONG urdf-->
-	<!-- head sensors mount positions | relative to head_3_link -->
-	<!--
-	<xacro:property name="def_sensorring_x" value="0.0"/>
-	<xacro:property name="def_sensorring_y" value="0.0"/>
-	<xacro:property name="def_sensorring_z" value="0.006"/>
-	<xacro:property name="def_sensorring_roll" value="0.0"/>
-	<xacro:property name="def_sensorring_pitch" value="0.0"/>
-	<xacro:property name="def_sensorring_yaw" value="0.0"/>
-	-->
 	<!-- head sensors mount positions | relative to head_2_link -->
 	<xacro:property name="def_sensorring_x" value="0.0"/>
