Commit message: update cob4-8 (is now running kinetic with d435 cams)

File: cob_hardware_config/robots/cob4-8/urdf/calibration_default.urdf.xacro (robot description, xacro)
@@ -11,5 +11,5 @@
 	<xacro:property name="def_laser_front_pitch" value="0.0"/>
 	<xacro:property name="def_laser_front_yaw" value="0.0"/>
-	<!-- laser rear mount positions | relative to base_link -->
+	<!-- laser left mount positions | relative to base_link -->
 	<xacro:property name="def_laser_left_x" value="-0.122"/>
 	<xacro:property name="def_laser_left_y" value="0.21131"/>
@@ -18,5 +18,5 @@
 	<xacro:property name="def_laser_left_pitch" value="0.0"/>
 	<xacro:property name="def_laser_left_yaw" value="2.094"/>
-	<!-- laser top mount positions | relative to base_link -->
+	<!-- laser right mount positions | relative to base_link -->
 	<xacro:property name="def_laser_right_x" value="-0.122"/>
 	<xacro:property name="def_laser_right_y" value="-0.21131"/>
@@ -77,30 +77,29 @@
 	<xacro:property name="def_gripper_left_pitch" value="0.0"/>
 	<xacro:property name="def_gripper_left_yaw" value="3.14159"/>
-	<!-- *********************************** -->
-	<!-- kinematic chain reference positions -->
-	<!-- *********************************** -->
-	<!-- this feature is no longer supported as urdfdom does not parse the according 'calibration_rising' tag -->
-	<!-- cam3d left | handeye calibration | relative to torso_3_link -->
-	<xacro:property name="def_torso_cam3d_left_x" value="0.125"/>
-	<xacro:property name="def_torso_cam3d_left_y" value="0.01802"/>
-	<xacro:property name="def_torso_cam3d_left_z" value="0.24214"/>
-	<xacro:property name="def_torso_cam3d_left_roll" value="1.57079"/>
+	<!-- ***************************** -->
+	<!-- extrinsic camera calibration  -->
+	<!-- ***************************** -->
+	<!-- torso cam3d left mount positions | relative to torso_3_link -->
+	<xacro:property name="def_torso_cam3d_left_x" value="0.14873"/>
+	<xacro:property name="def_torso_cam3d_left_y" value="0.01293"/>
+	<xacro:property name="def_torso_cam3d_left_z" value="0.27008"/>
+	<xacro:property name="def_torso_cam3d_left_roll" value="-1.57079"/>
 	<xacro:property name="def_torso_cam3d_left_pitch" value="0.0"/>
-	<xacro:property name="def_torso_cam3d_left_yaw" value="0.418879"/>
-	<!-- cam3d right | handeye calibration | relative to torso_3_link -->
-	<xacro:property name="def_torso_cam3d_right_x" value="0.12839"/>
-	<xacro:property name="def_torso_cam3d_right_y" value="-0.01802"/>
-	<xacro:property name="def_torso_cam3d_right_z" value="0.24214"/>
-	<xacro:property name="def_torso_cam3d_right_roll" value="1.57079"/>
+	<xacro:property name="def_torso_cam3d_left_yaw" value="0.61"/>
+	<!-- torso cam3d right mount positions | relative to torso_3_link -->
+	<xacro:property name="def_torso_cam3d_right_x" value="0.14873"/>
+	<xacro:property name="def_torso_cam3d_right_y" value="-0.01293"/>
+	<xacro:property name="def_torso_cam3d_right_z" value="0.27008"/>
+	<xacro:property name="def_torso_cam3d_right_roll" value="-1.57079"/>
 	<xacro:property name="def_torso_cam3d_right_pitch" value="0.0"/>
-	<xacro:property name="def_torso_cam3d_right_yaw" value="-0.418879"/>
-	<!-- cam3d down | handeye calibration | relative to torso_3_link -->
-	<xacro:property name="def_torso_cam3d_down_x" value="0.15908"/>
+	<xacro:property name="def_torso_cam3d_right_yaw" value="-0.61"/>
+	<!-- torso cam3d down mount positions | relative to torso_3_link -->
+	<xacro:property name="def_torso_cam3d_down_x" value="0.15203"/>
 	<xacro:property name="def_torso_cam3d_down_y" value="0.0"/>
-	<xacro:property name="def_torso_cam3d_down_z" value="0.14005"/>
+	<xacro:property name="def_torso_cam3d_down_z" value="0.1307"/>
 	<xacro:property name="def_torso_cam3d_down_roll" value="0.0"/>
-	<xacro:property name="def_torso_cam3d_down_pitch" value="0.61086"/>
+	<xacro:property name="def_torso_cam3d_down_pitch" value="0.56"/>
 	<xacro:property name="def_torso_cam3d_down_yaw" value="0.0"/>
-	<!-- cam3d | handeye calibration | relative to sensorring_link -->
+	<!-- sensorring cam3d | handeye calibration | relative to sensorring_link -->
 	<xacro:property name="def_sensorring_cam3d_x" value="0.096"/>
 	<xacro:property name="def_sensorring_cam3d_y" value="0.0"/>
@@ -109,5 +108,5 @@
 	<xacro:property name="def_sensorring_cam3d_pitch" value="0.0"/>
 	<xacro:property name="def_sensorring_cam3d_yaw" value="0.0"/>
-	<!-- cam | handeye calibration | relative to head_3_link -->
+	<!-- head cam mount positions | relative to head_3_link -->
 	<xacro:property name="def_head_cam_x" value="-0.181"/>
 	<xacro:property name="def_head_cam_y" value="0.0"/>

File: cob_hardware_config/robots/cob4-8/urdf/cob4-8.urdf.xacro (robot description, xacro)
@@ -20,5 +20,5 @@
   <xacro:include filename="$(find cob_description)/urdf/cob4_sensorring/sensorring.urdf.xacro" />
   <!-- sensors -->
-  <xacro:include filename="$(find cob_description)/urdf/sensors/realsense.urdf.xacro" />
+  <xacro:include filename="$(find cob_description)/urdf/sensors/realsense_d435.urdf.xacro" />
   <xacro:include filename="$(find cob_description)/urdf/sensors/kinect.urdf.xacro" />
   <xacro:include filename="$(find cob_description)/urdf/sensors/usb_cam.urdf.xacro" />
@@ -39,16 +39,13 @@
     <origin xyz="${torso_x} ${torso_y} ${torso_z}" rpy="${torso_roll} ${torso_pitch} ${torso_yaw}" />
   </xacro:torso>
-  <!-- left camera -->
-  <xacro:cob_kinect_v0 name="torso_cam3d_left" ros_topic="torso_cam3d_left" parent="torso_3_link" update_rate="30" data_skip="9">
+  <xacro:realsense_d435 name="torso_cam3d_left" parent="torso_3_link">
     <origin xyz="${torso_cam3d_left_x} ${torso_cam3d_left_y} ${torso_cam3d_left_z}" rpy="${torso_cam3d_left_roll} ${torso_cam3d_left_pitch} ${torso_cam3d_left_yaw}" />
-  </xacro:cob_kinect_v0>
-  <!-- right camera -->
-  <xacro:cob_kinect_v0 name="torso_cam3d_right" ros_topic="torso_cam3d_right" parent="torso_3_link" update_rate="30" data_skip="9">
+  </xacro:realsense_d435>
+  <xacro:realsense_d435 name="torso_cam3d_right" parent="torso_3_link">
     <origin xyz="${torso_cam3d_right_x} ${torso_cam3d_right_y} ${torso_cam3d_right_z}" rpy="${torso_cam3d_right_roll} ${torso_cam3d_right_pitch} ${torso_cam3d_right_yaw}" />
-  </xacro:cob_kinect_v0>
-  <!-- down camera -->
-  <xacro:realsense name="torso_cam3d_down" ros_topic="torso_cam3d_down" parent="torso_3_link">
+  </xacro:realsense_d435>
+  <xacro:realsense_d435 name="torso_cam3d_down" parent="torso_3_link">
     <origin xyz="${torso_cam3d_down_x} ${torso_cam3d_down_y} ${torso_cam3d_down_z}" rpy="${torso_cam3d_down_roll} ${torso_cam3d_down_pitch} ${torso_cam3d_down_yaw}" />
-  </xacro:realsense>
+  </xacro:realsense_d435>
   <xacro:head name="head" parent="torso_3_link" dof1="${True}" dof2="${True}" dof3="${True}">
     <origin xyz="${head_x} ${head_y} ${head_z}" rpy="${head_roll} ${head_pitch} ${head_yaw}" />
@@ -60,5 +57,4 @@
     <origin xyz="${sensorring_x} ${sensorring_y} ${sensorring_z}" rpy="${sensorring_roll} ${sensorring_pitch} ${sensorring_yaw}" />
   </xacro:sensorring>
-  <!-- cameras -->
   <xacro:cob_kinect_v0 name="sensorring_cam3d" ros_topic="sensorring_cam3d" parent="sensorring_link" update_rate="30" data_skip="9">
     <origin xyz="${sensorring_cam3d_x} ${sensorring_cam3d_y} ${sensorring_cam3d_z}" rpy="${sensorring_cam3d_roll} ${sensorring_cam3d_pitch} ${sensorring_cam3d_yaw}" />

File: cob_hardware_config/robots/cob4-8/urdf/properties.urdf.xacro (robot description, xacro)
@@ -14,5 +14,5 @@
 	<xacro:property name="laser_front_pitch" value="${def_laser_front_pitch+offset_laser_front_pitch}"/>
 	<xacro:property name="laser_front_yaw" value="${def_laser_front_yaw+offset_laser_front_yaw}"/>
-	<!-- laser rear mount positions | relative to base_link -->
+	<!-- laser left mount positions | relative to base_link -->
 	<xacro:property name="laser_left_x" value="${def_laser_left_x+offset_laser_left_x}"/>
 	<xacro:property name="laser_left_y" value="${def_laser_left_y+offset_laser_left_y}"/>
@@ -21,5 +21,5 @@
 	<xacro:property name="laser_left_pitch" value="${def_laser_left_pitch+offset_laser_left_pitch}"/>
 	<xacro:property name="laser_left_yaw" value="${def_laser_left_yaw+offset_laser_left_yaw}"/>
-	<!-- laser top mount positions | relative to base_link -->
+	<!-- laser right mount positions | relative to base_link -->
 	<xacro:property name="laser_right_x" value="${def_laser_right_x+offset_laser_right_x}"/>
 	<xacro:property name="laser_right_y" value="${def_laser_right_y+offset_laser_right_y}"/>
@@ -45,5 +45,5 @@
 	<xacro:property name="head_pitch" value="${def_head_pitch+offset_head_pitch}"/>
 	<xacro:property name="head_yaw" value="${def_head_yaw+offset_head_yaw}"/>
-	<!-- head sensors mount positions | relative to head_3_link -->
+	<!-- sensorring mount positions | relative to head_3_link -->
 	<xacro:property name="sensorring_x" value="${def_sensorring_x+offset_sensorring_x}"/>
 	<xacro:property name="sensorring_y" value="${def_sensorring_y+offset_sensorring_y}"/>
@@ -52,5 +52,5 @@
 	<xacro:property name="sensorring_pitch" value="${def_sensorring_pitch+offset_sensorring_pitch}"/>
 	<xacro:property name="sensorring_yaw" value="${def_sensorring_yaw+offset_sensorring_yaw}"/>
-	<!-- arm mount positions | relative to torso_3_link -->
+	<!-- arm right mount positions | relative to torso_3_link -->
 	<xacro:property name="arm_right_x" value="${def_arm_right_x+offset_arm_right_x}"/>
 	<xacro:property name="arm_right_y" value="${def_arm_right_y+offset_arm_right_y}"/>
@@ -59,5 +59,5 @@
 	<xacro:property name="arm_right_pitch" value="${def_arm_right_pitch+offset_arm_right_pitch}"/>
 	<xacro:property name="arm_right_yaw" value="${def_arm_right_yaw+offset_arm_right_yaw}"/>
-	<!-- arm mount positions | relative to torso_3_link -->
+	<!-- arm left mount positions | relative to torso_3_link -->
 	<xacro:property name="arm_left_x" value="${def_arm_left_x+offset_arm_left_x}"/>
 	<xacro:property name="arm_left_y" value="${def_arm_left_y+offset_arm_left_y}"/>
@@ -66,5 +66,5 @@
 	<xacro:property name="arm_left_pitch" value="${def_arm_left_pitch+offset_arm_left_pitch}"/>
 	<xacro:property name="arm_left_yaw" value="${def_arm_left_yaw+offset_arm_left_yaw}"/>
-	<!-- gripper mount positions | relative to arm_7_link -->
+	<!-- gripper right mount positions | relative to arm_7_link -->
 	<xacro:property name="gripper_right_x" value="${def_gripper_right_x+offset_gripper_right_x}"/>
 	<xacro:property name="gripper_right_y" value="${def_gripper_right_y+offset_gripper_right_y}"/>
@@ -73,5 +73,5 @@
 	<xacro:property name="gripper_right_pitch" value="${def_gripper_right_pitch+offset_gripper_right_pitch}"/>
 	<xacro:property name="gripper_right_yaw" value="${def_gripper_right_yaw+offset_gripper_right_yaw}"/>
-	<!-- gripper mount positions | relative to arm_7_link -->
+	<!-- gripper left mount positions | relative to arm_7_link -->
 	<xacro:property name="gripper_left_x" value="${def_gripper_left_x+offset_gripper_left_x}"/>
 	<xacro:property name="gripper_left_y" value="${def_gripper_left_y+offset_gripper_left_y}"/>
@@ -80,9 +80,8 @@
 	<xacro:property name="gripper_left_pitch" value="${def_gripper_left_pitch+offset_gripper_left_pitch}"/>
 	<xacro:property name="gripper_left_yaw" value="${def_gripper_left_yaw+offset_gripper_left_yaw}"/>
-	<!-- *********************************** -->
-	<!-- kinematic chain reference positions -->
-	<!-- *********************************** -->
-	<!-- this feature is no longer supported as urdfdom does not parse the according 'calibration_rising' tag -->
-	<!-- cam3d left | handeye calibration | relative to torso_3_link -->
+	<!-- ***************************** -->
+	<!-- extrinsic camera calibration  -->
+	<!-- ***************************** -->
+	<!-- torso cam3d left mount positions | relative to torso_3_link -->
 	<xacro:property name="torso_cam3d_left_x" value="${def_torso_cam3d_left_x+offset_torso_cam3d_left_x}"/>
 	<xacro:property name="torso_cam3d_left_y" value="${def_torso_cam3d_left_y+offset_torso_cam3d_left_y}"/>
@@ -91,5 +90,5 @@
 	<xacro:property name="torso_cam3d_left_pitch" value="${def_torso_cam3d_left_pitch+offset_torso_cam3d_left_pitch}"/>
 	<xacro:property name="torso_cam3d_left_yaw" value="${def_torso_cam3d_left_yaw+offset_torso_cam3d_left_yaw}"/>
-	<!-- cam3d right | handeye calibration | relative to torso_3_link -->
+	<!-- torso cam3d right mount positions | relative to torso_3_link -->
 	<xacro:property name="torso_cam3d_right_x" value="${def_torso_cam3d_right_x+offset_torso_cam3d_right_x}"/>
 	<xacro:property name="torso_cam3d_right_y" value="${def_torso_cam3d_right_y+offset_torso_cam3d_right_y}"/>
@@ -98,5 +97,5 @@
 	<xacro:property name="torso_cam3d_right_pitch" value="${def_torso_cam3d_right_pitch+offset_torso_cam3d_right_pitch}"/>
 	<xacro:property name="torso_cam3d_right_yaw" value="${def_torso_cam3d_right_yaw+offset_torso_cam3d_right_yaw}"/>
-	<!-- cam3d down | handeye calibration | relative to torso_3_link -->
+	<!-- torso cam3d down mount positions | relative to torso_3_link -->
 	<xacro:property name="torso_cam3d_down_x" value="${def_torso_cam3d_down_x+offset_torso_cam3d_down_x}"/>
 	<xacro:property name="torso_cam3d_down_y" value="${def_torso_cam3d_down_y+offset_torso_cam3d_down_y}"/>
@@ -105,5 +104,5 @@
 	<xacro:property name="torso_cam3d_down_pitch" value="${def_torso_cam3d_down_pitch+offset_torso_cam3d_down_pitch}"/>
 	<xacro:property name="torso_cam3d_down_yaw" value="${def_torso_cam3d_down_yaw+offset_torso_cam3d_down_yaw}"/>
-	<!-- cam3d | handeye calibration | relative to sensorring_link -->
+	<!-- sensorring cam3d mount positions | relative to sensorring_link -->
 	<xacro:property name="sensorring_cam3d_x" value="${def_sensorring_cam3d_x+offset_sensorring_cam3d_x}"/>
 	<xacro:property name="sensorring_cam3d_y" value="${def_sensorring_cam3d_y+offset_sensorring_cam3d_y}"/>
@@ -112,5 +111,5 @@
 	<xacro:property name="sensorring_cam3d_pitch" value="${def_sensorring_cam3d_pitch+offset_sensorring_cam3d_pitch}"/>
 	<xacro:property name="sensorring_cam3d_yaw" value="${def_sensorring_cam3d_yaw+offset_sensorring_cam3d_yaw}"/>
-	<!-- cam | handeye calibration | relative to head_3_link -->
+	<!-- head cam mount positions | relative to head_3_link -->
 	<xacro:property name="head_cam_x" value="${def_head_cam_x+offset_head_cam_x}"/>
 	<xacro:property name="head_cam_y" value="${def_head_cam_y+offset_head_cam_y}"/>

Commit message: correct mount position for sensorring

File: cob_hardware_config/robots/cob4-8/urdf/calibration_default.urdf.xacro (robot description, xacro)
@@ -44,9 +44,9 @@
 	<!-- head sensors mount positions | relative to head_2_link -->
 	<xacro:property name="def_sensorring_x" value="0.0"/>
-	<xacro:property name="def_sensorring_y" value="-0.098"/>
-	<xacro:property name="def_sensorring_z" value="0.051"/>
+	<xacro:property name="def_sensorring_y" value="0.09849"/>
+	<xacro:property name="def_sensorring_z" value="0.04476"/>
 	<xacro:property name="def_sensorring_roll" value="0.349"/>
 	<xacro:property name="def_sensorring_pitch" value="0.0"/>
-	<xacro:property name="def_sensorring_yaw" value="0.0"/>
+	<xacro:property name="def_sensorring_yaw" value="-${M_PI}"/>
 	<!-- arm right mount positions | relative to torso_3_link -->
 	<xacro:property name="def_arm_right_x" value="0.0"/>
