Commit message: dummy beverage robot for navigation - cob4-18 with torso cam3d bottom and top

File: cob_hardware_config/robots/cob4-18/urdf/cob4-18.urdf.xacro (robot description, xacro)
@@ -11,4 +11,5 @@
   <!-- sensors -->
   <xacro:include filename="$(find cob_description)/urdf/sensors/sick_s300_laser.urdf.xacro"/>
+  <xacro:include filename="$(find cob_description)/urdf/sensors/realsense_d435.urdf.xacro" />
   <!-- composition of the robot -->
   <xacro:base name="base"/>
@@ -23,3 +24,9 @@
     <origin xyz="${laser_right_x} ${laser_right_y} ${laser_right_z}" rpy="${laser_right_roll} ${laser_right_pitch} ${laser_right_yaw}" />
   </xacro:sick_s300_laser_v0>
+  <xacro:realsense_d435 name="torso_cam3d_bottom" parent="base_link">
+    <origin xyz="0.296 0.018 0.272" rpy="0.000 -0.490 0.000" />
+  </xacro:realsense_d435>
+  <xacro:realsense_d435 name="torso_cam3d_top" parent="base_link">
+    <origin xyz="0.318 0.018 0.905" rpy="0.000 0.975 0.000" />
+  </xacro:realsense_d435>
 </robot>
